File: HARDWARE/ETH1CSMU2/Trigger.kicad_sch (KiCad schematic)
At the start: 22 parts, among them U26 TXB0104PW, U27 ADuM5402, U28 74AC125

Commit message: Hardware design
Parts:
- renumbered R58 to R59, R59 to R60, R60 to R61, R61 to R62, R62 to R63, R63 to R64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
