File: HARDWARE/ETH1CSMU2/Trigger.kicad_sch (KiCad schematic)
At the start: 22 parts, among them U28 TXB0104PW, U29 ADuM5402, U30 74AC125

Commit message: Hardware design
Parts:
- renumbered C51 to C701, C52 to C702, C53 to C703, C54 to C704, C55 to C705, C56 to C706, C57 to C707, C58 to C708, C59 to C709, D6 to D701, D7 to D702, D8 to D703, L2 to L701, R59 to R701, R60 to R702, R61 to R703, R62 to R704, R63 to R705, R64 to R706, U28 to U701, U29 to U702, U30 to U703

Commit message: Hardware design.
Parts:
- renumbered C701 to C71, C702 to C72, C703 to C73, C704 to C74, C705 to C75, C706 to C76, C707 to C77, C708 to C78, C709 to C79, D701 to D6, D702 to D7, D703 to D8, L701 to L2, R701 to R59, R702 to R60, R703 to R61, R704 to R62, R705 to R63, R706 to R64, U701 to U28, U702 to U29, U703 to U30

Commit message: Hardware design
Parts:
- L701: renamed from L2; footprint ETH1CLCR2:CW252016 -> ETH1CSMU2:CW252016
- U703: renamed from U30; symbol ETH1CLCR2:74AC125 -> ETH1CSMU2:74AC125
- renumbered C71 to C701, C72 to C702, C73 to C703, C74 to C704, C75 to C705, C76 to C706, C77 to C707, C78 to C708, C79 to C709, D6 to D701, D7 to D702, D8 to D703, R59 to R701, R60 to R702, R61 to R703, R62 to R704, R63 to R705, R64 to R706, U28 to U701, U29 to U702

Commit message: PCB layout
Connections:
- net +3V3 renamed +3.3V
