File: HARDWARE/ETH1CSMU2/Connect.kicad_sch (KiCad schematic)
At the start: 8 parts, among them J1 C64AC, K1 HE3621A0510, K2 HE3621A0510, K3 HE3621A0510, K4 HE3621A0510, K5 HE3621A0510, U4 ULN2003AS16

Commit message: Hardware design
Parts:
- J301: renamed from J1; footprint ETH1CSMU1:Socket_DIN41612-CaseC1-AC-Male-64Pin-2rows -> ETH1CSMU2:Socket_DIN41612-CaseC1-AC-Male-64Pin-2rows
- K301: renamed from K1; footprint ETH1CSMU1:HE360_x-5050462-8 -> ETH1CSMU2:HE360_x-5050462-8
- K302: renamed from K2; footprint ETH1CSMU1:HE360_x-5050462-8 -> ETH1CSMU2:HE360_x-5050462-8
- K303: renamed from K3; footprint ETH1CSMU1:HE360_x-5050462-8 -> ETH1CSMU2:HE360_x-5050462-8
- K304: renamed from K4; footprint ETH1CSMU1:HE360_x-5050462-8 -> ETH1CSMU2:HE360_x-5050462-8
- K305: renamed from K5; footprint ETH1CSMU1:HE360_x-5050462-8 -> ETH1CSMU2:HE360_x-5050462-8
- renumbered C15 to C301, U4 to U301
Changed lines of the file:
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@@
   (symbol (lib_id "ETH1CSMU2:HE3621A0510") (at 77.47 58.42 90) (unit 1)
     (in_bom yes) (on_board yes)
-    (property "Reference" "K4" (id 0) (at 77.47 52.959 90))
+    (property "Reference" "K304" (id 0) (at 77.47 52.959 90))
     (property "Value" "HE3621A0510" (id 1) (at 77.47 55.2704 90))
-    (property "Footprint" "ETH1CSMU1:HE360_x-5050462-8" (id 2) (at 78.74 52.07 0)
+    (property "Footprint" "ETH1CSMU2:HE360_x-5050462-8" (id 2) (at 78.74 52.07 0)
       (effects (font (size 1.27 1.27)) hide)
     )
@@
   (symbol (lib_id "power:+24V") (at 113.03 181.61 90) (unit 1)
     (in_bom yes) (on_board yes)
-    (property "Reference" "#PWR027" (id 0) (at 116.84 181.61 0)
+    (property "Reference" "#PWR0304" (id 0) (at 116.84 181.61 0)
       (effects (font (size 1.27 1.27)) hide)
     )
@@
   (symbol (lib_id "Transistor_Array:ULN2003A") (at 243.84 55.88 0) (mirror y) (unit 1)
     (in_bom yes) (on_board yes)
-    (property "Reference" "U4" (id 0) (at 243.84 38.9382 0))
+    (property "Reference" "U301" (id 0) (at 243.84 38.9382 0))
     (property "Value" "ULN2003AS16" (id 1) (at 243.84 41.2496 0))
     (property "Footprint" "Package_SO:TSSOP-16_4.4x5mm_P0.65mm" (id 2) (at 242.57 69.85 0)
@@
   (symbol (lib_id "ETH1CSMU2:HE3621A0510") (at 77.47 67.31 90) (unit 1)
     (in_bom yes) (on_board yes)
-    (property "Reference" "K5" (id 0) (at 77.47 61.849 90))
+    (property "Reference" "K305" (id 0) (at 77.47 61.849 90))
     (property "Value" "HE3621A0510" (id 1) (at 77.47 64.1604 90))
-    (property "Footprint" "ETH1CSMU1:HE360_x-5050462-8" (id 2) (at 78.74 60.96 0)
+    (property "Footprint" "ETH1CSMU2:HE360_x-5050462-8" (id 2) (at 78.74 60.96 0)
       (effects (font (size 1.27 1.27)) hide)
     )
@@
   (symbol (lib_id "ETH1CSMU2:HE3621A0510") (at 208.28 45.72 0) (unit 2)
     (in_bom yes) (on_board yes)
-    (property "Reference" "K5" (id 0) (at 210.2612 44.5516 0)
+    (property "Reference" "K305" (id 0) (at 210.2612 44.5516 0)
       (effects (font (size 1.27 1.27)) (justify left))
     )
@@
       (effects (font (size 1.27 1.27)) (justify left))
     )
-    (property "Footprint" "ETH1CSMU1:HE360_x-5050462-8" (id 2) (at 214.63 46.99 0)
+    (property "Footprint" "ETH1CSMU2:HE360_x-5050462-8" (id 2) (at 214.63 46.99 0)
       (effects (font (size 1.27 1.27)) hide)
     )
@@
   (symbol (lib_id "ETH1CSMU2:HE3621A0510") (at 77.47 40.64 90) (unit 1)
     (in_bom yes) (on_board yes)
-    (property "Reference" "K2" (id 0) (at 77.47 35.179 90))
+    (property "Reference" "K302" (id 0) (at 77.47 35.179 90))
     (property "Value" "HE3621A0510" (id 1) (at 77.47 37.4904 90))
-    (property "Footprint" "ETH1CSMU1:HE360_x-5050462-8" (id 2) (at 78.74 34.29 0)
+    (property "Footprint" "ETH1CSMU2:HE360_x-5050462-8" (id 2) (at 78.74 34.29 0)
       (effects (font (size 1.27 1.27)) hide)
     )
@@
   (symbol (lib_id "ETH1CSMU2:HE3621A0510") (at 77.47 49.53 90) (unit 1)
     (in_bom yes) (on_board yes)
-    (property "Reference" "K3" (id 0) (at 77.47 44.069 90))
+    (property "Reference" "K303" (id 0) (at 77.47 44.069 90))
     (property "Value" "HE3621A0510" (id 1) (at 77.47 46.3804 90))
-    (property "Footprint" "ETH1CSMU1:HE360_x-5050462-8" (id 2) (at 78.74 43.18 0)
+    (property "Footprint" "ETH1CSMU2:HE360_x-5050462-8" (id 2) (at 78.74 43.18 0)
       (effects (font (size 1.27 1.27)) hide)
     )
@@
   (symbol (lib_id "ETH1CSMU2:HE3621A0510") (at 172.72 45.72 0) (unit 2)
     (in_bom yes) (on_board yes)
-    (property "Reference" "K3" (id 0) (at 174.7012 44.5516 0)
+    (property "Reference" "K303" (id 0) (at 174.7012 44.5516 0)
       (effects (font (size 1.27 1.27)) (justify left))
     )
@@
       (effects (font (size 1.27 1.27)) (justify left))
     )
-    (property "Footprint" "ETH1CSMU1:HE360_x-5050462-8" (id 2) (at 179.07 46.99 0)
+    (property "Footprint" "ETH1CSMU2:HE360_x-5050462-8" (id 2) (at 179.07 46.99 0)
       (effects (font (size 1.27 1.27)) hide)
     )
@@
   (symbol (lib_id "power:+5V") (at 172.72 39.37 0) (unit 1)
     (in_bom yes) (on_board yes)
-    (property "Reference" "#PWR029" (id 0) (at 172.72 43.18 0)
+    (property "Reference" "#PWR0306" (id 0) (at 172.72 43.18 0)
       (effects (font (size 1.27 1.27)) hide)
     )
@@
   (symbol (lib_id "ETH1CSMU2:HE3621A0510") (at 137.16 45.72 0) (unit 2)
     (in_bom yes) (on_board yes)
-    (property "Reference" "K1" (id 0) (at 139.1412 44.5516 0)
+    (property "Reference" "K301" (id 0) (at 139.1412 44.5516 0)
       (effects (font (size 1.27 1.27)) (justify left))
     )
@@
       (effects (font (size 1.27 1.27)) (justify left))
     )
-    (property "Footprint" "ETH1CSMU1:HE360_x-5050462-8" (id 2) (at 143.51 46.99 0)
+    (property "Footprint" "ETH1CSMU2:HE360_x-5050462-8" (id 2) (at 143.51 46.99 0)
       (effects (font (size 1.27 1.27)) hide)
     )
@@
   (symbol (lib_id "power:GND") (at 243.84 71.12 0) (unit 1)
     (in_bom yes) (on_board yes)
-    (property "Reference" "#PWR031" (id 0) (at 243.84 77.47 0)
+    (property "Reference" "#PWR0308" (id 0) (at 243.84 77.47 0)
       (effects (font (size 1.27 1.27)) hide)
     )
@@
   (symbol (lib_id "power:GNDPWR") (at 113.03 161.29 270) (unit 1)
     (in_bom yes) (on_board yes)
-    (property "Reference" "#PWR026" (id 0) (at 107.95 161.29 0)
+    (property "Reference" "#PWR0303" (id 0) (at 107.95 161.29 0)
       (effects (font (size 1.27 1.27)) hide)
     )
@@
   (symbol (lib_id "power:Earth") (at 113.03 133.35 270) (unit 1)
     (in_bom yes) (on_board yes)
-    (property "Reference" "#PWR025" (id 0) (at 106.68 133.35 0)
+    (property "Reference" "#PWR0302" (id 0) (at 106.68 133.35 0)
       (effects (font (size 1.27 1.27)) hide)
     )
@@
   (symbol (lib_id "ETH1CSMU2:HE3621A0510") (at 190.5 45.72 0) (unit 2)
     (in_bom yes) (on_board yes)
-    (property "Reference" "K4" (id 0) (at 192.4812 44.5516 0)
+    (property "Reference" "K304" (id 0) (at 192.4812 44.5516 0)
       (effects (font (size 1.27 1.27)) (justify left))
     )
@@
       (effects (font (size 1.27 1.27)) (justify left))
     )
-    (property "Footprint" "ETH1CSMU1:HE360_x-5050462-8" (id 2) (at 196.85 46.99 0)
+    (property "Footprint" "ETH1CSMU2:HE360_x-5050462-8" (id 2) (at 196.85 46.99 0)
       (effects (font (size 1.27 1.27)) hide)
     )
@@
   (symbol (lib_id "power:Earth") (at 113.03 113.03 270) (unit 1)
     (in_bom yes) (on_board yes)
-    (property "Reference" "#PWR024" (id 0) (at 106.68 113.03 0)
+    (property "Reference" "#PWR0301" (id 0) (at 106.68 113.03 0)
       (effects (font (size 1.27 1.27)) hide)
     )
@@
   (symbol (lib_id "Device:C") (at 276.86 54.61 0) (unit 1)
     (in_bom yes) (on_board yes)
-    (property "Reference" "C15" (id 0) (at 279.781 53.4416 0)
+    (property "Reference" "C301" (id 0) (at 279.781 53.4416 0)
       (effects (font (size 1.27 1.27)) (justify left))
     )
@@
   (symbol (lib_id "power:GND") (at 276.86 58.42 0) (unit 1)
     (in_bom yes) (on_board yes)
-    (property "Reference" "#PWR033" (id 0) (at 276.86 64.77 0)
+    (property "Reference" "#PWR0310" (id 0) (at 276.86 64.77 0)
       (effects (font (size 1.27 1.27)) hide)
     )
@@
   (symbol (lib_id "ETH1CSMU2:GND_TRIG") (at 114.3 104.14 270) (unit 1)
     (in_bom yes) (on_board yes)
-    (property "Reference" "#PWR028" (id 0) (at 107.95 104.14 0)
+    (property "Reference" "#PWR0305" (id 0) (at 107.95 104.14 0)
       (effects (font (size 1.27 1.27)) hide)
     )
@@
   (symbol (lib_id "power:+5V") (at 233.68 45.72 90) (unit 1)
     (in_bom yes) (on_board yes)
-    (property "Reference" "#PWR030" (id 0) (at 237.49 45.72 0)
+    (property "Reference" "#PWR0307" (id 0) (at 237.49 45.72 0)
       (effects (font (size 1.27 1.27)) hide)
     )
@@
   (symbol (lib_id "Connector:C64AC") (at 123.19 106.68 0) (unit 1)
     (in_bom yes) (on_board yes)
-    (property "Reference" "J1" (id 0) (at 127.762 104.2416 0)
+    (property "Reference" "J301" (id 0) (at 127.762 104.2416 0)
       (effects (font (size 1.27 1.27)) (justify left))
     )
@@
       (effects (font (size 1.27 1.27)) (justify left))
     )
-    (property "Footprint" "ETH1CSMU1:Socket_DIN41612-CaseC1-AC-Male-64Pin-2rows" (id 2) (at 123.19 105.41 0)
+    (property "Footprint" "ETH1CSMU2:Socket_DIN41612-CaseC1-AC-Male-64Pin-2rows" (id 2) (at 123.19 105.41 0)
       (effects (font (size 1.27 1.27)) hide)
     )
@@
   (symbol (lib_id "power:+5V") (at 276.86 50.8 0) (unit 1)
     (in_bom yes) (on_board yes)
-    (property "Reference" "#PWR032" (id 0) (at 276.86 54.61 0)
+    (property "Reference" "#PWR0309" (id 0) (at 276.86 54.61 0)
       (effects (font (size 1.27 1.27)) hide)
     )
@@
   (symbol (lib_id "ETH1CSMU2:HE3621A0510") (at 154.94 45.72 0) (unit 2)
     (in_bom yes) (on_board yes)
-    (property "Reference" "K2" (id 0) (at 156.9212 44.5516 0)
+    (property "Reference" "K302" (id 0) (at 156.9212 44.5516 0)
       (effects (font (size 1.27 1.27)) (justify left))
     )
@@
       (effects (font (size 1.27 1.27)) (justify left))
     )
-    (property "Footprint" "ETH1CSMU1:HE360_x-5050462-8" (id 2) (at 161.29 46.99 0)
+    (property "Footprint" "ETH1CSMU2:HE360_x-5050462-8" (id 2) (at 161.29 46.99 0)
       (effects (font (size 1.27 1.27)) hide)
     )
@@
   (symbol (lib_id "ETH1CSMU2:HE3621A0510") (at 77.47 31.75 90) (unit 1)
     (in_bom yes) (on_board yes)
-    (property "Reference" "K1" (id 0) (at 77.47 26.289 90))
+    (property "Reference" "K301" (id 0) (at 77.47 26.289 90))
     (property "Value" "HE3621A0510" (id 1) (at 77.47 28.6004 90))
-    (property "Footprint" "ETH1CSMU1:HE360_x-5050462-8" (id 2) (at 78.74 25.4 0)
-      (effects (font (size 1.27 1.27)) hide)
-    )
+    (property "Footprint" "ETH1CSMU2:HE360_x-5050462-8" (id 2) (at 78.74 25.4 0)
+      (effects (font (size 1.27 1.27)) hide)
+    )

Commit message: CRC check
Connections:
- net VOUT_OUT: now reaches K301.1
Changed lines of the file:
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@@
     (effects (font (size 1.27 1.27)) (justify left))
+  )
+  (hierarchical_label "VOUT_OUT" (shape input) (at 66.04 31.75 180)
+    (effects (font (size 1.27 1.27)) (justify right))
   )
   (hierarchical_label "CXN_REL3" (shape input) (at 255.27 55.88 0)
@@
     (pin "2")
     (pin "3")
+  )
+  (symbol (lib_id "power:PWR_FLAG") (at 140.97 181.61 180) (unit 1)
+    (in_bom yes) (on_board yes) (fields_autoplaced)
+    (property "Reference" "#FLG0301" (id 0) (at 140.97 183.515 0)
+      (effects (font (size 1.27 1.27)) hide)
+    )
+    (property "Value" "PWR_FLAG" (id 1) (at 140.97 186.0534 0))
+    (property "Footprint" "" (id 2) (at 140.97 181.61 0)
+      (effects (font (size 1.27 1.27)) hide)
+    )
+    (property "Datasheet" "~" (id 3) (at 140.97 181.61 0)
+      (effects (font (size 1.27 1.27)) hide)
+    )
+    (pin "1")
   )
   (symbol (lib_id "power:+24V") (at 113.03 181.61 90) (unit 1)
@@
   (symbol (lib_id "power:+5V") (at 172.72 39.37 0) (unit 1)
     (in_bom yes) (on_board yes)
-    (property "Reference" "#PWR0306" (id 0) (at 172.72 43.18 0)
+    (property "Reference" "#PWR0307" (id 0) (at 172.72 43.18 0)
       (effects (font (size 1.27 1.27)) hide)
     )
@@
   (symbol (lib_id "power:GND") (at 243.84 71.12 0) (unit 1)
     (in_bom yes) (on_board yes)
-    (property "Reference" "#PWR0308" (id 0) (at 243.84 77.47 0)
+    (property "Reference" "#PWR0309" (id 0) (at 243.84 77.47 0)
       (effects (font (size 1.27 1.27)) hide)
     )
@@
   (symbol (lib_id "power:GND") (at 276.86 58.42 0) (unit 1)
     (in_bom yes) (on_board yes)
-    (property "Reference" "#PWR0310" (id 0) (at 276.86 64.77 0)
+    (property "Reference" "#PWR0311" (id 0) (at 276.86 64.77 0)
       (effects (font (size 1.27 1.27)) hide)
     )
@@
   (symbol (lib_id "power:+5V") (at 233.68 45.72 90) (unit 1)
     (in_bom yes) (on_board yes)
-    (property "Reference" "#PWR0307" (id 0) (at 237.49 45.72 0)
+    (property "Reference" "#PWR0308" (id 0) (at 237.49 45.72 0)
       (effects (font (size 1.27 1.27)) hide)
     )
@@
   (symbol (lib_id "power:+5V") (at 276.86 50.8 0) (unit 1)
     (in_bom yes) (on_board yes)
-    (property "Reference" "#PWR0309" (id 0) (at 276.86 54.61 0)
+    (property "Reference" "#PWR0310" (id 0) (at 276.86 54.61 0)
       (effects (font (size 1.27 1.27)) hide)
     )
@@
     (pin "3")
   )
+  (symbol (lib_id "power:+24V") (at 140.97 181.61 0) (unit 1)
+    (in_bom yes) (on_board yes) (fields_autoplaced)
+    (property "Reference" "#PWR0306" (id 0) (at 140.97 185.42 0)
+      (effects (font (size 1.27 1.27)) hide)
+    )
+    (property "Value" "+24V" (id 1) (at 140.97 178.0342 0))
+    (property "Footprint" "" (id 2) (at 140.97 181.61 0)
+      (effects (font (size 1.27 1.27)) hide)
+    )
+    (property "Datasheet" "" (id 3) (at 140.97 181.61 0)
+      (effects (font (size 1.27 1.27)) hide)
+    )
+    (pin "1")
+  )
 )

Commit message: Hardware design
Parts:
- added K304: HE3621A0510, ETH1CSMU2:HE360_x-5050462-8, symbol ETH1CSMU2:HE3621A0510
- renumbered K304 to K305, K305 to K306
Connections:
- net GNDPWR is gone; now on net GND: J301.A27 (27A), J301.A28 (28A), J301.C27 (27C), J301.C28 (28C)
- net +5V: now also K304.2
- net CXN_REL1: now also U301.6 (I6); no longer U301.5 (I5)
- net CXN_REL2: now also U301.5 (I5); no longer U301.4 (I4)
- net CXN_REL3: now also U301.4 (I4); no longer U301.3 (I3)
- net CXN_REL4: now also U301.3 (I3); no longer U301.2 (I2)
- net CXN_REL5: now also U301.2 (I2); no longer U301.1 (I1)
- net D: now also K304.4
- net GND: now also K302.1, K306.1
- net VOLT_MEAS_SENS: now reaches K305.1
- net at U301.11 (O6): now also K304.3
- net GUARD: now reaches K303.1
- net GUARD: now also K304.1
- new net CXN_REL6: U301.1 (I1)
- no-connect marks 38 -> 36
Other:
- moved on the sheet: J301, K301A, K302A, K303A, K305A, K306A

Commit message: Hardware design
Parts:
- U301: value ULN2003AS16 -> ULN2003AIDE4; footprint Package_SO:TSSOP-16_4.4x5mm_P0.65mm -> Package_SO:SOIC-16_3.9x9.9mm_P1.27mm
Changed lines of the file:
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@@
     (in_bom yes) (on_board yes)
     (property "Reference" "U301" (id 0) (at 243.84 38.9382 0))
-    (property "Value" "ULN2003AS16" (id 1) (at 243.84 41.2496 0))
-    (property "Footprint" "Package_SO:TSSOP-16_4.4x5mm_P0.65mm" (id 2) (at 242.57 69.85 0)
+    (property "Value" "ULN2003AIDE4" (id 1) (at 243.84 41.2496 0))
+    (property "Footprint" "Package_SO:SOIC-16_3.9x9.9mm_P1.27mm" (id 2) (at 242.57 69.85 0)
       (effects (font (size 1.27 1.27)) (justify left) hide)
     )
