File: HARDWARE/ETH1CSMU2/Ethernet.kicad_sch (KiCad schematic)
At the start: 43 parts, among them U201 LAN8742A, U202 LC03-3.3, U203 LC03-3.3, Y201 NX5032GA-25.000M-LN-CD-1

Commit message: Hardware design
Parts:
- Y201: value NX5032GA-25.000M-LN-CD-1 -> NX5032GA-25.000000MHZ-LN-CD-1
Other:
- moved on the sheet: C201, Y201
Changed lines of the file:
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@@
   (junction (at 185.42 26.67) (diameter 0) (color 0 0 0 0)
   )
-  (junction (at 27.94 120.65) (diameter 0) (color 0 0 0 0)
+  (junction (at 25.4 120.65) (diameter 0) (color 0 0 0 0)
   )
   (junction (at 152.4 76.2) (diameter 0) (color 0 0 0 0)
@@
     (stroke (width 0) (type default) (color 0 0 0 0))
   )
-  (wire (pts (xy 49.53 120.65) (xy 63.5 120.65))
+  (wire (pts (xy 48.26 120.65) (xy 63.5 120.65))
     (stroke (width 0) (type default) (color 0 0 0 0))
   )
@@
     (stroke (width 0) (type default) (color 0 0 0 0))
   )
-  (wire (pts (xy 27.94 129.54) (xy 27.94 130.81))
+  (wire (pts (xy 25.4 129.54) (xy 25.4 130.81))
     (stroke (width 0) (type default) (color 0 0 0 0))
   )
@@
     (stroke (width 0) (type default) (color 0 0 0 0))
   )
-  (wire (pts (xy 27.94 104.14) (xy 27.94 120.65))
+  (wire (pts (xy 25.4 104.14) (xy 25.4 120.65))
     (stroke (width 0) (type default) (color 0 0 0 0))
   )
@@
     (stroke (width 0) (type default) (color 0 0 0 0))
   )
-  (wire (pts (xy 27.94 121.92) (xy 27.94 120.65))
+  (wire (pts (xy 25.4 121.92) (xy 25.4 120.65))
     (stroke (width 0) (type default) (color 0 0 0 0))
   )
@@
     (stroke (width 0) (type default) (color 0 0 0 0))
   )
-  (wire (pts (xy 27.94 120.65) (xy 41.91 120.65))
+  (wire (pts (xy 25.4 120.65) (xy 40.64 120.65))
     (stroke (width 0) (type default) (color 0 0 0 0))
   )
@@
     (stroke (width 0) (type default) (color 0 0 0 0))
   )
-  (wire (pts (xy 66.04 104.14) (xy 27.94 104.14))
+  (wire (pts (xy 66.04 104.14) (xy 25.4 104.14))
     (stroke (width 0) (type default) (color 0 0 0 0))
   )
@@
     (pin "1")
   )
-  (symbol (lib_id "Device:C") (at 27.94 125.73 0) (unit 1)
-    (in_bom yes) (on_board yes)
-    (property "Reference" "C201" (id 0) (at 30.861 124.5616 0)
-      (effects (font (size 1.27 1.27)) (justify left))
-    )
-    (property "Value" "8p" (id 1) (at 30.861 126.873 0)
-      (effects (font (size 1.27 1.27)) (justify left))
-    )
-    (property "Footprint" "" (id 2) (at 28.9052 129.54 0)
-      (effects (font (size 1.27 1.27)) hide)
-    )
-    (property "Datasheet" "~" (id 3) (at 27.94 125.73 0)
+  (symbol (lib_id "Device:C") (at 25.4 125.73 0) (unit 1)
+    (in_bom yes) (on_board yes)
+    (property "Reference" "C201" (id 0) (at 28.321 124.5616 0)
+      (effects (font (size 1.27 1.27)) (justify left))
+    )
+    (property "Value" "8p" (id 1) (at 28.321 126.873 0)
+      (effects (font (size 1.27 1.27)) (justify left))
+    )
+    (property "Footprint" "" (id 2) (at 26.3652 129.54 0)
+      (effects (font (size 1.27 1.27)) hide)
+    )
+    (property "Datasheet" "~" (id 3) (at 25.4 125.73 0)
       (effects (font (size 1.27 1.27)) hide)
     )
@@
     (pin "1")
   )
-  (symbol (lib_id "Device:Crystal") (at 45.72 120.65 180) (unit 1)
-    (in_bom yes) (on_board yes)
-    (property "Reference" "Y201" (id 0) (at 45.72 113.8428 0))
-    (property "Value" "NX5032GA-25.000M-LN-CD-1" (id 1) (at 45.72 116.1542 0))
-    (property "Footprint" "" (id 2) (at 45.72 120.65 0)
-      (effects (font (size 1.27 1.27)) hide)
-    )
-    (property "Datasheet" "~" (id 3) (at 45.72 120.65 0)
-      (effects (font (size 1.27 1.27)) hide)
-    )
-    (pin "1")
-    (pin "2")
-  )
-  (symbol (lib_id "power:GND") (at 27.94 130.81 0) (unit 1)
-    (in_bom yes) (on_board yes)
-    (property "Reference" "#PWR0202" (id 0) (at 27.94 137.16 0)
-      (effects (font (size 1.27 1.27)) hide)
-    )
-    (property "Value" "GND" (id 1) (at 28.067 135.2042 0))
-    (property "Footprint" "" (id 2) (at 27.94 130.81 0)
-      (effects (font (size 1.27 1.27)) hide)
-    )
-    (property "Datasheet" "" (id 3) (at 27.94 130.81 0)
-      (effects (font (size 1.27 1.27)) hide)
-    )
+  (symbol (lib_id "Device:Crystal") (at 44.45 120.65 180) (unit 1)
+    (in_bom yes) (on_board yes)
+    (property "Reference" "Y201" (id 0) (at 44.45 113.8428 0))
+    (property "Value" "NX5032GA-25.000000MHZ-LN-CD-1" (id 1) (at 44.45 116.1542 0))
+    (property "Footprint" "" (id 2) (at 44.45 120.65 0)
+      (effects (font (size 1.27 1.27)) hide)
+    )
+    (property "Datasheet" "~" (id 3) (at 44.45 120.65 0)
+      (effects (font (size 1.27 1.27)) hide)
+    )
+    (pin "1")
+    (pin "2")
+  )
+  (symbol (lib_id "power:GND") (at 25.4 130.81 0) (unit 1)
+    (in_bom yes) (on_board yes)
+    (property "Reference" "#PWR0202" (id 0) (at 25.4 137.16 0)
+      (effects (font (size 1.27 1.27)) hide)
+    )
+    (property "Value" "GND" (id 1) (at 25.527 135.2042 0))
+    (property "Footprint" "" (id 2) (at 25.4 130.81 0)
+      (effects (font (size 1.27 1.27)) hide)
+    )
+    (property "Datasheet" "" (id 3) (at 25.4 130.81 0)
+      (effects (font (size 1.27 1.27)) hide)
+    )

Commit message: Hardware design
Parts:
- renumbered C201 to C1, C210 to C10, C211 to C11, C212 to C12, C213 to C13, C214 to C14, C202 to C2, C203 to C3, C204 to C4, C205 to C5, C206 to C6, C207 to C7, C208 to C8, C209 to C9, D201 to D1, D202 to D2, FB201 to FB1, L201 to L1, R201 to R1, R210 to R10, R211 to R11, R212 to R12, R213 to R13, R214 to R14, R215 to R15, R216 to R16, R217 to R17, R218 to R18, R219 to R19, R202 to R2, R220 to R20, R221 to R21, R203 to R3, R204 to R4, R205 to R5, R206 to R6, R207 to R7, R208 to R8, R209 to R9, U201 to U1, U202 to U2, U203 to U3, Y201 to Y1

Commit message: Hardware design
Parts:
- renumbered C1 to C201, C2 to C202, C3 to C203, C4 to C204, C5 to C205, C6 to C206, C7 to C207, C8 to C208, C9 to C209, C10 to C210, C11 to C211, C12 to C212, C13 to C213, C14 to C214, D1 to D201, D2 to D202, FB1 to FB201, L1 to L201, R1 to R201, R2 to R202, R3 to R203, R4 to R204, R5 to R205, R6 to R206, R7 to R207, R8 to R208, R9 to R209, R10 to R210, R11 to R211, R12 to R212, R13 to R213, R14 to R214, R15 to R215, R16 to R216, R17 to R217, R18 to R218, R19 to R219, R20 to R220, R21 to R221, U1 to U201, U2 to U202, U3 to U203, Y1 to Y201
