File: HARDWARE/ETH1CSMU2/Ethernet.kicad_sch (KiCad schematic)
At the start: 43 parts, among them U1 LAN8742A, U2 LC03-3.3, U3 LC03-3.3, Y1 NX5032GA-25.000000MHZ-LN-CD-1

Commit message: Hardware design
Parts:
- renumbered C1 to C201, C2 to C202, C3 to C203, C4 to C204, C5 to C205, C6 to C206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

Commit message: CRC check
Connections:
- net RMII_MDIO: no longer R210.2
- new net MDIO: R210.2
