File: HARDWARE/ETH1CSMU2/ETH1CSMU2.kicad_sch (KiCad schematic)
At the start: 0 parts

Commit message: Hardware design
Other:
- removed sheet VREF
- added sheet MCU (MCU.kicad_sch)
- added sheet Power (Power.kicad_sch)
- added sheet Source (Source.kicad_sch)
- added sheet Trigger (Trigger.kicad_sch)
- sheet Connect ports: added CXN_REL1, CXN_REL2, CXN_REL3, CXN_REL4, CXN_REL5, EXT_TRIG, RX+, RX-, TX+, TX-; removed none
- sheet Frontend ports: added none; removed VOLT_MEAS

Commit message: Hardware design
Other:
- sheet Frontend ports: added CURR_MEAS, VOLT_MEAS; removed none

Commit message: Hardware design
Other:
- sheet Control ports: added SING_SEL, VMEAS_SEL; removed none
- sheet Frontend ports: added FGEN, SING_SEL; removed none

Commit message: Hardware design
Other:
- sheet Control ports: added ATT_A0, ATT_A1, DDS_LPF; removed none
- sheet MCU ports: added CXN_REL1, CXN_REL2, CXN_REL3, CXN_REL4, CXN_REL5, NRST, REF_CLK, RMII_CRS_DV, RMII_MDC, RMII_MDIO, RMII_RXD0, RMII_RXD1, RMII_TXD0, RMII_TXD1, RMII_TXEN, TRIG_EN, TRIG_IN, TRIG_OUT; removed none
- sheet Source ports: added ATT_A0, ATT_A1, DDS_LPF, FGEN; removed none

Commit message: Schematic
Other:
- sheet Measure ports: added VMEAS_SEL, VOLT_MEAS_SENS; removed none
- sheet Source ports: added DAC1_DIN, DAC1_LDAC, DAC1_SCLK, DAC1_~{RST}, DAC1_~{SYNC}, DAC2_DIN, DAC2_SCLK, DAC2_~{LDAC}, DAC2_~{SYNC}, DDS_CS, DDS_SCLK, DDS_SDATA; removed DAC_DIN, DAC_LDAC, DAC_SCLK, DAC_~{RST}, DAC_~{SYNC}
