File: HARDWARE/ETH1CSMU2/ETH1CSMU2.kicad_sch (KiCad schematic)
At the start: 0 parts

Commit message: Hardware design
Other:
- sheet Source ports: added DDS_DIV2, DDS_DIV4, DDS_DIV8, ~{DDS_DIV10}; removed none

Commit message: Hardware design
Other:
- sheet Control ports: added ADC_SEL; removed none
- sheet Measure ports: added ADC1_MISO, ADC1_MOSI, ADC1_RVS1, ADC1_RVS2, ADC1_SCLK, ADC1_~{CS}, ADC2_CNV, ADC2_MISO, ADC2_SCLK, ADC_SEL; removed ADC_HS_MISO, ADC_HS_MOSI, ADC_HS_RVS1, ADC_HS_RVS2, ADC_HS_SCLK, ADC_HS_~{CS}

Commit message: Hardware and software development
Connections:
- no-connect marks 0 -> 2
Other:
- sheet Control ports: added SR_CLK, SR_DAT, SR_LAT, SR_OUT; removed GPIO_SPI_MISO, GPIO_SPI_MOSI, GPIO_SPI_NSS, GPIO_SPI_SCK
- sheet MCU ports: added ADC1_RVS1, ADC1_RVS2, DDS_DIV2, DDS_DIV4, DDS_DIV8, MCU_nISNK, MCU_nISRC, MCU_nTDS, SPI1_MISO, SPI1_MOSI, SPI1_NSS, SPI1_SCK, SPI2_MISO, SPI2_MOSI, SPI2_NSS, SPI2_SCK, SPI3_MISO, SPI3_MOSI, SPI3_NSS, SPI3_SCK, SPI4_MISO, SPI4_MOSI, SPI4_NSS, SPI4_SCK, SPI5_MISO, SPI5_MOSI, SPI5_NSS, SPI5_SCK, SR_CLK, SR_DAT, SR_LAT, SR_OUT, ~{DDS_DIV10}; removed none

Commit message: CRC check
Connections:
- no-connect marks 2 -> 4
Other:
- sheet Connect ports: added VOUT_OUT; removed none
- sheet MCU ports: added DAC1_LDAC, DAC1_~{RST}, DAC2_~{LDAC}; removed none

Commit message: Hardware design.
Other:
- sheet Frontend ports: added MCU_CURR_SENS_100R, MCU_CURR_SENS_10R, MCU_CURR_SENS_1R; removed none
- sheet MCU ports: added MCU_CURR_SENS_100R, MCU_CURR_SENS_10R, MCU_CURR_SENS_1R; removed none

Commit message: Hardware design
Other:
- sheet Frontend ports: added MCU_CURR_SENS_1kR; removed none
- sheet MCU ports: added MCU_CURR_SENS_1kR; removed none

Commit message: Hardware design
Other:
- sheet Connect ports: added CXN_REL6, GUARD, VOLT_MEAS_SENS; removed none
- sheet Frontend ports: added GUARD; removed none
- sheet MCU ports: added CXN_REL6; removed none

Commit message: Hardware design
Other:
- sheet Frontend ports: added VOUT_OFFSET; removed none
- sheet MCU ports: added DAC_OFFS_SCL, DAC_OFFS_SDA; removed none
- sheet Source ports: added DAC_OFFS_SCL, DAC_OFFS_SDA, VOUT_OFFSET; removed none
