File: HARDWARE/ETH1CSMU2/Control.kicad_sch (KiCad schematic)
At the start: 7 parts, among them U15 74HCT595, U16 74HCT595, U17 SN74LVC1T45DPKR, U18 SN74LVC1T45DPKR, U19 SN74LVC1T45DPKR, U20 SN74LVC1T45DPKR

Commit message: Hardware design
Connections:
- net SING_SEL: now reaches U16.2 (QC)
Changed lines of the file:
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@@
+    (effects (font (size 1.27 1.27)) (justify right))
+  )
+  (hierarchical_label "SING_SEL" (shape output) (at 78.74 90.17 180)
     (effects (font (size 1.27 1.27)) (justify right))
   )
@@
   (symbol (lib_id "power:+5V") (at 100.33 44.45 270) (unit 1)
     (in_bom yes) (on_board yes)
-    (property "Reference" "#PWR095" (id 0) (at 96.52 44.45 0)
+    (property "Reference" "#PWR099" (id 0) (at 96.52 44.45 0)
       (effects (font (size 1.27 1.27)) hide)
     )
@@
   (symbol (lib_id "power:+5V") (at 100.33 92.71 270) (unit 1)
     (in_bom yes) (on_board yes)
-    (property "Reference" "#PWR097" (id 0) (at 96.52 92.71 0)
+    (property "Reference" "#PWR0101" (id 0) (at 96.52 92.71 0)
       (effects (font (size 1.27 1.27)) hide)
     )
@@
   (symbol (lib_id "power:+3.3V") (at 157.48 95.25 0) (unit 1)
     (in_bom yes) (on_board yes)
-    (property "Reference" "#PWR0110" (id 0) (at 157.48 99.06 0)
+    (property "Reference" "#PWR0114" (id 0) (at 157.48 99.06 0)
       (effects (font (size 1.27 1.27)) hide)
     )
@@
   (symbol (lib_id "power:+5V") (at 152.4 95.25 0) (unit 1)
     (in_bom yes) (on_board yes)
-    (property "Reference" "#PWR0102" (id 0) (at 152.4 99.06 0)
+    (property "Reference" "#PWR0106" (id 0) (at 152.4 99.06 0)
       (effects (font (size 1.27 1.27)) hide)
     )
@@
   (symbol (lib_id "power:GND") (at 90.17 64.77 0) (unit 1)
     (in_bom yes) (on_board yes)
-    (property "Reference" "#PWR092" (id 0) (at 90.17 71.12 0)
+    (property "Reference" "#PWR096" (id 0) (at 90.17 71.12 0)
       (effects (font (size 1.27 1.27)) hide)
     )
@@
   (symbol (lib_id "power:GND") (at 90.17 113.03 0) (unit 1)
     (in_bom yes) (on_board yes)
-    (property "Reference" "#PWR094" (id 0) (at 90.17 119.38 0)
+    (property "Reference" "#PWR098" (id 0) (at 90.17 119.38 0)
       (effects (font (size 1.27 1.27)) hide)
     )
@@
   (symbol (lib_id "power:+5V") (at 152.4 26.67 0) (unit 1)
     (in_bom yes) (on_board yes)
-    (property "Reference" "#PWR0100" (id 0) (at 152.4 30.48 0)
+    (property "Reference" "#PWR0104" (id 0) (at 152.4 30.48 0)
       (effects (font (size 1.27 1.27)) hide)
     )
@@
   (symbol (lib_id "power:+5V") (at 152.4 129.54 0) (unit 1)
     (in_bom yes) (on_board yes)
-    (property "Reference" "#PWR0103" (id 0) (at 152.4 133.35 0)
+    (property "Reference" "#PWR0107" (id 0) (at 152.4 133.35 0)
       (effects (font (size 1.27 1.27)) hide)
     )
@@
   (symbol (lib_id "power:GND") (at 154.94 83.82 0) (unit 1)
     (in_bom yes) (on_board yes)
-    (property "Reference" "#PWR0105" (id 0) (at 154.94 90.17 0)
+    (property "Reference" "#PWR0109" (id 0) (at 154.94 90.17 0)
       (effects (font (size 1.27 1.27)) hide)
     )
@@
   (symbol (lib_id "power:GND") (at 100.33 100.33 90) (unit 1)
     (in_bom yes) (on_board yes)
-    (property "Reference" "#PWR098" (id 0) (at 106.68 100.33 0)
+    (property "Reference" "#PWR0102" (id 0) (at 106.68 100.33 0)
       (effects (font (size 1.27 1.27)) hide)
     )
@@
   (symbol (lib_id "power:+3.3V") (at 157.48 26.67 0) (unit 1)
     (in_bom yes) (on_board yes)
-    (property "Reference" "#PWR0108" (id 0) (at 157.48 30.48 0)
+    (property "Reference" "#PWR0112" (id 0) (at 157.48 30.48 0)
       (effects (font (size 1.27 1.27)) hide)
     )
@@
   (symbol (lib_id "power:+5V") (at 90.17 80.01 0) (unit 1)
     (in_bom yes) (on_board yes)
-    (property "Reference" "#PWR093" (id 0) (at 90.17 83.82 0)
+    (property "Reference" "#PWR097" (id 0) (at 90.17 83.82 0)
       (effects (font (size 1.27 1.27)) hide)
     )
@@
   (symbol (lib_id "power:+5V") (at 152.4 60.96 0) (unit 1)
     (in_bom yes) (on_board yes)
-    (property "Reference" "#PWR0101" (id 0) (at 152.4 64.77 0)
+    (property "Reference" "#PWR0105" (id 0) (at 152.4 64.77 0)
       (effects (font (size 1.27 1.27)) hide)
     )
@@
   (symbol (lib_id "power:GND") (at 154.94 118.11 0) (unit 1)
     (in_bom yes) (on_board yes)
-    (property "Reference" "#PWR0106" (id 0) (at 154.94 124.46 0)
+    (property "Reference" "#PWR0110" (id 0) (at 154.94 124.46 0)
       (effects (font (size 1.27 1.27)) hide)
     )
@@
   (symbol (lib_id "power:+5V") (at 135.89 144.78 90) (unit 1)
     (in_bom yes) (on_board yes)
-    (property "Reference" "#PWR099" (id 0) (at 139.7 144.78 0)
+    (property "Reference" "#PWR0103" (id 0) (at 139.7 144.78 0)
       (effects (font (size 1.27 1.27)) hide)
     )
@@
   (symbol (lib_id "power:+5V") (at 90.17 31.75 0) (unit 1)
     (in_bom yes) (on_board yes)
-    (property "Reference" "#PWR091" (id 0) (at 90.17 35.56 0)
+    (property "Reference" "#PWR095" (id 0) (at 90.17 35.56 0)
       (effects (font (size 1.27 1.27)) hide)
     )
@@
   (symbol (lib_id "power:+3.3V") (at 157.48 60.96 0) (unit 1)
     (in_bom yes) (on_board yes)
-    (property "Reference" "#PWR0109" (id 0) (at 157.48 64.77 0)
+    (property "Reference" "#PWR0113" (id 0) (at 157.48 64.77 0)
       (effects (font (size 1.27 1.27)) hide)
     )
@@
   (symbol (lib_id "power:GND") (at 100.33 52.07 90) (unit 1)
     (in_bom yes) (on_board yes)
-    (property "Reference" "#PWR096" (id 0) (at 106.68 52.07 0)
+    (property "Reference" "#PWR0100" (id 0) (at 106.68 52.07 0)
       (effects (font (size 1.27 1.27)) hide)
     )
@@
   (symbol (lib_id "power:GND") (at 154.94 152.4 0) (unit 1)
     (in_bom yes) (on_board yes)
-    (property "Reference" "#PWR0107" (id 0) (at 154.94 158.75 0)
+    (property "Reference" "#PWR0111" (id 0) (at 154.94 158.75 0)
       (effects (font (size 1.27 1.27)) hide)
     )
@@
   (symbol (lib_id "power:GND") (at 154.94 49.53 0) (unit 1)
     (in_bom yes) (on_board yes)
-    (property "Reference" "#PWR0104" (id 0) (at 154.94 55.88 0)
+    (property "Reference" "#PWR0108" (id 0) (at 154.94 55.88 0)
       (effects (font (size 1.27 1.27)) hide)
     )
@@
   (symbol (lib_id "power:+3.3V") (at 157.48 129.54 0) (unit 1)
     (in_bom yes) (on_board yes)
-    (property "Reference" "#PWR0111" (id 0) (at 157.48 133.35 0)
-      (effects (font (size 1.27 1.27)) hide)
-    )
+    (property "Reference" "#PWR0115" (id 0) (at 157.48 133.35 0)
+      (effects (font (size 1.27 1.27)) hide)
+    )

Commit message: Hardware design
Parts:
- renumbered R43 to R501, U15 to U501, U16 to U502, U17 to U503, U18 to U504, U19 to U505, U20 to U506
Connections:
- net ATT_A0: now reaches U502.3 (QD)
- net ATT_A1: now reaches U502.4 (QE)
- net DDS_LPF: now reaches U502.5 (QF)
Changed lines of the file:
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@@
     (stroke (width 0) (type default) (color 0 0 0 0))
+  )
+  (hierarchical_label "ATT_A1" (shape output) (at 78.74 95.25 180)
+    (effects (font (size 1.27 1.27)) (justify right))
   )
   (hierarchical_label "VMEAS_SEL" (shape output) (at 78.74 87.63 180)
@@
     (effects (font (size 1.27 1.27)) (justify right))
   )
+  (hierarchical_label "ATT_A0" (shape output) (at 78.74 92.71 180)
+    (effects (font (size 1.27 1.27)) (justify right))
+  )
   (hierarchical_label "V_AZ" (shape output) (at 78.74 44.45 180)
+    (effects (font (size 1.27 1.27)) (justify right))
+  )
+  (hierarchical_label "DDS_LPF" (shape output) (at 78.74 97.79 180)
     (effects (font (size 1.27 1.27)) (justify right))
   )
@@
   (symbol (lib_id "power:+5V") (at 100.33 44.45 270) (unit 1)
     (in_bom yes) (on_board yes)
-    (property "Reference" "#PWR099" (id 0) (at 96.52 44.45 0)
+    (property "Reference" "#PWR0505" (id 0) (at 96.52 44.45 0)
       (effects (font (size 1.27 1.27)) hide)
     )
@@
   (symbol (lib_id "power:+5V") (at 100.33 92.71 270) (unit 1)
     (in_bom yes) (on_board yes)
-    (property "Reference" "#PWR0101" (id 0) (at 96.52 92.71 0)
+    (property "Reference" "#PWR0507" (id 0) (at 96.52 92.71 0)
       (effects (font (size 1.27 1.27)) hide)
     )
@@
   (symbol (lib_id "power:+3.3V") (at 157.48 95.25 0) (unit 1)
     (in_bom yes) (on_board yes)
-    (property "Reference" "#PWR0114" (id 0) (at 157.48 99.06 0)
+    (property "Reference" "#PWR0520" (id 0) (at 157.48 99.06 0)
       (effects (font (size 1.27 1.27)) hide)
     )
@@
   (symbol (lib_id "Logic_LevelTranslator:SN74LVC1T45DBV") (at 154.94 139.7 0) (unit 1)
     (in_bom yes) (on_board yes)
-    (property "Reference" "U20" (id 0) (at 167.64 128.27 0)
+    (property "Reference" "U506" (id 0) (at 167.64 128.27 0)
       (effects (font (size 1.27 1.27)) (justify left))
     )
@@
   (symbol (lib_id "power:+5V") (at 152.4 95.25 0) (unit 1)
     (in_bom yes) (on_board yes)
-    (property "Reference" "#PWR0106" (id 0) (at 152.4 99.06 0)
+    (property "Reference" "#PWR0512" (id 0) (at 152.4 99.06 0)
       (effects (font (size 1.27 1.27)) hide)
     )
@@
   (symbol (lib_id "power:GND") (at 90.17 64.77 0) (unit 1)
     (in_bom yes) (on_board yes)
-    (property "Reference" "#PWR096" (id 0) (at 90.17 71.12 0)
+    (property "Reference" "#PWR0502" (id 0) (at 90.17 71.12 0)
       (effects (font (size 1.27 1.27)) hide)
     )
@@
   (symbol (lib_id "74xx:74HCT595") (at 90.17 46.99 0) (mirror y) (unit 1)
     (in_bom yes) (on_board yes)
-    (property "Reference" "U15" (id 0) (at 96.52 30.48 0))
+    (property "Reference" "U501" (id 0) (at 96.52 30.48 0))
     (property "Value" "74HCT595" (id 1) (at 96.52 33.02 0))
     (property "Footprint" "Package_SO:TSSOP-16_4.4x5mm_P0.65mm" (id 2) (at 90.17 46.99 0)
@@
   (symbol (lib_id "power:GND") (at 90.17 113.03 0) (unit 1)
     (in_bom yes) (on_board yes)
-    (property "Reference" "#PWR098" (id 0) (at 90.17 119.38 0)
+    (property "Reference" "#PWR0504" (id 0) (at 90.17 119.38 0)
       (effects (font (size 1.27 1.27)) hide)
     )
@@
   (symbol (lib_id "power:+5V") (at 152.4 26.67 0) (unit 1)
     (in_bom yes) (on_board yes)
-    (property "Reference" "#PWR0104" (id 0) (at 152.4 30.48 0)
+    (property "Reference" "#PWR0510" (id 0) (at 152.4 30.48 0)
       (effects (font (size 1.27 1.27)) hide)
     )
@@
   (symbol (lib_id "power:+5V") (at 152.4 129.54 0) (unit 1)
     (in_bom yes) (on_board yes)
-    (property "Reference" "#PWR0107" (id 0) (at 152.4 133.35 0)
+    (property "Reference" "#PWR0513" (id 0) (at 152.4 133.35 0)
       (effects (font (size 1.27 1.27)) hide)
     )
@@
   (symbol (lib_id "power:GND") (at 154.94 83.82 0) (unit 1)
     (in_bom yes) (on_board yes)
-    (property "Reference" "#PWR0109" (id 0) (at 154.94 90.17 0)
+    (property "Reference" "#PWR0515" (id 0) (at 154.94 90.17 0)
       (effects (font (size 1.27 1.27)) hide)
     )
@@
   (symbol (lib_id "power:GND") (at 100.33 100.33 90) (unit 1)
     (in_bom yes) (on_board yes)
-    (property "Reference" "#PWR0102" (id 0) (at 106.68 100.33 0)
+    (property "Reference" "#PWR0508" (id 0) (at 106.68 100.33 0)
       (effects (font (size 1.27 1.27)) hide)
     )
@@
   (symbol (lib_id "power:+3.3V") (at 157.48 26.67 0) (unit 1)
     (in_bom yes) (on_board yes)
-    (property "Reference" "#PWR0112" (id 0) (at 157.48 30.48 0)
+    (property "Reference" "#PWR0518" (id 0) (at 157.48 30.48 0)
       (effects (font (size 1.27 1.27)) hide)
     )
@@
   (symbol (lib_id "Logic_LevelTranslator:SN74LVC1T45DBV") (at 154.94 36.83 0) (unit 1)
     (in_bom yes) (on_board yes)
-    (property "Reference" "U17" (id 0) (at 167.64 25.4 0)
+    (property "Reference" "U503" (id 0) (at 167.64 25.4 0)
       (effects (font (size 1.27 1.27)) (justify left))
     )
@@
   (symbol (lib_id "power:+5V") (at 90.17 80.01 0) (unit 1)
     (in_bom yes) (on_board yes)
-    (property "Reference" "#PWR097" (id 0) (at 90.17 83.82 0)
+    (property "Reference" "#PWR0503" (id 0) (at 90.17 83.82 0)
       (effects (font (size 1.27 1.27)) hide)
     )
@@
   (symbol (lib_id "power:+5V") (at 152.4 60.96 0) (unit 1)
     (in_bom yes) (on_board yes)
-    (property "Reference" "#PWR0105" (id 0) (at 152.4 64.77 0)
+    (property "Reference" "#PWR0511" (id 0) (at 152.4 64.77 0)
       (effects (font (size 1.27 1.27)) hide)
     )
@@
   (symbol (lib_id "power:GND") (at 154.94 118.11 0) (unit 1)
     (in_bom yes) (on_board yes)
-    (property "Reference" "#PWR0110" (id 0) (at 154.94 124.46 0)
+    (property "Reference" "#PWR0516" (id 0) (at 154.94 124.46 0)
       (effects (font (size 1.27 1.27)) hide)
     )
@@
   (symbol (lib_id "power:+5V") (at 135.89 144.78 90) (unit 1)
     (in_bom yes) (on_board yes)
-    (property "Reference" "#PWR0103" (id 0) (at 139.7 144.78 0)
+    (property "Reference" "#PWR0509" (id 0) (at 139.7 144.78 0)
       (effects (font (size 1.27 1.27)) hide)
     )
@@
   (symbol (lib_id "power:+5V") (at 90.17 31.75 0) (unit 1)
     (in_bom yes) (on_board yes)
-    (property "Reference" "#PWR095" (id 0) (at 90.17 35.56 0)
+    (property "Reference" "#PWR0501" (id 0) (at 90.17 35.56 0)
       (effects (font (size 1.27 1.27)) hide)
     )
@@
   (symbol (lib_id "power:+3.3V") (at 157.48 60.96 0) (unit 1)
     (in_bom yes) (on_board yes)
-    (property "Reference" "#PWR0113" (id 0) (at 157.48 64.77 0)
+    (property "Reference" "#PWR0519" (id 0) (at 157.48 64.77 0)
       (effects (font (size 1.27 1.27)) hide)
     )
@@
   (symbol (lib_id "Device:R") (at 139.7 144.78 270) (unit 1)
     (in_bom yes) (on_board yes)
-    (property "Reference" "R43" (id 0) (at 139.7 142.24 90))
+    (property "Reference" "R501" (id 0) (at 139.7 142.24 90))
     (property "Value" "1k" (id 1) (at 139.7 144.78 90))
     (property "Footprint" "Resistor_SMD:R_0603_1608Metric_Pad0.98x0.95mm_HandSolder" (id 2) (at 139.7 143.002 90)
@@
   (symbol (lib_id "Logic_LevelTranslator:SN74LVC1T45DBV") (at 154.94 105.41 0) (unit 1)
     (in_bom yes) (on_board yes)
-    (property "Reference" "U19" (id 0) (at 167.64 93.98 0)
+    (property "Reference" "U505" (id 0) (at 167.64 93.98 0)
       (effects (font (size 1.27 1.27)) (justify left))
     )
@@
   (symbol (lib_id "power:GND") (at 100.33 52.07 90) (unit 1)
     (in_bom yes) (on_board yes)
-    (property "Reference" "#PWR0100" (id 0) (at 106.68 52.07 0)
+    (property "Reference" "#PWR0506" (id 0) (at 106.68 52.07 0)
       (effects (font (size 1.27 1.27)) hide)
     )
@@
   (symbol (lib_id "Logic_LevelTranslator:SN74LVC1T45DBV") (at 154.94 71.12 0) (unit 1)
     (in_bom yes) (on_board yes)
-    (property "Reference" "U18" (id 0) (at 167.64 59.69 0)
+    (property "Reference" "U504" (id 0) (at 167.64 59.69 0)
       (effects (font (size 1.27 1.27)) (justify left))
     )
@@
   (symbol (lib_id "power:GND") (at 154.94 152.4 0) (unit 1)
     (in_bom yes) (on_board yes)
-    (property "Reference" "#PWR0111" (id 0) (at 154.94 158.75 0)
+    (property "Reference" "#PWR0517" (id 0) (at 154.94 158.75 0)
       (effects (font (size 1.27 1.27)) hide)
     )
@@
   (symbol (lib_id "power:GND") (at 154.94 49.53 0) (unit 1)
     (in_bom yes) (on_board yes)
-    (property "Reference" "#PWR0108" (id 0) (at 154.94 55.88 0)
+    (property "Reference" "#PWR0514" (id 0) (at 154.94 55.88 0)
       (effects (font (size 1.27 1.27)) hide)
     )
@@
   (symbol (lib_id "74xx:74HCT595") (at 90.17 95.25 0) (mirror y) (unit 1)
     (in_bom yes) (on_board yes)
-    (property "Reference" "U16" (id 0) (at 96.52 78.74 0))
+    (property "Reference" "U502" (id 0) (at 96.52 78.74 0))
     (property "Value" "74HCT595" (id 1) (at 96.52 81.28 0))
     (property "Footprint" "Package_SO:TSSOP-16_4.4x5mm_P0.65mm" (id 2) (at 90.17 95.25 0)
@@
   (symbol (lib_id "power:+3.3V") (at 157.48 129.54 0) (unit 1)
     (in_bom yes) (on_board yes)
-    (property "Reference" "#PWR0115" (id 0) (at 157.48 133.35 0)
-      (effects (font (size 1.27 1.27)) hide)
-    )
+    (property "Reference" "#PWR0521" (id 0) (at 157.48 133.35 0)
+      (effects (font (size 1.27 1.27)) hide)
+    )

Commit message: Hardware design.
Parts:
- added C45, C46, C47, C48, C49, C50, C51, C52, C53, C54: 100n, symbol Device:C
- U15: renamed from U501; value 74HCT595 -> 74HCT595PW
- U16: renamed from U502; value 74HCT595 -> 74HCT595PW
- renumbered R501 to R43, U503 to U17, U504 to U18, U505 to U19, U506 to U20
Connections:
- net +3.3V: now also C51.1, C52.1, C53.1, C54.1
- net +5V: now also C45.1, C46.1, C47.1, C48.1, C49.1, C50.1
- net GND: now also C45.2, C46.2, C47.2, C48.2, C49.2, C50.2, C51.2, C52.2, C53.2, C54.2

Commit message: Hardware design
Parts:
- C45, C46, C47, C48, C49, C50, C51, C52, C53, C54: footprint (none) -> Capacitor_SMD:C_0603_1608Metric_Pad1.08x0.95mm_HandSolder
- U17, U18, U19, U20: value SN74LVC1T45DPKR -> SN74LVC1T45DRLR; footprint Package_TO_SOT_SMD:SOT-23-6 -> Package_TO_SOT_SMD:SOT-563
Changed lines of the file:
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@@
       (effects (font (size 1.27 1.27)) (justify left))
     )
-    (property "Value" "SN74LVC1T45DPKR" (id 1) (at 161.29 130.81 0)
-      (effects (font (size 1.27 1.27)) (justify left))
-    )
-    (property "Footprint" "Package_TO_SOT_SMD:SOT-23-6" (id 2) (at 154.94 151.13 0)
+    (property "Value" "SN74LVC1T45DRLR" (id 1) (at 161.29 130.81 0)
+      (effects (font (size 1.27 1.27)) (justify left))
+    )
+    (property "Footprint" "Package_TO_SOT_SMD:SOT-563" (id 2) (at 154.94 151.13 0)
       (effects (font (size 1.27 1.27)) hide)
     )
@@
       (effects (font (size 1.27 1.27)) (justify left))
     )
-    (property "Footprint" "" (id 2) (at 20.0152 185.42 0)
+    (property "Footprint" "Capacitor_SMD:C_0603_1608Metric_Pad1.08x0.95mm_HandSolder" (id 2) (at 20.0152 185.42 0)
       (effects (font (size 1.27 1.27)) hide)
     )
@@
       (effects (font (size 1.27 1.27)) (justify left))
     )
-    (property "Footprint" "" (id 2) (at 73.3552 185.42 0)
+    (property "Footprint" "Capacitor_SMD:C_0603_1608Metric_Pad1.08x0.95mm_HandSolder" (id 2) (at 73.3552 185.42 0)
       (effects (font (size 1.27 1.27)) hide)
     )
@@
       (effects (font (size 1.27 1.27)) (justify left))
     )
-    (property "Footprint" "" (id 2) (at 46.6852 185.42 0)
+    (property "Footprint" "Capacitor_SMD:C_0603_1608Metric_Pad1.08x0.95mm_HandSolder" (id 2) (at 46.6852 185.42 0)
       (effects (font (size 1.27 1.27)) hide)
     )
@@
       (effects (font (size 1.27 1.27)) (justify left))
     )
-    (property "Footprint" "" (id 2) (at 87.3252 185.42 0)
+    (property "Footprint" "Capacitor_SMD:C_0603_1608Metric_Pad1.08x0.95mm_HandSolder" (id 2) (at 87.3252 185.42 0)
       (effects (font (size 1.27 1.27)) hide)
     )
@@
       (effects (font (size 1.27 1.27)) (justify left))
     )
-    (property "Value" "SN74LVC1T45DPKR" (id 1) (at 161.29 27.94 0)
-      (effects (font (size 1.27 1.27)) (justify left))
-    )
-    (property "Footprint" "Package_TO_SOT_SMD:SOT-23-6" (id 2) (at 154.94 48.26 0)
+    (property "Value" "SN74LVC1T45DRLR" (id 1) (at 161.29 27.94 0)
+      (effects (font (size 1.27 1.27)) (justify left))
+    )
+    (property "Footprint" "Package_TO_SOT_SMD:SOT-563" (id 2) (at 154.94 48.26 0)
       (effects (font (size 1.27 1.27)) hide)
     )
@@
       (effects (font (size 1.27 1.27)) (justify left))
     )
-    (property "Footprint" "" (id 2) (at 32.7152 185.42 0)
+    (property "Footprint" "Capacitor_SMD:C_0603_1608Metric_Pad1.08x0.95mm_HandSolder" (id 2) (at 32.7152 185.42 0)
       (effects (font (size 1.27 1.27)) hide)
     )
@@
       (effects (font (size 1.27 1.27)) (justify left))
     )
-    (property "Footprint" "" (id 2) (at 103.8352 185.42 0)
+    (property "Footprint" "Capacitor_SMD:C_0603_1608Metric_Pad1.08x0.95mm_HandSolder" (id 2) (at 103.8352 185.42 0)
       (effects (font (size 1.27 1.27)) hide)
     )
@@
       (effects (font (size 1.27 1.27)) (justify left))
     )
-    (property "Footprint" "" (id 2) (at 143.2052 185.42 0)
+    (property "Footprint" "Capacitor_SMD:C_0603_1608Metric_Pad1.08x0.95mm_HandSolder" (id 2) (at 143.2052 185.42 0)
       (effects (font (size 1.27 1.27)) hide)
     )
@@
       (effects (font (size 1.27 1.27)) (justify left))
     )
-    (property "Value" "SN74LVC1T45DPKR" (id 1) (at 161.29 96.52 0)
-      (effects (font (size 1.27 1.27)) (justify left))
-    )
-    (property "Footprint" "Package_TO_SOT_SMD:SOT-23-6" (id 2) (at 154.94 116.84 0)
+    (property "Value" "SN74LVC1T45DRLR" (id 1) (at 161.29 96.52 0)
+      (effects (font (size 1.27 1.27)) (justify left))
+    )
+    (property "Footprint" "Package_TO_SOT_SMD:SOT-563" (id 2) (at 154.94 116.84 0)
       (effects (font (size 1.27 1.27)) hide)
     )
@@
       (effects (font (size 1.27 1.27)) (justify left))
     )
-    (property "Footprint" "" (id 2) (at 116.5352 185.42 0)
+    (property "Footprint" "Capacitor_SMD:C_0603_1608Metric_Pad1.08x0.95mm_HandSolder" (id 2) (at 116.5352 185.42 0)
       (effects (font (size 1.27 1.27)) hide)
     )
@@
       (effects (font (size 1.27 1.27)) (justify left))
     )
-    (property "Footprint" "" (id 2) (at 130.5052 185.42 0)
+    (property "Footprint" "Capacitor_SMD:C_0603_1608Metric_Pad1.08x0.95mm_HandSolder" (id 2) (at 130.5052 185.42 0)
       (effects (font (size 1.27 1.27)) hide)
     )
@@
       (effects (font (size 1.27 1.27)) (justify left))
     )
-    (property "Value" "SN74LVC1T45DPKR" (id 1) (at 161.29 62.23 0)
-      (effects (font (size 1.27 1.27)) (justify left))
-    )
-    (property "Footprint" "Package_TO_SOT_SMD:SOT-23-6" (id 2) (at 154.94 82.55 0)
+    (property "Value" "SN74LVC1T45DRLR" (id 1) (at 161.29 62.23 0)
+      (effects (font (size 1.27 1.27)) (justify left))
+    )
+    (property "Footprint" "Package_TO_SOT_SMD:SOT-563" (id 2) (at 154.94 82.55 0)
       (effects (font (size 1.27 1.27)) hide)
     )
@@
       (effects (font (size 1.27 1.27)) (justify left))
     )
-    (property "Footprint" "" (id 2) (at 59.3852 185.42 0)
-      (effects (font (size 1.27 1.27)) hide)
-    )
+    (property "Footprint" "Capacitor_SMD:C_0603_1608Metric_Pad1.08x0.95mm_HandSolder" (id 2) (at 59.3852 185.42 0)
+      (effects (font (size 1.27 1.27)) hide)
+    )

Commit message: Hardware design
Parts:
- renumbered C45 to C501, C46 to C502, C47 to C503, C48 to C504, C49 to C505, C50 to C506, C51 to C507, C52 to C508, C53 to C509, C54 to C510, R43 to R501, U15 to U501, U16 to U502, U17 to U503, U18 to U504, U19 to U505, U20 to U506
