File: HARDWARE/ETH1CSMU2/Control.kicad_sch (KiCad schematic)
At the start: 17 parts, among them U501 74HCT595PW, U502 74HCT595PW, U503 SN74LVC1T45DRLR, U504 SN74LVC1T45DRLR, U505 SN74LVC1T45DRLR, U506 SN74LVC1T45DRLR

Commit message: Hardware design
Connections:
- net ADC_SEL: now reaches U502.6 (QG)
Changed lines of the file:
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@@
     (effects (font (size 1.27 1.27)) (justify left))
+  )
+  (hierarchical_label "ADC_SEL" (shape output) (at 78.74 100.33 180)
+    (effects (font (size 1.27 1.27)) (justify right))
   )
   (hierarchical_label "GPIO_SPI_SCK" (shape input) (at 166.37 71.12 0)

Commit message: Hardware and software development
Connections:
- net GPIO_SPI_MISO renamed SR_OUT
- net GPIO_SPI_MOSI renamed SR_DAT
- net GPIO_SPI_NSS renamed SR_LAT
- net GPIO_SPI_SCK renamed SR_CLK
- no-connect marks 0 -> 1
Changed lines of the file:
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@@
   (junction (at 129.54 186.69) (diameter 0) (color 0 0 0 0)
   )
+  (no_connect (at 80.01 102.87))
   (wire (pts (xy 129.54 185.42) (xy 129.54 186.69))
     (stroke (width 0) (type default) (color 0 0 0 0))
@@
     (stroke (width 0) (type default) (color 0 0 0 0))
   )
-  (wire (pts (xy 80.01 102.87) (xy 78.74 102.87))
-    (stroke (width 0) (type default) (color 0 0 0 0))
-  )
   (wire (pts (xy 129.54 176.53) (xy 142.24 176.53))
     (stroke (width 0) (type default) (color 0 0 0 0))
@@
     (effects (font (size 1.27 1.27)) (justify right))
   )
-  (hierarchical_label "GPIO_SPI_MOSI" (shape input) (at 166.37 36.83 0)
+  (hierarchical_label "SR_DAT" (shape input) (at 166.37 36.83 0)
     (effects (font (size 1.27 1.27)) (justify left))
   )
@@
     (effects (font (size 1.27 1.27)) (justify right))
   )
-  (hierarchical_label "GPIO_SPI_NSS" (shape input) (at 166.37 105.41 0)
+  (hierarchical_label "SR_LAT" (shape input) (at 166.37 105.41 0)
     (effects (font (size 1.27 1.27)) (justify left))
   )
@@
     (effects (font (size 1.27 1.27)) (justify right))
   )
-  (hierarchical_label "GPIO_SPI_MISO" (shape output) (at 166.37 139.7 0)
+  (hierarchical_label "SR_OUT" (shape output) (at 166.37 139.7 0)
     (effects (font (size 1.27 1.27)) (justify left))
   )
@@
     (effects (font (size 1.27 1.27)) (justify right))
   )
-  (hierarchical_label "GPIO_SPI_SCK" (shape input) (at 166.37 71.12 0)
+  (hierarchical_label "SR_CLK" (shape input) (at 166.37 71.12 0)
     (effects (font (size 1.27 1.27)) (justify left))
   )

Commit message: PCB layout
Connections:
- net C_G1: now also U501.1 (QB); no longer U501.4 (QE)
- net C_G10: now also U501.2 (QC); no longer U501.5 (QF)
- net C_G100: now also U501.15 (QA); no longer U501.6 (QG)
- net V_G1: now also U501.5 (QF); no longer U501.15 (QA)
- net V_G10: now also U501.6 (QG); no longer U501.1 (QB)
- net V_G100: now also U501.4 (QE); no longer U501.2 (QC)
Changed lines of the file:
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@@
     (effects (font (size 1.27 1.27)) (justify right))
   )
-  (hierarchical_label "C_G1" (shape output) (at 78.74 46.99 180)
+  (hierarchical_label "C_G1" (shape output) (at 78.74 39.37 180)
     (effects (font (size 1.27 1.27)) (justify right))
   )
@@
     (effects (font (size 1.27 1.27)) (justify left))
   )
-  (hierarchical_label "C_G10" (shape output) (at 78.74 49.53 180)
+  (hierarchical_label "C_G10" (shape output) (at 78.74 41.91 180)
     (effects (font (size 1.27 1.27)) (justify right))
   )
@@
     (effects (font (size 1.27 1.27)) (justify left))
   )
-  (hierarchical_label "V_G100" (shape output) (at 78.74 41.91 180)
+  (hierarchical_label "V_G100" (shape output) (at 78.74 46.99 180)
     (effects (font (size 1.27 1.27)) (justify right))
   )
@@
     (effects (font (size 1.27 1.27)) (justify right))
   )
-  (hierarchical_label "V_G1" (shape output) (at 78.74 36.83 180)
+  (hierarchical_label "V_G1" (shape output) (at 78.74 49.53 180)
     (effects (font (size 1.27 1.27)) (justify right))
   )
@@
     (effects (font (size 1.27 1.27)) (justify left))
   )
-  (hierarchical_label "V_G10" (shape output) (at 78.74 39.37 180)
+  (hierarchical_label "V_G10" (shape output) (at 78.74 52.07 180)
     (effects (font (size 1.27 1.27)) (justify right))
   )
-  (hierarchical_label "C_G100" (shape output) (at 78.74 52.07 180)
+  (hierarchical_label "C_G100" (shape output) (at 78.74 36.83 180)
     (effects (font (size 1.27 1.27)) (justify right))
   )

Commit message: Software development
Connections:
- net SING_SEL renamed SIGN_SEL
Changed lines of the file:
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@@
     (effects (font (size 1.27 1.27)) (justify right))
   )
-  (hierarchical_label "SING_SEL" (shape output) (at 78.74 90.17 180) (fields_autoplaced)
+  (hierarchical_label "SIGN_SEL" (shape output) (at 78.74 90.17 180) (fields_autoplaced)
     (effects (font (size 1.27 1.27)) (justify right))
   )

Commit message: Software development and hardware changes. FGEN code works.
Connections:
- net DDS_LPF renamed FGEN_LPF
Changed lines of the file:
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@@
     (effects (font (size 1.27 1.27)) (justify right))
   )
-  (hierarchical_label "DDS_LPF" (shape output) (at 78.74 97.79 180) (fields_autoplaced)
+  (hierarchical_label "FGEN_LPF" (shape output) (at 78.74 97.79 180) (fields_autoplaced)
     (effects (font (size 1.27 1.27)) (justify right))
   )

Commit message: AD7980 test works.
Parts:
- R501, U506: now not fitted
Changed lines of the file:
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@@
   )
   (symbol (lib_id "Logic_LevelTranslator:SN74LVC1T45DBV") (at 154.94 139.7 0) (unit 1)
-    (in_bom yes) (on_board yes) (dnp no)
+    (in_bom yes) (on_board yes) (dnp yes)
     (property "Reference" "U506" (at 167.64 128.27 0)
       (effects (font (size 1.27 1.27)) (justify left))
@@
   )
   (symbol (lib_id "Device:R") (at 139.7 144.78 270) (unit 1)
-    (in_bom yes) (on_board yes) (dnp no)
+    (in_bom yes) (on_board yes) (dnp yes)
     (property "Reference" "R501" (at 139.7 142.24 90)
       (effects (font (size 1.27 1.27)))
