File: HARDWARE/ETH1CSMU2/Frontend.kicad_sch (KiCad schematic)
At the start: 22 parts, among them U701 SN74LVC1T45DPKR, U702 LT1970, U703 SN74LVC1T45DPKR, U704 SN74LVC1T45DPKR

Commit message: Hardware design
Parts:
- removed R710, R711, R713, R714: 5, symbol Device:R
- added C601, C602, C603, C604, C605, C606: 100n, symbol Device:C
- added R610, R613: 0, symbol Device:R
- R611: renamed from R712; value 5 -> 1
- renumbered D701 to D601, D702 to D602, D703 to D603, R701 to R601, R702 to R602, R703 to R603, R707 to R604, R704 to R605, R705 to R606, R706 to R607, R709 to R608, R708 to R609, R715 to R612, U701 to U601, U702 to U602, U703 to U603, U704 to U604
Connections:
- net +3.3V: now also C604.1, C605.1, C606.1
- net +5V: now also C601.1, C602.1, C603.1
- net GND: now also C601.2, C602.2, C603.2, C604.2, C605.2, C606.2
- net at R611.1, U602.3 (OUT): now also R610.1; no longer U602.4 (SENSE+)
- net VOLT_MEAS: no longer names the net of U602.5 (FILTER), U602.6 (SENSE-)
- net VOLT_MEAS: now also R613.2; no longer R609.2, R611.2
- new net: R610.2, U602.4 (SENSE+)
- new net VOUT_OUT: R609.2, R611.2, R613.1
Other:
- moved on the sheet: R611

Commit message: Hardware design
Parts:
- added R54: OPT, symbol Device:R
- added U24: INA823, symbol ETH1CSMU2:INA823
- renumbered C601 to C45, C602 to C46, C603 to C47, C604 to C48, C605 to C49, C606 to C50, D601 to D3, D602 to D4, D603 to D5, R601 to R44, R602 to R45, R603 to R46, R604 to R47, R605 to R48, R606 to R49, R607 to R50, R608 to R51, R609 to R52, R610 to R53, R611 to R55, R612 to R56, R613 to R57, U601 to U21, U602 to U22, U603 to U23, U604 to U25
Connections:
- net +15V: now also U24.7 (V+)
- net -15V: now also U24.4 (V-)
- net GND: now also U24.5 (Ref)
- net at R53.1, R55.1, U22.3 (OUT): now also U24.3 (+)
- net VOUT_OUT renamed VOLT_MEAS
- net VOLT_MEAS: now also U24.2 (-)
- new net: R54.1, U24.1 (Rg)
- new net: R54.2, U24.8 (Rg)
- new net CURR_MEAS: U24.6
Other:
- moved on the sheet: R48, R49, R50, R52, R53, R55, R57, U22

Commit message: Hardware design
Parts:
- added R51: 10k2, symbol Device:R
- added U21, U22: DG419DY, Package_SO:SOIC-8_3.9x4.9mm_P1.27mm, symbol Analog_Switch:DG419xY
- renumbered C48 to C45, C45 to C46, C49 to C47, C46 to C48, C50 to C49, C47 to C50, R49 to R48, R48 to R49, R51 to R52, R52 to R53, R56 to R54, R53 to R55, R54 to R56, R55 to R57, R57 to R58, U21 to U23, U23 to U24, U22 to U25, U25 to U26, U24 to U27
Connections:
- net +15V: now also U21.4 (V+), U22.4 (V+)
- net +5V: now also U21.5 (VL), U22.5 (VL)
- net -15V: now also U21.7 (V-), U22.7 (V-)
- net GND: now also R51.1, U21.3 (GND), U22.3 (GND)
- net at R49.2, R50.1: now also U22.2; no longer U25.9 (+IN)
- net at R53.1, U25.8 (-IN): now also U21.1; no longer R48.2
- new net: R48.2, U21.2
- new net: R51.2, U21.8
- new net: U22.1, U25.9 (+IN)
- new net FGEN: U22.8
- new net SING_SEL: U21.6, U22.6
Other:
- moved on the sheet: C45, C46, C47, C48, C49, C50, R48, R49, R50, R53, R55, R56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

Commit message: Hardware design
Parts:
- renumbered C45 to C601, C46 to C602, C47 to C603, C48 to C604, C49 to C605, C50 to C606, D3 to D601, D4 to D602, D5 to D603, R44 to R601, R45 to R602, R46 to R603, R47 to R604, R48 to R605, R49 to R606, R50 to R607, R51 to R608, R52 to R609, R53 to R610, R54 to R611, R55 to R612, R56 to R613, R57 to R614, R58 to R615, U21 to U601, U22 to U602, U23 to U603, U24 to U604, U25 to U605, U26 to U606, U27 to U607

Commit message: Hardware design.
Parts:
- added C55, C57, C59, C61, C63, C65, C67, C68, C69, C70: 100n, symbol Device:C
- U25: renamed from U605; value LT1970 -> LT1970ACFE
- U27: renamed from U607; value INA823 -> INA823DT
- renumbered C601 to C56, C603 to C58, C605 to C60, C602 to C62, C604 to C64, C606 to C66, D601 to D3, D602 to D4, D603 to D5, R601 to R44, R602 to R45, R603 to R46, R604 to R47, R605 to R48, R606 to R49, R607 to R50, R608 to R51, R609 to R52, R610 to R53, R611 to R54, R612 to R55, R613 to R56, R614 to R57, R615 to R58, U601 to U21, U602 to U22, U603 to U23, U604 to U24, U606 to U26
Connections:
- net +15V: now also C55.1, C57.1, C59.1, C61.1
- net +5V: now also C68.1, C70.1
- net -15V: now also C63.1, C65.1, C67.1, C69.1
- net GND: now also C55.2, C57.2, C59.2, C61.2, C63.2, C65.2, C67.2, C68.2, C69.2, C70.2
Other:
- moved on the sheet: C56, C58, C60, C62, C64, C66, U21B, U22B

Commit message: Hardware design
Parts:
- C55, C56, C57, C58, C59, C60, C61, C62, C63, C64, C65, C66, C67, C68, C69, C70: footprint (none) -> Capacitor_SMD:C_0603_1608Metric_Pad1.08x0.95mm_HandSolder
- D3, D4, D5: footprint (none) -> LED_SMD:LED_0603_1608Metric_Pad1.05x0.95mm_HandSolder
- R44, R45, R46, R48, R49, R50, R51, R53, R55, R56, R58: footprint (none) -> Resistor_SMD:R_0603_1608Metric_Pad0.98x0.95mm_HandSolder
- R57: value 1 -> LCS2512; footprint (none) -> Resistor_SMD:R_2512_6332Metric_Pad1.40x3.35mm_HandSolder
- U23, U24, U26: value SN74LVC1T45DPKR -> SN74LVC1T45DRLR; footprint Package_TO_SOT_SMD:SOT-23-6 -> Package_TO_SOT_SMD:SOT-563
- U25: footprint (none) -> Package_SO:HTSSOP-20-1EP_4.4x6.5mm_P0.65mm_EP3.4x6.5mm_ThermalVias
- U27: footprint (none) -> Package_SO:SOIC-8_3.9x4.9mm_P1.27mm

Commit message: Hardware design
Parts:
- R613: renamed from R56; value OPT -> 5k23
- renumbered C55 to C601, C56 to C602, C57 to C603, C58 to C604, C59 to C605, C60 to C606, C61 to C607, C62 to C608, C63 to C609, C64 to C610, C65 to C611, C66 to C612, C67 to C613, C68 to C614, C69 to C615, C70 to C616, D3 to D601, D4 to D602, D5 to D603, R44 to R601, R45 to R602, R46 to R603, R47 to R604, R48 to R605, R49 to R606, R50 to R607, R51 to R608, R52 to R609, R53 to R610, R54 to R611, R55 to R612, R57 to R614, R58 to R615, U21 to U601, U22 to U602, U23 to U603, U24 to U604, U25 to U605, U26 to U606, U27 to U607
