File: HARDWARE/ETH1CSMU2/Frontend.kicad_sch (KiCad schematic)
At the start: 41 parts, among them U601 DG419DY, U602 DG419DY, U603 SN74LVC1T45DRLR, U604 SN74LVC1T45DRLR, U605 LT1970ACFE, U606 SN74LVC1T45DRLR, U607 INA823DT

Commit message: Hardware design
Other:
- moved on the sheet: C601, C602, C603, C604, C605, C606, C607, C608, C609, C610, C611, C612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

Commit message: Hardware and software development
Parts:
- renumbered C608 to C601, C601 to C602, C609 to C603, C610 to C604, C602 to C605, C603 to C606, C611 to C607, C612 to C608, C604 to C609, C605 to C610, C613 to C611, C614 to C612, C606 to C613, C607 to C614
Changed lines of the file:
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@@
   (symbol (lib_id "power:+5V") (at 49.53 128.27 0) (mirror y) (unit 1)
     (in_bom yes) (on_board yes) (fields_autoplaced)
-    (property "Reference" "#PWR0606" (id 0) (at 49.53 132.08 0)
+    (property "Reference" "#PWR0614" (id 0) (at 49.53 132.08 0)
       (effects (font (size 1.27 1.27)) hide)
     )
@@
   (symbol (lib_id "power:GND") (at 121.92 50.8 0) (unit 1)
     (in_bom yes) (on_board yes)
-    (property "Reference" "#PWR0616" (id 0) (at 121.92 57.15 0)
+    (property "Reference" "#PWR0620" (id 0) (at 121.92 57.15 0)
       (effects (font (size 1.27 1.27)) hide)
     )
@@
   (symbol (lib_id "Device:C") (at 17.78 29.21 0) (unit 1)
     (in_bom yes) (on_board yes) (fields_autoplaced)
-    (property "Reference" "C608" (id 0) (at 20.701 28.3753 0)
+    (property "Reference" "C601" (id 0) (at 20.701 28.3753 0)
       (effects (font (size 1.27 1.27)) (justify left))
     )
@@
   (symbol (lib_id "Device:C") (at 43.18 29.21 0) (unit 1)
     (in_bom yes) (on_board yes) (fields_autoplaced)
-    (property "Reference" "C612" (id 0) (at 46.101 28.3753 0)
+    (property "Reference" "C608" (id 0) (at 46.101 28.3753 0)
       (effects (font (size 1.27 1.27)) (justify left))
     )
@@
   (symbol (lib_id "power:+3.3V") (at 124.46 27.94 0) (unit 1)
     (in_bom yes) (on_board yes)
-    (property "Reference" "#PWR0617" (id 0) (at 124.46 31.75 0)
+    (property "Reference" "#PWR0621" (id 0) (at 124.46 31.75 0)
       (effects (font (size 1.27 1.27)) hide)
     )
@@
   (symbol (lib_id "power:-15V") (at 43.18 101.6 0) (unit 1)
     (in_bom yes) (on_board yes) (fields_autoplaced)
-    (property "Reference" "#PWR0620" (id 0) (at 43.18 99.06 0)
+    (property "Reference" "#PWR0611" (id 0) (at 43.18 99.06 0)
       (effects (font (size 1.27 1.27)) hide)
     )
@@
   (symbol (lib_id "Device:C") (at 50.8 81.28 0) (unit 1)
     (in_bom yes) (on_board yes) (fields_autoplaced)
-    (property "Reference" "C605" (id 0) (at 53.721 80.4453 0)
+    (property "Reference" "C610" (id 0) (at 53.721 80.4453 0)
       (effects (font (size 1.27 1.27)) (justify left))
     )
@@
   (symbol (lib_id "Device:C") (at 25.4 81.28 0) (unit 1)
     (in_bom yes) (on_board yes)
-    (property "Reference" "C601" (id 0) (at 28.321 80.4453 0)
+    (property "Reference" "C602" (id 0) (at 28.321 80.4453 0)
       (effects (font (size 1.27 1.27)) (justify left))
     )
@@
   (symbol (lib_id "Device:C") (at 25.4 107.95 0) (unit 1)
     (in_bom yes) (on_board yes) (fields_autoplaced)
-    (property "Reference" "C609" (id 0) (at 28.321 107.1153 0)
+    (property "Reference" "C603" (id 0) (at 28.321 107.1153 0)
       (effects (font (size 1.27 1.27)) (justify left))
     )
@@
   (symbol (lib_id "power:-15V") (at 49.53 156.21 0) (mirror x) (unit 1)
     (in_bom yes) (on_board yes)
-    (property "Reference" "#PWR0607" (id 0) (at 49.53 158.75 0)
+    (property "Reference" "#PWR0615" (id 0) (at 49.53 158.75 0)
       (effects (font (size 1.27 1.27)) hide)
     )
@@
   (symbol (lib_id "power:+3.3V") (at 43.18 48.26 0) (unit 1)
     (in_bom yes) (on_board yes)
-    (property "Reference" "#PWR0610" (id 0) (at 43.18 52.07 0)
+    (property "Reference" "#PWR0607" (id 0) (at 43.18 52.07 0)
       (effects (font (size 1.27 1.27)) hide)
     )
@@
   (symbol (lib_id "power:+5V") (at 43.18 22.86 0) (unit 1)
     (in_bom yes) (on_board yes) (fields_autoplaced)
-    (property "Reference" "#PWR0618" (id 0) (at 43.18 26.67 0)
+    (property "Reference" "#PWR0605" (id 0) (at 43.18 26.67 0)
       (effects (font (size 1.27 1.27)) hide)
     )
@@
   (symbol (lib_id "Device:C") (at 43.18 54.61 0) (unit 1)
     (in_bom yes) (on_board yes) (fields_autoplaced)
-    (property "Reference" "C604" (id 0) (at 46.101 53.7753 0)
+    (property "Reference" "C609" (id 0) (at 46.101 53.7753 0)
       (effects (font (size 1.27 1.27)) (justify left))
     )
@@
   (symbol (lib_id "power:GND") (at 43.18 114.3 0) (unit 1)
     (in_bom yes) (on_board yes) (fields_autoplaced)
-    (property "Reference" "#PWR0621" (id 0) (at 43.18 120.65 0)
+    (property "Reference" "#PWR0612" (id 0) (at 43.18 120.65 0)
       (effects (font (size 1.27 1.27)) hide)
     )
@@
   (symbol (lib_id "power:GND") (at 59.69 156.21 0) (mirror y) (unit 1)
     (in_bom yes) (on_board yes)
-    (property "Reference" "#PWR0609" (id 0) (at 59.69 162.56 0)
+    (property "Reference" "#PWR0617" (id 0) (at 59.69 162.56 0)
       (effects (font (size 1.27 1.27)) hide)
     )
@@
   (symbol (lib_id "Device:C") (at 50.8 107.95 0) (unit 1)
     (in_bom yes) (on_board yes) (fields_autoplaced)
-    (property "Reference" "C613" (id 0) (at 53.721 107.1153 0)
+    (property "Reference" "C611" (id 0) (at 53.721 107.1153 0)
       (effects (font (size 1.27 1.27)) (justify left))
     )
@@
   (symbol (lib_id "power:+15V") (at 43.18 74.93 0) (unit 1)
     (in_bom yes) (on_board yes)
-    (property "Reference" "#PWR0612" (id 0) (at 43.18 78.74 0)
+    (property "Reference" "#PWR0609" (id 0) (at 43.18 78.74 0)
       (effects (font (size 1.27 1.27)) hide)
     )
@@
   (symbol (lib_id "power:+5V") (at 102.87 43.18 90) (unit 1)
     (in_bom yes) (on_board yes)
-    (property "Reference" "#PWR0614" (id 0) (at 106.68 43.18 0)
+    (property "Reference" "#PWR0618" (id 0) (at 106.68 43.18 0)
       (effects (font (size 1.27 1.27)) hide)
     )
@@
   (symbol (lib_id "Device:C") (at 30.48 29.21 0) (unit 1)
     (in_bom yes) (on_board yes) (fields_autoplaced)
-    (property "Reference" "C610" (id 0) (at 33.401 28.3753 0)
+    (property "Reference" "C604" (id 0) (at 33.401 28.3753 0)
       (effects (font (size 1.27 1.27)) (justify left))
     )
@@
   (symbol (lib_id "power:GND") (at 43.18 87.63 0) (unit 1)
     (in_bom yes) (on_board yes) (fields_autoplaced)
-    (property "Reference" "#PWR0613" (id 0) (at 43.18 93.98 0)
+    (property "Reference" "#PWR0610" (id 0) (at 43.18 93.98 0)
       (effects (font (size 1.27 1.27)) hide)
     )
@@
   (symbol (lib_id "Device:C") (at 38.1 81.28 0) (unit 1)
     (in_bom yes) (on_board yes) (fields_autoplaced)
-    (property "Reference" "C603" (id 0) (at 41.021 80.4453 0)
+    (property "Reference" "C606" (id 0) (at 41.021 80.4453 0)
       (effects (font (size 1.27 1.27)) (justify left))
     )
@@
   (symbol (lib_id "power:GND") (at 43.18 60.96 0) (unit 1)
     (in_bom yes) (on_board yes) (fields_autoplaced)
-    (property "Reference" "#PWR0611" (id 0) (at 43.18 67.31 0)
+    (property "Reference" "#PWR0608" (id 0) (at 43.18 67.31 0)
       (effects (font (size 1.27 1.27)) hide)
     )
@@
   (symbol (lib_id "Device:C") (at 55.88 29.21 0) (unit 1)
     (in_bom yes) (on_board yes) (fields_autoplaced)
-    (property "Reference" "C614" (id 0) (at 58.801 28.3753 0)
+    (property "Reference" "C612" (id 0) (at 58.801 28.3753 0)
       (effects (font (size 1.27 1.27)) (justify left))
     )
@@
   (symbol (lib_id "power:+5V") (at 43.18 167.64 0) (unit 1)
     (in_bom yes) (on_board yes) (fields_autoplaced)
-    (property "Reference" "#PWR0605" (id 0) (at 43.18 171.45 0)
+    (property "Reference" "#PWR0613" (id 0) (at 43.18 171.45 0)
       (effects (font (size 1.27 1.27)) hide)
     )
@@
   (symbol (lib_id "power:+15V") (at 59.69 128.27 0) (mirror y) (unit 1)
     (in_bom yes) (on_board yes)
-    (property "Reference" "#PWR0608" (id 0) (at 59.69 132.08 0)
+    (property "Reference" "#PWR0616" (id 0) (at 59.69 132.08 0)
       (effects (font (size 1.27 1.27)) hide)
     )
@@
   (symbol (lib_id "power:GND") (at 43.18 35.56 0) (unit 1)
     (in_bom yes) (on_board yes) (fields_autoplaced)
-    (property "Reference" "#PWR0619" (id 0) (at 43.18 41.91 0)
+    (property "Reference" "#PWR0606" (id 0) (at 43.18 41.91 0)
       (effects (font (size 1.27 1.27)) hide)
     )
@@
   (symbol (lib_id "power:+5V") (at 119.38 27.94 0) (unit 1)
     (in_bom yes) (on_board yes)
-    (property "Reference" "#PWR0615" (id 0) (at 119.38 31.75 0)
+    (property "Reference" "#PWR0619" (id 0) (at 119.38 31.75 0)
       (effects (font (size 1.27 1.27)) hide)
     )
@@
   (symbol (lib_id "Device:C") (at 30.48 54.61 0) (unit 1)
     (in_bom yes) (on_board yes) (fields_autoplaced)
-    (property "Reference" "C602" (id 0) (at 33.401 53.7753 0)
+    (property "Reference" "C605" (id 0) (at 33.401 53.7753 0)
       (effects (font (size 1.27 1.27)) (justify left))
     )
@@
   (symbol (lib_id "Device:C") (at 38.1 107.95 0) (unit 1)
     (in_bom yes) (on_board yes) (fields_autoplaced)
-    (property "Reference" "C611" (id 0) (at 41.021 107.1153 0)
+    (property "Reference" "C607" (id 0) (at 41.021 107.1153 0)
       (effects (font (size 1.27 1.27)) (justify left))
     )
@@
   (symbol (lib_id "Device:C") (at 63.5 81.28 0) (unit 1)
     (in_bom yes) (on_board yes) (fields_autoplaced)
-    (property "Reference" "C607" (id 0) (at 66.421 80.4453 0)
+    (property "Reference" "C614" (id 0) (at 66.421 80.4453 0)
       (effects (font (size 1.27 1.27)) (justify left))
     )
@@
   (symbol (lib_id "Device:C") (at 55.88 54.61 0) (unit 1)
     (in_bom yes) (on_board yes) (fields_autoplaced)
-    (property "Reference" "C606" (id 0) (at 58.801 53.7753 0)
-      (effects (font (size 1.27 1.27)) (justify left))
-    )
+    (property "Reference" "C613" (id 0) (at 58.801 53.7753 0)
+      (effects (font (size 1.27 1.27)) (justify left))
+    )

Commit message: Hardware design.
Parts:
- removed R612: 0, Resistor_SMD:R_0603_1608Metric_Pad0.98x0.95mm_HandSolder, symbol Device:R
- added C617, C618, C619: 10p, Capacitor_SMD:C_0603_1608Metric_Pad1.08x0.95mm_HandSolder, symbol Device:C
- added Q601, Q602, Q603: MMBT3904, Package_TO_SOT_SMD:SOT-23, symbol Transistor_BJT:MMBT3904
- added R611, R625: 10k, Resistor_SMD:R_0603_1608Metric_Pad0.98x0.95mm_HandSolder, symbol Device:R
- added R613: 0, Resistor_SMD:R_0603_1608Metric_Pad0.98x0.95mm_HandSolder, symbol Device:R
- added R615, R616, R617: 1k, Resistor_SMD:R_0603_1608Metric_Pad0.98x0.95mm_HandSolder, symbol Device:R
- added R618: OPT, Resistor_SMD:R_0603_1608Metric_Pad0.98x0.95mm_HandSolder, symbol Device:R
- added R620: WSR2R8000FEK, Resistor_SMD:R_Shunt_Vishay_WSR2_WSR3_KelvinConnection, symbol Device:R
- added R621: WSR21R000FEK, Resistor_SMD:R_Shunt_Vishay_WSR2_WSR3_KelvinConnection, symbol Device:R
- added R622: RP73D2B10RBTG, Resistor_SMD:R_1206_3216Metric_Pad1.30x1.75mm_HandSolder, symbol Device:R
- added R623: RQ73C2B100RBT, Resistor_SMD:R_1206_3216Metric_Pad1.30x1.75mm_HandSolder, symbol Device:R
- added U607, U608, U609: AQY212G2SX, ETH1CSMU2:AQY212GS, symbol ETH1CSMU2:AQY212GS
- R614: value LCS2512 -> 10k; footprint Resistor_SMD:R_2512_6332Metric_Pad1.40x3.35mm_HandSolder -> Resistor_SMD:R_0603_1608Metric_Pad0.98x0.95mm_HandSolder
- R619: renamed from R613; value 5k23 -> 11k
- renumbered R611 to R605, R609 to R606, R605 to R607, R606 to R608, R607 to R609, R608 to R610, R610 to R612, R615 to R624, U606 to U604, U604 to U605, U605 to U606, U607 to U610
Connections:
- net +5V: now also R615.1, R616.1, R617.1
- net GND: now also C617.2, C618.2, C619.2, Q601.2 (E), Q602.2 (E), Q603.2 (E)
- net VOLT_MEAS: now also R620.2, R621.2, R622.2, R623.2; no longer R612.2, R614.2
- net at U606.3 (OUT), U610.3 (+): now also R613.2, R618.1, U607.4, U608.4, U609.4; no longer R614.1
- net at U606.4 (SENSE+): now also R613.1
- net at R624.2, U606.5 (FILTER), U606.6 (SENSE-): now also R612.2
- new net: C619.1, Q603.1 (B), R625.2
- new net: R623.1, U609.3
- new net: R616.2, U608.1
- new net: C618.1, Q602.1 (B), R614.2
- new net: R618.2, R620.1, R621.1, U607.3
- new net: C617.1, Q601.1 (B), R611.2
- new net: R615.2, U607.1
- new net: R617.2, U609.1
- new net: R622.1, U608.3
- new net CURR_SENS_100R: Q603.3 (C), U609.2
- new net CURR_SENS_10R: Q602.3 (C), U608.2
- new net CURR_SENS_1R: Q601.3 (C), U607.2
- new net MCU_CURR_SENS_100R: R625.1
- new net MCU_CURR_SENS_10R: R614.1
- new net MCU_CURR_SENS_1R: R611.1
Other:
- moved on the sheet: R604, R605, R606, R607, R608, R609, R610, R612, R619, R624, U601A, U602A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

Commit message: Hardware design
Parts:
- added C620: 10p, Capacitor_SMD:C_0603_1608Metric_Pad1.08x0.95mm_HandSolder, symbol Device:C
- added Q604: MMBT3904, Package_TO_SOT_SMD:SOT-23, symbol Transistor_BJT:MMBT3904
- added R619: 1k, Resistor_SMD:R_0603_1608Metric_Pad0.98x0.95mm_HandSolder, symbol Device:R
- added R626: PHPA1206E1001BST, Resistor_SMD:R_1206_3216Metric_Pad1.30x1.75mm_HandSolder, symbol Device:R
- added R628: 10k, Resistor_SMD:R_0603_1608Metric_Pad0.98x0.95mm_HandSolder, symbol Device:R
- added U610: AQY212G2SX, ETH1CSMU2:AQY212GS, symbol ETH1CSMU2:AQY212GS
- renumbered R611 to R609, R609 to R610, R610 to R611, R614 to R612, R612 to R613, R613 to R614, R625 to R615, R615 to R616, R616 to R617, R617 to R618, R618 to R620, R619 to R621, R620 to R622, R621 to R623, R622 to R624, R623 to R625, R624 to R627, U610 to U611
Connections:
- net +5V: now also R619.1
- net GND: now also C620.2, Q604.2 (E)
- net VOLT_MEAS: now also R626.2
- net at R614.2, R620.1, U606.3 (OUT)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: now also U610.4
- new net: C620.1, Q604.1 (B), R628.2
- new net: R619.2, U610.1
- new net: R626.1, U610.3
- new net CURR_SENS_1kR: Q604.3 (C), U610.2
- new net MCU_CURR_SENS_1kR: R628.1
Other:
- moved on the sheet: C617, C618, C619, Q601, Q602, Q603, R606, R607, R608, R609, R610, R611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

Commit message: Hardware design
Parts:
- added C617, C618: 100n, Capacitor_SMD:C_0603_1608Metric_Pad1.08x0.95mm_HandSolder, symbol Device:C
- added R613: 0, Resistor_SMD:R_0603_1608Metric_Pad0.98x0.95mm_HandSolder, symbol Device:R
- added U612: LM7171BIM, Package_SO:SOIC-8_3.9x4.9mm_P1.27mm, symbol Amplifier_Operational:LM7171xIM
- R601, R602, R603: value 10k -> 1k
- R606: renamed from R607; value 3k4 -> 3k4/.1%
- R607: renamed from R608; value 3k4 -> 3k4/.1%
- R608: renamed from R610; value 10k2 -> 10k2/.1%
- R610: renamed from R611; value 10k2 -> 10k2/.1%
- R612: renamed from R613; value 10k2 -> 10k2/.1%
- R621: value 11k -> 11k/.1%
- renumbered C617 to C619, C618 to C620, C619 to C621, C620 to C622, R606 to R609, R609 to R611, R612 to R614, R614 to R615, R615 to R622, R622 to R623, R623 to R624, R624 to R625, R625 to R626, R626 to R627, R627 to R628, R628 to R629
Connections:
- net +15V: now also C617.1, U612.7 (V+)
- net -15V: now also C618.1, U612.4 (V-)
- net GND: now also C617.2, C618.2
- net VOLT_MEAS: now also R612.2, U612.3 (+)
- net at R628.2, U606.6 (SENSE-): now also R613.1; no longer R612.2, U606.5 (FILTER)
- new net: R613.2, U606.5 (FILTER)
- new net GUARD: U612.2 (-), U612.6
Other:
- note added: "GPIO"
- note added: "MISC"
- moved on the sheet: C602, C603, C606, C607, C610, C611, C614, C615, D601, D602, D603, R601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

Commit message: Hardware design
Parts:
- added R623, R630: 0, Resistor_SMD:R_0603_1608Metric_Pad0.98x0.95mm_HandSolder, symbol Device:R
- renumbered R623 to R624, R624 to R625, R625 to R626, R626 to R627, R627 to R628, R628 to R629, R629 to R631
Connections:
- net GND: now also R623.2; no longer U611.5 (Ref)
- new net: R623.1, R630.1, U611.5 (Ref)
- new net VOUT_OFFSET: R630.2
Other:
- moved on the sheet: U612

Commit message: Hardware design
Parts:
- removed R624: WSR2R8000FEK, Resistor_SMD:R_Shunt_Vishay_WSR2_WSR3_KelvinConnection, symbol Device:R
- R625: value WSR21R000FEK -> RT1206BRD071RL; footprint Resistor_SMD:R_Shunt_Vishay_WSR2_WSR3_KelvinConnection -> Resistor_SMD:R_1206_3216Metric_Pad1.30x1.75mm_HandSolder
- renumbered R621 to R616, R616 to R617, R617 to R618, R618 to R619, R619 to R620, R620 to R621, R630 to R622, R622 to R624, R631 to R630, U611 to U607, U607 to U608, U608 to U609, U609 to U610, U610 to U611
Other:
- moved on the sheet: R616, R622, R623, U607

Commit message: Changes in schematic.
Parts:
- added C619: 1n, Capacitor_SMD:C_0603_1608Metric_Pad1.08x0.95mm_HandSolder, symbol Device:C
- added D604: BAV99, Package_TO_SOT_SMD:SOT-23, symbol Diode:BAV99
- added R611: 100, Resistor_SMD:R_0603_1608Metric_Pad0.98x0.95mm_HandSolder, symbol Device:R
- renumbered C619 to C620, C620 to C621, C621 to C622, C622 to C623, R611 to R612, R612 to R613, R613 to R614, R614 to R615, R615 to R616, R616 to R617, R617 to R618, R618 to R619, R619 to R620, R620 to R621, R621 to R622, R622 to R623, R623 to R624, R624 to R625, R625 to R626, R626 to R627, R627 to R628, R628 to R629, R629 to R630, R630 to R631
Connections:
- net SENS+_LIM: now reaches R616.1, U606.4 (SENSE+)
- net SENS+_LIM: now also D604.3 (K)
- net FILTER_LIM: now reaches R614.2, U606.5 (FILTER)
- net FILTER_LIM: now also C619.1, D604.1 (K), D604.2 (A), R611.1
- net SENS-_LIM: now reaches R614.1, R630.2, U606.6 (SENSE-)
- net SENS-_LIM: now also C619.2, R611.2
Other:
- note added: "Protection from abrust load shorts"
- moved on the sheet: R614, R630
