File: HARDWARE/ETH1CSMU2/MCU.kicad_sch (KiCad schematic)
At the start: 4 parts

Commit message: Hardware design
Parts:
- gave numbers to parts that had none: 4
Other:
- moved on the sheet: J2, R66, R67, U35

Commit message: Hardware design
Parts:
- added U?: STM32F746ZG, symbol ETH1CSMU2:STM32F746ZG
- renumbered R66 to R73, R67 to R74, U35 to U39
Changed lines of the file:
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@@
   (symbol (lib_id "power:+3.3V") (at 246.38 260.35 0) (unit 1)
     (in_bom yes) (on_board yes)
-    (property "Reference" "#PWR0195" (id 0) (at 246.38 264.16 0)
+    (property "Reference" "#PWR0219" (id 0) (at 246.38 264.16 0)
       (effects (font (size 1.27 1.27)) hide)
     )
@@
   (symbol (lib_id "power:+3.3V") (at 281.94 254 0) (unit 1)
     (in_bom yes) (on_board yes)
-    (property "Reference" "#PWR0197" (id 0) (at 281.94 257.81 0)
+    (property "Reference" "#PWR0221" (id 0) (at 281.94 257.81 0)
       (effects (font (size 1.27 1.27)) hide)
     )
@@
   (symbol (lib_id "Device:R") (at 281.94 260.35 0) (unit 1)
     (in_bom yes) (on_board yes)
-    (property "Reference" "R67" (id 0) (at 283.718 259.1816 0)
+    (property "Reference" "R74" (id 0) (at 283.718 259.1816 0)
       (effects (font (size 1.27 1.27)) (justify left))
     )
@@
   (symbol (lib_id "power:GND") (at 199.39 274.32 0) (unit 1)
     (in_bom yes) (on_board yes)
-    (property "Reference" "#PWR0193" (id 0) (at 199.39 280.67 0)
+    (property "Reference" "#PWR0217" (id 0) (at 199.39 280.67 0)
       (effects (font (size 1.27 1.27)) hide)
     )
@@
   (symbol (lib_id "Device:R") (at 271.78 260.35 0) (unit 1)
     (in_bom yes) (on_board yes)
-    (property "Reference" "R66" (id 0) (at 273.558 259.1816 0)
+    (property "Reference" "R73" (id 0) (at 273.558 259.1816 0)
       (effects (font (size 1.27 1.27)) (justify left))
     )
@@
   (symbol (lib_id "Memory_EEPROM:24LC08") (at 246.38 267.97 0) (unit 1)
     (in_bom yes) (on_board yes)
-    (property "Reference" "U35" (id 0) (at 255.27 259.08 0))
+    (property "Reference" "U39" (id 0) (at 255.27 259.08 0))
     (property "Value" "24LC08B-E/MS" (id 1) (at 255.27 261.62 0))
     (property "Footprint" "Package_SO:MSOP-8_3x3mm_P0.65mm" (id 2) (at 246.38 267.97 0)
@@
   (symbol (lib_id "power:+3.3V") (at 199.39 260.35 0) (unit 1)
     (in_bom yes) (on_board yes)
-    (property "Reference" "#PWR0192" (id 0) (at 199.39 264.16 0)
+    (property "Reference" "#PWR0216" (id 0) (at 199.39 264.16 0)
       (effects (font (size 1.27 1.27)) hide)
     )
@@
     (pin "1")
   )
+  (symbol (lib_id "ETH1CSMU2:STM32F746ZG") (at 224.79 132.08 0) (unit 1)
+    (in_bom yes) (on_board yes)
+    (property "Reference" "U?" (id 0) (at 86.36 33.02 0)
+      (effects (font (size 1.27 1.27)) (justify left))
+    )
+    (property "Value" "STM32F746ZG" (id 1) (at 350.52 33.02 0)
+      (effects (font (size 1.27 1.27)) (justify left))
+    )
+    (property "Footprint" "" (id 2) (at 628.65 93.98 0)
+      (effects (font (size 1.27 1.27)) hide)
+    )
+    (property "Datasheet" "" (id 3) (at 628.65 93.98 0)
+      (effects (font (size 1.27 1.27)) hide)
+    )
+    (pin "1")
+    (pin "10")
+    (pin "100")
+    (pin "101")
+    (pin "102")
+    (pin "103")
+    (pin "104")
+    (pin "105")
+    (pin "106")
+    (pin "107")
+    (pin "108")
+    (pin "109")
+    (pin "11")
+    (pin "110")
+    (pin "111")
+    (pin "112")
+    (pin "113")
+    (pin "114")
+    (pin "115")
+    (pin "116")
+    (pin "117")
+    (pin "118")
+    (pin "119")
+    (pin "12")
+    (pin "120")
+    (pin "121")
+    (pin "122")
+    (pin "123")
+    (pin "124")
+    (pin "125")
+    (pin "126")
+    (pin "127")
+    (pin "128")
+    (pin "129")
+    (pin "13")
+    (pin "130")
+    (pin "131")
+    (pin "132")
+    (pin "133")
+    (pin "134")
+    (pin "135")
+    (pin "136")
+    (pin "137")
+    (pin "138")
+    (pin "139")
+    (pin "14")
+    (pin "140")
+    (pin "141")
+    (pin "142")
+    (pin "143")
+    (pin "144")
+    (pin "15")
+    (pin "16")
+    (pin "17")
+    (pin "18")
+    (pin "19")
+    (pin "2")
+    (pin "20")
+    (pin "21")
+    (pin "22")
+    (pin "23")
+    (pin "24")
+    (pin "25")
+    (pin "26")
+    (pin "27")
+    (pin "28")
+    (pin "29")
+    (pin "3")
+    (pin "30")
+    (pin "31")
+    (pin "32")
+    (pin "33")
+    (pin "34")
+    (pin "35")
+    (pin "36")
+    (pin "37")
+    (pin "38")
+    (pin "39")
+    (pin "4")
+    (pin "40")
+    (pin "41")
+    (pin "42")
+    (pin "43")
+    (pin "44")
+    (pin "45")
+    (pin "46")
+    (pin "47")
+    (pin "48")
+    (pin "49")
+    (pin "5")
+    (pin "50")
+    (pin "51")
+    (pin "52")
+    (pin "53")
+    (pin "54")
+    (pin "55")
+    (pin "56")
+    (pin "57")
+    (pin "58")
+    (pin "59")
+    (pin "6")
+    (pin "60")
+    (pin "61")
+    (pin "62")
+    (pin "63")
+    (pin "64")
+    (pin "65")
+    (pin "66")
+    (pin "67")
+    (pin "68")
+    (pin "69")
+    (pin "7")
+    (pin "70")
+    (pin "71")
+    (pin "72")
+    (pin "73")
+    (pin "74")
+    (pin "75")
+    (pin "76")
+    (pin "77")
+    (pin "78")
+    (pin "79")
+    (pin "8")
+    (pin "80")
+    (pin "81")
+    (pin "82")
+    (pin "83")
+    (pin "84")
+    (pin "85")
+    (pin "86")
+    (pin "87")
+    (pin "88")
+    (pin "89")
+    (pin "9")
+    (pin "90")
+    (pin "91")
+    (pin "92")
+    (pin "93")
+    (pin "94")
+    (pin "95")
+    (pin "96")
+    (pin "97")
+    (pin "98")
+    (pin "99")
+  )
   (symbol (lib_id "power:GND") (at 246.38 275.59 0) (unit 1)
     (in_bom yes) (on_board yes)
-    (property "Reference" "#PWR0196" (id 0) (at 246.38 281.94 0)
+    (property "Reference" "#PWR0220" (id 0) (at 246.38 281.94 0)
       (effects (font (size 1.27 1.27)) hide)
     )
@@
   (symbol (lib_id "power:GND") (at 234.95 275.59 0) (unit 1)
     (in_bom yes) (on_board yes)
-    (property "Reference" "#PWR0194" (id 0) (at 234.95 281.94 0)
-      (effects (font (size 1.27 1.27)) hide)
-    )
+    (property "Reference" "#PWR0218" (id 0) (at 234.95 281.94 0)
+      (effects (font (size 1.27 1.27)) hide)
+    )

Commit message: Hardware design
Parts:
- added C1001, C1002, C1003, C1006, C1009, C1011, C1012, C1013, C1014, C1015, C1016, C1017, C1018, C1019, C1020, C1022: 100n, Capacitor_SMD:C_0603_1608Metric_Pad1.08x0.95mm_HandSolder, symbol Device:C
- added C1004, C1007: 8p, Capacitor_SMD:C_0603_1608Metric_Pad1.08x0.95mm_HandSolder, symbol Device:C
- added C1005, C1008: 2u2, Capacitor_SMD:C_0603_1608Metric_Pad1.08x0.95mm_HandSolder, symbol Device:C
- added C1010, C1021: 1u, Capacitor_SMD:C_0603_1608Metric_Pad1.08x0.95mm_HandSolder, symbol Device:C
- added D1001: BLUE, LED_SMD:LED_0603_1608Metric_Pad1.05x0.95mm_HandSolder, symbol Device:LED
- added D1002: RED, LED_SMD:LED_0603_1608Metric_Pad1.05x0.95mm_HandSolder, symbol Device:LED
- added D1003: GREEN, LED_SMD:LED_0603_1608Metric_Pad1.05x0.95mm_HandSolder, symbol Device:LED
- added FB1001: 742792031, Inductor_SMD:L_0805_2012Metric_Pad1.15x1.40mm_HandSolder, symbol Device:Ferrite_Bead
- added J1001: Conn_02x01, Connector_PinHeader_2.54mm:PinHeader_1x02_P2.54mm_Vertical, symbol Connector_Generic:Conn_02x01
- added R1001, R1005: 680, Resistor_SMD:R_0603_1608Metric_Pad0.98x0.95mm_HandSolder, symbol Device:R
- added R1002, R1009, R1010: 10k, Resistor_SMD:R_0603_1608Metric_Pad0.98x0.95mm_HandSolder, symbol Device:R
- added R1003: 560, Resistor_SMD:R_0603_1608Metric_Pad0.98x0.95mm_HandSolder, symbol Device:R
- added R1004, R1006: 4k7, Resistor_SMD:R_0603_1608Metric_Pad0.98x0.95mm_HandSolder, symbol Device:R
- added U1001: HDC1080, Package_SON:Texas_PWSON-N6, symbol Sensor_Humidity:HDC1080
- added Y1001: X, ETH1CLCR2:NX3225GD, symbol Device:Crystal
- gave numbers to parts that had none: 1
- renumbered J2 to J1002, R73 to R1007, R74 to R1008, U39 to U1003
Connections:
- net +3.3V: now also U1002.108 (VDD), U1002.121 (VDD), U1002.131 (VDD), U1002.143 (PDR_ON), U1002.144 (VDD), U1002.17 (VDD), U1002.30 (VDD), U1002.39 (VDD), U1002.52 (VDD), U1002.6 (VBAT), U1002.62 (VDD), U1002.72 (VDD), U1002.84 (VDD), U1002.95 (VDDUSB), C1001.1, C1002.1, C1003.1, C1006.1, C1009.1, C1010.1, C1011.1, C1012.1, C1013.1, C1014.1, C1015.1, C1016.1, C1017.1, C1018.1, C1019.1, C1020.1, D1001.2 (A), D1002.2 (A), D1003.2 (A), FB1001.2, R1002.2, R1004.1, R1006.1, R1010.1, U1001.5 (VCC)
- net EEPROM_SCL: now also U1002.81 (PD12,TIM4_CH1,LPTIM1_IN1,I2C4_SCL,USART3_RTS,QUADSPI_BK1_IO1,SAI2_FS_A,FMC_A17,FMC_ALE,EVENTOUT)
- net EEPROM_SDA: now also U1002.82 (PD13,TIM4_CH2,LPTIM1_OUT,I2C4_SDA,QUADSPI_BK1_IO3,SAI2_SCK_A,FMC_A18,EVENTOUT)
- net EEPROM_WP: now also U1002.80 (PD11,I2C4_SMBA,USART3_CTS,QUADSPI_BK1_IO0,SAI2_SD_A,FMC_A16,FMC_CLE,EVENTOUT)
- net GND: now also U1002.107 (VSS), U1002.120 (VSS), U1002.130 (VSS), U1002.16 (VSS), U1002.31 (VSSA), U1002.38 (VSS), U1002.51 (VSS), U1002.61 (VSS), U1002.83 (VSS), U1002.94 (VSS), C1001.2, C1002.2, C1003.2, C1004.2, C1005.2, C1006.2, C1007.2, C1008.2, C1009.2, C1010.2, C1011.2, C1012.2, C1013.2, C1014.2, C1015.2, C1016.2, C1017.2, C1018.2, C1019.2, C1020.2, C1021.2, C1022.2, J1001.2 (Pin_2), R1009.2, U1001.2 (GND)
- net NRST: now also U1002.25 (NRST), C1022.1, R1010.2
- net TCK_SWCLK: now also U1002.109 (PA14,JTCK-SWCLK,EVENTOUT)
- net TMS_SWDIO: now also U1002.105 (PA13,JTMS-SWDIO,EVENTOUT)
- net SENS_SCL: now reaches U1002.100 (PA8,MCO1,TIM1_CH1,TIM8_BKIN2,I2C3_SCL,USART1_CK,OTG_FS_SOF,CAN3_RX,UART7_RX,LCD_B3,LCD_R6,EVENTOUT)
- net SENS_SCL: now also R1004.2, U1001.6 (SCL)
- net at U1002.106 (VCAP_2): now also C1008.1
- net MCU_DEFAULT: now reaches U1002.116 (PD2,TRACED2,TIM3_ETR,UART5_RX,SDMMC1_CMD,DCMI_D11,EVENTOUT)
- net MCU_DEFAULT: now also J1001.1 (Pin_1), R1002.1
- net LED_BLUE: now reaches U1002.123 (PD7,DFSDM1_DATIN4,SPI1_MOSI,I2S1_SD,DFSDM1_CKIN1,USART2_CK,SPDIF_RX0,SDMMC2_CMD,FMC_NE1,EVENTOUT)
- net LED_BLUE: now also R1001.1
- net LED_RED: now reaches U1002.124 (PG9,SPI1_MISO,SPDIF_RX3,USART6_RX,QUADSPI_BK2_IO2,SAI2_FS_B,SDMMC2_D0,FMC_NE2,FMC_NCE,DCMI_VSYNC,EVENTOUT)
- net LED_RED: now also R1003.1
- net LED_GREEN: now reaches U1002.125 (PG10,SPI1_NSS,I2S1_WS,LCD_G3,SAI2_SD_B,SDMMC2_D1,FMC_NE3,DCMI_D2,LCD_B2,EVENTOUT)
- net LED_GREEN: now also R1005.1
- net RMII_TXEN: now reaches U1002.126 (PG11,SPI1_SCK,I2S1_CK,SPDIF_RX0,SDMMC2_D2,ETH_MII_TX_EN,ETH_RMII_TX_EN,DCMI_D3,LCD_B3,EVENTOUT)
- net RMII_TXD0: now reaches U1002.128 (PG13,TRACED0,LPTIM1_OUT,SPI6_SCK,USART6_CTS,ETH_MII_TXD0,ETH_RMII_TXD0,FMC_A24,LCD_R0,EVENTOUT)
- net RMII_TXD1: now reaches U1002.129 (PG14,TRACED1,LPTIM1_ETR,SPI6_MOSI,USART6_TX,QUADSPI_BK2_IO3,ETH_MII_TXD1,ETH_RMII_TXD1,FMC_A25,LCD_B0,EVENTOUT)
- net at U1002.138 (BOOT0): now also R1009.1
- net at U1002.23 (PH0,EVENTOUT,OSC_IN): now also C1004.1, Y1001.1
- net at U1002.24 (PH1,EVENTOUT,OSC_OUT): now also C1007.1, Y1001.2
- net RMII_MDC: now reaches U1002.27 (PC1,TRACED0,_DFSDM1_DATIN0,SPI2_MOSI,I2S2_SD,SAI1_SD_A,DFSDM1_CKIN4,ETH_MDC,MDIOS_MDC,EVENTOUT,ADC1_IN11,ADC2_IN11,ADC3_IN11,RTC_TAMP3,WKUP3)
- net MCU_VDDA: now reaches U1002.32 (VREF+)
- net MCU_VDDA: now also U1002.33 (VDDA), C1021.1, FB1001.1
- net REF_CLK: now reaches U1002.35 (PA1,TIM2_CH2,TIM5_CH2,UART2_RTS,UART4_RX,QUADSPI_BK1_IO3,SAI2_MCLK_B,ETH_MII_RX_CLK,ETH_RMII_REF_CLK,LCD_R2,EVENTOUT,ADC1_IN1,ADC2_IN1,ADC3_IN1)
- net RMII_MDIO: now reaches U1002.36 (PA2,TIM2_CH3,TIM5_CH3,TIM9_CH1,USART2_TX,SAI2_SCK_B,ETH_MDIO,MDIOS_MDIO,LCD_R1,EVENTOUT,ADC1_IN2,ADC2_IN2,ADC3_IN2,WKUP2)
- net RMII_CRS_DV: now reaches U1002.43 (PA7,TIM1_CH1N,TIM3_CH2,TIM8_CH1N,SPI1_MOSI,I2S1_SD,SPI6_MOSI,TIM14_CH1,ETH_MII_RX_DV,ETH_RMII_CRS_DV,FMC_SDNWE,EVENTOUT,ADC1_IN7,ADC2_IN7)
- net RMII_RXD0: now reaches U1002.44 (PC4,DFSDM1_CKIN2,I2S1_MCK,SPDIF_RX2,ETH_MII_RXD0,ETH_RMII_RXD0,FMC_SDNE0,EVENTOUT,ADC1_IN14,ADC2_IN14)
- net RMII_RXD1: now reaches U1002.45 (PC5,DFSDM1_DATIN2,SPDIF_RX3,ETH_MII_RXD1,ETH_RMII_RXD1,FMC_SDCKE0,EVENTOUT,ADC1_IN15,ADC2_IN15)
- net TRIG_EN: now reaches U1002.60 (PE9,TIM1_CH1,DFSDM1_CKOUT,UART7_RTS,QUADSPI_BK2_IO2,FMC_D6,EVENTOUT)
- net TRIG_OUT: now reaches U1002.63 (PE10,TIM1_CH2N,DFSDM1_DATIN4,UART7_CTS,QUADSPI_BK2_IO3,FMC_D7,EVENTOUT)
- net TRIG_IN: now reaches U1002.64 (PE11,TIM1_CH2,SPI4_NSS,DFSDM1_CKIN4,SAI2_SD_B,FMC_D8,LCD_G3,EVENTOUT)
- net CXN_REL5: now reaches U1002.66 (PE13,TIM1_CH3,SPI4_MISO,DFSDM1_CKIN5,SAI2_FS_B,FMC_D10,LCD_DE,EVENTOUT)
- net CXN_REL4: now reaches U1002.67 (PE14,TIM1_CH4,SPI4_MOSI,SAI2_MCLK_B,FMC_D11,LCD_CLK,EVENTOUT)
- net CXN_REL3: now reaches U1002.68 (PE15,TIM1_BKIN,FMC_D12,LCD_R7,EVENTOUT)
- net CXN_REL2: now reaches U1002.69 (PB10,TIM2_CH3,I2C2_SCL,SPI2_SCK,I2S2_CK,DFSDM1_DATIN7,USART3_TX,QUADSPI_BK1_NCS,OTG_HS_ULPI_D3,ETH_MII_RX_ER,LCD_G4,EVENTOUT)
- net CXN_REL1: now reaches U1002.70 (PB11,TIM2_CH4,I2C2_SDA,DFSDM1_CKIN7,USART3_RX,OTG_HS_ULPI_D4,ETH_MII_TX_EN,ETH_RMII_TX_EN,_DSI_TE,LCD_G5,EVENTOUT)
- net at U1002.71 (VCAP_1): now also C1005.1
- net SENS_SDA: now reaches U1002.99 (PC9,MCO2,TIM3_CH4,TIM8_CH4,I2C3_SDA,I2S_CKIN,UART5_CTS,QUADSPI_BK1_IO0,LCD_G3,SDMMC1_D1,DCMI_D3,LCD_B2,EVENTOUT)
- net SENS_SDA: now also R1006.2, U1001.1 (SDA)
- new net: D1003.1 (K), R1005.2
- new net: D1001.1 (K), R1001.2
- new net: D1002.1 (K), R1003.2
Other:
- moved on the sheet: U1002

Commit message: Hardware design.
Parts:
- renumbered C1001 to C134, C1002 to C135, C1003 to C136, C1004 to C137, C1005 to C138, C1006 to C139, C1007 to C140, C1008 to C141, C1009 to C142, C1010 to C143, C1011 to C144, C1012 to C145, C1013 to C146, C1014 to C147, C1015 to C148, C1016 to C149, C1017 to C150, C1018 to C151, C1019 to C152, C1020 to C153, C1021 to C154, C1022 to C155, D1001 to D12, D1002 to D13, D1003 to D14, FB1001 to FB2, J1001 to J2, J1002 to J3, R1008 to R100, R1009 to R101, R1010 to R102, R1001 to R93, R1002 to R94, R1003 to R95, R1004 to R96, R1005 to R97, R1006 to R98, R1007 to R99, U1001 to U43, U1002 to U44, U1003 to U45, Y1001 to Y2

Commit message: Hardware design.
Parts:
- renumbered R99 to R100, R100 to R101, R101 to R102, R102 to R103, R93 to R94, R94 to R95, R95 to R96, R96 to R97, R97 to R98, R98 to R99
Changed lines of the file:
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@@
   (symbol (lib_id "Device:R") (at 39.37 247.65 180) (unit 1)
     (in_bom yes) (on_board yes)
-    (property "Reference" "R97" (id 0) (at 44.6278 247.65 90))
+    (property "Reference" "R98" (id 0) (at 44.6278 247.65 90))
     (property "Value" "680" (id 1) (at 42.3164 247.65 90))
     (property "Footprint" "Resistor_SMD:R_0603_1608Metric_Pad0.98x0.95mm_HandSolder" (id 2) (at 41.148 247.65 90)
@@
   (symbol (lib_id "Device:R") (at 19.05 247.65 180) (unit 1)
     (in_bom yes) (on_board yes)
-    (property "Reference" "R93" (id 0) (at 24.3078 247.65 90))
+    (property "Reference" "R94" (id 0) (at 24.3078 247.65 90))
     (property "Value" "680" (id 1) (at 21.9964 247.65 90))
     (property "Footprint" "Resistor_SMD:R_0603_1608Metric_Pad0.98x0.95mm_HandSolder" (id 2) (at 20.828 247.65 90)
@@
   (symbol (lib_id "Device:R") (at 372.11 226.06 0) (unit 1)
     (in_bom yes) (on_board yes)
-    (property "Reference" "R101" (id 0) (at 373.888 224.8916 0)
+    (property "Reference" "R102" (id 0) (at 373.888 224.8916 0)
       (effects (font (size 1.27 1.27)) (justify left))
     )
@@
   (symbol (lib_id "Device:R") (at 43.18 157.48 0) (unit 1)
     (in_bom yes) (on_board yes)
-    (property "Reference" "R98" (id 0) (at 44.958 156.3116 0)
+    (property "Reference" "R99" (id 0) (at 44.958 156.3116 0)
       (effects (font (size 1.27 1.27)) (justify left))
     )
@@
   (symbol (lib_id "Device:R") (at 281.94 260.35 0) (unit 1)
     (in_bom yes) (on_board yes)
-    (property "Reference" "R100" (id 0) (at 283.718 259.1816 0)
+    (property "Reference" "R101" (id 0) (at 283.718 259.1816 0)
       (effects (font (size 1.27 1.27)) (justify left))
     )
@@
   (symbol (lib_id "Device:R") (at 271.78 260.35 0) (unit 1)
     (in_bom yes) (on_board yes)
-    (property "Reference" "R99" (id 0) (at 273.558 259.1816 0)
+    (property "Reference" "R100" (id 0) (at 273.558 259.1816 0)
       (effects (font (size 1.27 1.27)) (justify left))
     )
@@
   (symbol (lib_id "Device:R") (at 29.21 247.65 180) (unit 1)
     (in_bom yes) (on_board yes)
-    (property "Reference" "R95" (id 0) (at 34.4678 247.65 90))
+    (property "Reference" "R96" (id 0) (at 34.4678 247.65 90))
     (property "Value" "560" (id 1) (at 32.1564 247.65 90))
     (property "Footprint" "Resistor_SMD:R_0603_1608Metric_Pad0.98x0.95mm_HandSolder" (id 2) (at 30.988 247.65 90)
@@
   (symbol (lib_id "Device:R") (at 33.02 157.48 0) (unit 1)
     (in_bom yes) (on_board yes)
-    (property "Reference" "R96" (id 0) (at 34.798 156.3116 0)
+    (property "Reference" "R97" (id 0) (at 34.798 156.3116 0)
       (effects (font (size 1.27 1.27)) (justify left))
     )
@@
   (symbol (lib_id "Device:R") (at 383.54 215.9 0) (unit 1)
     (in_bom yes) (on_board yes)
-    (property "Reference" "R102" (id 0) (at 385.318 214.7316 0)
+    (property "Reference" "R103" (id 0) (at 385.318 214.7316 0)
       (effects (font (size 1.27 1.27)) (justify left))
     )
@@
   (symbol (lib_id "Device:R") (at 20.32 194.31 180) (unit 1)
     (in_bom yes) (on_board yes)
-    (property "Reference" "R94" (id 0) (at 22.098 193.1416 0)
+    (property "Reference" "R95" (id 0) (at 22.098 193.1416 0)
       (effects (font (size 1.27 1.27)) (justify right))
     )
