File: HARDWARE/ETH1CSMU2/MCU.kicad_sch (KiCad schematic)
At the start: 42 parts, among them J2 Conn_02x01, J3 20021111-00010T4LF, U43 HDC1080, U44 STM32F746ZG, U45 24LC08B-E/MS, Y2 X

Commit message: Hardware design
Parts:
- C137, C140: value 8p -> 6p
- U44: footprint (none) -> ETH1CSMU2:TQFP-144_20x20mm_P0.5mm
- Y2: value X -> ECS-080-18-23A-JGN-TR; footprint ETH1CLCR2:NX3225GD -> Crystal:Crystal_SMD_0603-2Pin_6.0x3.5mm_HandSoldering
Other:
- moved on the sheet: C137, C140, Y2
Changed lines of the file:
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@@
   (junction (at 252.73 21.59) (diameter 0) (color 0 0 0 0)
   )
-  (junction (at 53.34 43.18) (diameter 0) (color 0 0 0 0)
+  (junction (at 43.18 43.18) (diameter 0) (color 0 0 0 0)
   )
   (junction (at 207.01 21.59) (diameter 0) (color 0 0 0 0)
@@
   (junction (at 106.68 266.7) (diameter 0) (color 0 0 0 0)
   )
-  (junction (at 59.69 33.02) (diameter 0) (color 0 0 0 0)
+  (junction (at 49.53 33.02) (diameter 0) (color 0 0 0 0)
   )
   (junction (at 234.95 267.97) (diameter 0) (color 0 0 0 0)
@@
   (junction (at 30.48 276.86) (diameter 0) (color 0 0 0 0)
   )
-  (junction (at 59.69 22.86) (diameter 0) (color 0 0 0 0)
+  (junction (at 49.53 22.86) (diameter 0) (color 0 0 0 0)
   )
   (junction (at 281.94 255.27) (diameter 0) (color 0 0 0 0)
@@
     (stroke (width 0) (type default) (color 0 0 0 0))
   )
-  (wire (pts (xy 82.55 33.02) (xy 59.69 33.02))
+  (wire (pts (xy 82.55 33.02) (xy 49.53 33.02))
     (stroke (width 0) (type default) (color 0 0 0 0))
   )
@@
     (stroke (width 0) (type default) (color 0 0 0 0))
   )
-  (wire (pts (xy 81.28 22.86) (xy 59.69 22.86))
+  (wire (pts (xy 81.28 22.86) (xy 49.53 22.86))
     (stroke (width 0) (type default) (color 0 0 0 0))
   )
@@
     (stroke (width 0) (type default) (color 0 0 0 0))
   )
-  (wire (pts (xy 46.99 43.18) (xy 53.34 43.18))
+  (wire (pts (xy 36.83 43.18) (xy 43.18 43.18))
     (stroke (width 0) (type default) (color 0 0 0 0))
   )
@@
     (stroke (width 0) (type default) (color 0 0 0 0))
   )
-  (wire (pts (xy 59.69 31.75) (xy 59.69 33.02))
+  (wire (pts (xy 49.53 31.75) (xy 49.53 33.02))
     (stroke (width 0) (type default) (color 0 0 0 0))
   )
@@
     (stroke (width 0) (type default) (color 0 0 0 0))
   )
-  (wire (pts (xy 59.69 43.18) (xy 59.69 41.91))
+  (wire (pts (xy 49.53 43.18) (xy 49.53 41.91))
     (stroke (width 0) (type default) (color 0 0 0 0))
   )
@@
     (stroke (width 0) (type default) (color 0 0 0 0))
   )
-  (wire (pts (xy 59.69 33.02) (xy 59.69 34.29))
+  (wire (pts (xy 49.53 33.02) (xy 49.53 34.29))
     (stroke (width 0) (type default) (color 0 0 0 0))
   )
@@
     (stroke (width 0) (type default) (color 0 0 0 0))
   )
-  (wire (pts (xy 53.34 43.18) (xy 59.69 43.18))
+  (wire (pts (xy 43.18 43.18) (xy 49.53 43.18))
     (stroke (width 0) (type default) (color 0 0 0 0))
   )
@@
     (stroke (width 0) (type default) (color 0 0 0 0))
   )
-  (wire (pts (xy 53.34 44.45) (xy 53.34 43.18))
+  (wire (pts (xy 43.18 44.45) (xy 43.18 43.18))
     (stroke (width 0) (type default) (color 0 0 0 0))
   )
@@
     (stroke (width 0) (type default) (color 0 0 0 0))
   )
-  (wire (pts (xy 59.69 22.86) (xy 46.99 22.86))
-    (stroke (width 0) (type default) (color 0 0 0 0))
-  )
-  (wire (pts (xy 46.99 22.86) (xy 46.99 34.29))
+  (wire (pts (xy 49.53 22.86) (xy 36.83 22.86))
+    (stroke (width 0) (type default) (color 0 0 0 0))
+  )
+  (wire (pts (xy 36.83 22.86) (xy 36.83 34.29))
     (stroke (width 0) (type default) (color 0 0 0 0))
   )
@@
     (stroke (width 0) (type default) (color 0 0 0 0))
   )
-  (wire (pts (xy 59.69 24.13) (xy 59.69 22.86))
+  (wire (pts (xy 49.53 24.13) (xy 49.53 22.86))
     (stroke (width 0) (type default) (color 0 0 0 0))
   )
@@
     (stroke (width 0) (type default) (color 0 0 0 0))
   )
-  (wire (pts (xy 46.99 41.91) (xy 46.99 43.18))
+  (wire (pts (xy 36.83 41.91) (xy 36.83 43.18))
     (stroke (width 0) (type default) (color 0 0 0 0))
   )
@@
     (pin "2")
   )
-  (symbol (lib_id "power:GND") (at 53.34 44.45 0) (unit 1)
-    (in_bom yes) (on_board yes)
-    (property "Reference" "#PWR0258" (id 0) (at 53.34 50.8 0)
-      (effects (font (size 1.27 1.27)) hide)
-    )
-    (property "Value" "GND" (id 1) (at 53.467 48.8442 0))
-    (property "Footprint" "" (id 2) (at 53.34 44.45 0)
-      (effects (font (size 1.27 1.27)) hide)
-    )
-    (property "Datasheet" "" (id 3) (at 53.34 44.45 0)
-      (effects (font (size 1.27 1.27)) hide)
-    )
-    (pin "1")
-  )
-  (symbol (lib_id "Device:C") (at 46.99 38.1 0) (unit 1)
-    (in_bom yes) (on_board yes)
-    (property "Reference" "C137" (id 0) (at 49.911 36.9316 0)
-      (effects (font (size 1.27 1.27)) (justify left))
-    )
-    (property "Value" "8p" (id 1) (at 49.911 39.243 0)
-      (effects (font (size 1.27 1.27)) (justify left))
-    )
-    (property "Footprint" "Capacitor_SMD:C_0603_1608Metric_Pad1.08x0.95mm_HandSolder" (id 2) (at 47.9552 41.91 0)
-      (effects (font (size 1.27 1.27)) hide)
-    )
-    (property "Datasheet" "~" (id 3) (at 46.99 38.1 0)
-      (effects (font (size 1.27 1.27)) hide)
-    )
-    (pin "1")
-    (pin "2")
-  )
-  (symbol (lib_id "Device:C") (at 59.69 38.1 0) (unit 1)
-    (in_bom yes) (on_board yes)
-    (property "Reference" "C140" (id 0) (at 62.611 36.9316 0)
-      (effects (font (size 1.27 1.27)) (justify left))
-    )
-    (property "Value" "8p" (id 1) (at 62.611 39.243 0)
-      (effects (font (size 1.27 1.27)) (justify left))
-    )
-    (property "Footprint" "Capacitor_SMD:C_0603_1608Metric_Pad1.08x0.95mm_HandSolder" (id 2) (at 60.6552 41.91 0)
-      (effects (font (size 1.27 1.27)) hide)
-    )
-    (property "Datasheet" "~" (id 3) (at 59.69 38.1 0)
+  (symbol (lib_id "power:GND") (at 43.18 44.45 0) (unit 1)
+    (in_bom yes) (on_board yes)
+    (property "Reference" "#PWR0258" (id 0) (at 43.18 50.8 0)
+      (effects (font (size 1.27 1.27)) hide)
+    )
+    (property "Value" "GND" (id 1) (at 43.307 48.8442 0))
+    (property "Footprint" "" (id 2) (at 43.18 44.45 0)
+      (effects (font (size 1.27 1.27)) hide)
+    )
+    (property "Datasheet" "" (id 3) (at 43.18 44.45 0)
+      (effects (font (size 1.27 1.27)) hide)
+    )
+    (pin "1")
+  )
+  (symbol (lib_id "Device:C") (at 36.83 38.1 0) (unit 1)
+    (in_bom yes) (on_board yes)
+    (property "Reference" "C137" (id 0) (at 39.751 36.9316 0)
+      (effects (font (size 1.27 1.27)) (justify left))
+    )
+    (property "Value" "6p" (id 1) (at 39.751 39.243 0)
+      (effects (font (size 1.27 1.27)) (justify left))
+    )
+    (property "Footprint" "Capacitor_SMD:C_0603_1608Metric_Pad1.08x0.95mm_HandSolder" (id 2) (at 37.7952 41.91 0)
+      (effects (font (size 1.27 1.27)) hide)
+    )
+    (property "Datasheet" "~" (id 3) (at 36.83 38.1 0)
+      (effects (font (size 1.27 1.27)) hide)
+    )
+    (pin "1")
+    (pin "2")
+  )
+  (symbol (lib_id "Device:C") (at 49.53 38.1 0) (unit 1)
+    (in_bom yes) (on_board yes)
+    (property "Reference" "C140" (id 0) (at 52.451 36.9316 0)
+      (effects (font (size 1.27 1.27)) (justify left))
+    )
+    (property "Value" "6p" (id 1) (at 52.451 39.243 0)
+      (effects (font (size 1.27 1.27)) (justify left))
+    )
+    (property "Footprint" "Capacitor_SMD:C_0603_1608Metric_Pad1.08x0.95mm_HandSolder" (id 2) (at 50.4952 41.91 0)
+      (effects (font (size 1.27 1.27)) hide)
+    )
+    (property "Datasheet" "~" (id 3) (at 49.53 38.1 0)
       (effects (font (size 1.27 1.27)) hide)
     )
@@
       (effects (font (size 1.27 1.27)) (justify left))
     )
-    (property "Footprint" "" (id 2) (at 631.19 87.63 0)
+    (property "Footprint" "ETH1CSMU2:TQFP-144_20x20mm_P0.5mm" (id 2) (at 631.19 87.63 0)
       (effects (font (size 1.27 1.27)) hide)
     )
@@
     (pin "2")
   )
-  (symbol (lib_id "Device:Crystal") (at 59.69 27.94 270) (unit 1)
-    (in_bom yes) (on_board yes)
-    (property "Reference" "Y2" (id 0) (at 63.0174 26.7716 90)
-      (effects (font (size 1.27 1.27)) (justify left))
-    )
-    (property "Value" "X" (id 1) (at 63.0174 29.083 90)
-      (effects (font (size 1.27 1.27)) (justify left))
-    )
-    (property "Footprint" "ETH1CLCR2:NX3225GD" (id 2) (at 59.69 27.94 0)
-      (effects (font (size 1.27 1.27)) hide)
-    )
-    (property "Datasheet" "~" (id 3) (at 59.69 27.94 0)
-      (effects (font (size 1.27 1.27)) hide)
-    )
+  (symbol (lib_id "Device:Crystal") (at 49.53 27.94 270) (unit 1)
+    (in_bom yes) (on_board yes)
+    (property "Reference" "Y2" (id 0) (at 52.8574 26.7716 90)
+      (effects (font (size 1.27 1.27)) (justify left))
+    )
+    (property "Value" "ECS-080-18-23A-JGN-TR" (id 1) (at 52.8574 29.083 90)
+      (effects (font (size 1.27 1.27)) (justify left))
+    )
+    (property "Footprint" "Crystal:Crystal_SMD_0603-2Pin_6.0x3.5mm_HandSoldering" (id 2) (at 49.53 27.94 0)
+      (effects (font (size 1.27 1.27)) hide)
+    )
+    (property "Datasheet" "~" (id 3) (at 49.53 27.94 0)
+      (effects (font (size 1.27 1.27)) hide)
+    )

Commit message: Hardware design
Parts:
- renumbered C134 to C1001, C135 to C1002, C137 to C1003, C136 to C1004, C140 to C1005, C138 to C1006, C139 to C1007, C141 to C1008, C142 to C1009, C143 to C1010, C144 to C1011, C145 to C1012, C146 to C1013, C147 to C1014, C148 to C1015, C149 to C1016, C150 to C1017, C151 to C1018, C152 to C1019, C153 to C1020, C154 to C1021, C155 to C1022, D12 to D1001, D13 to D1002, D14 to D1003, FB2 to FB1001, J2 to J1001, J3 to J1002, R94 to R1001, R95 to R1002, R96 to R1003, R97 to R1004, R98 to R1005, R99 to R1006, R100 to R1007, R101 to R1008, R102 to R1009, R103 to R1010, U43 to U1001, U44 to U1002, U45 to U1003, Y2 to Y1001
