File: HARDWARE/ETH1CSMU2/MCU.kicad_sch (KiCad schematic)
At the start: 42 parts, among them J1001 Conn_02x01, J1002 20021111-00010T4LF, U1001 HDC1080, U1002 STM32F746ZG, U1003 24LC08B-E/MS, Y1001 ECS-080-18-23A-JGN-TR

Commit message: Hardware and software development
Connections:
- net SPI4_SCK: now reaches U1002.1 (PE2,TRACECLK,SPI4_SCK,SAI1_MCLK_A,QUADSPI_BK1_IO2,ETH_MII_TXD3,FMC_A23,EVENTOUT)
- net MCU_nISNK: now reaches U1002.10 (PF0,I2C2_SDA,FMC_A0,EVENTOUT)
- net MCU_nISRC: now reaches U1002.11 (PF1,I2C2_SCL,FMC_A1,EVENTOUT)
- net SPI3_NSS: now reaches U1002.110 (PA15,JTDI,TIM2_CH1,TIM2_ETR,HDMI_CEC,SPI1_NSS,I2S1_WS,SPI3_NSS,I2S3_WS,SPI6_NSS,UART4_RTS,CAN3_TX,UART7_TX,EVENTOUT)
- net SPI3_SCK: now reaches U1002.111 (PC10,DFSDM1_CKIN5,SPI3_SCK,I2S3_CK,USART3_TX,UART4_TX,QUADSPI_BK1_IO1,SDMMC1_D2,DCMI_D8,LCD_R2,EVENTOUT)
- net SPI3_MISO: now reaches U1002.112 (PC11,DFSDM1_DATIN5,SPI3_MISO,USART3_RX,UART4_RX,QUADSPI_BK2_NCS,SDMMC1_D3,DCMI_D4,EVENTOUT)
- net SPI3_MOSI: now reaches U1002.113 (PC12,TRACED3,SPI3_MOSI,I2S3_SD,USART3_CK,UART5_TX,SDMMC1_CK,DCMI_D9,EVENTOUT)
- net MCU_nTDS: now reaches U1002.12 (PF2,I2C2_SMBA,FMC_A2,EVENTOUT)
- net SPI1_MOSI: now reaches U1002.135 (PB5,UART5_RX,TIM3_CH2,I2C1_SMBA,SPI1_MOSI,I2S1_SD,SPI3_MOSI,I2S3_SD,SPI6_MOSI,CAN2_RX,OTG_HS_ULPI_D7,ETH_PPS_OUT,FMC_SDCKE1,DCMI_D10,LCD_G7,EVENTOUT)
- net ADC1_RVS2: now reaches U1002.15 (PF5,FMC_A5,EVENTOUT,ADC3_IN15)
- net SPI5_NSS: now reaches U1002.18 (PF6,TIM10_CH1,SPI5_NSS,SAI1_SD_B,UART7_RX,QUADSPI_BK1_IO3,EVENTOUT,ADC3_IN4)
- net SPI5_SCK: now reaches U1002.19 (PF7,TIM11_CH1,SPI5_SCK,SAI1_MCLK_B,UART7_TX,QUADSPI_BK1_IO2,EVENTOUT,ADC3_IN5)
- net SPI5_MISO: now reaches U1002.20 (PF8,SPI5_MISO,SAI1_SCK_B,UART7_RTS,TIM13_CH1,QUADSPI_BK1_IO0,EVENTOUT,ADC3_IN6)
- net SPI5_MOSI: now reaches U1002.21 (PF9,SPI5_MOSI,SAI1_FS_B,UART7_CTS,TIM14_CH1,QUADSPI_BK1_IO1,EVENTOUT,ADC3_IN7)
- net ADC1_RVS1: now reaches U1002.22 (PF10,QUADSPI_CLK,DCMI_D11,LCD_DE,EVENTOUT,ADC3_IN8)
- net SPI4_NSS: now reaches U1002.3 (PE4,TRACED1,SPI4_NSS,SAI1_FS_A,DFSDM1_DATIN3,FMC_A20,DCMI_D4,LCD_B0,EVENTOUT)
- net SPI4_MISO: now reaches U1002.4 (PE5,TRACED2,TIM9_CH1,SPI4_MISO,SAI1_SCK_A,DFSDM1_CKIN3,FMC_A21,DCMI_D6,LCD_G0,EVENTOUT)
- net SPI1_NSS: now reaches U1002.40 (PA4,SPI1_NSS,I2S1_WS,SPI3_NSS,I2S3_WS,USART2_CK,SPI6_NSS,OTG_HS_SOF,DCMI_HSYNC,LCD_VSYNC,EVENTOUT,ADC1_IN4,ADC2_IN4,DAC_OUT1)
- net SPI1_SCK: now reaches U1002.41 (PA5,TIM2_CH1,TIM2_ETR,TIM8_CH1N,SPI1_SCK,I2S1_CK,SPI6_SCK,OTG_HS_ULPI_CK,LCD_R4,EVENTOUT,ADC1_IN5,ADC2_IN5,DAC_OUT2)
- net SPI1_MISO: now reaches U1002.42 (PA6,TIM1_BKIN,TIM3_CH1,TIM8_BKIN,SPI1_MISO,SPI6_MISO,TIM13_CH1,MDIOS_MDC,DCMI_PIXCLK,LCD_G2,EVENTOUT,ADC1_IN6,ADC2_IN6)
- net SPI4_MOSI: now reaches U1002.5 (PE6,TRACED3,TIM1_BKIN2,TIM9_CH2,SPI4_MOSI,SAI1_SD_A,SAI2_MCLK_B,FMC_A22,DCMI_D7,LCD_G1,EVENTOUT)
- net DDS_DIV2: now reaches U1002.50 (PF12,FMC_A6,EVENTOUT)
- net DDS_DIV4: now reaches U1002.53 (PF13,I2C4_SMBA,DFSDM1_DATIN6,FMC_A7,EVENTOUT)
- net DDS_DIV8: now reaches U1002.54 (PF14,I2C4_SCL,DFSDM1_CKIN6,FMC_A8,EVENTOUT)
- net ~{DDS_DIV10}: now reaches U1002.55 (PF15,I2C4_SDA,FMC_A9,EVENTOUT)
- net SPI2_NSS: now reaches U1002.73 (PB12,TIM1_BKIN,I2C2_SMBA,SPI2_NSS,I2S2_WS,DFSDM1_DATIN1,USART3_CK,UART5_RX,CAN2_RX,OTG_HS_ULPI_D5,ETH_MII_TXD0,ETH_RMII_TXD0,OTG_HS_ID,EVENTOUT)
- net SPI2_SCK: now reaches U1002.74 (PB13,TIM1_CH1N,SPI2_SCK,I2S2_CK,DFSDM1_CKIN1,USART3_CTS,UART5_TX,CAN2_TX,OTG_HS_ULPI_D6,ETH_MII_TXD1,ETH_RMII_TXD1,EVENTOUT,OTG_HS_VBUS)
- net SPI2_MISO: now reaches U1002.75 (PB14,TIM1_CH2N,TIM8_CH2N,USART1_TX,SPI2_MISO,DFSDM1_DATIN2,USART3_RTS,UART4_RTS,TIM12_CH1,SDMMC2_D0,OTG_HS_DM,EVENTOUT)
- net SPI2_MOSI: now reaches U1002.76 (PB15,RTC_REFIN,TIM1_CH3N,TIM8_CH3N,USART1_RX,SPI2_MOSI,I2S2_SD,DFSDM1_CKIN2,UART4_CTS,TIM12_CH2,SDMMC2_D1,OTG_HS_DP,EVENTOUT)
- net SR_CLK: now reaches U1002.87 (PG2,FMC_A12,EVENTOUT)
- net SR_DAT: now reaches U1002.88 (PG3,FMC_A13,EVENTOUT)
- net SR_LAT: now reaches U1002.89 (PG4,FMC_A14,FMC_BA0,EVENTOUT)
- net SR_OUT: now reaches U1002.90 (PG5,FMC_A15,FMC_BA1,EVENTOUT)

Commit message: CRC check
Connections:
- net ADC1_RVS1: now also U1002.34 (PA0,TIM2_CH1,TIM2_ETR,TIM5_CH1,TIM8_ETR,USART2_CTS,UART4_TX,SAI2_SD_B,ETH_MII_CRS,EVENTOUT,ADC1_IN0,ADC2_IN0,ADC3_IN0,WKUP1); no longer U1002.22 (PF10,QUADSPI_CLK,DCMI_D11,LCD_DE,EVENTOUT,ADC3_IN8)
- net ADC1_RVS2: now also U1002.37 (PA3,TIM2_CH4,TIM5_CH4,TIM9_CH2,USART2_RX,LCD_B2,OTG_HS_ULPI_D0,ETH_MII_COL,LCD_B5,EVENTOUT,ADC1_IN3,ADC2_IN3,ADC3_IN3); no longer U1002.15 (PF5,FMC_A5,EVENTOUT,ADC3_IN15)
- net CXN_REL1: now also U1002.65 (PE12,TIM1_CH3N,SPI4_SCK,DFSDM1_DATIN5,SAI2_SCK_B,FMC_D9,LCD_B4,EVENTOUT); no longer U1002.70 (PB11,TIM2_CH4,I2C2_SDA,DFSDM1_CKIN7,USART3_RX,OTG_HS_ULPI_D4,ETH_MII_TX_EN,ETH_RMII_TX_EN,_DSI_TE,LCD_G5,EVENTOUT)
- net CXN_REL2: now also U1002.64 (PE11,TIM1_CH2,SPI4_NSS,DFSDM1_CKIN4,SAI2_SD_B,FMC_D8,LCD_G3,EVENTOUT); no longer U1002.69 (PB10,TIM2_CH3,I2C2_SCL,SPI2_SCK,I2S2_CK,DFSDM1_DATIN7,USART3_TX,QUADSPI_BK1_NCS,OTG_HS_ULPI_D3,ETH_MII_RX_ER,LCD_G4,EVENTOUT)
- net TRIG_EN: now also U1002.59 (PE8,TIM1_CH1N,DFSDM1_CKIN2,UART7_TX,QUADSPI_BK2_IO1,FMC_D5,EVENTOUT); no longer U1002.60 (PE9,TIM1_CH1,DFSDM1_CKOUT,UART7_RTS,QUADSPI_BK2_IO2,FMC_D6,EVENTOUT)
- net TRIG_IN: now also U1002.63 (PE10,TIM1_CH2N,DFSDM1_DATIN4,UART7_CTS,QUADSPI_BK2_IO3,FMC_D7,EVENTOUT); no longer U1002.64 (PE11,TIM1_CH2,SPI4_NSS,DFSDM1_CKIN4,SAI2_SD_B,FMC_D8,LCD_G3,EVENTOUT)
- net TRIG_OUT: now also U1002.60 (PE9,TIM1_CH1,DFSDM1_CKOUT,UART7_RTS,QUADSPI_BK2_IO2,FMC_D6,EVENTOUT); no longer U1002.63 (PE10,TIM1_CH2N,DFSDM1_DATIN4,UART7_CTS,QUADSPI_BK2_IO3,FMC_D7,EVENTOUT)
- new net DAC1_LDAC: U1002.69 (PB10,TIM2_CH3,I2C2_SCL,SPI2_SCK,I2S2_CK,DFSDM1_DATIN7,USART3_TX,QUADSPI_BK1_NCS,OTG_HS_ULPI_D3,ETH_MII_RX_ER,LCD_G4,EVENTOUT)
- new net DAC1_~{RST}: U1002.70 (PB11,TIM2_CH4,I2C2_SDA,DFSDM1_CKIN7,USART3_RX,OTG_HS_ULPI_D4,ETH_MII_TX_EN,ETH_RMII_TX_EN,_DSI_TE,LCD_G5,EVENTOUT)
- new net DAC2_~{LDAC}: U1002.22 (PF10,QUADSPI_CLK,DCMI_D11,LCD_DE,EVENTOUT,ADC3_IN8)
- no-connect marks 4 -> 52
Changed lines of the file:
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@@
   )
   (no_connect (at 218.44 267.97))
+  (no_connect (at 372.11 33.02))
+  (no_connect (at 372.11 30.48))
+  (no_connect (at 372.11 48.26))
+  (no_connect (at 372.11 45.72))
+  (no_connect (at 82.55 66.04))
+  (no_connect (at 82.55 50.8))
+  (no_connect (at 82.55 45.72))
+  (no_connect (at 82.55 48.26))
+  (no_connect (at 82.55 104.14))
+  (no_connect (at 82.55 106.68))
+  (no_connect (at 82.55 109.22))
+  (no_connect (at 82.55 111.76))
+  (no_connect (at 82.55 124.46))
+  (no_connect (at 82.55 129.54))
+  (no_connect (at 82.55 132.08))
+  (no_connect (at 82.55 139.7))
+  (no_connect (at 82.55 142.24))
   (no_connect (at 218.44 270.51))
+  (no_connect (at 372.11 68.58))
+  (no_connect (at 372.11 60.96))
+  (no_connect (at 372.11 88.9))
+  (no_connect (at 372.11 86.36))
+  (no_connect (at 372.11 83.82))
+  (no_connect (at 372.11 50.8))
+  (no_connect (at 372.11 81.28))
+  (no_connect (at 372.11 76.2))
+  (no_connect (at 372.11 73.66))
+  (no_connect (at 372.11 162.56))
+  (no_connect (at 372.11 165.1))
+  (no_connect (at 372.11 167.64))
+  (no_connect (at 372.11 170.18))
+  (no_connect (at 372.11 175.26))
+  (no_connect (at 372.11 177.8))
+  (no_connect (at 372.11 180.34))
+  (no_connect (at 372.11 182.88))
+  (no_connect (at 372.11 96.52))
+  (no_connect (at 372.11 93.98))
+  (no_connect (at 372.11 134.62))
+  (no_connect (at 372.11 124.46))
+  (no_connect (at 372.11 119.38))
+  (no_connect (at 372.11 116.84))
+  (no_connect (at 372.11 109.22))
+  (no_connect (at 372.11 111.76))
+  (no_connect (at 372.11 99.06))
   (no_connect (at 205.74 270.51))
+  (no_connect (at 372.11 160.02))
+  (no_connect (at 82.55 144.78))
+  (no_connect (at 82.55 157.48))
+  (no_connect (at 82.55 160.02))
+  (no_connect (at 82.55 162.56))
   (no_connect (at 205.74 273.05))
   (wire (pts (xy 20.32 199.39) (xy 34.29 199.39))
@@
     (stroke (width 0) (type default) (color 0 0 0 0))
   )
+  (wire (pts (xy 372.11 185.42) (xy 373.38 185.42))
+    (stroke (width 0) (type default) (color 0 0 0 0))
+  )
   (wire (pts (xy 106.68 266.7) (xy 119.38 266.7))
     (stroke (width 0) (type default) (color 0 0 0 0))
@@
     (stroke (width 0) (type default) (color 0 0 0 0))
   )
+  (wire (pts (xy 372.11 187.96) (xy 373.38 187.96))
+    (stroke (width 0) (type default) (color 0 0 0 0))
+  )
   (wire (pts (xy 144.78 276.86) (xy 157.48 276.86))
     (stroke (width 0) (type default) (color 0 0 0 0))
@@
     (stroke (width 0) (type default) (color 0 0 0 0))
   )
-  (wire (pts (xy 373.38 142.24) (xy 372.11 142.24))
+  (wire (pts (xy 373.38 139.7) (xy 372.11 139.7))
     (stroke (width 0) (type default) (color 0 0 0 0))
   )
@@
     (stroke (width 0) (type default) (color 0 0 0 0))
   )
-  (wire (pts (xy 373.38 187.96) (xy 372.11 187.96))
+  (wire (pts (xy 373.38 147.32) (xy 372.11 147.32))
     (stroke (width 0) (type default) (color 0 0 0 0))
   )
@@
     (stroke (width 0) (type default) (color 0 0 0 0))
   )
-  (wire (pts (xy 373.38 185.42) (xy 372.11 185.42))
+  (wire (pts (xy 373.38 144.78) (xy 372.11 144.78))
     (stroke (width 0) (type default) (color 0 0 0 0))
   )
@@
     (stroke (width 0) (type default) (color 0 0 0 0))
   )
-  (wire (pts (xy 373.38 139.7) (xy 372.11 139.7))
-    (stroke (width 0) (type default) (color 0 0 0 0))
-  )
-  (wire (pts (xy 81.28 50.8) (xy 82.55 50.8))
+  (wire (pts (xy 373.38 137.16) (xy 372.11 137.16))
+    (stroke (width 0) (type default) (color 0 0 0 0))
+  )
+  (wire (pts (xy 81.28 88.9) (xy 82.55 88.9))
     (stroke (width 0) (type default) (color 0 0 0 0))
   )
@@
     (stroke (width 0) (type default) (color 0 0 0 0))
   )
-  (wire (pts (xy 372.11 144.78) (xy 373.38 144.78))
+  (wire (pts (xy 372.11 142.24) (xy 373.38 142.24))
     (stroke (width 0) (type default) (color 0 0 0 0))
   )
@@
     (stroke (width 0) (type default) (color 0 0 0 0))
   )
+  (wire (pts (xy 81.28 63.5) (xy 82.55 63.5))
+    (stroke (width 0) (type default) (color 0 0 0 0))
+  )
   (wire (pts (xy 170.18 276.86) (xy 170.18 275.59))
     (stroke (width 0) (type default) (color 0 0 0 0))
@@
     (stroke (width 0) (type default) (color 0 0 0 0))
   )
-  (wire (pts (xy 81.28 63.5) (xy 82.55 63.5))
+  (wire (pts (xy 81.28 81.28) (xy 82.55 81.28))
     (stroke (width 0) (type default) (color 0 0 0 0))
   )
@@
     (effects (font (size 1.27 1.27)) (justify right bottom))
   )
-  (hierarchical_label "ADC1_RVS1" (shape input) (at 81.28 63.5 180)
+  (hierarchical_label "ADC1_RVS1" (shape input) (at 81.28 81.28 180)
     (effects (font (size 1.27 1.27)) (justify right))
   )
@@
     (effects (font (size 1.27 1.27)) (justify right))
   )
-  (hierarchical_label "CXN_REL2" (shape output) (at 373.38 185.42 0)
-    (effects (font (size 1.27 1.27)) (justify left))
-  )
-  (hierarchical_label "ADC1_RVS2" (shape input) (at 81.28 50.8 180)
+  (hierarchical_label "CXN_REL2" (shape output) (at 373.38 144.78 0)
+    (effects (font (size 1.27 1.27)) (justify left))
+  )
+  (hierarchical_label "ADC1_RVS2" (shape input) (at 81.28 88.9 180)
     (effects (font (size 1.27 1.27)) (justify right))
   )
@@
     (effects (font (size 1.27 1.27)) (justify left))
   )
-  (hierarchical_label "CXN_REL1" (shape output) (at 373.38 187.96 0)
+  (hierarchical_label "CXN_REL1" (shape output) (at 373.38 147.32 0)
     (effects (font (size 1.27 1.27)) (justify left))
   )
@@
     (effects (font (size 1.27 1.27)) (justify right))
   )
-  (hierarchical_label "TRIG_EN" (shape output) (at 373.38 139.7 0)
+  (hierarchical_label "TRIG_EN" (shape output) (at 373.38 137.16 0)
     (effects (font (size 1.27 1.27)) (justify left))
   )
@@
     (effects (font (size 1.27 1.27)) (justify right))
   )
+  (hierarchical_label "DAC1_LDAC" (shape output) (at 373.38 185.42 0)
+    (effects (font (size 1.27 1.27)) (justify left))
+  )
   (hierarchical_label "DDS_DIV8" (shape output) (at 81.28 73.66 180)
     (effects (font (size 1.27 1.27)) (justify right))
@@
     (effects (font (size 1.27 1.27)) (justify left))
   )
+  (hierarchical_label "DAC2_~{LDAC}" (shape output) (at 81.28 63.5 180)
+    (effects (font (size 1.27 1.27)) (justify right))
+  )
   (hierarchical_label "DDS_DIV4" (shape output) (at 81.28 71.12 180)
     (effects (font (size 1.27 1.27)) (justify right))
@@
     (effects (font (size 1.27 1.27)) (justify left))
   )
-  (hierarchical_label "TRIG_OUT" (shape output) (at 373.38 142.24 0)
+  (hierarchical_label "TRIG_OUT" (shape output) (at 373.38 139.7 0)
+    (effects (font (size 1.27 1.27)) (justify left))
+  )
+  (hierarchical_label "DAC1_~{RST}" (shape output) (at 373.38 187.96 0)
     (effects (font (size 1.27 1.27)) (justify left))
   )
@@
     (effects (font (size 1.27 1.27)) (justify left))
   )
-  (hierarchical_label "TRIG_IN" (shape input) (at 373.38 144.78 0)
-    (effects (font (size 1.27 1.27)) (justify left))
-  )
+  (hierarchical_label "TRIG_IN" (shape input) (at 373.38 142.24 0)
+    (effects (font (size 1.27 1.27)) (justify left))
+  )

Commit message: Hardware design.
Connections:
- net MCU_CURR_SENS_100R: now reaches U1002.91 (PG6,FMC_NE3,DCMI_D12,LCD_R7,EVENTOUT)
- net MCU_CURR_SENS_10R: now reaches U1002.92 (PG7,SAI1_MCLK_A,USART6_CK,FMC_INT,DCMI_D13,LCD_CLK,EVENTOUT)
- net MCU_CURR_SENS_1R: now reaches U1002.93 (PG8,SPI6_NSS,SPDIF_RX2,USART6_RTS,ETH_PPS_OUT,FMC_SDCLK,LCD_G7,EVENTOUT)
- no-connect marks 52 -> 49
Changed lines of the file:
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@@
   (no_connect (at 372.11 33.02))
   (no_connect (at 372.11 30.48))
-  (no_connect (at 372.11 48.26))
-  (no_connect (at 372.11 45.72))
   (no_connect (at 82.55 66.04))
   (no_connect (at 82.55 50.8))
@@
   (no_connect (at 372.11 86.36))
   (no_connect (at 372.11 83.82))
-  (no_connect (at 372.11 50.8))
   (no_connect (at 372.11 81.28))
   (no_connect (at 372.11 76.2))
@@
     (stroke (width 0) (type default) (color 0 0 0 0))
   )
+  (wire (pts (xy 372.11 50.8) (xy 373.38 50.8))
+    (stroke (width 0) (type default) (color 0 0 0 0))
+  )
   (wire (pts (xy 68.58 266.7) (xy 81.28 266.7))
     (stroke (width 0) (type default) (color 0 0 0 0))
@@
     (stroke (width 0) (type default) (color 0 0 0 0))
   )
+  (wire (pts (xy 372.11 45.72) (xy 373.38 45.72))
+    (stroke (width 0) (type default) (color 0 0 0 0))
+  )
   (wire (pts (xy 247.65 21.59) (xy 252.73 21.59))
     (stroke (width 0) (type default) (color 0 0 0 0))
@@
   )
   (wire (pts (xy 212.09 22.86) (xy 212.09 21.59))
+    (stroke (width 0) (type default) (color 0 0 0 0))
+  )
+  (wire (pts (xy 372.11 48.26) (xy 373.38 48.26))
     (stroke (width 0) (type default) (color 0 0 0 0))
   )
@@
     (effects (font (size 1.27 1.27)) (justify left))
   )
+  (hierarchical_label "MCU_CURR_SENS_1R" (shape output) (at 373.38 50.8 0)
+    (effects (font (size 1.27 1.27)) (justify left))
+  )
   (hierarchical_label "RMII_MDIO" (shape bidirectional) (at 81.28 86.36 180)
     (effects (font (size 1.27 1.27)) (justify right))
@@
     (effects (font (size 1.27 1.27)) (justify left))
   )
+  (hierarchical_label "MCU_CURR_SENS_10R" (shape output) (at 373.38 48.26 0)
+    (effects (font (size 1.27 1.27)) (justify left))
+  )
   (hierarchical_label "DDS_DIV8" (shape output) (at 81.28 73.66 180)
     (effects (font (size 1.27 1.27)) (justify right))
@@
     (effects (font (size 1.27 1.27)) (justify left))
   )
+  (hierarchical_label "MCU_CURR_SENS_100R" (shape output) (at 373.38 45.72 0)
+    (effects (font (size 1.27 1.27)) (justify left))
+  )

Commit message: Hardware design
Connections:
- net SR_CLK: now also U1002.117 (PD3,DFSDM1_CKOUT,SPI2_SCK,I2S2_CK,DFSDM1_DATIN0,USART2_CTS,FMC_CLK,DCMI_D5,LCD_G7,EVENTOUT); no longer U1002.87 (PG2,FMC_A12,EVENTOUT)
- net SR_DAT: now also U1002.118 (PD4,DFSDM1_CKIN0,USART2_RTS,FMC_NOE,EVENTOUT); no longer U1002.88 (PG3,FMC_A13,EVENTOUT)
- net SR_LAT: now also U1002.119 (PD5,USART2_TX,FMC_NWE,EVENTOUT); no longer U1002.89 (PG4,FMC_A14,FMC_BA0,EVENTOUT)
- net SR_OUT: now also U1002.122 (PD6,DFSDM1_CKIN4,SPI3_MOSI,I2S3_SD,SAI1_SD_A,USART2_RX,DFSDM1_DATIN1,SDMMC2_CK,FMC_NWAIT,DCMI_D10,LCD_B2,EVENTOUT); no longer U1002.90 (PG5,FMC_A15,FMC_BA1,EVENTOUT)
- new net MCU_CURR_SENS_1kR: U1002.90 (PG5,FMC_A15,FMC_BA1,EVENTOUT)
- no-connect marks 49 -> 48
Changed lines of the file:
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@@
   )
   (no_connect (at 218.44 267.97))
-  (no_connect (at 372.11 33.02))
   (no_connect (at 372.11 30.48))
   (no_connect (at 82.55 66.04))
@@
   (no_connect (at 82.55 142.24))
   (no_connect (at 218.44 270.51))
+  (no_connect (at 372.11 33.02))
+  (no_connect (at 372.11 40.64))
+  (no_connect (at 372.11 38.1))
+  (no_connect (at 372.11 35.56))
   (no_connect (at 372.11 68.58))
   (no_connect (at 372.11 60.96))
-  (no_connect (at 372.11 88.9))
-  (no_connect (at 372.11 86.36))
-  (no_connect (at 372.11 83.82))
-  (no_connect (at 372.11 81.28))
   (no_connect (at 372.11 76.2))
   (no_connect (at 372.11 73.66))
@@
     (stroke (width 0) (type default) (color 0 0 0 0))
   )
-  (wire (pts (xy 372.11 38.1) (xy 373.38 38.1))
+  (wire (pts (xy 372.11 83.82) (xy 373.38 83.82))
     (stroke (width 0) (type default) (color 0 0 0 0))
   )
@@
     (stroke (width 0) (type default) (color 0 0 0 0))
   )
-  (wire (pts (xy 372.11 35.56) (xy 373.38 35.56))
+  (wire (pts (xy 372.11 81.28) (xy 373.38 81.28))
     (stroke (width 0) (type default) (color 0 0 0 0))
   )
@@
     (stroke (width 0) (type default) (color 0 0 0 0))
   )
-  (wire (pts (xy 372.11 40.64) (xy 373.38 40.64))
+  (wire (pts (xy 372.11 86.36) (xy 373.38 86.36))
     (stroke (width 0) (type default) (color 0 0 0 0))
   )
@@
     (stroke (width 0) (type default) (color 0 0 0 0))
   )
+  (wire (pts (xy 372.11 43.18) (xy 373.38 43.18))
+    (stroke (width 0) (type default) (color 0 0 0 0))
+  )
   (wire (pts (xy 82.55 116.84) (xy 71.12 116.84))
     (stroke (width 0) (type default) (color 0 0 0 0))
@@
     (stroke (width 0) (type default) (color 0 0 0 0))
   )
-  (wire (pts (xy 372.11 43.18) (xy 373.38 43.18))
+  (wire (pts (xy 372.11 88.9) (xy 373.38 88.9))
     (stroke (width 0) (type default) (color 0 0 0 0))
   )
@@
     (effects (font (size 1.27 1.27)) (justify right))
   )
-  (hierarchical_label "SR_CLK" (shape output) (at 373.38 35.56 0)
+  (hierarchical_label "SR_CLK" (shape output) (at 373.38 81.28 0)
+    (effects (font (size 1.27 1.27)) (justify left))
+  )
+  (hierarchical_label "MCU_CURR_SENS_1kR" (shape output) (at 373.38 43.18 0)
     (effects (font (size 1.27 1.27)) (justify left))
   )
@@
     (effects (font (size 1.27 1.27)) (justify right))
   )
-  (hierarchical_label "SR_DAT" (shape output) (at 373.38 38.1 0)
+  (hierarchical_label "SR_DAT" (shape output) (at 373.38 83.82 0)
     (effects (font (size 1.27 1.27)) (justify left))
   )
@@
     (effects (font (size 1.27 1.27)) (justify right))
   )
-  (hierarchical_label "SR_OUT" (shape input) (at 373.38 43.18 0)
+  (hierarchical_label "SR_OUT" (shape input) (at 373.38 88.9 0)
     (effects (font (size 1.27 1.27)) (justify left))
   )
@@
     (effects (font (size 1.27 1.27)) (justify right))
   )
-  (hierarchical_label "SR_LAT" (shape output) (at 373.38 40.64 0)
-    (effects (font (size 1.27 1.27)) (justify left))
-  )
+  (hierarchical_label "SR_LAT" (shape output) (at 373.38 86.36 0)
+    (effects (font (size 1.27 1.27)) (justify left))
+  )

Commit message: Hardware design
Parts:
- Y1001: value ECS-080-18-23A-JGN-TR -> NX3225GD-16MHZ; footprint Crystal:Crystal_SMD_0603-2Pin_6.0x3.5mm_HandSoldering -> ETH1CSMU2:NX3225GD
Connections:
- net CXN_REL6: now reaches U1002.58 (PE7,TIM1_ETR,DFSDM1_DATIN2,UART7_RX,QUADSPI_BK2_IO0,FMC_D4,EVENTOUT)
- no-connect marks 48 -> 47
Changed lines of the file:
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@@
   (no_connect (at 372.11 96.52))
   (no_connect (at 372.11 93.98))
-  (no_connect (at 372.11 134.62))
   (no_connect (at 372.11 124.46))
   (no_connect (at 372.11 119.38))
@@
     (stroke (width 0) (type default) (color 0 0 0 0))
   )
+  (wire (pts (xy 372.11 134.62) (xy 373.38 134.62))
+    (stroke (width 0) (type default) (color 0 0 0 0))
+  )
   (wire (pts (xy 144.78 276.86) (xy 157.48 276.86))
     (stroke (width 0) (type default) (color 0 0 0 0))
@@
   (hierarchical_label "MCU_nTDS" (shape input) (at 81.28 43.18 180)
     (effects (font (size 1.27 1.27)) (justify right))
+  )
+  (hierarchical_label "CXN_REL6" (shape output) (at 373.38 134.62 0)
+    (effects (font (size 1.27 1.27)) (justify left))
   )
   (hierarchical_label "SPI3_MISO" (shape input) (at 81.28 152.4 180)
@@
     )
     (property "Datasheet" "~" (id 3) (at 271.78 260.35 0)
+      (effects (font (size 1.27 1.27)) hide)
+    )
+    (pin "1")
+    (pin "2")
+  )
+  (symbol (lib_id "Device:Crystal") (at 49.53 27.94 270) (unit 1)
+    (in_bom yes) (on_board yes)
+    (property "Reference" "Y1001" (id 0) (at 52.8574 26.7716 90)
+      (effects (font (size 1.27 1.27)) (justify left))
+    )
+    (property "Value" "NX3225GD-16MHZ" (id 1) (at 52.8574 29.083 90)
+      (effects (font (size 1.27 1.27)) (justify left))
+    )
+    (property "Footprint" "ETH1CSMU2:NX3225GD" (id 2) (at 49.53 27.94 0)
+      (effects (font (size 1.27 1.27)) hide)
+    )
+    (property "Datasheet" "~" (id 3) (at 49.53 27.94 0)
       (effects (font (size 1.27 1.27)) hide)
     )
@@
       (effects (font (size 1.27 1.27)) hide)
     )
-    (pin "1")
-    (pin "2")
-  )
-  (symbol (lib_id "Device:Crystal") (at 49.53 27.94 270) (unit 1)
-    (in_bom yes) (on_board yes)
-    (property "Reference" "Y1001" (id 0) (at 52.8574 26.7716 90)
-      (effects (font (size 1.27 1.27)) (justify left))
-    )
-    (property "Value" "ECS-080-18-23A-JGN-TR" (id 1) (at 52.8574 29.083 90)
-      (effects (font (size 1.27 1.27)) (justify left))
-    )
-    (property "Footprint" "Crystal:Crystal_SMD_0603-2Pin_6.0x3.5mm_HandSoldering" (id 2) (at 49.53 27.94 0)
-      (effects (font (size 1.27 1.27)) hide)
-    )
-    (property "Datasheet" "~" (id 3) (at 49.53 27.94 0)
-      (effects (font (size 1.27 1.27)) hide)
-    )

Commit message: Hardware design
Connections:
- net SENS_SCL renamed DAC_OFFS_SCL
- net SENS_SDA renamed DAC_OFFS_SDA
Changed lines of the file:
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@@
     (effects (font (size 1.27 1.27)) (justify left))
+  )
+  (hierarchical_label "DAC_OFFS_SDA" (shape bidirectional) (at 71.12 147.32 180)
+    (effects (font (size 1.27 1.27)) (justify right))
   )
   (hierarchical_label "SPI1_SCK" (shape output) (at 81.28 93.98 180)
     (effects (font (size 1.27 1.27)) (justify right))
   )
+  (hierarchical_label "DAC_OFFS_SCL" (shape bidirectional) (at 71.12 101.6 180)
+    (effects (font (size 1.27 1.27)) (justify right))
+  )

Commit message: Hardware design
Parts:
- C1003, C1005: value 6p -> 8p
- Y1001: value NX3225GD-16MHZ -> NX5032GA-16.000M
Changed lines of the file:
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@@
       (effects (font (size 1.27 1.27)) (justify left))
     )
-    (property "Value" "6p" (id 1) (at 39.751 39.243 0)
+    (property "Value" "8p" (id 1) (at 39.751 39.243 0)
       (effects (font (size 1.27 1.27)) (justify left))
     )
@@
       (effects (font (size 1.27 1.27)) (justify left))
     )
-    (property "Value" "6p" (id 1) (at 52.451 39.243 0)
+    (property "Value" "8p" (id 1) (at 52.451 39.243 0)
       (effects (font (size 1.27 1.27)) (justify left))
     )
@@
       (effects (font (size 1.27 1.27)) (justify left))
     )
-    (property "Value" "NX3225GD-16MHZ" (id 1) (at 52.8574 29.083 90)
-      (effects (font (size 1.27 1.27)) (justify left))
-    )
+    (property "Value" "NX5032GA-16.000M" (id 1) (at 52.8574 29.083 90)
+      (effects (font (size 1.27 1.27)) (justify left))
+    )
