File: HARDWARE/ETH1CSMU2/MCU.kicad_sch (KiCad schematic)
At the start: 42 parts, among them J1001 Conn_02x01, J1002 20021111-00010T4LF, U1001 HDC1080, U1002 STM32F746ZG, U1003 24LC08B-E/MS, Y1001 NX5032GA-16.000M

Commit message: PCB layout
Changed lines of the file:
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@@
   )
   (symbol (lib_id "power:+3.3V") (at 227.33 20.32 0) (unit 1)
-    (in_bom yes) (on_board yes)
+    (in_bom yes) (on_board yes) (fields_autoplaced)
     (property "Reference" "#PWR01021" (id 0) (at 227.33 24.13 0)
       (effects (font (size 1.27 1.27)) hide)
     )
-    (property "Value" "+3.3V" (id 1) (at 227.711 15.9258 0))
+    (property "Value" "+3.3V" (id 1) (at 227.33 16.7442 0))
     (property "Footprint" "" (id 2) (at 227.33 20.32 0)
       (effects (font (size 1.27 1.27)) hide)

Commit message: PCB layout
Connections:
- net CXN_REL1: now also U1002.70 (PB11,TIM2_CH4,I2C2_SDA,DFSDM1_CKIN7,USART3_RX,OTG_HS_ULPI_D4,ETH_MII_TX_EN,ETH_RMII_TX_EN,_DSI_TE,LCD_G5,EVENTOUT); no longer U1002.65 (PE12,TIM1_CH3N,SPI4_SCK,DFSDM1_DATIN5,SAI2_SCK_B,FMC_D9,LCD_B4,EVENTOUT)
- net CXN_REL2: now also U1002.69 (PB10,TIM2_CH3,I2C2_SCL,SPI2_SCK,I2S2_CK,DFSDM1_DATIN7,USART3_TX,QUADSPI_BK1_NCS,OTG_HS_ULPI_D3,ETH_MII_RX_ER,LCD_G4,EVENTOUT); no longer U1002.64 (PE11,TIM1_CH2,SPI4_NSS,DFSDM1_CKIN4,SAI2_SD_B,FMC_D8,LCD_G3,EVENTOUT)
- net CXN_REL6: now also U1002.65 (PE12,TIM1_CH3N,SPI4_SCK,DFSDM1_DATIN5,SAI2_SCK_B,FMC_D9,LCD_B4,EVENTOUT); no longer U1002.58 (PE7,TIM1_ETR,DFSDM1_DATIN2,UART7_RX,QUADSPI_BK2_IO0,FMC_D4,EVENTOUT)
- net DAC1_LDAC: now also U1002.58 (PE7,TIM1_ETR,DFSDM1_DATIN2,UART7_RX,QUADSPI_BK2_IO0,FMC_D4,EVENTOUT); no longer U1002.69 (PB10,TIM2_CH3,I2C2_SCL,SPI2_SCK,I2S2_CK,DFSDM1_DATIN7,USART3_TX,QUADSPI_BK1_NCS,OTG_HS_ULPI_D3,ETH_MII_RX_ER,LCD_G4,EVENTOUT)
- net DAC1_~{RST}: now also U1002.64 (PE11,TIM1_CH2,SPI4_NSS,DFSDM1_CKIN4,SAI2_SD_B,FMC_D8,LCD_G3,EVENTOUT); no longer U1002.70 (PB11,TIM2_CH4,I2C2_SDA,DFSDM1_CKIN7,USART3_RX,OTG_HS_ULPI_D4,ETH_MII_TX_EN,ETH_RMII_TX_EN,_DSI_TE,LCD_G5,EVENTOUT)
- net DDS_DIV2: now also U1002.10 (PF0,I2C2_SDA,FMC_A0,EVENTOUT); no longer U1002.50 (PF12,FMC_A6,EVENTOUT)
- net DDS_DIV4: now also U1002.9 (PC15,EVENTOUT,OSC32_OUT); no longer U1002.53 (PF13,I2C4_SMBA,DFSDM1_DATIN6,FMC_A7,EVENTOUT)
- net DDS_DIV8: now also U1002.8 (PC14,EVENTOUT,OSC32_IN); no longer U1002.54 (PF14,I2C4_SCL,DFSDM1_CKIN6,FMC_A8,EVENTOUT)
- net MCU_nISNK: now also U1002.53 (PF13,I2C4_SMBA,DFSDM1_DATIN6,FMC_A7,EVENTOUT); no longer U1002.10 (PF0,I2C2_SDA,FMC_A0,EVENTOUT)
- net MCU_nISRC: now also U1002.54 (PF14,I2C4_SCL,DFSDM1_CKIN6,FMC_A8,EVENTOUT); no longer U1002.11 (PF1,I2C2_SCL,FMC_A1,EVENTOUT)
- net MCU_nTDS: now also U1002.55 (PF15,I2C4_SDA,FMC_A9,EVENTOUT); no longer U1002.12 (PF2,I2C2_SMBA,FMC_A2,EVENTOUT)
- net ~{DDS_DIV10}: now also U1002.7 (PC13,EVENTOUT,RTC_TAMP2,RTC_TS,WKUP5); no longer U1002.55 (PF15,I2C4_SDA,FMC_A9,EVENTOUT)

Commit message: PCB layout
Connections:
- net DAC1_LDAC: now also U1002.2 (PE3,TRACED0,SAI1_SD_B,FMC_A19,EVENTOUT); no longer U1002.58 (PE7,TIM1_ETR,DFSDM1_DATIN2,UART7_RX,QUADSPI_BK2_IO0,FMC_D4,EVENTOUT)
- net EEPROM_WP: now also U1002.89 (PG4,FMC_A14,FMC_BA0,EVENTOUT); no longer U1002.80 (PD11,I2C4_SMBA,USART3_CTS,QUADSPI_BK1_IO0,SAI2_SD_A,FMC_A16,FMC_CLE,EVENTOUT)
- net LED_BLUE: now also U1002.48 (PB2,SAI1_SD_A,SPI3_MOSI,I2S3_SD,QUADSPI_CLK,DFSDM1_CKIN1,EVENTOUT); no longer U1002.123 (PD7,DFSDM1_DATIN4,SPI1_MOSI,I2S1_SD,DFSDM1_CKIN1,USART2_CK,SPDIF_RX0,SDMMC2_CMD,FMC_NE1,EVENTOUT)
- net LED_GREEN: now also U1002.50 (PF12,FMC_A6,EVENTOUT); no longer U1002.125 (PG10,SPI1_NSS,I2S1_WS,LCD_G3,SAI2_SD_B,SDMMC2_D1,FMC_NE3,DCMI_D2,LCD_B2,EVENTOUT)
- net LED_RED: now also U1002.49 (PF11,SPI5_MOSI,SAI2_SD_B,FMC_SDNRAS,_DCMI_D12,EVENTOUT); no longer U1002.124 (PG9,SPI1_MISO,SPDIF_RX3,USART6_RX,QUADSPI_BK2_IO2,SAI2_FS_B,SDMMC2_D0,FMC_NE2,FMC_NCE,DCMI_VSYNC,EVENTOUT)
- net MCU_DEFAULT: now also U1002.63 (PE10,TIM1_CH2N,DFSDM1_DATIN4,UART7_CTS,QUADSPI_BK2_IO3,FMC_D7,EVENTOUT); no longer U1002.116 (PD2,TRACED2,TIM3_ETR,UART5_RX,SDMMC1_CMD,DCMI_D11,EVENTOUT)
- net MCU_nISNK: now also U1002.79 (PD10,DFSDM1_CKOUT,USART3_CK,FMC_D15,LCD_B3,EVENTOUT); no longer U1002.53 (PF13,I2C4_SMBA,DFSDM1_DATIN6,FMC_A7,EVENTOUT)
- net MCU_nISRC: now also U1002.80 (PD11,I2C4_SMBA,USART3_CTS,QUADSPI_BK1_IO0,SAI2_SD_A,FMC_A16,FMC_CLE,EVENTOUT); no longer U1002.54 (PF14,I2C4_SCL,DFSDM1_CKIN6,FMC_A8,EVENTOUT)
- net MCU_nTDS: now also U1002.78 (PD9,DFSDM1_DATIN3,USART3_RX,FMC_D14,EVENTOUT); no longer U1002.55 (PF15,I2C4_SDA,FMC_A9,EVENTOUT)
- net SR_CLK: now also U1002.87 (PG2,FMC_A12,EVENTOUT); no longer U1002.117 (PD3,DFSDM1_CKOUT,SPI2_SCK,I2S2_CK,DFSDM1_DATIN0,USART2_CTS,FMC_CLK,DCMI_D5,LCD_G7,EVENTOUT)
- net SR_DAT: now also U1002.88 (PG3,FMC_A13,EVENTOUT); no longer U1002.118 (PD4,DFSDM1_CKIN0,USART2_RTS,FMC_NOE,EVENTOUT)
- net SR_LAT: now also U1002.86 (PD15,TIM4_CH4,UART8_RTS,FMC_D1,EVENTOUT); no longer U1002.119 (PD5,USART2_TX,FMC_NWE,EVENTOUT)
- net SR_OUT: now also U1002.85 (PD14,TIM4_CH3,UART8_CTS,FMC_D0,EVENTOUT); no longer U1002.122 (PD6,DFSDM1_CKIN4,SPI3_MOSI,I2S3_SD,SAI1_SD_A,USART2_RX,DFSDM1_DATIN1,SDMMC2_CK,FMC_NWAIT,DCMI_D10,LCD_B2,EVENTOUT)
- net TRIG_EN: now also U1002.60 (PE9,TIM1_CH1,DFSDM1_CKOUT,UART7_RTS,QUADSPI_BK2_IO2,FMC_D6,EVENTOUT); no longer U1002.59 (PE8,TIM1_CH1N,DFSDM1_CKIN2,UART7_TX,QUADSPI_BK2_IO1,FMC_D5,EVENTOUT)
- net TRIG_IN: now also U1002.58 (PE7,TIM1_ETR,DFSDM1_DATIN2,UART7_RX,QUADSPI_BK2_IO0,FMC_D4,EVENTOUT); no longer U1002.63 (PE10,TIM1_CH2N,DFSDM1_DATIN4,UART7_CTS,QUADSPI_BK2_IO3,FMC_D7,EVENTOUT)
- net TRIG_OUT: now also U1002.59 (PE8,TIM1_CH1N,DFSDM1_CKIN2,UART7_TX,QUADSPI_BK2_IO1,FMC_D5,EVENTOUT); no longer U1002.60 (PE9,TIM1_CH1,DFSDM1_CKOUT,UART7_RTS,QUADSPI_BK2_IO2,FMC_D6,EVENTOUT)
- no-connect marks 47 -> 46

Commit message: PCB layout
Parts:
- removed R1009: 10k, Resistor_SMD:R_0603_1608Metric_Pad0.98x0.95mm_HandSolder, symbol Device:R
Connections:
- net ADC1_RVS1: now also U1002.114 (PD0,DFSDM1_CKIN6,DFSDM1_DATIN7,UART4_RX,CAN1_RX,FMC_D2,EVENTOUT); no longer U1002.34 (PA0,TIM2_CH1,TIM2_ETR,TIM5_CH1,TIM8_ETR,USART2_CTS,UART4_TX,SAI2_SD_B,ETH_MII_CRS,EVENTOUT,ADC1_IN0,ADC2_IN0,ADC3_IN0,WKUP1)
- net ADC1_RVS2: now also U1002.115 (PD1,DFSDM1_DATIN6,DFSDM1_CKIN7,UART4_TX,CAN1_TX,FMC_D3,EVENTOUT); no longer U1002.37 (PA3,TIM2_CH4,TIM5_CH4,TIM9_CH2,USART2_RX,LCD_B2,OTG_HS_ULPI_D0,ETH_MII_COL,LCD_B5,EVENTOUT,ADC1_IN3,ADC2_IN3,ADC3_IN3)
- net DAC1_LDAC: now also U1002.104 (PA12,TIM1_ETR,SPI2_SCK,I2S2_CK,UART4_TX,USART1_RTS,SAI2_FS_B,CAN1_TX,OTG_FS_DP,LCD_R5,EVENTOUT); no longer U1002.2 (PE3,TRACED0,SAI1_SD_B,FMC_A19,EVENTOUT)
- net DAC1_~{RST}: now also U1002.103 (PA11,TIM1_CH4,SPI2_NSS,I2S2_WS,UART4_RX,USART1_CTS,CAN1_RX,OTG_FS_DM,LCD_R4,EVENTOUT); no longer U1002.64 (PE11,TIM1_CH2,SPI4_NSS,DFSDM1_CKIN4,SAI2_SD_B,FMC_D8,LCD_G3,EVENTOUT)
- net DAC2_~{LDAC}: now also U1002.127 (PG12,LPTIM1_IN1,SPI6_MISO,SPDIF_RX1,USART6_RTS,LCD_B4,SDMMC2_D3,FMC_NE4,LCD_B1,EVENTOUT); no longer U1002.22 (PF10,QUADSPI_CLK,DCMI_D11,LCD_DE,EVENTOUT,ADC3_IN8)
Changed lines of the file:
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@@
   )
   (no_connect (at 218.44 267.97))
+  (no_connect (at 82.55 63.5))
   (no_connect (at 372.11 88.9))
   (no_connect (at 372.11 86.36))
@@
   (no_connect (at 372.11 55.88))
   (no_connect (at 372.11 53.34))
+  (no_connect (at 82.55 88.9))
+  (no_connect (at 372.11 78.74))
+  (no_connect (at 372.11 144.78))
   (no_connect (at 82.55 43.18))
   (no_connect (at 372.11 30.48))
@@
   (no_connect (at 82.55 104.14))
   (no_connect (at 82.55 106.68))
-  (no_connect (at 82.55 109.22))
-  (no_connect (at 82.55 111.76))
   (no_connect (at 82.55 124.46))
   (no_connect (at 82.55 129.54))
@@
   (no_connect (at 372.11 33.02))
   (no_connect (at 372.11 68.58))
-  (no_connect (at 372.11 60.96))
-  (no_connect (at 372.11 76.2))
-  (no_connect (at 372.11 73.66))
   (no_connect (at 372.11 162.56))
   (no_connect (at 372.11 167.64))
@@
   (no_connect (at 372.11 160.02))
   (no_connect (at 82.55 144.78))
+  (no_connect (at 82.55 81.28))
   (no_connect (at 82.55 73.66))
   (no_connect (at 82.55 76.2))
@@
     (stroke (width 0) (type default) (color 0 0 0 0))
   )
-  (wire (pts (xy 372.11 124.46) (xy 373.38 124.46))
+  (wire (pts (xy 82.55 111.76) (xy 81.28 111.76))
     (stroke (width 0) (type default) (color 0 0 0 0))
   )
@@
     (stroke (width 0) (type default) (color 0 0 0 0))
   )
-  (wire (pts (xy 372.11 144.78) (xy 373.38 144.78))
+  (wire (pts (xy 82.55 109.22) (xy 81.28 109.22))
     (stroke (width 0) (type default) (color 0 0 0 0))
   )
@@
     (stroke (width 0) (type default) (color 0 0 0 0))
   )
-  (wire (pts (xy 81.28 88.9) (xy 82.55 88.9))
+  (wire (pts (xy 373.38 76.2) (xy 372.11 76.2))
     (stroke (width 0) (type default) (color 0 0 0 0))
   )
@@
     (stroke (width 0) (type default) (color 0 0 0 0))
   )
-  (wire (pts (xy 81.28 63.5) (xy 82.55 63.5))
+  (wire (pts (xy 373.38 60.96) (xy 372.11 60.96))
     (stroke (width 0) (type default) (color 0 0 0 0))
   )
@@
     (stroke (width 0) (type default) (color 0 0 0 0))
   )
-  (wire (pts (xy 81.28 81.28) (xy 82.55 81.28))
+  (wire (pts (xy 373.38 73.66) (xy 372.11 73.66))
     (stroke (width 0) (type default) (color 0 0 0 0))
   )
@@
     (effects (font (size 1.27 1.27)) (justify right bottom))
   )
-  (hierarchical_label "ADC1_RVS1" (shape input) (at 81.28 81.28 180)
-    (effects (font (size 1.27 1.27)) (justify right))
+  (hierarchical_label "ADC1_RVS1" (shape input) (at 373.38 73.66 0)
+    (effects (font (size 1.27 1.27)) (justify left))
   )
   (hierarchical_label "SR_CLK" (shape output) (at 373.38 35.56 0)
@@
     (effects (font (size 1.27 1.27)) (justify left))
   )
-  (hierarchical_label "ADC1_RVS2" (shape input) (at 81.28 88.9 180)
-    (effects (font (size 1.27 1.27)) (justify right))
+  (hierarchical_label "ADC1_RVS2" (shape input) (at 373.38 76.2 0)
+    (effects (font (size 1.27 1.27)) (justify left))
   )
   (hierarchical_label "SPI4_MOSI" (shape output) (at 373.38 132.08 0)
@@
     (effects (font (size 1.27 1.27)) (justify right))
   )
-  (hierarchical_label "DAC1_LDAC" (shape output) (at 373.38 124.46 0)
-    (effects (font (size 1.27 1.27)) (justify left))
+  (hierarchical_label "DAC1_LDAC" (shape output) (at 81.28 111.76 180)
+    (effects (font (size 1.27 1.27)) (justify right))
   )
   (hierarchical_label "MCU_CURR_SENS_10R" (shape output) (at 373.38 48.26 0)
@@
     (effects (font (size 1.27 1.27)) (justify left))
   )
-  (hierarchical_label "DAC2_~{LDAC}" (shape output) (at 81.28 63.5 180)
-    (effects (font (size 1.27 1.27)) (justify right))
+  (hierarchical_label "DAC2_~{LDAC}" (shape output) (at 373.38 60.96 0)
+    (effects (font (size 1.27 1.27)) (justify left))
   )
   (hierarchical_label "DDS_DIV4" (shape output) (at 81.28 162.56 180)
@@
     (effects (font (size 1.27 1.27)) (justify left))
   )
-  (hierarchical_label "DAC1_~{RST}" (shape output) (at 373.38 144.78 0)
-    (effects (font (size 1.27 1.27)) (justify left))
+  (hierarchical_label "DAC1_~{RST}" (shape output) (at 81.28 109.22 180)
+    (effects (font (size 1.27 1.27)) (justify right))
   )
   (hierarchical_label "RMII_MDC" (shape bidirectional) (at 81.28 127 180)
@@
     (pin "1")
   )
-  (symbol (lib_id "Device:R") (at 372.11 226.06 0) (unit 1)
-    (in_bom yes) (on_board yes)
-    (property "Reference" "R1009" (id 0) (at 373.888 224.8916 0)
-      (effects (font (size 1.27 1.27)) (justify left))
-    )
-    (property "Value" "10k" (id 1) (at 373.888 227.203 0)
-      (effects (font (size 1.27 1.27)) (justify left))
-    )
-    (property "Footprint" "Resistor_SMD:R_0603_1608Metric_Pad0.98x0.95mm_HandSolder" (id 2) (at 370.332 226.06 90)
-      (effects (font (size 1.27 1.27)) hide)
-    )
-    (property "Datasheet" "~" (id 3) (at 372.11 226.06 0)
-      (effects (font (size 1.27 1.27)) hide)
-    )
-    (pin "1")
-    (pin "2")
-  )
   (symbol (lib_id "power:+3.3V") (at 227.33 20.32 0) (unit 1)

Commit message: Bug fixes.
Parts:
- added R1009: 10k, Resistor_SMD:R_0603_1608Metric_Pad0.98x0.95mm_HandSolder, symbol Device:R
Connections:
- net GND: now also R1009.2
- net at U1002.138 (BOOT0): now also R1009.1
- no-connect marks 46 -> 47
Changed lines of the file:
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@@
   (junction (at 281.94 255.27) (diameter 0) (color 0 0 0 0)
   )
+  (no_connect (at 372.11 124.46))
   (no_connect (at 218.44 267.97))
   (no_connect (at 82.55 63.5))
@@
     (pin "1")
   )
+  (symbol (lib_id "Device:R") (at 372.11 226.06 0) (unit 1)
+    (in_bom yes) (on_board yes)
+    (property "Reference" "R1009" (id 0) (at 373.888 224.8916 0)
+      (effects (font (size 1.27 1.27)) (justify left))
+    )
+    (property "Value" "10k" (id 1) (at 373.888 227.203 0)
+      (effects (font (size 1.27 1.27)) (justify left))
+    )
+    (property "Footprint" "Resistor_SMD:R_0603_1608Metric_Pad0.98x0.95mm_HandSolder" (id 2) (at 370.332 226.06 90)
+      (effects (font (size 1.27 1.27)) hide)
+    )
+    (property "Datasheet" "~" (id 3) (at 372.11 226.06 0)
+      (effects (font (size 1.27 1.27)) hide)
+    )
+    (pin "1")
+    (pin "2")
+  )
   (symbol (lib_id "Device:R") (at 271.78 260.35 0) (unit 1)
