File: HARDWARE/ETH1CSMU2/Measure.kicad_sch (KiCad schematic)
At the start: 34 parts, among them U401 DG444DY+, U402 DG444DY+, U403 DG419DY, U404 DG419DY, U405 OPA140/OPA141, U406 OPA140/OPA141, U407 ADS8681IRUMT, U408 ADS8681IRUMT

Commit message: Hardware design
Parts:
- added C401, C402, C403, C405, C406, C407, C410, C411, C412, C413, C415, C416, C417, C418, C422, C423, C424, C425, C426, C427: 100n, symbol Device:C
- added C404, C414: 1u, Capacitor_SMD:C_0603_1608Metric_Pad1.08x0.95mm_HandSolder, symbol Device:C
- added C420: 10u, Resistor_SMD:R_0805_2012Metric_Pad1.20x1.40mm_HandSolder, symbol Device:C
- added R405: 0R22, Resistor_SMD:R_0603_1608Metric_Pad0.98x0.95mm_HandSolder, symbol Device:R
- added U402: REF5040ID, Package_SO:SOIC-8_3.9x4.9mm_P1.27mm, symbol Reference_Voltage:REF5040ID
- added unit 2 of U404
- added unit 2 of U405
- renumbered C401 to C408, C402 to C409, C403 to C419, C404 to C421, C405 to C428, C406 to C429, R405 to R406, R406 to R407, R407 to R408, R408 to R409, R409 to R410, R410 to R411, R411 to R412, R412 to R413, R413 to R414, R414 to R415, R415 to R416, R416 to R417, R417 to R418, R418 to R419, R419 to R420, R420 to R421, U402 to U403, U403 to U404, U404 to U405, U405 to U406, U406 to U407, U407 to U408, U408 to U409
Connections:
- net +15V: now also U401.13 (V+), U403.13 (V+), C403.1, C407.1, C413.1, C418.1, C424.1, C427.1, U404.5 (VL), U405.4 (V+)
- net +3.3V: now also C410.1, C415.1
- net +4V: now also R405.1, U402.6 (Vout)
- net +5V: now also C401.1, C404.1, C405.1, C411.1, C416.1, C422.1, C425.1, U402.2 (Vin), U404.4 (V+), U405.5 (VL)
- net -15V: now also U401.4 (V-), U403.4 (V-), C402.1, C406.1, C412.1, C417.1, C423.1, C426.1, U404.7 (V-), U405.7 (V-)
- net GND: now also C401.2, C402.2, C403.2, C404.2, C405.2, C406.2, C407.2, C410.2, C411.2, C412.2, C413.2, C414.2, C415.2, C416.2, C417.2, C418.2, C420.2, C422.2, C423.2, C424.2, C425.2, C426.2, C427.2, U402.4 (GND), U404.3 (GND), U405.3 (GND)
- new net: C420.1, R405.2
- new net: C414.1, U402.5 (Trim/NR)
- no-connect marks 2 -> 3
Other:
- moved on the sheet: C408, C409, C419, C421, C428, C429, R401, R402, R403, R404, R406, R407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

Commit message: Hardware design
Parts:
- added U10: DG419DY, Package_SO:SOIC-8_3.9x4.9mm_P1.27mm, symbol Analog_Switch:DG419xY
- renumbered C401 to C16, C402 to C17, C403 to C18, C404 to C19, C405 to C20, C406 to C21, C407 to C22, C408 to C23, C409 to C24, C410 to C25, C411 to C26, C412 to C27, C413 to C28, C414 to C29, C415 to C30, C416 to C31, C417 to C32, C418 to C33, C419 to C34, C420 to C35, C421 to C36, C422 to C37, C423 to C38, C424 to C39, C425 to C40, C426 to C41, C427 to C42, C428 to C43, C429 to C44, R401 to R22, R402 to R23, R403 to R24, R404 to R25, R405 to R26, R406 to R27, R407 to R28, R408 to R29, R409 to R30, R410 to R31, R411 to R32, R412 to R33, R413 to R34, R414 to R35, R415 to R36, R416 to R37, R417 to R38, R418 to R39, R419 to R40, R420 to R41, R421 to R42, U406 to U11, U407 to U12, U408 to U13, U409 to U14, U401 to U5, U402 to U6, U403 to U7, U404 to U8, U405 to U9
Connections:
- net +15V: now also U10.4 (V+)
- net +5V: now also U10.5 (VL)
- net -15V: now also U10.7 (V-)
- net GND: now also U10.3 (GND)
- net VOLT_MEAS: now also U10.2; no longer R27.2
- new net: R27.2, U10.1
- new net VMEAS_SEL: U10.6
- new net VOLT_MEAS_SENS: U10.8

Commit message: Hardware design
Parts:
- renumbered C16 to C401, C17 to C402, C18 to C403, C19 to C404, C20 to C405, C21 to C406, C22 to C407, C23 to C408, C24 to C409, C25 to C410, C26 to C411, C27 to C412, C28 to C413, C29 to C414, C30 to C415, C31 to C416, C32 to C417, C33 to C418, C34 to C419, C35 to C420, C36 to C421, C37 to C422, C38 to C423, C39 to C424, C40 to C425, C41 to C426, C42 to C427, C43 to C428, C44 to C429, R22 to R401, R23 to R402, R24 to R403, R25 to R404, R26 to R405, R27 to R406, R28 to R407, R29 to R408, R30 to R409, R31 to R410, R32 to R411, R33 to R412, R34 to R413, R35 to R414, R36 to R415, R37 to R416, R38 to R417, R39 to R418, R40 to R419, R41 to R420, R42 to R421, U5 to U401, U6 to U402, U7 to U403, U8 to U404, U9 to U405, U10 to U406, U11 to U407, U12 to U408, U13 to U409, U14 to U410

Commit message: Hardware design.
Parts:
- U11: renamed from U407; value OPA140/OPA141 -> OPA141AID
- U12: renamed from U408; value OPA140/OPA141 -> OPA141AID
- renumbered C401 to C16, C402 to C17, C403 to C18, C404 to C19, C405 to C20, C406 to C21, C407 to C22, C408 to C23, C409 to C24, C410 to C25, C411 to C26, C412 to C27, C413 to C28, C414 to C29, C415 to C30, C416 to C31, C417 to C32, C418 to C33, C419 to C34, C420 to C35, C421 to C36, C422 to C37, C423 to C38, C424 to C39, C425 to C40, C426 to C41, C427 to C42, C428 to C43, C429 to C44, R401 to R22, R402 to R23, R403 to R24, R404 to R25, R405 to R26, R406 to R27, R407 to R28, R408 to R29, R409 to R30, R410 to R31, R411 to R32, R412 to R33, R413 to R34, R414 to R35, R415 to R36, R416 to R37, R417 to R38, R418 to R39, R419 to R40, R420 to R41, R421 to R42, U406 to U10, U409 to U13, U410 to U14, U401 to U5, U402 to U6, U403 to U7, U404 to U8, U405 to U9

Commit message: Hardware design
Parts:
- C16, C17, C18, C20, C21, C22, C25, C26, C27, C28, C30, C31, C32, C33, C37, C38, C39, C40, C41, C42: footprint (none) -> Capacitor_SMD:C_0603_1608Metric_Pad1.08x0.95mm_HandSolder
- R37, R38: footprint (none) -> Resistor_SMD:R_0603_1608Metric_Pad0.98x0.95mm_HandSolder
- U5, U7: footprint (none) -> Package_SO:SOIC-16_3.9x9.9mm_P1.27mm
Changed lines of the file:
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@@
     (property "Reference" "U7" (id 0) (at 246.38 194.4202 0))
     (property "Value" "DG444DY+" (id 1) (at 246.38 196.9571 0))
-    (property "Footprint" "" (id 2) (at 246.38 203.2 0)
+    (property "Footprint" "Package_SO:SOIC-16_3.9x9.9mm_P1.27mm" (id 2) (at 246.38 203.2 0)
       (effects (font (size 1.27 1.27)) hide)
     )
@@
     (property "Reference" "R38" (id 0) (at 278.13 156.5742 90))
     (property "Value" "0" (id 1) (at 278.13 159.1111 90))
-    (property "Footprint" "" (id 2) (at 278.13 163.068 90)
+    (property "Footprint" "Resistor_SMD:R_0603_1608Metric_Pad0.98x0.95mm_HandSolder" (id 2) (at 278.13 163.068 90)
       (effects (font (size 1.27 1.27)) hide)
     )
@@
       (effects (font (size 1.27 1.27)) (justify left))
     )
-    (property "Footprint" "" (id 2) (at 23.8252 245.11 0)
+    (property "Footprint" "Capacitor_SMD:C_0603_1608Metric_Pad1.08x0.95mm_HandSolder" (id 2) (at 23.8252 245.11 0)
       (effects (font (size 1.27 1.27)) hide)
     )
@@
     (property "Reference" "U5" (id 0) (at 246.38 110.6002 0))
     (property "Value" "DG444DY+" (id 1) (at 246.38 113.1371 0))
-    (property "Footprint" "" (id 2) (at 246.38 119.38 0)
+    (property "Footprint" "Package_SO:SOIC-16_3.9x9.9mm_P1.27mm" (id 2) (at 246.38 119.38 0)
       (effects (font (size 1.27 1.27)) hide)
     )
@@
     (property "Reference" "U5" (id 0) (at 246.38 77.5802 0))
     (property "Value" "DG444DY+" (id 1) (at 246.38 80.1171 0))
-    (property "Footprint" "" (id 2) (at 246.38 86.36 0)
+    (property "Footprint" "Package_SO:SOIC-16_3.9x9.9mm_P1.27mm" (id 2) (at 246.38 86.36 0)
       (effects (font (size 1.27 1.27)) hide)
     )
@@
       (effects (font (size 1.27 1.27)) (justify left))
     )
-    (property "Footprint" "" (id 2) (at 50.4952 245.11 0)
+    (property "Footprint" "Capacitor_SMD:C_0603_1608Metric_Pad1.08x0.95mm_HandSolder" (id 2) (at 50.4952 245.11 0)
       (effects (font (size 1.27 1.27)) hide)
     )
@@
       (effects (font (size 1.27 1.27)) (justify left))
     )
-    (property "Footprint" "" (id 2) (at 23.8252 219.71 0)
+    (property "Footprint" "Capacitor_SMD:C_0603_1608Metric_Pad1.08x0.95mm_HandSolder" (id 2) (at 23.8252 219.71 0)
       (effects (font (size 1.27 1.27)) hide)
     )
@@
       (effects (font (size 1.27 1.27)) (justify left))
     )
-    (property "Footprint" "" (id 2) (at 63.1952 245.11 0)
+    (property "Footprint" "Capacitor_SMD:C_0603_1608Metric_Pad1.08x0.95mm_HandSolder" (id 2) (at 63.1952 245.11 0)
       (effects (font (size 1.27 1.27)) hide)
     )
@@
     (property "Reference" "U7" (id 0) (at 69.85 99.1702 0))
     (property "Value" "DG444DY+" (id 1) (at 69.85 101.7071 0))
-    (property "Footprint" "" (id 2) (at 69.85 107.95 0)
+    (property "Footprint" "Package_SO:SOIC-16_3.9x9.9mm_P1.27mm" (id 2) (at 69.85 107.95 0)
       (effects (font (size 1.27 1.27)) hide)
     )
@@
     (property "Reference" "U7" (id 0) (at 125.73 215.9 0))
     (property "Value" "DG444DY+" (id 1) (at 125.73 218.44 0))
-    (property "Footprint" "" (id 2) (at 113.03 219.71 0)
+    (property "Footprint" "Package_SO:SOIC-16_3.9x9.9mm_P1.27mm" (id 2) (at 113.03 219.71 0)
       (effects (font (size 1.27 1.27)) hide)
     )
@@
     (property "Reference" "U5" (id 0) (at 125.73 257.81 0))
     (property "Value" "DG444DY+" (id 1) (at 125.73 260.35 0))
-    (property "Footprint" "" (id 2) (at 113.03 261.62 0)
+    (property "Footprint" "Package_SO:SOIC-16_3.9x9.9mm_P1.27mm" (id 2) (at 113.03 261.62 0)
       (effects (font (size 1.27 1.27)) hide)
     )
@@
       (effects (font (size 1.27 1.27)) (justify left))
     )
-    (property "Footprint" "" (id 2) (at 77.1652 219.71 0)
+    (property "Footprint" "Capacitor_SMD:C_0603_1608Metric_Pad1.08x0.95mm_HandSolder" (id 2) (at 77.1652 219.71 0)
       (effects (font (size 1.27 1.27)) hide)
     )
@@
       (effects (font (size 1.27 1.27)) (justify left))
     )
-    (property "Footprint" "" (id 2) (at 91.1352 270.51 0)
+    (property "Footprint" "Capacitor_SMD:C_0603_1608Metric_Pad1.08x0.95mm_HandSolder" (id 2) (at 91.1352 270.51 0)
       (effects (font (size 1.27 1.27)) hide)
     )
@@
       (effects (font (size 1.27 1.27)) (justify left))
     )
-    (property "Footprint" "" (id 2) (at 63.1952 219.71 0)
+    (property "Footprint" "Capacitor_SMD:C_0603_1608Metric_Pad1.08x0.95mm_HandSolder" (id 2) (at 63.1952 219.71 0)
       (effects (font (size 1.27 1.27)) hide)
     )
@@
       (effects (font (size 1.27 1.27)) (justify left))
     )
-    (property "Footprint" "" (id 2) (at 36.5252 245.11 0)
+    (property "Footprint" "Capacitor_SMD:C_0603_1608Metric_Pad1.08x0.95mm_HandSolder" (id 2) (at 36.5252 245.11 0)
       (effects (font (size 1.27 1.27)) hide)
     )
@@
       (effects (font (size 1.27 1.27)) (justify left))
     )
-    (property "Footprint" "" (id 2) (at 63.1952 270.51 0)
+    (property "Footprint" "Capacitor_SMD:C_0603_1608Metric_Pad1.08x0.95mm_HandSolder" (id 2) (at 63.1952 270.51 0)
       (effects (font (size 1.27 1.27)) hide)
     )
@@
       (effects (font (size 1.27 1.27)) (justify left))
     )
-    (property "Footprint" "" (id 2) (at 63.1952 193.04 0)
+    (property "Footprint" "Capacitor_SMD:C_0603_1608Metric_Pad1.08x0.95mm_HandSolder" (id 2) (at 63.1952 193.04 0)
       (effects (font (size 1.27 1.27)) hide)
     )
@@
       (effects (font (size 1.27 1.27)) (justify left))
     )
-    (property "Footprint" "" (id 2) (at 36.5252 270.51 0)
+    (property "Footprint" "Capacitor_SMD:C_0603_1608Metric_Pad1.08x0.95mm_HandSolder" (id 2) (at 36.5252 270.51 0)
       (effects (font (size 1.27 1.27)) hide)
     )
@@
       (effects (font (size 1.27 1.27)) (justify left))
     )
-    (property "Footprint" "" (id 2) (at 50.4952 270.51 0)
+    (property "Footprint" "Capacitor_SMD:C_0603_1608Metric_Pad1.08x0.95mm_HandSolder" (id 2) (at 50.4952 270.51 0)
       (effects (font (size 1.27 1.27)) hide)
     )
@@
       (effects (font (size 1.27 1.27)) (justify left))
     )
-    (property "Footprint" "" (id 2) (at 77.1652 270.51 0)
+    (property "Footprint" "Capacitor_SMD:C_0603_1608Metric_Pad1.08x0.95mm_HandSolder" (id 2) (at 77.1652 270.51 0)
       (effects (font (size 1.27 1.27)) hide)
     )
@@
       (effects (font (size 1.27 1.27)) (justify left))
     )
-    (property "Footprint" "" (id 2) (at 77.1652 245.11 0)
+    (property "Footprint" "Capacitor_SMD:C_0603_1608Metric_Pad1.08x0.95mm_HandSolder" (id 2) (at 77.1652 245.11 0)
       (effects (font (size 1.27 1.27)) hide)
     )
@@
     (property "Reference" "U5" (id 0) (at 43.18 99.1702 0))
     (property "Value" "DG444DY+" (id 1) (at 43.18 101.7071 0))
-    (property "Footprint" "" (id 2) (at 43.18 107.95 0)
+    (property "Footprint" "Package_SO:SOIC-16_3.9x9.9mm_P1.27mm" (id 2) (at 43.18 107.95 0)
       (effects (font (size 1.27 1.27)) hide)
     )
@@
       (effects (font (size 1.27 1.27)) (justify left))
     )
-    (property "Footprint" "" (id 2) (at 50.4952 219.71 0)
+    (property "Footprint" "Capacitor_SMD:C_0603_1608Metric_Pad1.08x0.95mm_HandSolder" (id 2) (at 50.4952 219.71 0)
       (effects (font (size 1.27 1.27)) hide)
     )
@@
     (property "Reference" "U7" (id 0) (at 246.38 210.9302 0))
     (property "Value" "DG444DY+" (id 1) (at 246.38 213.4671 0))
-    (property "Footprint" "" (id 2) (at 246.38 219.71 0)
+    (property "Footprint" "Package_SO:SOIC-16_3.9x9.9mm_P1.27mm" (id 2) (at 246.38 219.71 0)
       (effects (font (size 1.27 1.27)) hide)
     )
@@
     (property "Reference" "U5" (id 0) (at 246.38 94.0902 0))
     (property "Value" "DG444DY+" (id 1) (at 246.38 96.6271 0))
-    (property "Footprint" "" (id 2) (at 246.38 102.87 0)
+    (property "Footprint" "Package_SO:SOIC-16_3.9x9.9mm_P1.27mm" (id 2) (at 246.38 102.87 0)
       (effects (font (size 1.27 1.27)) hide)
     )
@@
       (effects (font (size 1.27 1.27)) (justify left))
     )
-    (property "Footprint" "" (id 2) (at 91.1352 245.11 0)
+    (property "Footprint" "Capacitor_SMD:C_0603_1608Metric_Pad1.08x0.95mm_HandSolder" (id 2) (at 91.1352 245.11 0)
       (effects (font (size 1.27 1.27)) hide)
     )
@@
     (property "Reference" "R37" (id 0) (at 278.13 56.2442 90))
     (property "Value" "0" (id 1) (at 278.13 58.7811 90))
-    (property "Footprint" "" (id 2) (at 278.13 62.738 90)
+    (property "Footprint" "Resistor_SMD:R_0603_1608Metric_Pad0.98x0.95mm_HandSolder" (id 2) (at 278.13 62.738 90)
       (effects (font (size 1.27 1.27)) hide)
     )
@@
       (effects (font (size 1.27 1.27)) (justify left))
     )
-    (property "Footprint" "" (id 2) (at 36.5252 219.71 0)
+    (property "Footprint" "Capacitor_SMD:C_0603_1608Metric_Pad1.08x0.95mm_HandSolder" (id 2) (at 36.5252 219.71 0)
       (effects (font (size 1.27 1.27)) hide)
     )
@@
       (effects (font (size 1.27 1.27)) (justify left))
     )
-    (property "Footprint" "" (id 2) (at 91.1352 219.71 0)
+    (property "Footprint" "Capacitor_SMD:C_0603_1608Metric_Pad1.08x0.95mm_HandSolder" (id 2) (at 91.1352 219.71 0)
       (effects (font (size 1.27 1.27)) hide)
     )
@@
     (property "Reference" "U7" (id 0) (at 246.38 177.9102 0))
     (property "Value" "DG444DY+" (id 1) (at 246.38 180.4471 0))
-    (property "Footprint" "" (id 2) (at 246.38 186.69 0)
+    (property "Footprint" "Package_SO:SOIC-16_3.9x9.9mm_P1.27mm" (id 2) (at 246.38 186.69 0)
       (effects (font (size 1.27 1.27)) hide)
     )
@@
       (effects (font (size 1.27 1.27)) (justify left))
     )
-    (property "Footprint" "" (id 2) (at 50.4952 193.04 0)
+    (property "Footprint" "Capacitor_SMD:C_0603_1608Metric_Pad1.08x0.95mm_HandSolder" (id 2) (at 50.4952 193.04 0)
       (effects (font (size 1.27 1.27)) hide)
     )
@@
       (effects (font (size 1.27 1.27)) (justify left))
     )
-    (property "Footprint" "" (id 2) (at 23.8252 270.51 0)
-      (effects (font (size 1.27 1.27)) hide)
-    )
+    (property "Footprint" "Capacitor_SMD:C_0603_1608Metric_Pad1.08x0.95mm_HandSolder" (id 2) (at 23.8252 270.51 0)
+      (effects (font (size 1.27 1.27)) hide)
+    )

Commit message: Hardware design
Parts:
- added C?: 1u, Capacitor_SMD:C_0603_1608Metric_Pad1.08x0.95mm_HandSolder, symbol Device:C
- added R? (x4): 10k, symbol Device:R
- added R? (x4): 2k49, symbol Device:R
- added U409, U410: DG419DY, Package_SO:SOIC-8_3.9x4.9mm_P1.27mm, symbol Analog_Switch:DG419xY
- added U?: LT1790BCS6-2.5, Package_TO_SOT_SMD:TSOT-23-6, symbol Reference_Voltage:LT1790-2.5
- added U? (x2): TL071, symbol Amplifier_Operational:TL071
- added U?: TPS76925, Package_TO_SOT_SMD:SOT-23-5, symbol Regulator_Linear:TPS76925
- renumbered C16 to C401, C17 to C402, C18 to C403, C19 to C404, C20 to C405, C21 to C406, C22 to C407, C23 to C408, C24 to C409, C25 to C410, C26 to C411, C27 to C412, C28 to C413, C29 to C414, C30 to C415, C31 to C416, C32 to C417, C33 to C418, C34 to C419, C35 to C420, C36 to C421, C37 to C422, C38 to C423, C39 to C424, C40 to C425, C41 to C426, C42 to C427, C43 to C428, C44 to C429, R22 to R401, R23 to R402, R24 to R403, R25 to R404, R26 to R405, R27 to R406, R28 to R407, R29 to R408, R30 to R409, R31 to R410, R32 to R411, R33 to R412, R34 to R413, R35 to R414, R36 to R415, R37 to R416, R38 to R417, R39 to R418, R40 to R419, R41 to R420, R42 to R421, U5 to U401, U6 to U402, U7 to U403, U8 to U404, U9 to U405, U10 to U406, U11 to U407, U12 to U408, U13 to U411, U14 to U412
Connections:
- net +15V: now also U409.4 (V+), U410.4 (V+), U?.4 (Vin), U?.7 (V+), U?.7 (V+)
- net +5V: now also U409.5 (VL), U410.5 (VL), U?.1 (IN), U?.3 (~{EN})
- net -15V: now also U409.3 (GND), U410.3 (GND), U?.4 (V-), U?.4 (V-)
- net GND: now also C?.2, R?.1, R?.1, U409.7 (V-), U410.7 (V-), U?.1 (GND), U?.2 (GND), U?.2 (GND)
- net at R413.1, U403.3, U408.6: now also U410.1; no longer R417.1
- net at R410.1, U401.3, U407.6: now also U409.1; no longer R416.1
- new net: R?.2, R?.2, U?.3 (+) (x2)
- new net: R?.1, R?.2, U?.2 (-) (x2)
- new net: R?.2, U?.6 (x2)
- new net ADC1_CURR: R417.1, U410.2
- new net ADC1_VOLT: R416.1, U409.2
- new net ADC2_CURR: R?.1, U410.8
- new net ADC2_VOLT: R?.1, U409.8
- new net VDDF: C?.1, R?.1, R?.1, U?.6 (Vout)
- no-connect marks 3 -> 7
Other:
- note added: "ad7980"
- moved on the sheet: C428, C429, R406, R407, R408, R409, R410, R411, R412, R413, R414, R415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
