File: HARDWARE/ETH1CSMU2/Measure.kicad_sch (KiCad schematic)
At the start: 75 parts, among them U401 DG444DY+, U402 REF5040ID, U403 DG444DY+, U404 DG419DY, U405 DG419DY, U406 DG419DY, U407 OPA141AID, U408 OPA141AID, U409 DG419DY, U410 DG419DY, U411 ADS8681IRUMT, U412 ADS8681IRUMT

Commit message: Hardware design
Parts:
- removed C402, C406, C412, C417, C423: 100n, Capacitor_SMD:C_0603_1608Metric_Pad1.08x0.95mm_HandSolder, symbol Device:C
- removed U? (x2): TL071, symbol Amplifier_Operational:TL071
- added C401, C405, C409, C413, C419, C422, C427, C430, C431, C434, C435, C436, C437, C438, C439, C440, C441, C442, C443, C444, C445, C446, C? (x3): 100n, Capacitor_SMD:C_0603_1608Metric_Pad1.08x0.95mm_HandSolder, symbol Device:C
- added C433: 10n, Capacitor_SMD:C_0603_1608Metric_Pad1.08x0.95mm_HandSolder, symbol Device:C
- added C449, C450: 2n7, Capacitor_SMD:C_0603_1608Metric_Pad1.08x0.95mm_HandSolder, symbol Device:C
- added C451, C452: 1u, Capacitor_SMD:C_0603_1608Metric_Pad1.08x0.95mm_HandSolder, symbol Device:C
- added R406: 82k, Resistor_SMD:R_0603_1608Metric_Pad0.98x0.95mm_HandSolder, symbol Device:R
- added R427, R428: 20, Resistor_SMD:R_0603_1608Metric_Pad0.98x0.95mm_HandSolder, symbol Device:R
- added R433: OPT, Resistor_SMD:R_0603_1608Metric_Pad0.98x0.95mm_HandSolder, symbol Device:R
- added R434: 0, Resistor_SMD:R_0603_1608Metric_Pad0.98x0.95mm_HandSolder, symbol Device:R
- added U405: ADR435ARM, Package_SO:MSOP-8_3x3mm_P0.65mm, symbol ETH1CSMU2:ADR435ARM
- added U413, U414: OPA141AID, Package_SO:SOIC-8_3.9x4.9mm_P1.27mm, symbol ETH3CDAQ1:OPA140
- added U417, U418: AD7980ARM, Package_SO:MSOP-10_3x3mm_P0.5mm, symbol ETH1CSMU2:AD7980ARM
- R417, R420, R425, R426: renamed from R?; value 2k49 -> 2k49/.1%; footprint (none) -> Resistor_SMD:R_0603_1608Metric_Pad0.98x0.95mm_HandSolder
- R418, R419, R421, R422: renamed from R?; value 10k -> 12k/.1%; footprint (none) -> Resistor_SMD:R_0603_1608Metric_Pad0.98x0.95mm_HandSolder
- gave numbers to parts that had none: 3
- renumbered C403 to C402, C401 to C403, C407 to C406, C408 to C407, C405 to C408, C413 to C410, C409 to C411, C411 to C412, C418 to C414, C414 to C416, C419 to C417, C416 to C418, C424 to C420, C420 to C421, C427 to C423, C421 to C424, C422 to C425, C410 to C428, C425 to C429, C415 to C432, C428 to C447, C429 to C448, R406 to R407, R407 to R408, R408 to R409, R409 to R410, R410 to R411, R411 to R412, R412 to R413, R413 to R414, R414 to R415, R415 to R416, R416 to R423, R417 to R424, R418 to R429, R419 to R430, R420 to R431, R421 to R432, U401 to U402, U402 to U403, U403 to U404, U404 to U407, U405 to U408, U407 to U409, U408 to U410, U409 to U411, U410 to U412, U411 to U415, U412 to U416
Connections:
- net +15V: now also U407.4 (V+), C427.1, C431.1, C435.1, C438.1, C442.1, C444.1, C446.1, U405.2 (VIN), U413.7 (V+), U414.7 (V+); no longer U407.5 (VL)
- net +3.3V: now also C436.1, C440.1
- net +5V: now also U407.5 (VL), C451.1, C?.1, C?.1, C?.1; no longer U407.4 (V+)
- net -15V: now also U411.7 (V-), U412.7 (V-), C401.1, C405.1, C409.1, C413.1, C419.1, C422.1, C430.1, C434.1, C437.1, C441.1, C443.1, C445.1, U413.4 (V-), U414.4 (V-); no longer U411.3 (GND), U412.3 (GND)
- net GND: now also U411.3 (GND), U412.3 (GND), C401.2, C405.2, C409.2, C413.2, C419.2, C422.2, C427.2, C430.2, C431.2, C434.2, C435.2, C436.2, C437.2, C438.2, C439.2, C440.2, C441.2, C442.2, C443.2, C444.2, C445.2, C446.2, C449.2, C450.2, C451.2, C452.2, C?.2, C?.2, C?.2, R434.2, U405.4 (GND), U417.4 (IN-), U417.5 (GND), U418.4 (IN-), U418.5 (GND); no longer U411.7 (V-), U412.7 (V-)
- net VDDF: no longer C415.1, U401.6 (Vout)
- net at R417.2, R418.2: now also U413.3 (+)
- net ADC_SEL: now reaches U411.6
- net ADC_SEL: now also U412.6
- net at R419.2, R425.1: now also U413.2 (-)
- net at R425.2: now also R427.1, U413.6
- net +2V5PWR: now reaches U419.5 (OUT)
- net +2V5PWR: now also C452.1, U417.2 (VDD), U418.2 (VDD)
- net at R422.2, R426.1: now also U414.2 (-)
- net at R420.2, R421.2: now also U414.3 (+)
- net at R426.2: now also R428.1, U414.6
- net ADC_HS_MISO renamed ADC1_MISO
- net ADC_HS_MOSI renamed ADC1_MOSI
- net ADC_HS_RVS1 renamed ADC1_RVS1
- net ADC_HS_RVS2 renamed ADC1_RVS2
- net ADC_HS_SCLK renamed ADC1_SCLK
- net ADC_HS_~{CS} renamed ADC1_~{CS}
- new net: C433.2, R406.2
- new net: C450.1, R428.2, U418.3 (IN+)
- new net: R433.2, R434.1, U417.9 (SDI)
- new net: R406.1, U405.7 (COMP)
- new net: U417.7 (SDO), U418.9 (SDI)
- new net: C449.1, R427.2, U417.3 (IN+)
- new net +2V5REF: C415.1, U401.6 (Vout)
- new net +3V3: U417.10 (VIO), U418.10 (VIO)
- new net +5VREF: C433.1, C439.1, U405.6 (VOUT), U417.1 (REF), U418.1 (REF)
- new net ADC2_CNV: R433.1, U417.6 (CNV), U418.6 (CNV)
- new net ADC2_MISO: U418.7 (SDO)
- new net ADC2_SCLK: U417.8 (SCLK), U418.8 (SCLK)
- no-connect marks 7 -> 4
Other:
- note added: "ADC1"
- note added: "ADC2"
- note added: "GAIN AND ADC SELECTION"
- note added: "MISC"
- note added: "REFERENCES"
- note removed: "ad7980"
- moved on the sheet: C402, C403, C406, C407, C408, C410, C411, C412, C414, C415, C417, C418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

Commit message: Hardware and software development
Parts:
- gave numbers to parts that had none: 3
- renumbered C404 to C403, C405 to C404, C406 to C405, C407 to C406, C403 to C407, C409 to C408, C410 to C409, C411 to C410, C408 to C411, C413 to C412, C414 to C413, C415 to C414, C416 to C415, C417 to C416, C412 to C417, C419 to C418, C420 to C419, C421 to C420, C424 to C421, C418 to C422, C422 to C423, C423 to C424, C428 to C425, C425 to C426, C426 to C427, C427 to C428, C432 to C429, C429 to C432, C437 to C438, C438 to C439, C439 to C440, C440 to C441, C441 to C443, C442 to C444, C443 to C446, C444 to C447, C445 to C448, C446 to C449, C447 to C450, C448 to C451, C449 to C452, C450 to C453, C451 to C454, C452 to C455
Connections:
- net VDDF is gone; now on net +2V5REF: R417.1, R420.1

Commit message: CRC check
Parts:
- U409, U410, U413, U414: symbol ETH3CDAQ1:OPA140 -> ETH1CSMU2:OPA140
Connections:
- net GND: now also U415.17 (PAD), U416.17 (PAD)
- net +2V5REF renamed MEAS_2.5VREF
Other:
- moved on the sheet: C414

Commit message: PCB layout
Changed lines of the file:
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@@
     (pin "2")
   )
-  (symbol (lib_id "Device:R") (at 219.71 64.77 0) (unit 1)
+  (symbol (lib_id "Device:R") (at 219.71 64.77 0) (mirror y) (unit 1)
     (in_bom yes) (on_board yes)
-    (property "Reference" "R411" (id 0) (at 221.488 63.6016 0)
+    (property "Reference" "R411" (id 0) (at 217.932 63.6016 0)
       (effects (font (size 1.27 1.27)) (justify left))
     )
-    (property "Value" "180k/0.05%" (id 1) (at 221.488 65.913 0)
+    (property "Value" "180k/0.05%" (id 1) (at 217.932 65.913 0)
       (effects (font (size 1.27 1.27)) (justify left))
     )
-    (property "Footprint" "Resistor_SMD:R_0603_1608Metric_Pad0.98x0.95mm_HandSolder" (id 2) (at 217.932 64.77 90)
+    (property "Footprint" "Resistor_SMD:R_0603_1608Metric_Pad0.98x0.95mm_HandSolder" (id 2) (at 221.488 64.77 90)
       (effects (font (size 1.27 1.27)) hide)
     )

Commit message: PCB layout
Parts:
- removed C438, C446: 100n, Capacitor_SMD:C_0603_1608Metric_Pad1.08x0.95mm_HandSolder, symbol Device:C
- renumbered C443 to C438, C448 to C443, C447 to C446, C449 to C447, C450 to C448, C451 to C449, C452 to C450, C453 to C451, C454 to C452, C455 to C453
Other:
- moved on the sheet: C438, C443
Changed lines of the file:
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@@
   (junction (at 71.12 226.06) (diameter 0) (color 0 0 0 0)
   )
-  (junction (at 142.24 241.3) (diameter 0) (color 0 0 0 0)
-  )
   (junction (at 198.12 73.66) (diameter 0) (color 0 0 0 0)
   )
@@
   (junction (at 355.6 66.04) (diameter 0) (color 0 0 0 0)
   )
-  (junction (at 130.81 241.3) (diameter 0) (color 0 0 0 0)
-  )
   (junction (at 36.83 100.33) (diameter 0) (color 0 0 0 0)
   )
@@
   (junction (at 85.09 251.46) (diameter 0) (color 0 0 0 0)
   )
-  (junction (at 130.81 251.46) (diameter 0) (color 0 0 0 0)
-  )
   (junction (at 290.83 226.06) (diameter 0) (color 0 0 0 0)
   )
@@
   (junction (at 119.38 241.3) (diameter 0) (color 0 0 0 0)
   )
-  (junction (at 142.24 251.46) (diameter 0) (color 0 0 0 0)
-  )
   (junction (at 381 207.01) (diameter 0) (color 0 0 0 0)
   )
@@
     (stroke (width 0) (type default) (color 0 0 0 0))
   )
-  (wire (pts (xy 153.67 250.19) (xy 153.67 251.46))
-    (stroke (width 0) (type default) (color 0 0 0 0))
-  )
   (wire (pts (xy 349.25 21.59) (xy 349.25 20.32))
     (stroke (width 0) (type default) (color 0 0 0 0))
@@
     (stroke (width 0) (type default) (color 0 0 0 0))
   )
-  (wire (pts (xy 153.67 251.46) (xy 142.24 251.46))
-    (stroke (width 0) (type default) (color 0 0 0 0))
-  )
   (wire (pts (xy 222.25 276.86) (xy 222.25 275.59))
     (stroke (width 0) (type default) (color 0 0 0 0))
@@
     (stroke (width 0) (type default) (color 0 0 0 0))
   )
-  (wire (pts (xy 153.67 241.3) (xy 153.67 242.57))
-    (stroke (width 0) (type default) (color 0 0 0 0))
-  )
   (wire (pts (xy 96.52 251.46) (xy 85.09 251.46))
     (stroke (width 0) (type default) (color 0 0 0 0))
@@
     (stroke (width 0) (type default) (color 0 0 0 0))
   )
-  (wire (pts (xy 142.24 241.3) (xy 142.24 242.57))
-    (stroke (width 0) (type default) (color 0 0 0 0))
-  )
   (wire (pts (xy 120.65 93.98) (xy 120.65 101.6))
     (stroke (width 0) (type default) (color 0 0 0 0))
@@
     (stroke (width 0) (type default) (color 0 0 0 0))
   )
-  (wire (pts (xy 142.24 251.46) (xy 130.81 251.46))
-    (stroke (width 0) (type default) (color 0 0 0 0))
-  )
   (wire (pts (xy 73.66 251.46) (xy 62.23 251.46))
     (stroke (width 0) (type default) (color 0 0 0 0))
@@
     (stroke (width 0) (type default) (color 0 0 0 0))
   )
-  (wire (pts (xy 142.24 241.3) (xy 153.67 241.3))
-    (stroke (width 0) (type default) (color 0 0 0 0))
-  )
   (wire (pts (xy 349.25 34.29) (xy 349.25 29.21))
     (stroke (width 0) (type default) (color 0 0 0 0))
@@
     (stroke (width 0) (type default) (color 0 0 0 0))
   )
-  (wire (pts (xy 142.24 250.19) (xy 142.24 251.46))
-    (stroke (width 0) (type default) (color 0 0 0 0))
-  )
   (wire (pts (xy 83.82 187.96) (xy 96.52 187.96))
     (stroke (width 0) (type default) (color 0 0 0 0))
@@
     (stroke (width 0) (type default) (color 0 0 0 0))
   )
-  (wire (pts (xy 130.81 241.3) (xy 142.24 241.3))
-    (stroke (width 0) (type default) (color 0 0 0 0))
-  )
   (wire (pts (xy 325.12 26.67) (xy 325.12 16.51))
     (stroke (width 0) (type default) (color 0 0 0 0))
@@
   (symbol (lib_id "Device:C") (at 292.1 87.63 0) (unit 1)
     (in_bom yes) (on_board yes)
-    (property "Reference" "C451" (id 0) (at 295.021 86.4616 0)
+    (property "Reference" "C449" (id 0) (at 295.021 86.4616 0)
       (effects (font (size 1.27 1.27)) (justify left))
     )
@@
     (pin "12")
   )
-  (symbol (lib_id "Device:C") (at 153.67 246.38 0) (unit 1)
+  (symbol (lib_id "Device:C") (at 130.81 246.38 0) (unit 1)
     (in_bom yes) (on_board yes) (fields_autoplaced)
-    (property "Reference" "C448" (id 0) (at 156.591 245.5453 0)
+    (property "Reference" "C443" (id 0) (at 133.731 245.5453 0)
       (effects (font (size 1.27 1.27)) (justify left))
     )
-    (property "Value" "100n" (id 1) (at 156.591 248.0822 0)
+    (property "Value" "100n" (id 1) (at 133.731 248.0822 0)
       (effects (font (size 1.27 1.27)) (justify left))
     )
-    (property "Footprint" "Capacitor_SMD:C_0603_1608Metric_Pad1.08x0.95mm_HandSolder" (id 2) (at 154.6352 250.19 0)
+    (property "Footprint" "Capacitor_SMD:C_0603_1608Metric_Pad1.08x0.95mm_HandSolder" (id 2) (at 131.7752 250.19 0)
       (effects (font (size 1.27 1.27)) hide)
     )
-    (property "Datasheet" "~" (id 3) (at 153.67 246.38 0)
+    (property "Datasheet" "~" (id 3) (at 130.81 246.38 0)
       (effects (font (size 1.27 1.27)) hide)
     )
@@
   (symbol (lib_id "Device:C") (at 364.49 124.46 0) (unit 1)
     (in_bom yes) (on_board yes) (fields_autoplaced)
-    (property "Reference" "C454" (id 0) (at 368.3 123.1899 0)
+    (property "Reference" "C452" (id 0) (at 368.3 123.1899 0)
       (effects (font (size 1.27 1.27)) (justify left))
     )
@@
   (symbol (lib_id "Device:C") (at 142.24 270.51 0) (unit 1)
     (in_bom yes) (on_board yes) (fields_autoplaced)
-    (property "Reference" "C447" (id 0) (at 145.161 269.6753 0)
+    (property "Reference" "C446" (id 0) (at 145.161 269.6753 0)
       (effects (font (size 1.27 1.27)) (justify left))
     )
@@
   (symbol (lib_id "Device:C") (at 397.51 124.46 0) (unit 1)
     (in_bom yes) (on_board yes) (fields_autoplaced)
-    (property "Reference" "C455" (id 0) (at 401.32 123.1899 0)
+    (property "Reference" "C453" (id 0) (at 401.32 123.1899 0)
       (effects (font (size 1.27 1.27)) (justify left))
     )
@@
   (symbol (lib_id "Device:C") (at 321.31 210.82 0) (unit 1)
     (in_bom yes) (on_board yes) (fields_autoplaced)
-    (property "Reference" "C453" (id 0) (at 325.12 209.5499 0)
+    (property "Reference" "C451" (id 0) (at 325.12 209.5499 0)
       (effects (font (size 1.27 1.27)) (justify left))
     )
@@
   (symbol (lib_id "Device:C") (at 153.67 270.51 0) (unit 1)
     (in_bom yes) (on_board yes) (fields_autoplaced)
-    (property "Reference" "C449" (id 0) (at 156.591 269.6753 0)
+    (property "Reference" "C447" (id 0) (at 156.591 269.6753 0)
       (effects (font (size 1.27 1.27)) (justify left))
     )
@@
     (pin "9")
   )
-  (symbol (lib_id "Device:C") (at 142.24 246.38 0) (unit 1)
-    (in_bom yes) (on_board yes) (fields_autoplaced)
-    (property "Reference" "C446" (id 0) (at 145.161 245.5453 0)
-      (effects (font (size 1.27 1.27)) (justify left))
-    )
-    (property "Value" "100n" (id 1) (at 145.161 248.0822 0)
-      (effects (font (size 1.27 1.27)) (justify left))
-    )
-    (property "Footprint" "Capacitor_SMD:C_0603_1608Metric_Pad1.08x0.95mm_HandSolder" (id 2) (at 143.2052 250.19 0)
-      (effects (font (size 1.27 1.27)) hide)
-    )
-    (property "Datasheet" "~" (id 3) (at 142.24 246.38 0)
-      (effects (font (size 1.27 1.27)) hide)
-    )
-    (pin "1")
-    (pin "2")
-  )
   (symbol (lib_id "Analog_Switch:DG419xY") (at 190.5 115.57 0) (mirror y) (unit 1)
     (in_bom yes) (on_board yes)
@@
   (symbol (lib_id "Device:C") (at 292.1 41.91 0) (unit 1)
     (in_bom yes) (on_board yes)
-    (property "Reference" "C450" (id 0) (at 295.021 40.7416 0)
+    (property "Reference" "C448" (id 0) (at 295.021 40.7416 0)
       (effects (font (size 1.27 1.27)) (justify left))
     )
@@
   (symbol (lib_id "Device:C") (at 321.31 161.29 0) (unit 1)
     (in_bom yes) (on_board yes) (fields_autoplaced)
-    (property "Reference" "C452" (id 0) (at 325.12 160.0199 0)
+    (property "Reference" "C450" (id 0) (at 325.12 160.0199 0)
       (effects (font (size 1.27 1.27)) (justify left))
     )
@@
     (pin "7")
   )
-  (symbol (lib_id "Device:C") (at 119.38 246.38 0) (unit 1)
-    (in_bom yes) (on_board yes) (fields_autoplaced)
-    (property "Reference" "C438" (id 0) (at 122.301 245.5453 0)
-      (effects (font (size 1.27 1.27)) (justify left))
-    )
-    (property "Value" "100n" (id 1) (at 122.301 248.0822 0)
-      (effects (font (size 1.27 1.27)) (justify left))
-    )
-    (property "Footprint" "Capacitor_SMD:C_0603_1608Metric_Pad1.08x0.95mm_HandSolder" (id 2) (at 120.3452 250.19 0)
-      (effects (font (size 1.27 1.27)) hide)
-    )
-    (property "Datasheet" "~" (id 3) (at 119.38 246.38 0)
-      (effects (font (size 1.27 1.27)) hide)
-    )
-    (pin "1")
-    (pin "2")
-  )
   (symbol (lib_id "ETH1CSMU2:AD7980ARM") (at 355.6 158.75 0) (unit 1)
     (in_bom yes) (on_board yes)
@@
     (pin "7")
   )
-  (symbol (lib_id "Device:C") (at 130.81 246.38 0) (unit 1)
+  (symbol (lib_id "Device:C") (at 119.38 246.38 0) (unit 1)
     (in_bom yes) (on_board yes) (fields_autoplaced)
-    (property "Reference" "C443" (id 0) (at 133.731 245.5453 0)
+    (property "Reference" "C438" (id 0) (at 122.301 245.5453 0)
       (effects (font (size 1.27 1.27)) (justify left))
     )
-    (property "Value" "100n" (id 1) (at 133.731 248.0822 0)
+    (property "Value" "100n" (id 1) (at 122.301 248.0822 0)
       (effects (font (size 1.27 1.27)) (justify left))
     )
-    (property "Footprint" "Capacitor_SMD:C_0603_1608Metric_Pad1.08x0.95mm_HandSolder" (id 2) (at 131.7752 250.19 0)
+    (property "Footprint" "Capacitor_SMD:C_0603_1608Metric_Pad1.08x0.95mm_HandSolder" (id 2) (at 120.3452 250.19 0)
       (effects (font (size 1.27 1.27)) hide)
     )
-    (property "Datasheet" "~" (id 3) (at 130.81 246.38 0)
+    (property "Datasheet" "~" (id 3) (at 119.38 246.38 0)
       (effects (font (size 1.27 1.27)) hide)
     )

Commit message: PCB layout
Connections:
- net +3V3 is gone; now on net +3.3V: U417.10 (VIO), U418.10 (VIO)
Changed lines of the file:
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@@
     (stroke (width 0) (type default) (color 0 0 0 0))
   )
-  (wire (pts (xy 170.18 115.57) (xy 172.72 115.57))
+  (wire (pts (xy 360.68 144.78) (xy 360.68 146.05))
     (stroke (width 0) (type default) (color 0 0 0 0))
   )
-  (wire (pts (xy 38.1 187.96) (xy 44.45 187.96))
+  (wire (pts (xy 170.18 115.57) (xy 172.72 115.57))
     (stroke (width 0) (type default) (color 0 0 0 0))
   )
-  (wire (pts (xy 360.68 194.31) (xy 360.68 195.58))
+  (wire (pts (xy 38.1 187.96) (xy 44.45 187.96))
     (stroke (width 0) (type default) (color 0 0 0 0))
   )
@@
     (stroke (width 0) (type default) (color 0 0 0 0))
   )
-  (wire (pts (xy 360.68 144.78) (xy 360.68 146.05))
-    (stroke (width 0) (type default) (color 0 0 0 0))
-  )
   (wire (pts (xy 119.38 251.46) (xy 107.95 251.46))
     (stroke (width 0) (type default) (color 0 0 0 0))
@@
     (stroke (width 0) (type default) (color 0 0 0 0))
   )
-  (wire (pts (xy 364.49 144.78) (xy 360.68 144.78))
-    (stroke (width 0) (type default) (color 0 0 0 0))
-  )
   (wire (pts (xy 44.45 187.96) (xy 44.45 189.23))
     (stroke (width 0) (type default) (color 0 0 0 0))
@@
     (stroke (width 0) (type default) (color 0 0 0 0))
   )
+  (wire (pts (xy 364.49 194.31) (xy 360.68 194.31))
+    (stroke (width 0) (type default) (color 0 0 0 0))
+  )
   (wire (pts (xy 198.12 123.19) (xy 201.93 123.19))
     (stroke (width 0) (type default) (color 0 0 0 0))
@@
     (stroke (width 0) (type default) (color 0 0 0 0))
   )
+  (wire (pts (xy 364.49 144.78) (xy 360.68 144.78))
+    (stroke (width 0) (type default) (color 0 0 0 0))
+  )
   (wire (pts (xy 355.6 171.45) (xy 355.6 172.72))
     (stroke (width 0) (type default) (color 0 0 0 0))
@@
     (stroke (width 0) (type default) (color 0 0 0 0))
   )
+  (wire (pts (xy 360.68 194.31) (xy 360.68 195.58))
+    (stroke (width 0) (type default) (color 0 0 0 0))
+  )
   (wire (pts (xy 36.83 100.33) (xy 36.83 102.87))
     (stroke (width 0) (type default) (color 0 0 0 0))
@@
     (stroke (width 0) (type default) (color 0 0 0 0))
   )
-  (wire (pts (xy 364.49 194.31) (xy 360.68 194.31))
-    (stroke (width 0) (type default) (color 0 0 0 0))
-  )
   (wire (pts (xy 303.53 87.63) (xy 304.8 87.63))
     (stroke (width 0) (type default) (color 0 0 0 0))
@@
     (pin "2")
   )
-  (symbol (lib_name "+3.3V_1") (lib_id "power:+3.3V") (at 364.49 194.31 0) (unit 1)
-    (in_bom yes) (on_board yes)
-    (property "Reference" "#PWR0492" (id 0) (at 364.49 198.12 0)
-      (effects (font (size 1.27 1.27)) hide)
-    )
-    (property "Value" "+3.3V" (id 1) (at 364.49 190.5 0))
-    (property "Footprint" "" (id 2) (at 364.49 194.31 0)
-      (effects (font (size 1.27 1.27)) hide)
-    )
-    (property "Datasheet" "" (id 3) (at 364.49 194.31 0)
-      (effects (font (size 1.27 1.27)) hide)
-    )
-    (pin "1")
-  )
   (symbol (lib_id "Device:C") (at 96.52 270.51 0) (unit 1)
     (in_bom yes) (on_board yes) (fields_autoplaced)
@@
     (pin "2")
   )
+  (symbol (lib_id "power:+3.3V") (at 364.49 144.78 0) (unit 1)
+    (in_bom yes) (on_board yes) (fields_autoplaced)
+    (property "Reference" "#PWR0102" (id 0) (at 364.49 148.59 0)
+      (effects (font (size 1.27 1.27)) hide)
+    )
+    (property "Value" "+3.3V" (id 1) (at 364.49 141.2042 0))
+    (property "Footprint" "" (id 2) (at 364.49 144.78 0)
+      (effects (font (size 1.27 1.27)) hide)
+    )
+    (property "Datasheet" "" (id 3) (at 364.49 144.78 0)
+      (effects (font (size 1.27 1.27)) hide)
+    )
+    (pin "1")
+  )
   (symbol (lib_id "Device:R") (at 284.48 146.05 90) (unit 1)
     (in_bom yes) (on_board yes)
@@
     (pin "1")
   )
-  (symbol (lib_name "+3.3V_1") (lib_id "power:+3.3V") (at 364.49 144.78 0) (unit 1)
-    (in_bom yes) (on_board yes)
-    (property "Reference" "#PWR0491" (id 0) (at 364.49 148.59 0)
-      (effects (font (size 1.27 1.27)) hide)
-    )
-    (property "Value" "+3.3V" (id 1) (at 364.49 140.97 0))
-    (property "Footprint" "" (id 2) (at 364.49 144.78 0)
-      (effects (font (size 1.27 1.27)) hide)
-    )
-    (property "Datasheet" "" (id 3) (at 364.49 144.78 0)
-      (effects (font (size 1.27 1.27)) hide)
-    )
-    (pin "1")
-  )
   (symbol (lib_id "power:+5V") (at 372.11 116.84 0) (unit 1)
     (in_bom yes) (on_board yes)
@@
       (effects (font (size 1.27 1.27)) hide)
     )
+    (pin "1")
+  )
+  (symbol (lib_id "power:+3.3V") (at 364.49 194.31 0) (unit 1)
+    (in_bom yes) (on_board yes) (fields_autoplaced)
+    (property "Reference" "#PWR0101" (id 0) (at 364.49 198.12 0)
+      (effects (font (size 1.27 1.27)) hide)
+    )
+    (property "Value" "+3.3V" (id 1) (at 364.49 190.7342 0))
+    (property "Footprint" "" (id 2) (at 364.49 194.31 0)
+      (effects (font (size 1.27 1.27)) hide)
+    )
+    (property "Datasheet" "" (id 3) (at 364.49 194.31 0)
+      (effects (font (size 1.27 1.27)) hide)
+    )

Commit message: Bug fixes.
Parts:
- added R431: OPT, Resistor_SMD:R_0603_1608Metric_Pad0.98x0.95mm_HandSolder, symbol Device:R
- added R434: 0, Resistor_SMD:R_0603_1608Metric_Pad0.98x0.95mm_HandSolder, symbol Device:R
- renumbered R431 to R432, R432 to R433, R433 to R435, R434 to R436
Connections:
- net +5V: now also R431.1; no longer U419.3 (~{EN})
- net GND: now also R434.2
- new net: R431.2, R434.1, U419.3 (~{EN})
Other:
- moved on the sheet: C452
