File: HARDWARE/ETH1CSMU2/Measure.kicad_sch (KiCad schematic)
At the start: 108 parts, among them U401 LT1790BCS6-2.5, U402 DG444DY+, U403 REF5040ID, U404 DG444DY+, U405 ADR435ARM, U406 DG419DY, U407 DG419DY, U408 DG419DY, U409 OPA141AID, U410 OPA141AID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

Commit message: Software development
Parts:
- C406, C416: footprint Resistor_SMD:R_0805_2012Metric_Pad1.20x1.40mm_HandSolder -> Capacitor_SMD:C_0805_2012Metric_Pad1.18x1.45mm_HandSolder
Changed lines of the file:
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@@
       (effects (font (size 1.27 1.27)) (justify left))
     )
-    (property "Footprint" "Resistor_SMD:R_0805_2012Metric_Pad1.20x1.40mm_HandSolder" (id 2) (at 59.3852 196.85 0)
+    (property "Footprint" "Capacitor_SMD:C_0805_2012Metric_Pad1.18x1.45mm_HandSolder" (id 2) (at 59.3852 196.85 0)
       (effects (font (size 1.27 1.27)) hide)
     )
@@
       (effects (font (size 1.27 1.27)) (justify left))
     )
-    (property "Footprint" "Resistor_SMD:R_0805_2012Metric_Pad1.20x1.40mm_HandSolder" (id 2) (at 32.7152 196.85 0)
+    (property "Footprint" "Capacitor_SMD:C_0805_2012Metric_Pad1.18x1.45mm_HandSolder" (id 2) (at 32.7152 196.85 0)
       (effects (font (size 1.27 1.27)) hide)
     )

Commit message: Development
Changed lines of the file:
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@@
   )
   (polyline (pts (xy 172.72 203.2) (xy 149.86 203.2))
-    (stroke (width 0) (type default))
+    (stroke (width 0) (type dash))
   )
   (wire (pts (xy 290.83 82.55) (xy 292.1 82.55))
@@
   )
   (polyline (pts (xy 172.72 203.2) (xy 261.62 203.2))
-    (stroke (width 0) (type default))
+    (stroke (width 0) (type dash))
   )
   (wire (pts (xy 355.6 220.98) (xy 355.6 222.25))
@@
   )
   (polyline (pts (xy 172.72 281.94) (xy 172.72 203.2))
-    (stroke (width 0) (type default))
+    (stroke (width 0) (type dash))
   )
   (wire (pts (xy 199.39 90.17) (xy 198.12 90.17))
@@
   )
   (polyline (pts (xy 149.86 203.2) (xy 149.86 116.84))
-    (stroke (width 0) (type default))
+    (stroke (width 0) (type dash))
   )
   (polyline (pts (xy 261.62 13.97) (xy 261.62 236.22))
-    (stroke (width 0) (type default))
+    (stroke (width 0) (type dash))
   )
   (wire (pts (xy 320.04 26.67) (xy 316.23 26.67))
@@
   )
   (polyline (pts (xy 261.62 236.22) (xy 405.13 236.22))
-    (stroke (width 0) (type default))
+    (stroke (width 0) (type dash))
   )
   (wire (pts (xy 31.75 226.06) (xy 44.45 226.06))
@@
   )
   (polyline (pts (xy 149.86 116.84) (xy 132.08 116.84))
-    (stroke (width 0) (type default))
+    (stroke (width 0) (type dash))
   )
   (wire (pts (xy 69.85 87.63) (xy 71.12 87.63))
@@
   )
   (polyline (pts (xy 16.51 116.84) (xy 132.08 116.84))
-    (stroke (width 0) (type default))
+    (stroke (width 0) (type dash))
   )
   (wire (pts (xy 62.23 251.46) (xy 50.8 251.46))
@@
   )
   (polyline (pts (xy 132.08 13.97) (xy 132.08 116.84))
-    (stroke (width 0) (type default))
+    (stroke (width 0) (type dash))
   )
   (wire (pts (xy 294.64 176.53) (xy 290.83 176.53))
@@
   )
   (polyline (pts (xy 261.62 109.22) (xy 405.13 109.22))
-    (stroke (width 0) (type default))
+    (stroke (width 0) (type dash))
   )
   (wire (pts (xy 360.68 44.45) (xy 373.38 44.45))
@@
   )
   (text "MISC" (at 16.51 121.92 0)
-    (effects (font (size 1.27 1.27)) (justify left bottom))
+    (effects (font (size 2.54 2.54) (thickness 0.508) bold) (justify left bottom))
   )
   (text "ADC1" (at 265.43 17.78 0)
-    (effects (font (size 1.27 1.27)) (justify left bottom))
-  )
-  (text "ADC2\n" (at 264.16 114.3 0)
-    (effects (font (size 1.27 1.27)) (justify left bottom))
+    (effects (font (size 2.54 2.54) (thickness 0.508) bold) (justify left bottom))
+  )
+  (text "ADC2\n" (at 264.16 115.57 0)
+    (effects (font (size 2.54 2.54) (thickness 0.508) bold) (justify left bottom))
   )
   (text "GAIN AND ADC SELECTION" (at 134.62 17.78 0)
-    (effects (font (size 1.27 1.27)) (justify left bottom))
-  )
-  (text "REFERENCES" (at 13.97 15.24 0)
-    (effects (font (size 1.27 1.27)) (justify left bottom))
+    (effects (font (size 2.54 2.54) (thickness 0.508) bold) (justify left bottom))
+  )
+  (text "REFERENCES" (at 13.97 17.78 0)
+    (effects (font (size 2.54 2.54) (thickness 0.508) bold) (justify left bottom))
   )
   (label "ADC_SEL" (at 233.68 52.07 90) (fields_autoplaced)

Commit message: AD7980 test works.
Parts:
- R431, R435: now not fitted
Changed lines of the file:
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@@
   )
   (symbol (lib_id "Device:R") (at 388.62 154.94 90) (unit 1)
-    (in_bom yes) (on_board yes) (dnp no)
+    (in_bom yes) (on_board yes) (dnp yes)
     (property "Reference" "R435" (at 388.62 149.86 90)
       (effects (font (size 1.27 1.27)))
@@
   )
   (symbol (lib_id "Device:R") (at 359.41 121.92 90) (unit 1)
-    (in_bom yes) (on_board yes) (dnp no)
+    (in_bom yes) (on_board yes) (dnp yes)
     (property "Reference" "R431" (at 359.41 124.46 90)
       (effects (font (size 1.27 1.27)))

Commit message: Software development
Other:
- moved on the sheet: R408, R410, R414, R415, R416, U404A, U404B, U404C, U408A, U410, U412A
