File: HARDWARE/ETH1CSMU2/Source.kicad_sch (KiCad schematic)
At the start: 7 parts, among them U901 ADR425ARMZ, U902 DAC8565

Commit message: Hardware design
Parts:
- renumbered C901 to C87, C902 to C88, C903 to C89, C904 to C90, C905 to C91, U901 to U33, U902 to U34
Changed lines of the file:
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@@
   (symbol (lib_id "power:GND") (at 107.95 60.96 0) (unit 1)
     (in_bom yes) (on_board yes) (fields_autoplaced)
-    (property "Reference" "#PWR0907" (id 0) (at 107.95 67.31 0)
+    (property "Reference" "#PWR0186" (id 0) (at 107.95 67.31 0)
       (effects (font (size 1.27 1.27)) hide)
     )
@@
   (symbol (lib_id "power:+3.3V") (at 33.02 175.26 0) (unit 1)
     (in_bom yes) (on_board yes) (fields_autoplaced)
-    (property "Reference" "#PWR0903" (id 0) (at 33.02 179.07 0)
+    (property "Reference" "#PWR0182" (id 0) (at 33.02 179.07 0)
       (effects (font (size 1.27 1.27)) hide)
     )
@@
   (symbol (lib_id "power:+5V") (at 142.24 25.4 0) (unit 1)
     (in_bom yes) (on_board yes) (fields_autoplaced)
-    (property "Reference" "#PWR0910" (id 0) (at 142.24 29.21 0)
+    (property "Reference" "#PWR0189" (id 0) (at 142.24 29.21 0)
       (effects (font (size 1.27 1.27)) hide)
     )
@@
   (symbol (lib_id "Device:C") (at 20.32 180.34 0) (unit 1)
     (in_bom yes) (on_board yes) (fields_autoplaced)
-    (property "Reference" "C901" (id 0) (at 23.241 179.5053 0)
+    (property "Reference" "C87" (id 0) (at 23.241 179.5053 0)
       (effects (font (size 1.27 1.27)) (justify left))
     )
@@
   (symbol (lib_id "Device:C") (at 33.02 180.34 0) (unit 1)
     (in_bom yes) (on_board yes) (fields_autoplaced)
-    (property "Reference" "C902" (id 0) (at 35.941 179.5053 0)
+    (property "Reference" "C88" (id 0) (at 35.941 179.5053 0)
       (effects (font (size 1.27 1.27)) (justify left))
     )
@@
   (symbol (lib_id "Analog_DAC:DAC8565") (at 147.32 50.8 0) (unit 1)
     (in_bom yes) (on_board yes)
-    (property "Reference" "U902" (id 0) (at 156.21 25.4 0)
+    (property "Reference" "U34" (id 0) (at 156.21 25.4 0)
       (effects (font (size 1.27 1.27)) (justify left))
     )
@@
   (symbol (lib_id "Device:C") (at 76.2 53.34 0) (unit 1)
     (in_bom yes) (on_board yes)
-    (property "Reference" "C904" (id 0) (at 79.121 52.5053 0)
+    (property "Reference" "C90" (id 0) (at 79.121 52.5053 0)
       (effects (font (size 1.27 1.27)) (justify left))
     )
@@
   (symbol (lib_id "power:GND") (at 147.32 69.85 0) (unit 1)
     (in_bom yes) (on_board yes) (fields_autoplaced)
-    (property "Reference" "#PWR0911" (id 0) (at 147.32 76.2 0)
+    (property "Reference" "#PWR0190" (id 0) (at 147.32 76.2 0)
       (effects (font (size 1.27 1.27)) hide)
     )
@@
   (symbol (lib_id "power:+3.3V") (at 149.86 25.4 0) (unit 1)
     (in_bom yes) (on_board yes) (fields_autoplaced)
-    (property "Reference" "#PWR0912" (id 0) (at 149.86 29.21 0)
+    (property "Reference" "#PWR0191" (id 0) (at 149.86 29.21 0)
       (effects (font (size 1.27 1.27)) hide)
     )
@@
   (symbol (lib_id "power:GND") (at 132.08 53.34 270) (unit 1)
     (in_bom yes) (on_board yes)
-    (property "Reference" "#PWR0908" (id 0) (at 125.73 53.34 0)
+    (property "Reference" "#PWR0187" (id 0) (at 125.73 53.34 0)
       (effects (font (size 1.27 1.27)) hide)
     )
@@
   (symbol (lib_id "power:GND") (at 132.08 60.96 270) (unit 1)
     (in_bom yes) (on_board yes)
-    (property "Reference" "#PWR0909" (id 0) (at 125.73 60.96 0)
+    (property "Reference" "#PWR0188" (id 0) (at 125.73 60.96 0)
       (effects (font (size 1.27 1.27)) hide)
     )
@@
   (symbol (lib_id "power:GND") (at 63.5 62.23 0) (unit 1)
     (in_bom yes) (on_board yes) (fields_autoplaced)
-    (property "Reference" "#PWR0906" (id 0) (at 63.5 68.58 0)
+    (property "Reference" "#PWR0185" (id 0) (at 63.5 68.58 0)
       (effects (font (size 1.27 1.27)) hide)
     )
@@
   (symbol (lib_id "Reference_Voltage:ADR425ARMZ") (at 90.17 53.34 0) (unit 1)
     (in_bom yes) (on_board yes)
-    (property "Reference" "U901" (id 0) (at 99.06 44.45 0)
+    (property "Reference" "U33" (id 0) (at 99.06 44.45 0)
       (effects (font (size 1.27 1.27)) (justify right))
     )
@@
   (symbol (lib_id "Device:C") (at 107.95 55.88 0) (unit 1)
     (in_bom yes) (on_board yes) (fields_autoplaced)
-    (property "Reference" "C905" (id 0) (at 110.871 55.0453 0)
+    (property "Reference" "C91" (id 0) (at 110.871 55.0453 0)
       (effects (font (size 1.27 1.27)) (justify left))
     )
@@
   (symbol (lib_id "power:+5V") (at 63.5 44.45 0) (unit 1)
     (in_bom yes) (on_board yes) (fields_autoplaced)
-    (property "Reference" "#PWR0905" (id 0) (at 63.5 48.26 0)
+    (property "Reference" "#PWR0184" (id 0) (at 63.5 48.26 0)
       (effects (font (size 1.27 1.27)) hide)
     )
@@
   (symbol (lib_id "power:GND") (at 20.32 185.42 0) (unit 1)
     (in_bom yes) (on_board yes) (fields_autoplaced)
-    (property "Reference" "#PWR0902" (id 0) (at 20.32 191.77 0)
+    (property "Reference" "#PWR0181" (id 0) (at 20.32 191.77 0)
       (effects (font (size 1.27 1.27)) hide)
     )
@@
   (symbol (lib_id "power:GND") (at 33.02 185.42 0) (unit 1)
     (in_bom yes) (on_board yes) (fields_autoplaced)
-    (property "Reference" "#PWR0904" (id 0) (at 33.02 191.77 0)
+    (property "Reference" "#PWR0183" (id 0) (at 33.02 191.77 0)
       (effects (font (size 1.27 1.27)) hide)
     )
@@
   (symbol (lib_id "Device:C") (at 63.5 53.34 0) (unit 1)
     (in_bom yes) (on_board yes) (fields_autoplaced)
-    (property "Reference" "C903" (id 0) (at 66.421 52.5053 0)
+    (property "Reference" "C89" (id 0) (at 66.421 52.5053 0)
       (effects (font (size 1.27 1.27)) (justify left))
     )
@@
   (symbol (lib_id "power:+5V") (at 20.32 175.26 0) (unit 1)
     (in_bom yes) (on_board yes) (fields_autoplaced)
-    (property "Reference" "#PWR0901" (id 0) (at 20.32 179.07 0)
-      (effects (font (size 1.27 1.27)) hide)
-    )
+    (property "Reference" "#PWR0180" (id 0) (at 20.32 179.07 0)
+      (effects (font (size 1.27 1.27)) hide)
+    )

Commit message: Hardware design
Parts:
- added C92: 100n, symbol Device:C
- added C93, C94: 10n, symbol Device:C
- added C95, C?: 1p, symbol Device:C
- added R67, R68: 200, symbol Device:R
- added R69, R70, R71, R72, R? (x3): R, symbol Device:R
- added R?: 5k6, symbol Device:R
- added U36: AD9834, Package_SO:TSSOP-20_4.4x6.5mm_P0.65mm, symbol Interface:AD9834
- added U38, U?: LM7171xIM, Package_SO:SOIC-8_3.9x4.9mm_P1.27mm, symbol Amplifier_Operational:LM7171xIM
- added X1: SG-8002CE, Oscillator:Oscillator_SMD_SeikoEpson_SG8002CE-4Pin_3.2x2.5mm, symbol Oscillator:SG-8002CE
- renumbered C89 to C88, C88 to C89, U33 to U35, U34 to U37
Connections:
- net +5V: now also C93.1, U36.4 (AVDD)
- net GND: now also C92.1, C94.1, R67.2, R68.2, R71.1, U36.10 (PSELECT), U36.11 (RESET), U36.12 (SLEEP), U36.17 (VIN), U36.18 (AGND), U36.7 (DGND), U36.9 (FSELECT), U?.3 (+), X1.2 (GND)
- new net: R68.1, R70.1, U36.20 (IOUTB)
- new net: C95.1, R70.2, R72.1, U38.2 (-)
- new net: R67.1, R69.1, U36.19 (IOUT)
- new net: R69.2, R71.2, U38.3 (+)
- new net: C95.2, R72.2, U38.6
- new net: U36.8 (MCLK), X1.3 (OUT)
- new net: C92.2, U36.6 (CAP/2.5V)
- new net: C?.1, R?.1, R?.2, R?.2, U?.2 (-)
- new net: C94.2, U36.2 (REFOUT)
- new net: C?.2, R?.2, U?.6
- new net: R?.1, U36.1 (FS_ADJUST)
- new net: C93.2, U36.3 (COMP)
- new net +15V: U38.7 (V+), U?.7 (V+)
- new net +3V3: U36.5 (DVDD), X1.1 (OE), X1.4 (Vcc)
- new net -15V: U38.4 (V-), U?.4 (V-)
- no-connect marks 1 -> 2
Other:
- note added: "AD5322"
- moved on the sheet: C88, C90, C91, U35, U37

Commit message: Hardware design
Parts:
- removed R67, R68: 200, symbol Device:R
- added C904: 100n, symbol Device:C
- added C906: 1u, symbol Device:C
- added C910, C914: 100p, Capacitor_SMD:C_0603_1608Metric_Pad1.08x0.95mm_HandSolder, symbol Device:C
- added C912: 1000p, symbol Device:C
- added C913: 68p, Capacitor_SMD:C_0603_1608Metric_Pad1.08x0.95mm_HandSolder, symbol Device:C
- added C916: 4u7, symbol Device:C
- added C917: 10n, Capacitor_SMD:C_0603_1608Metric_Pad1.08x0.95mm_HandSolder, symbol Device:C
- added L901, L902, L903, L904: CBMF1608T100K, Inductor_SMD:L_0603_1608Metric_Pad1.05x0.95mm_HandSolder, symbol Device:L
- added Q901: FDV301N, Package_TO_SOT_SMD:SOT-23, symbol Device:Q_NMOS_GSD
- added R901, R902: 10k, symbol Device:R
- added R904: 24k9, symbol Device:R
- added R905: 33k2, symbol Device:R
- added R906: 100k, symbol Device:R
- added R907, R908: 200, symbol Device:R
- added R913: 4k7, Resistor_SMD:R_0603_1608Metric_Pad0.98x0.95mm_HandSolder, symbol Device:R
- added R914: 100k, Resistor_SMD:R_0603_1608Metric_Pad0.98x0.95mm_HandSolder, symbol Device:R
- added R915, R917: 220, Resistor_SMD:R_0603_1608Metric_Pad0.98x0.95mm_HandSolder, symbol Device:R
- added R916: 680, Resistor_SMD:R_0603_1608Metric_Pad0.98x0.95mm_HandSolder, symbol Device:R
- added R918: 68, Resistor_SMD:R_0603_1608Metric_Pad0.98x0.95mm_HandSolder, symbol Device:R
- added R919: 33, Resistor_SMD:R_0603_1608Metric_Pad0.98x0.95mm_HandSolder, symbol Device:R
- added R920: 100, Resistor_SMD:R_0603_1608Metric_Pad0.98x0.95mm_HandSolder, symbol Device:R
- added R921: 200, Resistor_SMD:R_0603_1608Metric_Pad0.98x0.95mm_HandSolder, symbol Device:R
- added R922: 1k, Resistor_SMD:R_0603_1608Metric_Pad0.98x0.95mm_HandSolder, symbol Device:R
- added U902: ADR421ARMZ, Package_SO:MSOP-8_3x3mm_P0.65mm, symbol Reference_Voltage:ADR421ARMZ
- added U905: AD5322, symbol ETH1CSMU2:AD5322
- added U906: TL071, symbol Amplifier_Operational:TL071
- added U908: DG409DY, Package_SO:SOIC-16_3.9x9.9mm_P1.27mm, symbol ETH1CLCR2:DG409
- C908: renamed from C92; value 100n -> 4u7
- R909: renamed from R69; value R -> 1k
- R910: renamed from R70; value R -> 1k
- R911: renamed from R71; value R -> 20k
- R912: renamed from R72; value R -> 20k
- R923, R924, R925: renamed from R?; value R -> 1k
- gave numbers to parts that had none: 3
- renumbered C87 to C901, C89 to C902, C88 to C903, C90 to C905, C91 to C907, C93 to C909, C94 to C911, C95 to C915, U35 to U901, U36 to U903, U37 to U904, U38 to U907, X1 to X901
Connections:
- net +15V: now also U906.7 (V+)
- net +3.3V: now also U905.2 (VDD)
- net +5V: now also C904.1, C906.1, U902.2 (VIN)
- net -15V: now also U906.4 (V-)
- net GND: now also C904.2, C906.2, Q901.2 (S), R902.1, R905.1, R907.2, R908.2, R919.2, R922.2, U902.4 (GND), U905.10 (GND), U908.15 (GND)
- net at U903.20 (IOUTB): now also C910.1, L901.1; no longer R910.1
- net at U903.19 (IOUT): now also C910.2, L902.1; no longer R909.1
- net at C915.2, R912.2, U907.6: now also C916.1
- net V_OFFS: now reaches R924.1
- net V_OFFS: now also C912.2, R906.2, U906.6
- net FGEN: now reaches C918.2, R925.2, U909.6
- net VOUTA: now reaches R903.2
- net VOUTA: now also U905.5 (VOUTA)
- net at R923.1: now also C917.1, U908.8 (DA)
- net DDS_SDATA: now reaches U903.13 (SDATA)
- net DDS_SCLK: now reaches U903.14 (SCLK)
- net DDS_CS: now reaches U903.15 (~{FSYNC})
- net DAC_DIN renamed DAC1_DIN
- net DAC_LDAC renamed DAC1_LDAC
- net DAC_SCLK renamed DAC1_SCLK
- net DAC_~{SYNC} renamed DAC1_~{SYNC}
- new net: R916.1, R917.1, U908.5 (S2A)
- new net: C916.2, R915.2, R916.2
- new net: C913.2, L902.2, L904.1
- new net: C914.2, L904.2, R907.1, R909.1
- new net: C914.1, L903.2, R908.1, R910.1
- new net: C912.1, R904.2, R905.2, R906.1, U906.2 (-)
- new net: R920.1, U908.6 (S3A)
- new net: R917.2, R918.1, R920.2
- new net: C917.2, Q901.3 (D), R914.2
- new net: R921.1, U908.7 (S4A)
- new net: R918.2, R919.1, R921.2
- new net: C913.1, L901.2, L903.1
- new net: U908.10 (S4B), U908.11 (S3B), U908.12 (S2B), U908.13 (S1B)
- new net: R915.1, U908.4 (S1A)
- new net: R922.1, U908.9 (DB)
- new net: Q901.1 (G), R913.1
- new net +1V25: R901.2, R902.2, U905.4 (VREFA)
- new net +2V5: R901.1, R904.1, U902.6 (OUT), U905.3 (VREFB)
- new net +5VA: R914.1, U908.14 (V+), U908.2 (EN)
- new net -5VA: U908.3 (V-)
- new net ATT_A0: U908.1 (A0)
- new net ATT_A1: U908.16 (A1)
- new net DAC2_DIN: U905.9 (DIN)
- new net DAC2_SCLK: U905.8 (SCLK)
- new net DAC2_~{LDAC}: U905.1 (~{LDAC})
- new net DAC2_~{SYNC}: U905.7 (~{SYNC})
- new net DDS_LPF: R913.2
- new net VOUTB: U905.6 (VOUTB), U906.3 (+)
- no-connect marks 2 -> 5
Other:
- note removed: "AD5322"
- moved on the sheet: C901, C902, C903, C905, C907, C908, C909, C911, C915, C918, R903, R909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

Commit message: Hardware design.
Parts:
- removed C901, C902, C903, C904: 100n, symbol Device:C
- removed C905, C906: 1u, symbol Device:C
- removed R905: 33k2, symbol Device:R
- removed U901: ADR425ARMZ, Package_SO:MSOP-8_3x3mm_P0.65mm, symbol Reference_Voltage:ADR425ARMZ
- removed U902: ADR421ARMZ, Package_SO:MSOP-8_3x3mm_P0.65mm, symbol Reference_Voltage:ADR421ARMZ
- added C107, C108, C109, C110, C111, C112, C114, C116, C117, C119, C122, C124, C126, C127: 100n, symbol Device:C
- added C132: 1u, symbol Device:C
- added R74: 26k4, symbol Device:R
- added R77: DNP, symbol Device:R
- added U40: LT1790BCS6-2.5, Package_TO_SOT_SMD:TSOT-23-6, symbol Reference_Voltage:LT1790-2.5
- C129: renamed from C912; value 1000p -> 1p
- R73: renamed from R904; value 24k9 -> 20k8
- U35: renamed from U903; value AD9834 -> AD9834BRUZ
- U36: renamed from U904; value DAC8565 -> DAC8565ICPW
- U37: renamed from U905; value AD5322 -> AD5322ARMZ
- U38: renamed from U907; value LM7171xIM -> LM7171BIM
- U39: renamed from U906; value TL071 -> TL071CDR
- U41: renamed from U908; value DG409DY -> DG409DY+
- U42: renamed from U909; value LM7171xIM -> LM7171BIM
- renumbered C907 to C113, C908 to C115, C909 to C118, C910 to C120, C911 to C121, C913 to C123, C914 to C125, C915 to C128, C916 to C130, C917 to C131, C918 to C133, L901 to L5, L902 to L6, L903 to L7, L904 to L8, Q901 to Q2, R903 to R67, R907 to R68, R908 to R69, R909 to R70, R910 to R71, R911 to R72, R912 to R75, R906 to R76, R913 to R78, R914 to R79, R915 to R80, R916 to R81, R917 to R82, R918 to R83, R919 to R84, R920 to R85, R921 to R86, R922 to R87, R901 to R88, R902 to R89, R923 to R90, R924 to R91, R925 to R92, X901 to X1
Connections:
- net +15V: now also C116.1, C117.1, C119.1, C122.1, U40.4 (Vin)
- net +2V5: now also C113.1, U36.3 (VREFH/VREFOUT), C132.1, U40.6 (Vout)
- net +3.3V: now also C110.1, C111.1, C112.1, C114.1
- net +5V: now also C107.1, C108.1, C109.1
- net -15V: now also C124.1, C126.1, C127.1
- net GND: now also C107.2, C108.2, C109.2, C110.2, C111.2, C112.2, C114.2, C116.2, C117.2, C119.2, C122.2, C124.2, C126.2, C127.2, C132.2, R74.1, U40.1 (GND), U40.2 (GND)
- net at C130.2, R80.2, R81.2: now also R77.2
- net at C128.2, C130.1, R75.2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: now also R77.1
- net at C129.1, R73.2, R76.1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: now also R74.2
- no-connect marks 5 -> 3
Other:
- moved on the sheet: C128, C129, R76, R88, R89

Commit message: Hardware design.
Parts:
- added R67: 0, symbol Device:R
- renumbered R67 to R68, R68 to R69, R69 to R70, R70 to R71, R71 to R72, R72 to R73, R73 to R74, R74 to R75, R75 to R76, R76 to R77, R77 to R78, R78 to R79, R79 to R80, R80 to R81, R81 to R82, R82 to R83, R83 to R84, R84 to R85, R85 to R86, R86 to R87, R87 to R88, R88 to R89, R89 to R90, R90 to R91, R91 to R92, R92 to R93
Connections:
- net +2V5: now also R67.1; no longer C113.1, U36.3 (VREFH/VREFOUT)
- new net: C113.1, R67.2, U36.3 (VREFH/VREFOUT)

Commit message: Hardware design
Parts:
- C107, C108, C109, C110, C111, C112, C113, C114, C116, C117, C118, C119, C121, C122, C124, C126, C127, C128, C129, C132, C133: footprint (none) -> Capacitor_SMD:C_0603_1608Metric_Pad1.08x0.95mm_HandSolder
- C115, C130: footprint (none) -> Capacitor_SMD:C_0805_2012Metric_Pad1.18x1.45mm_HandSolder
- R67, R68, R69, R70, R74, R75, R77, R78, R89, R90: footprint (none) -> Resistor_SMD:R_0603_1608Metric_Pad0.98x0.95mm_HandSolder
- R71, R72, R91, R92, R93: value 1k -> 1k/.1%; footprint (none) -> Resistor_SMD:R_0603_1608Metric_Pad0.98x0.95mm_HandSolder
- R73, R76: value 20k -> 20k/.1%; footprint (none) -> Resistor_SMD:R_0603_1608Metric_Pad0.98x0.95mm_HandSolder
- U37: footprint (none) -> Package_SO:MSOP-10_3x3mm_P0.5mm
- U39: footprint (none) -> Package_SO:SOIC-8_3.9x4.9mm_P1.27mm
Other:
- moved on the sheet: R71, R72, R73, R78

Commit message: Schematic
Connections:
- net DAC_~{RST} renamed DAC1_~{RST}
Changed lines of the file:
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@@
     (effects (font (size 1.27 1.27)) (justify right))
   )
-  (hierarchical_label "DAC_~{RST}" (shape input) (at 116.84 55.88 180)
+  (hierarchical_label "DAC1_~{RST}" (shape input) (at 116.84 55.88 180)
     (effects (font (size 1.27 1.27)) (justify right))
   )

Commit message: Hardware design
Parts:
- removed X1: SG-8002CE, Oscillator:Oscillator_SMD_SeikoEpson_SG8002CE-4Pin_3.2x2.5mm, symbol Oscillator:SG-8002CE
- added R901: 4k7, Resistor_SMD:R_0603_1608Metric_Pad0.98x0.95mm_HandSolder, symbol Device:R
- added R902, R909: 68, Resistor_SMD:R_0603_1608Metric_Pad0.98x0.95mm_HandSolder, symbol Device:R
- added U901, U905: MC74AC161DR2G, Package_SO:SOIC-16_3.9x9.9mm_P1.27mm, symbol ETH1CLCR2:74AC161
- added U903: SN74AHC1G14DBVT, Package_TO_SOT_SMD:SOT-23-5_HandSoldering, symbol 74xGxx:74AHC1G14
- added U906: SN74AUP1G79DCKR, Package_TO_SOT_SMD:SOT-353_SC-70-5_Handsoldering, symbol 74xGxx:74AUP1G79
- added X901: 830208220601, ETH1CSMU2:IQXO-791, symbol ETH1CLCR2:IQXO-791
- renumbered C107 to C901, C108 to C902, C109 to C903, C110 to C904, C111 to C905, C112 to C906, C113 to C907, C114 to C908, C115 to C909, C116 to C910, C117 to C911, C118 to C912, C119 to C913, C120 to C914, C121 to C915, C122 to C916, C123 to C917, C124 to C918, C125 to C919, C126 to C920, C127 to C921, C128 to C922, C130 to C923, C131 to C924, C132 to C925, C129 to C926, C133 to C927, L5 to L901, L6 to L902, L7 to L903, L8 to L904, Q2 to Q901, R67 to R903, R68 to R904, R69 to R905, R70 to R906, R71 to R907, R72 to R908, R73 to R910, R76 to R911, R78 to R912, R79 to R913, R80 to R914, R81 to R915, R82 to R916, R83 to R917, R84 to R918, R85 to R919, R86 to R920, R87 to R921, R74 to R922, R75 to R923, R88 to R924, R89 to R925, R77 to R926, R90 to R927, R91 to R928, R92 to R929, R93 to R930, U35 to U902, U36 to U904, U38 to U907, U37 to U908, U40 to U909, U41 to U910, U39 to U911, U42 to U912
Connections:
- net +3.3V: now also R901.1, U901.1 (~{MR}), U901.10 (CET), U901.16 (VCC), U901.7 (CEP), U903.5 (VCC), U905.1 (~{MR}), U905.16 (VCC), U905.3 (P0), U905.6 (P3), U905.7 (CEP), U906.5 (VCC), X901.4 (VDD)
- net GND: now also U901.3 (P0), U901.8 (GND), U903.3 (GND), U905.8 (GND), U906.3 (GND), X901.2 (GND)
- net MCLK: now reaches U902.8 (MCLK)
- net MCLK: now also R909.1
- new net: U903.2, U905.15 (TC), U906.1 (D)
- new net: R902.1, U901.2 (CP), U905.2 (CP), U906.2 (C)
- new net: R909.2, U906.4 (Q)
- new net: U901.9 (~{PE}), U903.4, U905.9 (~{PE})
- new net: U901.15 (TC), U905.10 (CET)
- new net: R901.2, X901.1 (EN)
- new net: R902.2, X901.3 (OUT)
- new net DDS_DIV2: U901.4 (P1)
- new net DDS_DIV4: U901.5 (P2)
- new net DDS_DIV8: U901.6 (P3)
- new net ~{DDS_DIV10}: U905.4 (P1), U905.5 (P2)
- no-connect marks 3 -> 11
Other:
- moved on the sheet: C926, R922, R923, R926, U908, U911
