File: HARDWARE/ETH1CSMU2/Source.kicad_sch (KiCad schematic)
At the start: 75 parts, among them Q901 FDV301N, U901 MC74AC161DR2G, U902 AD9834BRUZ, U903 SN74AHC1G14DBVT, U904 DAC8565ICPW, U905 MC74AC161DR2G, U906 SN74AUP1G79DCKR, U907 LM7171BIM, U908 AD5322ARMZ, U909 LT1790BCS6-2.5, U910 DG409DY+, U911 TL071CDR, U912 LM7171BIM, X901 830208220601

Commit message: Hardware design
Parts:
- R904: value 5k6 -> 7k5
Other:
- note added: "DAC"
- note added: "FGEN"
- moved on the sheet: C909, C912, C914, C915, C917, C919, C922, C923, C924, C926, C927, L901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

Commit message: Hardware and software development
Parts:
- renumbered C913 to C912, C912 to C913, C916 to C915, C915 to C916, C920 to C919, C919 to C920, R927 to R926, R926 to R927
Changed lines of the file:
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@@
   (symbol (lib_id "74xGxx:74AUP1G79") (at 172.72 201.93 0) (unit 1)
     (in_bom yes) (on_board yes)
-    (property "Reference" "U906" (id 0) (at 189.23 194.31 0))
-    (property "Value" "SN74AUP1G79DCKR" (id 1) (at 189.23 196.85 0))
+    (property "Reference" "U906" (id 0) (at 185.42 203.2 0))
+    (property "Value" "SN74AUP1G79DCKR" (id 1) (at 186.69 205.74 0))
     (property "Footprint" "Package_TO_SOT_SMD:SOT-353_SC-70-5_Handsoldering" (id 2) (at 172.72 201.93 0)
       (effects (font (size 1.27 1.27)) hide)
@@
   (symbol (lib_id "Device:C") (at 180.34 267.97 0) (unit 1)
     (in_bom yes) (on_board yes) (fields_autoplaced)
-    (property "Reference" "C920" (id 0) (at 184.15 266.6999 0)
+    (property "Reference" "C919" (id 0) (at 184.15 266.6999 0)
       (effects (font (size 1.27 1.27)) (justify left))
     )
@@
   (symbol (lib_id "power:+3.3V") (at 132.08 222.25 90) (unit 1)
     (in_bom yes) (on_board yes)
-    (property "Reference" "#PWR0926" (id 0) (at 135.89 222.25 0)
+    (property "Reference" "#PWR0927" (id 0) (at 135.89 222.25 0)
       (effects (font (size 1.27 1.27)) hide)
     )
@@
   (symbol (lib_id "Device:R") (at 325.12 226.06 90) (unit 1)
     (in_bom yes) (on_board yes)
-    (property "Reference" "R926" (id 0) (at 325.12 220.98 90))
+    (property "Reference" "R927" (id 0) (at 325.12 220.98 90))
     (property "Value" "100k" (id 1) (at 325.12 223.52 90))
     (property "Footprint" "Resistor_SMD:R_0603_1608Metric_Pad0.98x0.95mm_HandSolder" (id 2) (at 325.12 227.838 90)
@@
   (symbol (lib_id "Device:C") (at 181.61 144.78 0) (unit 1)
     (in_bom yes) (on_board yes)
-    (property "Reference" "C919" (id 0) (at 184.531 143.6116 0)
+    (property "Reference" "C920" (id 0) (at 184.531 143.6116 0)
       (effects (font (size 1.27 1.27)) (justify left))
     )
@@
   (symbol (lib_id "Device:C") (at 153.67 123.19 0) (unit 1)
     (in_bom yes) (on_board yes) (fields_autoplaced)
-    (property "Reference" "C915" (id 0) (at 157.48 121.9199 0)
+    (property "Reference" "C916" (id 0) (at 157.48 121.9199 0)
       (effects (font (size 1.27 1.27)) (justify left))
     )
@@
   (symbol (lib_id "power:GND") (at 132.08 67.31 0) (unit 1)
     (in_bom yes) (on_board yes) (fields_autoplaced)
-    (property "Reference" "#PWR0927" (id 0) (at 132.08 73.66 0)
+    (property "Reference" "#PWR0924" (id 0) (at 132.08 73.66 0)
       (effects (font (size 1.27 1.27)) hide)
     )
@@
   (symbol (lib_id "power:+3.3V") (at 132.08 214.63 90) (unit 1)
     (in_bom yes) (on_board yes)
-    (property "Reference" "#PWR0925" (id 0) (at 135.89 214.63 0)
+    (property "Reference" "#PWR0926" (id 0) (at 135.89 214.63 0)
       (effects (font (size 1.27 1.27)) hide)
     )
@@
   (symbol (lib_id "Device:C") (at 139.7 123.19 0) (unit 1)
     (in_bom yes) (on_board yes) (fields_autoplaced)
-    (property "Reference" "C912" (id 0) (at 143.51 121.9199 0)
+    (property "Reference" "C913" (id 0) (at 143.51 121.9199 0)
       (effects (font (size 1.27 1.27)) (justify left))
     )
@@
   (symbol (lib_id "Device:R") (at 325.12 50.8 180) (unit 1)
     (in_bom yes) (on_board yes) (fields_autoplaced)
-    (property "Reference" "R927" (id 0) (at 326.898 49.9653 0)
+    (property "Reference" "R926" (id 0) (at 326.898 49.9653 0)
       (effects (font (size 1.27 1.27)) (justify right))
     )
@@
   (symbol (lib_id "Device:C") (at 152.4 267.97 0) (unit 1)
     (in_bom yes) (on_board yes) (fields_autoplaced)
-    (property "Reference" "C916" (id 0) (at 156.21 266.6999 0)
+    (property "Reference" "C915" (id 0) (at 156.21 266.6999 0)
       (effects (font (size 1.27 1.27)) (justify left))
     )
@@
   (symbol (lib_id "power:+3.3V") (at 132.08 205.74 90) (unit 1)
     (in_bom yes) (on_board yes)
-    (property "Reference" "#PWR0924" (id 0) (at 135.89 205.74 0)
+    (property "Reference" "#PWR0925" (id 0) (at 135.89 205.74 0)
       (effects (font (size 1.27 1.27)) hide)
     )
@@
   (symbol (lib_id "Device:C") (at 138.43 267.97 0) (unit 1)
     (in_bom yes) (on_board yes) (fields_autoplaced)
-    (property "Reference" "C913" (id 0) (at 142.24 266.6999 0)
-      (effects (font (size 1.27 1.27)) (justify left))
-    )
+    (property "Reference" "C912" (id 0) (at 142.24 266.6999 0)
+      (effects (font (size 1.27 1.27)) (justify left))
+    )

Commit message: CRC check
Parts:
- U901, U905: symbol ETH1CLCR2:74AC161 -> ETH1CSMU2:74AC161
- U910: symbol ETH1CLCR2:DG409 -> ETH1CSMU2:DG409
- X901: symbol ETH1CLCR2:IQXO-791 -> ETH1CSMU2:IQXO-791
Connections:
- net -5VA is gone; now on net -15V: U910.3 (V-)
- net +15V: now also U910.14 (V+)
- net +5V: now also R914.1, U910.2 (EN)
- net +2V5 renamed SOUR_2V5
- removed net +5VA: R914.1, U910.14 (V+), U910.2 (EN)

Commit message: Hardware design
Parts:
- C923: value 4u7 -> 4u7/OPT
- R905, R906: value 200 -> 200/.1%
- R912: value DNP -> 0
Other:
- moved on the sheet: L903, L904, R905
Changed lines of the file:
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@@
   (junction (at 317.5 236.22) (diameter 0) (color 0 0 0 0)
   )
-  (junction (at 186.69 149.86) (diameter 0) (color 0 0 0 0)
+  (junction (at 182.88 149.86) (diameter 0) (color 0 0 0 0)
   )
   (junction (at 180.34 262.89) (diameter 0) (color 0 0 0 0)
@@
   (junction (at 334.01 226.06) (diameter 0) (color 0 0 0 0)
   )
-  (junction (at 190.5 161.29) (diameter 0) (color 0 0 0 0)
+  (junction (at 189.23 161.29) (diameter 0) (color 0 0 0 0)
   )
   (junction (at 118.11 58.42) (diameter 0) (color 0 0 0 0)
@@
     (stroke (width 0) (type default) (color 0 0 0 0))
   )
-  (wire (pts (xy 186.69 149.86) (xy 186.69 152.4))
+  (wire (pts (xy 182.88 149.86) (xy 182.88 152.4))
     (stroke (width 0) (type default) (color 0 0 0 0))
   )
@@
     (stroke (width 0) (type default) (color 0 0 0 0))
   )
-  (wire (pts (xy 179.07 149.86) (xy 181.61 149.86))
+  (wire (pts (xy 176.53 149.86) (xy 181.61 149.86))
     (stroke (width 0) (type default) (color 0 0 0 0))
   )
@@
     (stroke (width 0) (type default) (color 0 0 0 0))
   )
-  (wire (pts (xy 179.07 139.7) (xy 181.61 139.7))
+  (wire (pts (xy 176.53 139.7) (xy 181.61 139.7))
     (stroke (width 0) (type default) (color 0 0 0 0))
   )
@@
     (stroke (width 0) (type default) (color 0 0 0 0))
   )
-  (wire (pts (xy 186.69 160.02) (xy 186.69 161.29))
+  (wire (pts (xy 182.88 160.02) (xy 182.88 161.29))
     (stroke (width 0) (type default) (color 0 0 0 0))
   )
@@
     (stroke (width 0) (type default) (color 0 0 0 0))
   )
-  (wire (pts (xy 181.61 149.86) (xy 186.69 149.86))
+  (wire (pts (xy 181.61 149.86) (xy 182.88 149.86))
     (stroke (width 0) (type default) (color 0 0 0 0))
   )
@@
     (stroke (width 0) (type default) (color 0 0 0 0))
   )
-  (wire (pts (xy 190.5 161.29) (xy 190.5 162.56))
+  (wire (pts (xy 189.23 161.29) (xy 189.23 162.56))
     (stroke (width 0) (type default) (color 0 0 0 0))
   )
@@
     (stroke (width 0) (type default) (color 0 0 0 0))
   )
-  (wire (pts (xy 186.69 149.86) (xy 196.85 149.86))
+  (wire (pts (xy 182.88 149.86) (xy 196.85 149.86))
     (stroke (width 0) (type default) (color 0 0 0 0))
   )
@@
     (stroke (width 0) (type default) (color 0 0 0 0))
   )
-  (wire (pts (xy 186.69 161.29) (xy 190.5 161.29))
+  (wire (pts (xy 182.88 161.29) (xy 189.23 161.29))
     (stroke (width 0) (type default) (color 0 0 0 0))
   )
@@
     (stroke (width 0) (type default) (color 0 0 0 0))
   )
-  (wire (pts (xy 190.5 161.29) (xy 195.58 161.29))
+  (wire (pts (xy 189.23 161.29) (xy 195.58 161.29))
     (stroke (width 0) (type default) (color 0 0 0 0))
   )
@@
     (stroke (width 0) (type default) (color 0 0 0 0))
   )
-  (wire (pts (xy 163.83 139.7) (xy 171.45 139.7))
+  (wire (pts (xy 163.83 139.7) (xy 168.91 139.7))
     (stroke (width 0) (type default) (color 0 0 0 0))
   )
@@
     (stroke (width 0) (type default) (color 0 0 0 0))
   )
-  (wire (pts (xy 171.45 149.86) (xy 163.83 149.86))
+  (wire (pts (xy 168.91 149.86) (xy 163.83 149.86))
     (stroke (width 0) (type default) (color 0 0 0 0))
   )
@@
     (pin "1")
   )
-  (symbol (lib_id "power:GND") (at 190.5 162.56 0) (unit 1)
+  (symbol (lib_id "power:GND") (at 189.23 162.56 0) (unit 1)
     (in_bom yes) (on_board yes) (fields_autoplaced)
-    (property "Reference" "#PWR0938" (id 0) (at 190.5 168.91 0)
+    (property "Reference" "#PWR0938" (id 0) (at 189.23 168.91 0)
       (effects (font (size 1.27 1.27)) hide)
     )
-    (property "Value" "GND" (id 1) (at 190.5 167.64 0))
-    (property "Footprint" "" (id 2) (at 190.5 162.56 0)
+    (property "Value" "GND" (id 1) (at 189.23 167.64 0))
+    (property "Footprint" "" (id 2) (at 189.23 162.56 0)
       (effects (font (size 1.27 1.27)) hide)
     )
-    (property "Datasheet" "" (id 3) (at 190.5 162.56 0)
+    (property "Datasheet" "" (id 3) (at 189.23 162.56 0)
       (effects (font (size 1.27 1.27)) hide)
     )
@@
     (in_bom yes) (on_board yes)
     (property "Reference" "C923" (id 0) (at 247.65 138.43 90))
-    (property "Value" "4u7" (id 1) (at 247.65 140.97 90))
+    (property "Value" "4u7/OPT" (id 1) (at 247.65 140.97 90))
     (property "Footprint" "Capacitor_SMD:C_0805_2012Metric_Pad1.18x1.45mm_HandSolder" (id 2) (at 251.46 143.8148 0)
       (effects (font (size 1.27 1.27)) hide)
@@
     (pin "2")
   )
-  (symbol (lib_id "Device:L") (at 175.26 149.86 90) (unit 1)
+  (symbol (lib_id "Device:L") (at 172.72 149.86 90) (unit 1)
     (in_bom yes) (on_board yes)
-    (property "Reference" "L904" (id 0) (at 175.26 152.4 90))
-    (property "Value" "CBMF1608T100K" (id 1) (at 175.26 154.94 90))
-    (property "Footprint" "Inductor_SMD:L_0603_1608Metric_Pad1.05x0.95mm_HandSolder" (id 2) (at 175.26 149.86 0)
+    (property "Reference" "L904" (id 0) (at 172.72 152.4 90))
+    (property "Value" "CBMF1608T100K" (id 1) (at 172.72 154.94 90))
+    (property "Footprint" "Inductor_SMD:L_0603_1608Metric_Pad1.05x0.95mm_HandSolder" (id 2) (at 172.72 149.86 0)
       (effects (font (size 1.27 1.27)) hide)
     )
-    (property "Datasheet" "~" (id 3) (at 175.26 149.86 0)
+    (property "Datasheet" "~" (id 3) (at 172.72 149.86 0)
       (effects (font (size 1.27 1.27)) hide)
     )
@@
     (pin "1")
   )
-  (symbol (lib_id "Device:L") (at 175.26 139.7 90) (unit 1)
+  (symbol (lib_id "Device:L") (at 172.72 139.7 90) (unit 1)
     (in_bom yes) (on_board yes)
-    (property "Reference" "L903" (id 0) (at 175.26 134.874 90))
-    (property "Value" "CBMF1608T100K" (id 1) (at 175.26 137.1854 90))
-    (property "Footprint" "Inductor_SMD:L_0603_1608Metric_Pad1.05x0.95mm_HandSolder" (id 2) (at 175.26 139.7 0)
+    (property "Reference" "L903" (id 0) (at 172.72 134.874 90))
+    (property "Value" "CBMF1608T100K" (id 1) (at 172.72 137.1854 90))
+    (property "Footprint" "Inductor_SMD:L_0603_1608Metric_Pad1.05x0.95mm_HandSolder" (id 2) (at 172.72 139.7 0)
       (effects (font (size 1.27 1.27)) hide)
     )
-    (property "Datasheet" "~" (id 3) (at 175.26 139.7 0)
+    (property "Datasheet" "~" (id 3) (at 172.72 139.7 0)
       (effects (font (size 1.27 1.27)) hide)
     )
@@
       (effects (font (size 1.27 1.27)) (justify left))
     )
-    (property "Value" "200" (id 1) (at 197.358 157.9122 0)
+    (property "Value" "200/.1%" (id 1) (at 197.358 157.9122 0)
       (effects (font (size 1.27 1.27)) (justify left))
     )
@@
     (in_bom yes) (on_board yes)
     (property "Reference" "R912" (id 0) (at 247.65 130.81 90))
-    (property "Value" "DNP" (id 1) (at 247.65 133.35 90))
+    (property "Value" "0" (id 1) (at 247.65 133.35 90))
     (property "Footprint" "Resistor_SMD:R_0603_1608Metric_Pad0.98x0.95mm_HandSolder" (id 2) (at 247.65 137.668 90)
       (effects (font (size 1.27 1.27)) hide)
@@
     (pin "1")
   )
-  (symbol (lib_id "Device:R") (at 186.69 156.21 0) (unit 1)
+  (symbol (lib_id "Device:R") (at 182.88 156.21 0) (unit 1)
     (in_bom yes) (on_board yes) (fields_autoplaced)
-    (property "Reference" "R905" (id 0) (at 188.468 155.3753 0)
+    (property "Reference" "R905" (id 0) (at 184.658 155.3753 0)
       (effects (font (size 1.27 1.27)) (justify left))
     )
-    (property "Value" "200" (id 1) (at 188.468 157.9122 0)
+    (property "Value" "200/.1%" (id 1) (at 184.658 157.9122 0)
       (effects (font (size 1.27 1.27)) (justify left))
     )
-    (property "Footprint" "Resistor_SMD:R_0603_1608Metric_Pad0.98x0.95mm_HandSolder" (id 2) (at 184.912 156.21 90)
+    (property "Footprint" "Resistor_SMD:R_0603_1608Metric_Pad0.98x0.95mm_HandSolder" (id 2) (at 181.102 156.21 90)
       (effects (font (size 1.27 1.27)) hide)
     )
-    (property "Datasheet" "~" (id 3) (at 186.69 156.21 0)
+    (property "Datasheet" "~" (id 3) (at 182.88 156.21 0)
       (effects (font (size 1.27 1.27)) hide)
     )

Commit message: Hardware design
Parts:
- added C905, C906, C921, C922, C928, C929: 100n, Capacitor_SMD:C_0603_1608Metric_Pad1.08x0.95mm_HandSolder, symbol Device:C
- added R905, R906: 4k7, Resistor_SMD:R_0603_1608Metric_Pad0.98x0.95mm_HandSolder, symbol Device:R
- added R912, R914: 1k, Resistor_SMD:R_0603_1608Metric_Pad0.98x0.95mm_HandSolder, symbol Device:R
- added R916: 1Meg, Resistor_SMD:R_0603_1608Metric_Pad0.98x0.95mm_HandSolder, symbol Device:R
- added R917: 10k, Resistor_SMD:R_0603_1608Metric_Pad0.98x0.95mm_HandSolder, symbol Device:R
- added U906: MAX6102EUR, Package_TO_SOT_SMD:SOT-23, symbol Reference_Voltage:MAX6102
- added U908: MAX5217GUA+, Package_SO:MSOP-8_3x3mm_P0.65mm, symbol Analog_DAC:MAX5217
- added U909: OPA2141AID, Package_SO:SOIC-8_3.9x4.9mm_P1.27mm, symbol ETH1CSMU2:OPA2140
- added U911: OPA141AID, Package_SO:SOIC-8_3.9x4.9mm_P1.27mm, symbol ETH1CSMU2:OPA140
- renumbered C907 to C902, C902 to C903, C903 to C904, C904 to C907, C905 to C908, C906 to C909, C909 to C910, C908 to C911, C910 to C912, C911 to C915, C912 to C918, C915 to C919, C918 to C923, C922 to C924, C919 to C925, C921 to C926, C923 to C927, C924 to C930, C926 to C931, C927 to C932, C925 to C933, R903 to R902, R902 to R903, R905 to R907, R906 to R908, R907 to R909, R908 to R910, R909 to R911, R910 to R913, R911 to R915, R912 to R918, R913 to R919, R914 to R920, R915 to R921, R916 to R922, R917 to R923, R918 to R924, R919 to R925, R920 to R926, R921 to R927, R922 to R928, R923 to R929, R924 to R930, R927 to R931, R928 to R932, R929 to R933, R930 to R934, R925 to R935, R926 to R936, U904 to U901, U901 to U902, U902 to U903, U903 to U904, U906 to U907, U907 to U910, U908 to U912, U910 to U913, U911 to U914, U909 to U915, U912 to U916
Connections:
- net +15V: now also C921.1, C922.1, U909.8 (V+), U911.7 (V+)
- net +3.3V: now also C906.1, R905.1, R906.1, U908.5 (~{AUX}), U908.7 (VDD)
- net +5V: now also C905.1, U906.1 (IN)
- net -15V: now also C928.1, C929.1, U909.4 (V-), U911.4 (V-)
- net GND: now also C905.2, C906.2, C921.2, C922.2, C928.2, C929.2, R917.2, U906.3 (GND), U908.2 (ADDR), U908.8 (GND)
- new net: R912.2, R914.1, U909.6 (-)
- new net: R914.2, R916.1, U909.7
- new net: R912.1, U909.1, U909.2 (-)
- new net: U906.2 (OUT), U908.1 (REF), U909.3 (+)
- new net: R916.2, R917.1, U911.3 (+)
- new net: U908.6 (OUT), U909.5 (+)
- new net DAC_OFFS_SCL: R905.2, U908.3 (SCL)
- new net DAC_OFFS_SDA: R906.2, U908.4 (SDA)
- new net VOUT_OFFSET: U911.2 (-), U911.6
Other:
- note added: "OFFSET DAC"
- moved on the sheet: C902, C907, C908, C909, C911, C912, C915, C918, C919, C923, C925, C926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

Commit message: PCB layout
Parts:
- added R930: 300, Resistor_SMD:R_0603_1608Metric_Pad0.98x0.95mm_HandSolder, symbol Device:R
- R928: renamed from R929; value 26k4 -> 26k1
- renumbered R928 to R929, R930 to R931, R931 to R932, R932 to R933, R933 to R934, R934 to R935, R935 to R936, R936 to R937
Connections:
- net at C931.1, R929.2, R932.1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: now also R930.2; no longer R928.2
- new net: R928.2, R930.1
Other:
- moved on the sheet: R928
Changed lines of the file:
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@@
     (stroke (width 0) (type default) (color 0 0 0 0))
   )
+  (wire (pts (xy 316.23 236.22) (xy 317.5 236.22))
+    (stroke (width 0) (type default) (color 0 0 0 0))
+  )
   (wire (pts (xy 109.22 262.89) (xy 109.22 264.16))
     (stroke (width 0) (type default) (color 0 0 0 0))
@@
     (stroke (width 0) (type default) (color 0 0 0 0))
   )
-  (wire (pts (xy 316.23 236.22) (xy 317.5 236.22))
+  (wire (pts (xy 307.34 236.22) (xy 308.61 236.22))
     (stroke (width 0) (type default) (color 0 0 0 0))
   )
@@
     (stroke (width 0) (type default) (color 0 0 0 0))
   )
-  (wire (pts (xy 307.34 236.22) (xy 308.61 236.22))
+  (wire (pts (xy 298.45 236.22) (xy 299.72 236.22))
     (stroke (width 0) (type default) (color 0 0 0 0))
   )
@@
   (symbol (lib_id "ETH1CSMU2:+1V25") (at 299.72 207.01 270) (unit 1)
     (in_bom yes) (on_board yes) (fields_autoplaced)
-    (property "Reference" "#PWR0959" (id 0) (at 295.91 207.01 0)
+    (property "Reference" "#PWR0960" (id 0) (at 295.91 207.01 0)
       (effects (font (size 1.27 1.27)) hide)
     )
@@
     (pin "2")
   )
-  (symbol (lib_id "power:GND") (at 307.34 236.22 270) (unit 1)
+  (symbol (lib_id "power:GND") (at 298.45 236.22 270) (unit 1)
     (in_bom yes) (on_board yes) (fields_autoplaced)
-    (property "Reference" "#PWR0961" (id 0) (at 300.99 236.22 0)
+    (property "Reference" "#PWR0959" (id 0) (at 292.1 236.22 0)
       (effects (font (size 1.27 1.27)) hide)
     )
-    (property "Value" "GND" (id 1) (at 303.53 236.2199 90)
+    (property "Value" "GND" (id 1) (at 294.64 236.2199 90)
       (effects (font (size 1.27 1.27)) (justify right))
     )
-    (property "Footprint" "" (id 2) (at 307.34 236.22 0)
+    (property "Footprint" "" (id 2) (at 298.45 236.22 0)
       (effects (font (size 1.27 1.27)) hide)
     )
-    (property "Datasheet" "" (id 3) (at 307.34 236.22 0)
+    (property "Datasheet" "" (id 3) (at 298.45 236.22 0)
       (effects (font (size 1.27 1.27)) hide)
     )
@@
   (symbol (lib_id "Device:R") (at 325.12 226.06 90) (unit 1)
     (in_bom yes) (on_board yes)
-    (property "Reference" "R931" (id 0) (at 325.12 220.98 90))
+    (property "Reference" "R932" (id 0) (at 325.12 220.98 90))
     (property "Value" "100k" (id 1) (at 325.12 223.52 90))
     (property "Footprint" "Resistor_SMD:R_0603_1608Metric_Pad0.98x0.95mm_HandSolder" (id 2) (at 325.12 227.838 90)
@@
   (symbol (lib_id "Device:R") (at 340.36 157.48 90) (unit 1)
     (in_bom yes) (on_board yes)
-    (property "Reference" "R933" (id 0) (at 340.36 152.4 90))
+    (property "Reference" "R934" (id 0) (at 340.36 152.4 90))
     (property "Value" "1k/.1%" (id 1) (at 340.36 154.94 90))
     (property "Footprint" "Resistor_SMD:R_0603_1608Metric_Pad0.98x0.95mm_HandSolder" (id 2) (at 340.36 159.258 90)
@@
     (pin "1")
   )
-  (symbol (lib_id "Device:R") (at 312.42 236.22 90) (unit 1)
+  (symbol (lib_id "Device:R") (at 303.53 236.22 90) (unit 1)
     (in_bom yes) (on_board yes)
-    (property "Reference" "R929" (id 0) (at 312.42 231.14 90))
-    (property "Value" "26k4" (id 1) (at 312.42 233.68 90))
-    (property "Footprint" "Resistor_SMD:R_0603_1608Metric_Pad0.98x0.95mm_HandSolder" (id 2) (at 312.42 237.998 90)
+    (property "Reference" "R928" (id 0) (at 303.53 231.14 90))
+    (property "Value" "26k1" (id 1) (at 303.53 233.68 90))
+    (property "Footprint" "Resistor_SMD:R_0603_1608Metric_Pad0.98x0.95mm_HandSolder" (id 2) (at 303.53 237.998 90)
       (effects (font (size 1.27 1.27)) hide)
     )
-    (property "Datasheet" "~" (id 3) (at 312.42 236.22 0)
+    (property "Datasheet" "~" (id 3) (at 303.53 236.22 0)
       (effects (font (size 1.27 1.27)) hide)
     )
@@
     (pin "9")
   )
+  (symbol (lib_id "Device:R") (at 312.42 236.22 90) (unit 1)
+    (in_bom yes) (on_board yes)
+    (property "Reference" "R930" (id 0) (at 312.42 231.14 90))
+    (property "Value" "300" (id 1) (at 312.42 233.68 90))
+    (property "Footprint" "Resistor_SMD:R_0603_1608Metric_Pad0.98x0.95mm_HandSolder" (id 2) (at 312.42 237.998 90)
+      (effects (font (size 1.27 1.27)) hide)
+    )
+    (property "Datasheet" "~" (id 3) (at 312.42 236.22 0)
+      (effects (font (size 1.27 1.27)) hide)
+    )
+    (pin "1")
+    (pin "2")
+  )
   (symbol (lib_id "ETH1CSMU2:OPA2140") (at 284.48 267.97 0) (unit 3)
     (in_bom yes) (on_board yes) (fields_autoplaced)
@@
   (symbol (lib_id "Device:R") (at 354.33 157.48 90) (unit 1)
     (in_bom yes) (on_board yes)
-    (property "Reference" "R934" (id 0) (at 354.33 152.4 90))
+    (property "Reference" "R935" (id 0) (at 354.33 152.4 90))
     (property "Value" "1k/.1%" (id 1) (at 354.33 154.94 90))
     (property "Footprint" "Resistor_SMD:R_0603_1608Metric_Pad0.98x0.95mm_HandSolder" (id 2) (at 354.33 159.258 90)
@@
   (symbol (lib_id "Device:R") (at 312.42 226.06 90) (unit 1)
     (in_bom yes) (on_board yes)
-    (property "Reference" "R928" (id 0) (at 312.42 220.98 90))
+    (property "Reference" "R929" (id 0) (at 312.42 220.98 90))
     (property "Value" "20k8" (id 1) (at 312.42 223.52 90))
     (property "Footprint" "Resistor_SMD:R_0603_1608Metric_Pad0.98x0.95mm_HandSolder" (id 2) (at 312.42 227.838 90)
@@
   (symbol (lib_id "Device:R") (at 317.5 153.67 0) (unit 1)
     (in_bom yes) (on_board yes)
-    (property "Reference" "R930" (id 0) (at 319.278 152.5016 0)
+    (property "Reference" "R931" (id 0) (at 319.278 152.5016 0)
       (effects (font (size 1.27 1.27)) (justify left))
     )
@@
   (symbol (lib_id "Device:R") (at 378.46 53.34 180) (unit 1)
     (in_bom yes) (on_board yes) (fields_autoplaced)
-    (property "Reference" "R936" (id 0) (at 380.238 52.5053 0)
+    (property "Reference" "R937" (id 0) (at 380.238 52.5053 0)
       (effects (font (size 1.27 1.27)) (justify right))
     )
@@
   (symbol (lib_id "Device:R") (at 372.11 48.26 90) (unit 1)
     (in_bom yes) (on_board yes) (fields_autoplaced)
-    (property "Reference" "R935" (id 0) (at 372.11 43.5442 90))
+    (property "Reference" "R936" (id 0) (at 372.11 43.5442 90))
     (property "Value" "10k" (id 1) (at 372.11 46.0811 90))
     (property "Footprint" "Resistor_SMD:R_0603_1608Metric_Pad0.98x0.95mm_HandSolder" (id 2) (at 372.11 50.038 90)
@@
   (symbol (lib_id "Device:R") (at 340.36 146.05 90) (unit 1)
     (in_bom yes) (on_board yes)
-    (property "Reference" "R932" (id 0) (at 340.36 140.97 90))
+    (property "Reference" "R933" (id 0) (at 340.36 140.97 90))
     (property "Value" "1k/.1%" (id 1) (at 340.36 143.51 90))
     (property "Footprint" "Resistor_SMD:R_0603_1608Metric_Pad0.98x0.95mm_HandSolder" (id 2) (at 340.36 147.828 90)
@@
   (symbol (lib_id "power:GND") (at 303.53 158.75 0) (unit 1)
     (in_bom yes) (on_board yes)
-    (property "Reference" "#PWR0960" (id 0) (at 303.53 165.1 0)
+    (property "Reference" "#PWR0961" (id 0) (at 303.53 165.1 0)
       (effects (font (size 1.27 1.27)) hide)
     )
