File: HARDWARE/ETH1CSMU2/Power.kicad_sch (KiCad schematic)
At the start: 40 parts, among them Q801 IRFR5410, U801 MAX5902, U802 TMR 4-2411WI, U803 TEL 12-2423, U804 NCV1117DT33T5G

Commit message: Hardware design
Parts:
- renumbered C801 to C60, C802 to C61, C803 to C62, C804 to C63, C805 to C64, C806 to C65, C807 to C66, C808 to C67, C809 to C68, C810 to C69, C811 to C70, C812 to C71, C813 to C72, C814 to C73, C815 to C74, C816 to C75, C817 to C76, C818 to C77, C819 to C78, C820 to C79, C821 to C80, C822 to C81, C823 to C82, C824 to C83, C825 to C84, C826 to C85, C827 to C86, D802 to D10, D803 to D11, D801 to D9, F801 to F1, L801 to L3, L802 to L4, Q801 to Q1, R801 to R64, R802 to R65, U801 to U29, U802 to U30, U803 to U31, U804 to U32

Commit message: Hardware design
Parts:
- renumbered R64 to R65, R65 to R66, U29 to U31, U30 to U32, U31 to U33, U32 to U34
Changed lines of the file:
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@@
   (symbol (lib_id "power:+5V") (at 137.16 72.39 0) (unit 1)
     (in_bom yes) (on_board yes) (fields_autoplaced)
-    (property "Reference" "#PWR0174" (id 0) (at 137.16 76.2 0)
+    (property "Reference" "#PWR0187" (id 0) (at 137.16 76.2 0)
       (effects (font (size 1.27 1.27)) hide)
     )
@@
   (symbol (lib_id "power:VPP") (at 50.8 72.39 0) (unit 1)
     (in_bom yes) (on_board yes) (fields_autoplaced)
-    (property "Reference" "#PWR0171" (id 0) (at 50.8 76.2 0)
+    (property "Reference" "#PWR0184" (id 0) (at 50.8 76.2 0)
       (effects (font (size 1.27 1.27)) hide)
     )
@@
   (symbol (lib_id "Regulator_Linear:LM1117-3.3") (at 180.34 73.66 0) (unit 1)
     (in_bom yes) (on_board yes) (fields_autoplaced)
-    (property "Reference" "U32" (id 0) (at 180.34 68.0552 0))
+    (property "Reference" "U34" (id 0) (at 180.34 68.0552 0))
     (property "Value" "NCV1117DT33T5G" (id 1) (at 180.34 70.5921 0))
     (property "Footprint" "" (id 2) (at 180.34 73.66 0)
@@
   (symbol (lib_id "Device:R") (at 45.72 31.75 0) (unit 1)
     (in_bom yes) (on_board yes)
-    (property "Reference" "R64" (id 0) (at 47.498 30.5816 0)
+    (property "Reference" "R65" (id 0) (at 47.498 30.5816 0)
       (effects (font (size 1.27 1.27)) (justify left))
     )
@@
   (symbol (lib_id "power:+3.3V") (at 220.98 72.39 0) (unit 1)
     (in_bom yes) (on_board yes)
-    (property "Reference" "#PWR0178" (id 0) (at 220.98 76.2 0)
+    (property "Reference" "#PWR0191" (id 0) (at 220.98 76.2 0)
       (effects (font (size 1.27 1.27)) hide)
     )
@@
   (symbol (lib_id "power:VPP") (at 130.81 22.86 0) (unit 1)
     (in_bom yes) (on_board yes) (fields_autoplaced)
-    (property "Reference" "#PWR0173" (id 0) (at 130.81 26.67 0)
+    (property "Reference" "#PWR0186" (id 0) (at 130.81 26.67 0)
       (effects (font (size 1.27 1.27)) hide)
     )
@@
   (symbol (lib_id "power:VPP") (at 46.99 120.65 0) (unit 1)
     (in_bom yes) (on_board yes) (fields_autoplaced)
-    (property "Reference" "#PWR0169" (id 0) (at 46.99 124.46 0)
+    (property "Reference" "#PWR0182" (id 0) (at 46.99 124.46 0)
       (effects (font (size 1.27 1.27)) hide)
     )
@@
   (symbol (lib_id "power:+15V") (at 181.61 120.65 0) (unit 1)
     (in_bom yes) (on_board yes) (fields_autoplaced)
-    (property "Reference" "#PWR0175" (id 0) (at 181.61 124.46 0)
+    (property "Reference" "#PWR0188" (id 0) (at 181.61 124.46 0)
       (effects (font (size 1.27 1.27)) hide)
     )
@@
   (symbol (lib_id "ETH1CSMU2:TEL12_Dual") (at 95.25 137.16 0) (unit 1)
     (in_bom yes) (on_board yes)
-    (property "Reference" "U31" (id 0) (at 95.25 115.57 0))
+    (property "Reference" "U33" (id 0) (at 95.25 115.57 0))
     (property "Value" "TEL 12-2423" (id 1) (at 95.25 118.11 0))
     (property "Footprint" "" (id 2) (at 95.25 116.84 0)
@@
   (symbol (lib_id "power:GNDPWR") (at 50.8 86.36 0) (unit 1)
     (in_bom yes) (on_board yes)
-    (property "Reference" "#PWR0172" (id 0) (at 50.8 91.44 0)
+    (property "Reference" "#PWR0185" (id 0) (at 50.8 91.44 0)
       (effects (font (size 1.27 1.27)) hide)
     )
@@
   (symbol (lib_id "power:GND") (at 220.98 85.09 0) (unit 1)
     (in_bom yes) (on_board yes)
-    (property "Reference" "#PWR0179" (id 0) (at 220.98 91.44 0)
+    (property "Reference" "#PWR0192" (id 0) (at 220.98 91.44 0)
       (effects (font (size 1.27 1.27)) hide)
     )
@@
   (symbol (lib_id "Device:R") (at 100.33 36.83 0) (unit 1)
     (in_bom yes) (on_board yes)
-    (property "Reference" "R65" (id 0) (at 102.108 35.6616 0)
+    (property "Reference" "R66" (id 0) (at 102.108 35.6616 0)
       (effects (font (size 1.27 1.27)) (justify left))
     )
@@
   (symbol (lib_id "power:GNDPWR") (at 46.99 156.21 0) (unit 1)
     (in_bom yes) (on_board yes)
-    (property "Reference" "#PWR0170" (id 0) (at 46.99 161.29 0)
+    (property "Reference" "#PWR0183" (id 0) (at 46.99 161.29 0)
       (effects (font (size 1.27 1.27)) hide)
     )
@@
   (symbol (lib_id "power:GND") (at 182.88 137.16 90) (unit 1)
     (in_bom yes) (on_board yes)
-    (property "Reference" "#PWR0177" (id 0) (at 189.23 137.16 0)
+    (property "Reference" "#PWR0190" (id 0) (at 189.23 137.16 0)
       (effects (font (size 1.27 1.27)) hide)
     )
@@
   (symbol (lib_id "power:+24V") (at 17.78 20.32 0) (unit 1)
     (in_bom yes) (on_board yes)
-    (property "Reference" "#PWR0167" (id 0) (at 17.78 24.13 0)
+    (property "Reference" "#PWR0180" (id 0) (at 17.78 24.13 0)
       (effects (font (size 1.27 1.27)) hide)
     )
@@
   (symbol (lib_id "power:GNDPWR") (at 17.78 52.07 0) (unit 1)
     (in_bom yes) (on_board yes)
-    (property "Reference" "#PWR0168" (id 0) (at 17.78 57.15 0)
+    (property "Reference" "#PWR0181" (id 0) (at 17.78 57.15 0)
       (effects (font (size 1.27 1.27)) hide)
     )
@@
   (symbol (lib_id "Converter_DCDC:TMR-2411") (at 95.25 78.74 0) (unit 1)
     (in_bom yes) (on_board yes) (fields_autoplaced)
-    (property "Reference" "U30" (id 0) (at 95.25 67.4202 0))
+    (property "Reference" "U32" (id 0) (at 95.25 67.4202 0))
     (property "Value" "TMR 4-2411WI" (id 1) (at 95.25 69.9571 0))
     (property "Footprint" "" (id 2) (at 95.25 87.63 0)
@@
   (symbol (lib_id "ETH1CLCR2:MAX5902") (at 69.85 36.83 0) (unit 1)
     (in_bom yes) (on_board yes)
-    (property "Reference" "U29" (id 0) (at 69.85 27.559 0))
+    (property "Reference" "U31" (id 0) (at 69.85 27.559 0))
     (property "Value" "MAX5902" (id 1) (at 69.85 29.8704 0))
     (property "Footprint" "Package_TO_SOT_SMD:SOT-23-6_Handsoldering" (id 2) (at 69.85 36.83 0)
@@
   (symbol (lib_id "power:-15V") (at 181.61 153.67 180) (unit 1)
     (in_bom yes) (on_board yes) (fields_autoplaced)
-    (property "Reference" "#PWR0176" (id 0) (at 181.61 156.21 0)
-      (effects (font (size 1.27 1.27)) hide)
-    )
+    (property "Reference" "#PWR0189" (id 0) (at 181.61 156.21 0)
+      (effects (font (size 1.27 1.27)) hide)
+    )

Commit message: Hardware design
Parts:
- renumbered C60 to C801, C61 to C802, C62 to C803, C63 to C804, C64 to C805, C65 to C806, C66 to C807, C67 to C808, C68 to C809, C69 to C810, C70 to C811, C71 to C812, C72 to C813, C73 to C814, C74 to C815, C75 to C816, C76 to C817, C77 to C818, C78 to C819, C79 to C820, C80 to C821, C81 to C822, C82 to C823, C83 to C824, C84 to C825, C85 to C826, C86 to C827, D9 to D801, D10 to D802, D11 to D803, F1 to F801, L3 to L801, L4 to L802, Q1 to Q801, R65 to R801, R66 to R802, U31 to U801, U32 to U802, U33 to U803, U34 to U804

Commit message: Hardware design.
Parts:
- renumbered C821 to C100, C822 to C101, C823 to C102, C824 to C103, C825 to C104, C826 to C105, C827 to C106, C801 to C80, C802 to C81, C803 to C82, C804 to C83, C805 to C84, C806 to C85, C807 to C86, C808 to C87, C809 to C88, C810 to C89, C811 to C90, C812 to C91, C813 to C92, C814 to C93, C815 to C94, C816 to C95, C817 to C96, C818 to C97, C819 to C98, C820 to C99, D802 to D10, D803 to D11, D801 to D9, F801 to F1, L801 to L3, L802 to L4, Q801 to Q1, R801 to R65, R802 to R66, U801 to U31, U802 to U32, U803 to U33, U804 to U34
Other:
- note removed: "TMR 4-2411WI"

Commit message: Hardware design
Parts:
- C80, C82: value 470u/50V -> MAL214699108E3; footprint (none) -> Capacitor_SMD:CP_Elec_18x17.5
- C83, C84, C85, C86: footprint (none) -> Capacitor_SMD:C_1812_4532Metric_Pad1.57x3.40mm_HandSolder
- L3: footprint (none) -> ETH1CSMU2:74477410
- U32: footprint (none) -> ETH1CSMU2:TRM 4-SINGLE
- U33: footprint (none) -> ETH1CSMU2:TEL12-DUAL
- U34: footprint (none) -> Package_TO_SOT_SMD:TO-252-2
Other:
- moved on the sheet: C80, C82, L3

Commit message: Hardware design
Parts:
- removed C80, C82: MAL214699108E3, Capacitor_SMD:CP_Elec_18x17.5, symbol Device:C_Polarized
- removed L3: 74477410, ETH1CSMU2:74477410, symbol Device:L
- removed L4: PM1608S-100M-RC, ETH1CLCR2:PM1608S, symbol Device:L
- added C801, C802: 10u/50V, Capacitor_SMD:C_1206_3216Metric_Pad1.33x1.80mm_HandSolder, symbol Device:C
- added C803, C804, C805: 4u7/50V, Capacitor_SMD:C_1206_3216Metric_Pad1.33x1.80mm_HandSolder, symbol Device:C
- added C807, C808: 220p/2k, Capacitor_SMD:C_1812_4532Metric_Pad1.57x3.40mm_HandSolder, symbol Device:C
- D801: renamed from D9; footprint ETH1CLCR2:DO_214AA_REV -> ETH1CSMU2:DO_214AA_REV
- F801: renamed from F1; footprint ETH1CLCR2:Fuse_SMD2920 -> ETH1CSMU2:Fuse_SMD2920
- Q801: renamed from Q1; footprint ETH1CLCR2:TO-252-2_Rectifier -> ETH1CSMU2:TO-252-2_Rectifier
- U804: renamed from U31; symbol ETH1CLCR2:MAX5902 -> ETH1CSMU2:MAX5902
- renumbered C81 to C806, C83 to C809, C84 to C810, C85 to C811, C86 to C812, C87 to C813, C90 to C814, C91 to C815, C89 to C816, C94 to C817, C95 to C818, C93 to C819, C97 to C820, C98 to C821, C96 to C822, C100 to C823, C101 to C824, C99 to C825, C102 to C826, C103 to C827, C104 to C828, C105 to C829, C106 to C830, C88 to C831, C92 to C832, D10 to D802, D11 to D803, R65 to R801, R66 to R802, U32 to U801, U33 to U802, U34 to U803
Connections:
- net +15V: now also C812.2
- net +5V: now also C808.2
- net -15V: no longer C812.2
- net GND: now also C807.2
- net GNDPWR: now also C811.1, C812.1, U802.1 (-VIN), C801.2, C802.2, C803.2, C804.2, C805.2, C808.1
- net VPP: now also U801.2 (+VIN), C801.1, C802.1, C803.1, C804.1, C805.1, C807.1
Other:
- moved on the sheet: C806, C809, C810, C811, C812, C813, C814, C815, C816, C817, C818, C819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

Commit message: Hardware design
Other:
- moved on the sheet: C801, C802, C803, C804, C805, C806, C807, C808, C809, C810, C811, C812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
