File: HARDWARE/ETH1CSMU2/Power.kicad_sch (KiCad schematic)
At the start: 43 parts, among them Q801 IRFR5410, U801 TMR 4-2411WI, U802 TEL 12-2423, U803 NCV1117DT33T5G, U804 MAX5902

Commit message: CRC check
Changed lines of the file:
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@@
   (junction (at 194.31 25.4) (diameter 0) (color 0 0 0 0)
   )
+  (junction (at 210.82 82.55) (diameter 0) (color 0 0 0 0)
+  )
   (junction (at 101.6 140.97) (diameter 0) (color 0 0 0 0)
   )
@@
   )
   (junction (at 63.5 130.81) (diameter 0) (color 0 0 0 0)
-  )
-  (junction (at 210.82 82.55) (diameter 0) (color 0 0 0 0)
   )
   (no_connect (at 68.58 87.63))
@@
     (stroke (width 0) (type default) (color 0 0 0 0))
   )
-  (wire (pts (xy 223.52 82.55) (xy 210.82 82.55))
+  (wire (pts (xy 196.85 82.55) (xy 210.82 82.55))
     (stroke (width 0) (type default) (color 0 0 0 0))
   )
@@
     (stroke (width 0) (type default) (color 0 0 0 0))
   )
+  (wire (pts (xy 210.82 82.55) (xy 223.52 82.55))
+    (stroke (width 0) (type default) (color 0 0 0 0))
+  )
   (wire (pts (xy 36.83 160.02) (xy 36.83 171.45))
     (stroke (width 0) (type default) (color 0 0 0 0))
@@
     (stroke (width 0) (type default) (color 0 0 0 0))
   )
+  (wire (pts (xy 255.27 24.13) (xy 255.27 25.4))
+    (stroke (width 0) (type default) (color 0 0 0 0))
+  )
   (wire (pts (xy 24.13 95.25) (xy 24.13 92.71))
     (stroke (width 0) (type default) (color 0 0 0 0))
@@
     (stroke (width 0) (type default) (color 0 0 0 0))
   )
-  (wire (pts (xy 210.82 82.55) (xy 196.85 82.55))
-    (stroke (width 0) (type default) (color 0 0 0 0))
-  )
   (wire (pts (xy 99.06 171.45) (xy 104.14 171.45))
     (stroke (width 0) (type default) (color 0 0 0 0))
@@
     (stroke (width 0) (type default) (color 0 0 0 0))
   )
+  (wire (pts (xy 152.4 171.45) (xy 152.4 172.72))
+    (stroke (width 0) (type default) (color 0 0 0 0))
+  )
   (wire (pts (xy 114.3 152.4) (xy 114.3 160.02))
     (stroke (width 0) (type default) (color 0 0 0 0))
@@
   )
   (wire (pts (xy 53.34 160.02) (xy 53.34 171.45))
+    (stroke (width 0) (type default) (color 0 0 0 0))
+  )
+  (wire (pts (xy 152.4 139.7) (xy 152.4 140.97))
     (stroke (width 0) (type default) (color 0 0 0 0))
   )
@@
     (pin "1")
     (pin "2")
+  )
+  (symbol (lib_id "power:PWR_FLAG") (at 152.4 139.7 0) (unit 1)
+    (in_bom yes) (on_board yes) (fields_autoplaced)
+    (property "Reference" "#FLG0801" (id 0) (at 152.4 137.795 0)
+      (effects (font (size 1.27 1.27)) hide)
+    )
+    (property "Value" "PWR_FLAG" (id 1) (at 152.4 136.1242 0))
+    (property "Footprint" "" (id 2) (at 152.4 139.7 0)
+      (effects (font (size 1.27 1.27)) hide)
+    )
+    (property "Datasheet" "~" (id 3) (at 152.4 139.7 0)
+      (effects (font (size 1.27 1.27)) hide)
+    )
+    (pin "1")
   )
   (symbol (lib_id "Regulator_Linear:LM1117-3.3") (at 182.88 82.55 0) (unit 1)
@@
     (pin "2")
   )
+  (symbol (lib_id "power:PWR_FLAG") (at 255.27 24.13 0) (unit 1)
+    (in_bom yes) (on_board yes) (fields_autoplaced)
+    (property "Reference" "#FLG0804" (id 0) (at 255.27 22.225 0)
+      (effects (font (size 1.27 1.27)) hide)
+    )
+    (property "Value" "PWR_FLAG" (id 1) (at 255.27 20.5542 0))
+    (property "Footprint" "" (id 2) (at 255.27 24.13 0)
+      (effects (font (size 1.27 1.27)) hide)
+    )
+    (property "Datasheet" "~" (id 3) (at 255.27 24.13 0)
+      (effects (font (size 1.27 1.27)) hide)
+    )
+    (pin "1")
+  )
   (symbol (lib_id "power:GND") (at 167.64 156.21 90) (unit 1)
     (in_bom yes) (on_board yes)
@@
     (pin "1")
     (pin "2")
+  )
+  (symbol (lib_id "power:PWR_FLAG") (at 152.4 172.72 180) (unit 1)
+    (in_bom yes) (on_board yes) (fields_autoplaced)
+    (property "Reference" "#FLG0802" (id 0) (at 152.4 174.625 0)
+      (effects (font (size 1.27 1.27)) hide)
+    )
+    (property "Value" "PWR_FLAG" (id 1) (at 152.4 177.1634 0))
+    (property "Footprint" "" (id 2) (at 152.4 172.72 0)
+      (effects (font (size 1.27 1.27)) hide)
+    )
+    (property "Datasheet" "~" (id 3) (at 152.4 172.72 0)
+      (effects (font (size 1.27 1.27)) hide)
+    )
+    (pin "1")
   )
   (symbol (lib_id "power:GNDPWR") (at 157.48 53.34 0) (unit 1)
@@
   (symbol (lib_id "power:PWR_FLAG") (at 172.72 53.34 180) (unit 1)
     (in_bom yes) (on_board yes)
-    (property "Reference" "#FLG0801" (id 0) (at 172.72 55.245 0)
-      (effects (font (size 1.27 1.27)) hide)
-    )
+    (property "Reference" "#FLG0803" (id 0) (at 172.72 55.245 0)
+      (effects (font (size 1.27 1.27)) hide)
+    )

Commit message: Hardware design
Parts:
- removed C807, C808: 220p/2k, Capacitor_SMD:C_1812_4532Metric_Pad1.57x3.40mm_HandSolder, symbol Device:C
- removed U801: TMR 4-2411WI, ETH1CSMU2:TRM 4-SINGLE, symbol Converter_DCDC:TMR-2411
- added U802: TSR2-2450, ETH1CSMU2:TSR2, symbol ETH1CSMU2:TSR2
- renumbered C809 to C807, C810 to C808, C811 to C809, C812 to C810, C813 to C811, C816 to C812, C814 to C813, C815 to C814, C819 to C815, C831 to C816, C822 to C819, C832 to C820, C820 to C821, C821 to C822, C825 to C823, C823 to C824, C824 to C825, U804 to U801, U802 to U803, U803 to U804
Connections:
- net GNDPWR is gone; now on net GND: C801.2, C802.2, C803.2, C804.2, C805.2, C806.2, C809.1, C810.1, C816.2, C820.2, D801.2 (A), D803.1 (K), U801.4 (GND), U803.1 (-VIN)
- net +5V: now also U802.3 (VO)
- net GND: now also U802.2 (GND)
- net VPP: now also U802.1 (VI)
- no-connect marks 2 -> 1
Other:
- moved on the sheet: C801, C802, C803, C804, C805, C806, C807, C808, C809, C810, C811, C812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

Commit message: Hardware design
Parts:
- renumbered C803 to C802, C805 to C803, C802 to C804, C804 to C805, C807 to C806, C808 to C807, C809 to C808, C810 to C809, C806 to C810, C813 to C811, C814 to C812, C816 to C813, C811 to C814, C817 to C815, C818 to C816, C820 to C817, C812 to C818, C821 to C819, C822 to C820, C815 to C821, C824 to C822, C825 to C823, C819 to C824, C826 to C825, C827 to C826, C823 to C827, U803 to U802, U802 to U803

Commit message: Hardware design
Parts:
- removed C825, C826, C827: 1u, Capacitor_SMD:C_1206_3216Metric_Pad1.33x1.80mm_HandSolder, symbol Device:C
- C806, C807, C808, C809: footprint Capacitor_SMD:C_1812_4532Metric_Pad1.57x3.40mm_HandSolder -> Capacitor_SMD:C_1206_3216Metric_Pad1.33x1.80mm_HandSolder
- renumbered C828 to C825, C829 to C826, C830 to C827
Connections:
- net GND: now also C811.2, C812.1, C815.2, C816.1, C819.2, C820.1, C822.2, C823.1
Other:
- moved on the sheet: C825, C826, C827, U804
