File: HARDWARE/ETH1CSMU2/Power.kicad_sch (KiCad schematic)
At the start: 38 parts, among them Q801 IRFR5410, U801 MAX5902, U802 TEL 12-2423, U803 TSR2-2450, U804 NCV1117DT33T5G

Commit message: PCB layout
Parts:
- U801: value MAX5902 -> MAX5902ACEUT
Changed lines of the file:
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@@
     (in_bom yes) (on_board yes)
     (property "Reference" "U801" (id 0) (at 73.66 27.559 0))
-    (property "Value" "MAX5902" (id 1) (at 73.66 29.8704 0))
+    (property "Value" "MAX5902ACEUT" (id 1) (at 73.66 29.8704 0))
     (property "Footprint" "Package_TO_SOT_SMD:SOT-23-6_Handsoldering" (id 2) (at 73.66 36.83 0)
       (effects (font (size 1.524 1.524)) hide)

Commit message: PCB layout
Parts:
- removed C813, C817: 4u7/50V, Capacitor_SMD:C_1206_3216Metric_Pad1.33x1.80mm_HandSolder, symbol Device:C
- renumbered C814 to C813, C815 to C814, C816 to C815, C818 to C816, C819 to C817, C820 to C818, C821 to C819, C822 to C820, C823 to C821, C824 to C822, C825 to C823, C826 to C824, C827 to C825
Connections:
- net +3V3 renamed +3.3V
