File: HARDWARE/ETH1CSMU2/ETH1CSMU2.kicad_pcb (KiCad board)
At the start: 2 copper layers, 351 parts, among them J1001 Conn_02x01, J1002 20021111-00010T4LF, J301 C64AC, K301 HE3621A0510, K302 HE3621A0510, K303 HE3621A0510, K304 HE3621A0510, K305 HE3621A0510, Q801 IRFR5410, Q901 FDV301N, U1001 HDC1080, U1002 STM32F746ZG, U1003 24LC08B-E/MS, U201 LAN8742A, U202 LC03-3.3, U203 LC03-3.3, U301 ULN2003AS16, U401 DG444DY+, U402 REF5040ID, U403 DG444DY+, U404 DG419DY, U405 DG419DY, U406 DG419DY, U407 OPA141AID, U408 OPA141AID, U409 ADS8681IRUMT, U410 ADS8681IRUMT, U501 74HCT595PW, U502 74HCT595PW, U503 SN74LVC1T45DRLR, U504 SN74LVC1T45DRLR, U505 SN74LVC1T45DRLR, U506 SN74LVC1T45DRLR, U601 DG419DY, U602 DG419DY, U603 SN74LVC1T45DRLR, U604 SN74LVC1T45DRLR, U605 LT1970ACFE, U606 SN74LVC1T45DRLR, U607 INA823DT, U701 TXB0104PW, U702 ADuM5402, U703 74AC125, U801 TMR 4-2411WI, U802 TEL 12-2423, U803 NCV1117DT33T5G, U804 MAX5902, U901 MC74AC161DR2G, U902 AD9834BRUZ, U903 SN74AHC1G14DBVT, U904 DAC8565ICPW, U905 MC74AC161DR2G, U906 SN74AUP1G79DCKR, U907 LM7171BIM, U908 AD5322ARMZ, U909 LT1790BCS6-2.5, U910 DG409DY+, U911 TL071CDR, U912 LM7171BIM, X901 830208220601, Y1001 ECS-080-18-23A-JGN-TR, Y201 NX5032GA-25.000000MHZ-LN-CD-1

Commit message: Hardware design
Parts:
- removed the C402 at (127.3, 28.4)
- removed the C406 at (110.1, 36.3)
- removed the C417 at (118.8, 40.2)
- removed the C426 at (122.9, 28.9)
- removed the C807 at (-10.8, 77.4)
- removed the C808 at (-2.76, 69.3)
- removed the R612 at (79.8, 80.1)
- removed the U801 at (204.0, 108.0)
- added C401: 100n, Capacitor_SMD:C_0603_1608Metric_Pad1.08x0.95mm_HandSolder, F.Cu at (121.3, -29.2)
- added C404: 100n, Capacitor_SMD:C_0603_1608Metric_Pad1.08x0.95mm_HandSolder, F.Cu at (110.7, -19.2)
- added C408: 100n, Capacitor_SMD:C_0603_1608Metric_Pad1.08x0.95mm_HandSolder, F.Cu at (100.1, -10.8)
- added C414: 1u, Capacitor_SMD:C_0603_1608Metric_Pad1.08x0.95mm_HandSolder, F.Cu at (106.3, -16.7)
- added C418: 100n, Capacitor_SMD:C_0603_1608Metric_Pad1.08x0.95mm_HandSolder, F.Cu at (88.1, -13.8)
- added C427: 100n, Capacitor_SMD:C_0603_1608Metric_Pad1.08x0.95mm_HandSolder, F.Cu at (103.9, -29.2)
- added C428: 100n, Capacitor_SMD:C_0603_1608Metric_Pad1.08x0.95mm_HandSolder, F.Cu at (113.7, -24.2)
- added C430: 100n, Capacitor_SMD:C_0603_1608Metric_Pad1.08x0.95mm_HandSolder, F.Cu at (109.4, -24.2)
- added C431: 100n, Capacitor_SMD:C_0603_1608Metric_Pad1.08x0.95mm_HandSolder, F.Cu at (102.0, -19.2)
- added C433: 10n, Capacitor_SMD:C_0603_1608Metric_Pad1.08x0.95mm_HandSolder, F.Cu at (117.0, -29.2)
- added C434: 100n, Capacitor_SMD:C_0603_1608Metric_Pad1.08x0.95mm_HandSolder, F.Cu at (104.4, -11.7)
- added C435: 100n, Capacitor_SMD:C_0603_1608Metric_Pad1.08x0.95mm_HandSolder, F.Cu at (91.4, -11.3)
- added C436: 100n, Capacitor_SMD:C_0603_1608Metric_Pad1.08x0.95mm_HandSolder, F.Cu at (87.0, -9.89)
- added C437: 100n, Capacitor_SMD:C_0603_1608Metric_Pad1.08x0.95mm_HandSolder, F.Cu at (93.3, -18.2)
- added C438: 100n, Capacitor_SMD:C_0603_1608Metric_Pad1.08x0.95mm_HandSolder, F.Cu at (112.6, -29.2)
- added C439: 100n, Capacitor_SMD:C_0603_1608Metric_Pad1.08x0.95mm_HandSolder, F.Cu at (102.0, -16.7)
- added C440: 100n, Capacitor_SMD:C_0603_1608Metric_Pad1.08x0.95mm_HandSolder, F.Cu at (105.0, -26.7)
- added C441: 100n, Capacitor_SMD:C_0603_1608Metric_Pad1.08x0.95mm_HandSolder, F.Cu at (105.0, -24.2)
- added C442: 100n, Capacitor_SMD:C_0603_1608Metric_Pad1.08x0.95mm_HandSolder, F.Cu at (100.7, -22.0)
- added C443: 100n, Capacitor_SMD:C_0603_1608Metric_Pad1.08x0.95mm_HandSolder, F.Cu at (95.7, -13.2)
- added C444: 100n, Capacitor_SMD:C_0603_1608Metric_Pad1.08x0.95mm_HandSolder, F.Cu at (104.4, -9.16)
- added C445: 100n, Capacitor_SMD:C_0603_1608Metric_Pad1.08x0.95mm_HandSolder, F.Cu at (109.4, -26.7)
- added C446: 100n, Capacitor_SMD:C_0603_1608Metric_Pad1.08x0.95mm_HandSolder, F.Cu at (110.7, -16.7)
- added C447: 100n, Capacitor_SMD:C_0603_1608Metric_Pad1.08x0.95mm_HandSolder, F.Cu at (95.7, -8.21)
- added C448: 100n, Capacitor_SMD:C_0603_1608Metric_Pad1.08x0.95mm_HandSolder, F.Cu at (100.1, -5.79)
- added C449: 100n, Capacitor_SMD:C_0603_1608Metric_Pad1.08x0.95mm_HandSolder, F.Cu at (95.7, -5.70)
- added C452: 2n7, Capacitor_SMD:C_0603_1608Metric_Pad1.08x0.95mm_HandSolder, F.Cu at (97.6, -18.3)
- added C453: 2n7, Capacitor_SMD:C_0603_1608Metric_Pad1.08x0.95mm_HandSolder, F.Cu at (100.1, -13.3)
- added C454: 1u, Capacitor_SMD:C_0603_1608Metric_Pad1.08x0.95mm_HandSolder, F.Cu at (106.3, -19.2)
- added C455: 1u, Capacitor_SMD:C_0603_1608Metric_Pad1.08x0.95mm_HandSolder, F.Cu at (109.4, -21.7)
- added C617: 100n, Capacitor_SMD:C_0603_1608Metric_Pad1.08x0.95mm_HandSolder, F.Cu at (161.9, -26.7)
- added C618: 100n, Capacitor_SMD:C_0603_1608Metric_Pad1.08x0.95mm_HandSolder, F.Cu at (146.3, -10.0)
- added C619: 10p, Capacitor_SMD:C_0603_1608Metric_Pad1.08x0.95mm_HandSolder, F.Cu at (161.9, -29.2)
- added C620: 10p, Capacitor_SMD:C_0603_1608Metric_Pad1.08x0.95mm_HandSolder, F.Cu at (149.1, -15.8)
- added C621: 10p, Capacitor_SMD:C_0603_1608Metric_Pad1.08x0.95mm_HandSolder, F.Cu at (157.5, -29.2)
- added C622: 10p, Capacitor_SMD:C_0603_1608Metric_Pad1.08x0.95mm_HandSolder, F.Cu at (155.0, -21.7)
- added K304: HE3621A0510, ETH1CSMU2:HE360_x-5050462-8, F.Cu at (116.0, 82.0)
- added Q601: MMBT3904, Package_TO_SOT_SMD:SOT-23, F.Cu at (150.4, -21.8)
- added Q602: MMBT3904, Package_TO_SOT_SMD:SOT-23, F.Cu at (152.9, -28.3)
- added Q603: MMBT3904, Package_TO_SOT_SMD:SOT-23, F.Cu at (144.5, -18.5)
- added Q604: MMBT3904, Package_TO_SOT_SMD:SOT-23, F.Cu at (141.7, -11.2)
- added R406: 82k, Resistor_SMD:R_0603_1608Metric_Pad0.98x0.95mm_HandSolder, F.Cu at (104.4, -14.2)
- added R417: 2k49/.1%, Resistor_SMD:R_0603_1608Metric_Pad0.98x0.95mm_HandSolder, F.Cu at (105.0, -21.7)
- added R418: 12k/.1%, Resistor_SMD:R_0603_1608Metric_Pad0.98x0.95mm_HandSolder, F.Cu at (91.4, -6.26)
- added R419: 12k/.1%, Resistor_SMD:R_0603_1608Metric_Pad0.98x0.95mm_HandSolder, F.Cu at (93.3, -15.7)
- added R420: 2k49/.1%, Resistor_SMD:R_0603_1608Metric_Pad0.98x0.95mm_HandSolder, F.Cu at (87.0, -7.38)
- added R421: 12k/.1%, Resistor_SMD:R_0603_1608Metric_Pad0.98x0.95mm_HandSolder, F.Cu at (108.3, -29.2)
- added R422: 12k/.1%, Resistor_SMD:R_0603_1608Metric_Pad0.98x0.95mm_HandSolder, F.Cu at (118.1, -24.2)
- added R425: 2k49/.1%, Resistor_SMD:R_0603_1608Metric_Pad0.98x0.95mm_HandSolder, F.Cu at (97.6, -15.8)
- added R426: 2k49/.1%, Resistor_SMD:R_0603_1608Metric_Pad0.98x0.95mm_HandSolder, F.Cu at (100.7, -24.5)
- added R427: 20, Resistor_SMD:R_0603_1608Metric_Pad0.98x0.95mm_HandSolder, F.Cu at (95.7, -10.7)
- added R428: 20, Resistor_SMD:R_0603_1608Metric_Pad0.98x0.95mm_HandSolder, F.Cu at (100.1, -8.30)
- added R433: OPT, Resistor_SMD:R_0603_1608Metric_Pad0.98x0.95mm_HandSolder, F.Cu at (113.7, -26.7)
- added R434: 0, Resistor_SMD:R_0603_1608Metric_Pad0.98x0.95mm_HandSolder, F.Cu at (91.4, -8.78)
- added R611: 10k, Resistor_SMD:R_0603_1608Metric_Pad0.98x0.95mm_HandSolder, F.Cu at (155.0, -24.2)
- added R613: 0, Resistor_SMD:R_0603_1608Metric_Pad0.98x0.95mm_HandSolder, F.Cu at (146.2, 49.7)
- added R615: 0, Resistor_SMD:R_0603_1608Metric_Pad0.98x0.95mm_HandSolder, F.Cu at (159.4, -24.2)
- added R616: 1k, Resistor_SMD:R_0603_1608Metric_Pad0.98x0.95mm_HandSolder, F.Cu at (153.4, -18.3)
- added R617: 1k, Resistor_SMD:R_0603_1608Metric_Pad0.98x0.95mm_HandSolder, F.Cu at (149.1, -18.3)
- added R618: 1k, Resistor_SMD:R_0603_1608Metric_Pad0.98x0.95mm_HandSolder, F.Cu at (157.5, -26.7)
- added R619: 1k, Resistor_SMD:R_0603_1608Metric_Pad0.98x0.95mm_HandSolder, F.Cu at (144.2, -15.1)
- added R620: OPT, Resistor_SMD:R_0603_1608Metric_Pad0.98x0.95mm_HandSolder, F.Cu at (146.3, -12.5)
- added R622: 10k, Resistor_SMD:R_0603_1608Metric_Pad0.98x0.95mm_HandSolder, F.Cu at (150.7, -13.3)
- added R623: WSR2R8000FEK, Resistor_SMD:R_Shunt_Vishay_WSR2_WSR3_KelvinConnection, F.Cu at (176.0, 24.0)
- added R624: WSR21R000FEK, Resistor_SMD:R_Shunt_Vishay_WSR2_WSR3_KelvinConnection, F.Cu at (134.7, -25.9)
- added R625: RP73D2B10RBTG, Resistor_SMD:R_1206_3216Metric_Pad1.30x1.75mm_HandSolder, F.Cu at (145.0, -22.4)
- added R626: RQ73C2B100RBT, Resistor_SMD:R_1206_3216Metric_Pad1.30x1.75mm_HandSolder, F.Cu at (130.4, -11.8)
- added R627: PHPA1206E1001BST, Resistor_SMD:R_1206_3216Metric_Pad1.30x1.75mm_HandSolder, F.Cu at (136.3, -11.8)
- added R629: 10k, Resistor_SMD:R_0603_1608Metric_Pad0.98x0.95mm_HandSolder, F.Cu at (153.4, -15.8)
- added U401: LT1790BCS6-2.5, Package_TO_SOT_SMD:TSOT-23-6, F.Cu at (88.5, -17.3)
- added U405: ADR435ARM, Package_SO:MSOP-8_3x3mm_P0.65mm, F.Cu at (89.7, -21.8)
- added U411: DG419DY, Package_SO:SOIC-8_3.9x4.9mm_P1.27mm, F.Cu at (81.7, -20.8)
- added U412: DG419DY, Package_SO:SOIC-8_3.9x4.9mm_P1.27mm, F.Cu at (81.7, -14.4)
- added U413: OPA141AID, Package_SO:SOIC-8_3.9x4.9mm_P1.27mm, F.Cu at (90.2, -27.3)
- added U414: OPA141AID, Package_SO:SOIC-8_3.9x4.9mm_P1.27mm, F.Cu at (81.7, -27.3)
- added U417: AD7980ARM, Package_SO:MSOP-10_3x3mm_P0.5mm, F.Cu at (98.1, -28.1)
- added U418: AD7980ARM, Package_SO:MSOP-10_3x3mm_P0.5mm, F.Cu at (81.2, -8.78)
- added U419: TPS76925, Package_TO_SOT_SMD:SOT-23-5, F.Cu at (95.9, -21.8)
- added U607: AQY212G2SX, ETH1CSMU2:AQY212GS, F.Cu at (115.0, 64.4)
- added U608: AQY212G2SX, ETH1CSMU2:AQY212GS, F.Cu at (127.3, 64.4)
- added U609: AQY212G2SX, ETH1CSMU2:AQY212GS, F.Cu at (121.1, 64.4)
- added U610: AQY212G2SX, ETH1CSMU2:AQY212GS, F.Cu at (108.9, 64.4)
- added U612: LM7171BIM, Package_SO:SOIC-8_3.9x4.9mm_P1.27mm, F.Cu at (61.6, 25.0)
- added U802: TSR2-2450, ETH1CSMU2:TSR2, F.Cu at (199.3, 109.2)
- C923: value 4u7 -> 4u7/OPT
- R601, R602, R603: value 10k -> 1k
- R606: renamed from R605; value 3k4 -> 3k4/.1%
- R607: renamed from R606; value 3k4 -> 3k4/.1%
- R608: renamed from R607; value 10k2 -> 10k2/.1%
- R610: renamed from R608; value 10k2 -> 10k2/.1%
- R612: renamed from R610; value 10k2 -> 10k2/.1%
- R614: value LCS2512 -> 10k; footprint Resistor_SMD:R_2512_6332Metric_Pad1.40x3.35mm_HandSolder -> Resistor_SMD:R_0603_1608Metric_Pad0.98x0.95mm_HandSolder
- R621: renamed from R613; value OPT -> 11k/.1%
- R904: value 5k6 -> 7k5
- R905, R906: value 200 -> 200/.1%
- R912: value DNP -> 0
- Y1001: value ECS-080-18-23A-JGN-TR -> NX3225GD-16MHZ; footprint Crystal:Crystal_SMD_0603-2Pin_6.0x3.5mm_HandSoldering -> ETH1CSMU2:NX3225GD
- moved K305 239.3 mm to (217.9, 55.6)
- moved K302 218.4 mm to (217.9, 50.4)
- moved R614 127.4 mm to (159.4, -21.7)
- moved C412 69.7 mm to (118.1, -26.7)
- moved C423 60.7 mm to (113.7, -21.7)
- moved Y1001 56.2 mm to (74.6, 23.9)
- moved U606 9.26 mm to (194.0, 52.0)
- renumbered C403 to C402, C404 to C403, C407 to C405, C408 to C406, C401 to C407, C413 to C409, C409 to C410, C405 to C411, C418 to C413, C414 to C415, C419 to C416, C411 to C417, C424 to C419, C416 to C422, C427 to C424, C410 to C425, C422 to C426, C415 to C429, C425 to C432, C428 to C450, C429 to C451, C608 to C601, C601 to C602, C609 to C603, C610 to C604, C602 to C605, C603 to C606, C611 to C607, C612 to C608, C604 to C609, C605 to C610, C613 to C611, C614 to C612, C606 to C613, C607 to C614, C809 to C807, C810 to C808, C811 to C809, C812 to C810, C815 to C811, C818 to C812, C821 to C815, C831 to C816, C816 to C817, C817 to C818, C824 to C819, C832 to C820, C819 to C821, C820 to C822, C827 to C823, C822 to C824, C823 to C825, C825 to C826, C826 to C827, C913 to C912, C912 to C913, C916 to C915, C915 to C916, C920 to C919, C919 to C920, K304 to K305, K305 to K306, R406 to R407, R407 to R408, R408 to R409, R409 to R410, R410 to R411, R411 to R412, R412 to R413, R413 to R414, R414 to R415, R415 to R416, R416 to R423, R417 to R424, R418 to R429, R419 to R430, R420 to R431, R421 to R432, R611 to R605, R615 to R628, R927 to R926, R926 to R927, U401 to U402, U402 to U403, U403 to U404, U404 to U407, U405 to U408, U407 to U409, U408 to U410, U409 to U415, U410 to U416, U606 to U604, U604 to U605, U605 to U606, U607 to U611, U804 to U801, U802 to U803, U803 to U804
Connections:
- net +2V5 renamed /Source/SOUR_2V5
- C801 pad 2: GNDPWR -> GND
- C802 pad 2: GNDPWR -> GND
- C803 pad 2: GNDPWR -> GND
- C804 pad 2: GNDPWR -> GND
- C805 pad 2: GNDPWR -> GND
- C806 pad 2: GNDPWR -> GND
- C809 pad 1: GNDPWR -> GND
- C810 pad 1: GNDPWR -> GND
- C816 pad 2: GNDPWR -> GND
- C820 pad 2: GNDPWR -> GND
- C927 pad 2: /Source/FGEN -> /Frontend/FGEN
- D801 pad 2: GNDPWR -> GND
- D803 pad 1: GNDPWR -> GND
- J301 pad A27: GNDPWR -> GND
- J301 pad A28: GNDPWR -> GND
- J301 pad C27: GNDPWR -> GND
- J301 pad C28: GNDPWR -> GND
- K301 pad 1: unconnected-(K301-Pad1) -> /Connect/VOUT_OUT
- K302 pad 1: unconnected-(K302-Pad1) -> GND
- K303 pad 1: unconnected-(K303-Pad1) -> /Connect/GUARD
- K305 pad 1: unconnected-(K304-Pad1) -> /Connect/VOLT_MEAS_SENS
- K306 pad 1: unconnected-(K305-Pad1) -> GND
- R408 pad 2: /Measure/CURR_MEAS -> /Frontend/CURR_MEAS
- R411 pad 1: Net-(R410-Pad1) (its old number) -> Net-(R411-Pad1)
- R414 pad 1: Net-(R413-Pad1) -> Net-(R414-Pad1)
- R423 pad 1: Net-(R410-Pad1) (its old number) -> /Measure/ADC1_VOLT
- R424 pad 1: Net-(R413-Pad1) -> /Measure/ADC1_CURR
- R432 pad 2: /Measure/ADC_HS_MISO -> /MCU/SPI1_MISO
- R612 pad 2: /Frontend/VOLT_MEAS -> /Connect/VOUT_OUT
- R614 pad 1: Net-(R612-Pad1) (its old number) -> /Frontend/MCU_CURR_SENS_10R
- R614 pad 2: /Frontend/VOLT_MEAS -> Net-(C620-Pad1)
- R628 pad 1: /Frontend/VOLT_MEAS -> /Connect/VOUT_OUT
- R628 pad 2: Net-(R615-Pad2) -> Net-(R613-Pad1)
- R914 pad 1: +5VA -> +5V
- R930 pad 2: /Source/FGEN -> /Frontend/FGEN
- U1002 pad 1: unconnected-(U1002-Pad1) -> /MCU/SPI4_SCK
- U1002 pad 10: unconnected-(U1002-Pad10) -> /Frontend/MCU_nISNK
- U1002 pad 11: unconnected-(U1002-Pad11) -> /Frontend/MCU_nISRC
- U1002 pad 110: unconnected-(U1002-Pad110) -> /MCU/SPI3_NSS
- U1002 pad 111: unconnected-(U1002-Pad111) -> /MCU/SPI3_SCK
- U1002 pad 112: unconnected-(U1002-Pad112) -> /MCU/SPI3_MISO
- U1002 pad 113: unconnected-(U1002-Pad113) -> /MCU/SPI3_MOSI
- U1002 pad 117: unconnected-(U1002-Pad117) -> /Control/SR_CLK
- U1002 pad 118: unconnected-(U1002-Pad118) -> /Control/SR_DAT
- U1002 pad 119: unconnected-(U1002-Pad119) -> /Control/SR_LAT
- U1002 pad 12: unconnected-(U1002-Pad12) -> /Frontend/MCU_nTDS
- U1002 pad 122: unconnected-(U1002-Pad122) -> /Control/SR_OUT
- U1002 pad 135: unconnected-(U1002-Pad135) -> /MCU/SPI1_MOSI
- U1002 pad 18: unconnected-(U1002-Pad18) -> /MCU/SPI5_NSS
- U1002 pad 19: unconnected-(U1002-Pad19) -> /MCU/SPI5_SCK
- U1002 pad 20: unconnected-(U1002-Pad20) -> /MCU/SPI5_MISO
- U1002 pad 21: unconnected-(U1002-Pad21) -> /MCU/SPI5_MOSI
- U1002 pad 22: unconnected-(U1002-Pad22) -> /MCU/DAC2_~{LDAC}
- U1002 pad 3: unconnected-(U1002-Pad3) -> /MCU/SPI4_NSS
- U1002 pad 34: unconnected-(U1002-Pad34) -> /MCU/ADC1_RVS1
- U1002 pad 36: /Ethernet/MDIO -> /Ethernet/RMII_MDIO
- U1002 pad 37: unconnected-(U1002-Pad37) -> /MCU/ADC1_RVS2
- U1002 pad 4: unconnected-(U1002-Pad4) -> /MCU/SPI4_MISO
- U1002 pad 40: unconnected-(U1002-Pad40) -> /MCU/SPI1_NSS
- U1002 pad 41: unconnected-(U1002-Pad41) -> /MCU/SPI1_SCK
- U1002 pad 42: unconnected-(U1002-Pad42) -> /MCU/SPI1_MISO
- U1002 pad 5: unconnected-(U1002-Pad5) -> /MCU/SPI4_MOSI
- U1002 pad 50: unconnected-(U1002-Pad50) -> /MCU/DDS_DIV2
- U1002 pad 53: unconnected-(U1002-Pad53) -> /MCU/DDS_DIV4
- U1002 pad 54: unconnected-(U1002-Pad54) -> /MCU/DDS_DIV8
- U1002 pad 55: unconnected-(U1002-Pad55) -> /MCU/~{DDS_DIV10}
- U1002 pad 58: unconnected-(U1002-Pad58) -> /Connect/CXN_REL6
- U1002 pad 59: unconnected-(U1002-Pad59) -> /MCU/TRIG_EN
- U1002 pad 60: /MCU/TRIG_EN -> /MCU/TRIG_OUT
- U1002 pad 63: /MCU/TRIG_OUT -> /MCU/TRIG_IN
- U1002 pad 64: /MCU/TRIG_IN -> /Connect/CXN_REL2
- U1002 pad 65: unconnected-(U1002-Pad65) -> /Connect/CXN_REL1
- U1002 pad 69: /Connect/CXN_REL2 -> /MCU/DAC1_LDAC
- U1002 pad 70: /Connect/CXN_REL1 -> /MCU/DAC1_~{RST}
- U1002 pad 73: unconnected-(U1002-Pad73) -> /MCU/SPI2_NSS
- U1002 pad 74: unconnected-(U1002-Pad74) -> /MCU/SPI2_SCK
- U1002 pad 75: unconnected-(U1002-Pad75) -> /MCU/SPI2_MISO
- U1002 pad 76: unconnected-(U1002-Pad76) -> /MCU/SPI2_MOSI
- U1002 pad 90: unconnected-(U1002-Pad90) -> /Frontend/MCU_CURR_SENS_1kR
- U1002 pad 91: unconnected-(U1002-Pad91) -> /Frontend/MCU_CURR_SENS_100R
- U1002 pad 92: unconnected-(U1002-Pad92) -> /Frontend/MCU_CURR_SENS_10R
- U1002 pad 93: unconnected-(U1002-Pad93) -> /Frontend/MCU_CURR_SENS_1R
- U201 pad 12: /Ethernet/MDIO -> /Ethernet/RMII_MDIO
- U301 pad 1: /Connect/CXN_REL5 -> /Connect/CXN_REL6
- U301 pad 11: unconnected-(U301-Pad11) -> Net-(K304-Pad3)
- U301 pad 2: /Connect/CXN_REL4 -> /Connect/CXN_REL5
- U301 pad 3: /Connect/CXN_REL3 -> /Connect/CXN_REL4
- U301 pad 4: /Connect/CXN_REL2 -> /Connect/CXN_REL3
- U301 pad 5: /Connect/CXN_REL1 -> /Connect/CXN_REL2
- U301 pad 6: unconnected-(U301-Pad6) -> /Connect/CXN_REL1
- U402 pad 3: Net-(R410-Pad1) (its old number) -> Net-(R411-Pad1)
- U404 pad 3: Net-(R413-Pad1) -> Net-(R414-Pad1)
- U406 pad 2: /Measure/VOLT_MEAS -> /Connect/VOUT_OUT
- U406 pad 8: /Measure/VOLT_MEAS_SENS -> /Connect/VOLT_MEAS_SENS
- U407 pad 4: +5V -> +15V
- U407 pad 5: +15V -> +5V
- U409 pad 6: Net-(R410-Pad1) (its old number) -> Net-(R411-Pad1)
- U410 pad 6: Net-(R413-Pad1) -> Net-(R414-Pad1)
- U415 pad 10: /Measure/ADC_HS_SCLK -> /MCU/SPI1_SCK
- U415 pad 13: /Measure/ADC_HS_RVS1 -> /MCU/ADC1_RVS1
- U415 pad 17: unconnected-(U409-Pad17) -> GND
- U415 pad 8: /Measure/ADC_HS_MOSI -> /MCU/SPI1_MOSI
- U415 pad 9: /Measure/ADC_HS_~{CS} -> /MCU/SPI1_NSS
- U416 pad 10: /Measure/ADC_HS_SCLK -> /MCU/SPI1_SCK
- U416 pad 11: /Measure/ADC_HS_MISO -> /MCU/SPI1_MISO
- U416 pad 13: /Measure/ADC_HS_RVS2 -> /MCU/ADC1_RVS2
- U416 pad 17: unconnected-(U410-Pad17) -> GND
- U416 pad 9: /Measure/ADC_HS_~{CS} -> /MCU/SPI1_NSS
- U502 pad 6: unconnected-(U502-Pad6) -> /Measure/ADC_SEL
- U503 pad 4: /Control/GPIO_SPI_MOSI -> /Control/SR_DAT
- U504 pad 4: /Control/GPIO_SPI_SCK -> /Control/SR_CLK
- U505 pad 4: /Control/GPIO_SPI_NSS -> /Control/SR_LAT
- U506 pad 4: /Control/GPIO_SPI_MISO -> /Control/SR_OUT
- U606 pad 3: Net-(R612-Pad1) (its old number) -> Net-(R615-Pad2)
- U606 pad 5: Net-(R615-Pad2) -> Net-(R613-Pad2)
- U606 pad 6: Net-(R615-Pad2) -> Net-(R613-Pad1)
- U611 pad 2: /Frontend/VOLT_MEAS -> /Connect/VOUT_OUT
- U611 pad 3: Net-(R612-Pad1) (its old number) -> Net-(R615-Pad2)
- U801 pad 4: GNDPWR -> GND
- U803 pad 1: GNDPWR -> GND
- U901 pad 4: /Source/DDS_DIV2 -> /MCU/DDS_DIV2
- U901 pad 5: /Source/DDS_DIV4 -> /MCU/DDS_DIV4
- U901 pad 6: /Source/DDS_DIV8 -> /MCU/DDS_DIV8
- U902 pad 13: /Source/DDS_SDATA -> /MCU/SPI3_MOSI
- U902 pad 14: /Source/DDS_SCLK -> /MCU/SPI3_SCK
- U902 pad 15: /Source/DDS_CS -> /MCU/SPI3_NSS
- U904 pad 1: /Source/VC_+IN -> /Frontend/VC_+IN
- U904 pad 10: /Source/DAC1_SCLK -> /MCU/SPI2_SCK
- U904 pad 11: /Source/DAC1_DIN -> /MCU/SPI2_MOSI
- U904 pad 13: /Source/DAC1_~{RST} -> /MCU/DAC1_~{RST}
- U904 pad 16: /Source/DAC1_LDAC -> /MCU/DAC1_LDAC
- U904 pad 2: /Source/VC_-IN -> /Frontend/VC_-IN
- U904 pad 7: /Source/VC_SINK -> /Frontend/VC_SINK
- U904 pad 8: /Source/VC_SRC -> /Frontend/VC_SRC
- U904 pad 9: /Source/DAC1_~{SYNC} -> /MCU/SPI2_NSS
- U905 pad 4: /Source/~{DDS_DIV10} -> /MCU/~{DDS_DIV10}
- U905 pad 5: /Source/~{DDS_DIV10} -> /MCU/~{DDS_DIV10}
- U908 pad 1: /Source/DAC2_~{LDAC} -> /MCU/DAC2_~{LDAC}
- U908 pad 7: /Source/DAC2_~{SYNC} -> /MCU/SPI5_NSS
- U908 pad 8: /Source/DAC2_SCLK -> /MCU/SPI5_SCK
- U908 pad 9: /Source/DAC2_DIN -> /MCU/SPI5_MOSI
- U910 pad 14: +5VA -> +15V
- U910 pad 2: +5VA -> +5V
- U910 pad 3: -5VA -> -15V
- U912 pad 6: /Source/FGEN -> /Frontend/FGEN

Commit message: Hardware design
Parts:
- added C905: 100n, Capacitor_SMD:C_0603_1608Metric_Pad1.08x0.95mm_HandSolder, F.Cu at (128.0, 98.6)
- added C906: 100n, Capacitor_SMD:C_0603_1608Metric_Pad1.08x0.95mm_HandSolder, F.Cu at (123.1, 105.0)
- added C921: 100n, Capacitor_SMD:C_0603_1608Metric_Pad1.08x0.95mm_HandSolder, F.Cu at (114.7, 108.9)
- added C922: 100n, Capacitor_SMD:C_0603_1608Metric_Pad1.08x0.95mm_HandSolder, F.Cu at (119.0, 107.6)
- added C928: 100n, Capacitor_SMD:C_0603_1608Metric_Pad1.08x0.95mm_HandSolder, F.Cu at (110.3, 108.9)
- added C929: 100n, Capacitor_SMD:C_0603_1608Metric_Pad1.08x0.95mm_HandSolder, F.Cu at (118.8, 105.0)
- added R623: 0, Resistor_SMD:R_0603_1608Metric_Pad0.98x0.95mm_HandSolder, F.Cu at (110.3, 117.0)
- added R630: 0, Resistor_SMD:R_0603_1608Metric_Pad0.98x0.95mm_HandSolder, F.Cu at (110.3, 114.5)
- added R905: 4k7, Resistor_SMD:R_0603_1608Metric_Pad0.98x0.95mm_HandSolder, F.Cu at (130.5, 96.0)
- added R906: 4k7, Resistor_SMD:R_0603_1608Metric_Pad0.98x0.95mm_HandSolder, F.Cu at (123.7, 100.6)
- added R912: 1k, Resistor_SMD:R_0603_1608Metric_Pad0.98x0.95mm_HandSolder, F.Cu at (127.5, 103.6)
- added R914: 1k, Resistor_SMD:R_0603_1608Metric_Pad0.98x0.95mm_HandSolder, F.Cu at (126.2, 96.0)
- added R916: 1Meg, Resistor_SMD:R_0603_1608Metric_Pad0.98x0.95mm_HandSolder, F.Cu at (128.0, 101.1)
- added R917: 10k, Resistor_SMD:R_0603_1608Metric_Pad0.98x0.95mm_HandSolder, F.Cu at (132.4, 98.6)
- added U906: MAX6102EUR, Package_TO_SOT_SMD:SOT-23, F.Cu at (119.0, 101.6)
- added U908: MAX5217GUA+, Package_SO:MSOP-8_3x3mm_P0.65mm, F.Cu at (120.3, 97.1)
- added U909: OPA2141AID, Package_SO:SOIC-8_3.9x4.9mm_P1.27mm, F.Cu at (112.4, 104.5)
- added U911: OPA141AID, Package_SO:SOIC-8_3.9x4.9mm_P1.27mm, F.Cu at (112.4, 98.0)
- renumbered C803 to C802, C805 to C803, C802 to C804, C804 to C805, C807 to C806, C808 to C807, C809 to C808, C810 to C809, C806 to C810, C813 to C811, C814 to C812, C816 to C813, C811 to C814, C817 to C815, C818 to C816, C820 to C817, C812 to C818, C821 to C819, C822 to C820, C815 to C821, C824 to C822, C825 to C823, C819 to C824, C826 to C825, C827 to C826, C823 to C827, C907 to C902, C902 to C903, C903 to C904, C904 to C907, C905 to C908, C906 to C909, C909 to C910, C908 to C911, C910 to C912, C911 to C915, C912 to C918, C915 to C919, C918 to C923, C922 to C924, C919 to C925, C921 to C926, C923 to C927, C924 to C930, C926 to C931, C927 to C932, C925 to C933, R623 to R624, R624 to R625, R625 to R626, R626 to R627, R627 to R628, R628 to R629, R629 to R631, R903 to R902, R902 to R903, R905 to R907, R906 to R908, R907 to R909, R908 to R910, R909 to R911, R910 to R913, R911 to R915, R912 to R918, R913 to R919, R914 to R920, R915 to R921, R916 to R922, R917 to R923, R918 to R924, R919 to R925, R920 to R926, R921 to R927, R922 to R928, R923 to R929, R924 to R930, R927 to R931, R928 to R932, R929 to R933, R930 to R934, R925 to R935, R926 to R936, U803 to U802, U802 to U803, U904 to U901, U901 to U902, U902 to U903, U903 to U904, U906 to U907, U907 to U910, U908 to U912, U910 to U913, U911 to U914, U909 to U915, U912 to U916
Connections:
- U611 pad 5: GND -> Net-(R623-Pad1)

Commit message: Hardware design
Parts:
- removed the C825 at (-35.8, 107.0)
- removed the C826 at (-66.3, 107.8)
- removed the C827 at (9.96, 65.0)
- removed the R624 at (176.0, 24.0)
- C1003, C1005: value 6p -> 8p
- C619: moved to B.Cu
- C806, C807, C808: footprint Capacitor_SMD:C_1812_4532Metric_Pad1.57x3.40mm_HandSolder -> Capacitor_SMD:C_1206_3216Metric_Pad1.33x1.80mm_HandSolder; moved to B.Cu
- C809: footprint Capacitor_SMD:C_1812_4532Metric_Pad1.57x3.40mm_HandSolder -> Capacitor_SMD:C_1206_3216Metric_Pad1.33x1.80mm_HandSolder
- R616: renamed from R621; moved to B.Cu
- R617: renamed from R616; moved to B.Cu
- R621: renamed from R620; moved to B.Cu
- R625: value WSR21R000FEK -> RT1206BRD071RL; footprint Resistor_SMD:R_Shunt_Vishay_WSR2_WSR3_KelvinConnection -> Resistor_SMD:R_1206_3216Metric_Pad1.30x1.75mm_HandSolder
- U301: value ULN2003AS16 -> ULN2003AIDE4; footprint Package_SO:TSSOP-16_4.4x5mm_P0.65mm -> Package_SO:SOIC-16_3.9x9.9mm_P1.27mm
- Y1001: value NX3225GD-16MHZ -> NX5032GA-16.000M
- moved C801 300.0 mm to (209.0, 134.5), turned to -90 degrees
- moved C802 291.5 mm to (206.4, 134.5), turned to -90 degrees
- moved C803 289.5 mm to (203.7, 134.5), turned to -90 degrees
- moved C804 288.3 mm to (199.0, 120.0)
- moved K306 270.6 mm to (206.2, 71.8)
- moved K301 266.2 mm to (206.2, 45.7)
- moved D803 263.2 mm to (213.7, 122.2), turned to 90 degrees
- moved F801 259.3 mm to (216.5, 134.5)
- moved K303 247.9 mm to (206.2, 56.1)
- moved C818 234.1 mm to (179.5, 119.8), turned to -90 degrees
- moved C805 231.3 mm to (199.0, 116.7)
- moved U410 226.9 mm to (-62.5, -125.0)
- moved C901 226.8 mm to (-184.2, -114.5)
- moved C910 226.8 mm to (-211.2, -112.1)
- moved C913 226.8 mm to (-206.0, -114.5)
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- renumbered C828 to C825, C829 to C826, C830 to C827, R617 to R618, R618 to R619, R619 to R620, R630 to R622, R622 to R624, R631 to R630, U611 to U607, U607 to U608, U608 to U609, U609 to U610, U610 to U611
Connections:
- C811 pad 2: Net-(C811-Pad2) -> GND
- C812 pad 1: Net-(C811-Pad2) -> GND
- C815 pad 2: Net-(C815-Pad2) -> GND
- C816 pad 1: Net-(C815-Pad2) -> GND
- C819 pad 2: Net-(C819-Pad2) -> GND
- C820 pad 1: Net-(C819-Pad2) -> GND
- C822 pad 2: Net-(C822-Pad2) -> GND
- C823 pad 1: Net-(C822-Pad2) -> GND
Other:
- board outline added: 160 x 100 mm
- copper layers 2 -> 4

Commit message: PCB layout
Parts:
- added R930: 300, Resistor_SMD:R_0603_1608Metric_Pad0.98x0.95mm_HandSolder, F.Cu at (-187.2, -103.6)
- C1001, C1002, C1003, C1004, C1005, C1006, C1007, C1008, C1009, C1010, C1011, C1012, C1013, C1014, C1015, C1017, C1018, C1019, C1020, C1021, C1022, C213, C214, C602, C603, C620, C621, C622, C701, C702, C703, C704, C705, C706, C707, C708, FB1001, R1001, R1003, R1005, R1007, R1008, R1009, R1010, R206, R207, R208, R209, R212, R213, R214, R215, R216, R217, R218, R219, R220, R221, R601, R602, R603, R701, R704, R706, U1003, Y1001: moved to B.Cu
- C201, C202, C204, C205, C206, C207, C208, C209, C211, C212: footprint Capacitor_SMD:C_0201_0603Metric_Pad0.64x0.40mm_HandSolder -> Capacitor_SMD:C_0603_1608Metric_Pad1.08x0.95mm_HandSolder; moved to B.Cu
- C203, C210: footprint Capacitor_SMD:C_0201_0603Metric_Pad0.64x0.40mm_HandSolder -> Capacitor_SMD:C_0603_1608Metric_Pad1.08x0.95mm_HandSolder
- R617: moved to F.Cu
- R928: renamed from R929; value 26k4 -> 26k1
- U801: value MAX5902 -> MAX5902ACEUT
- moved L701 400.9 mm to (213.7, 88.1), turned to 180 degrees
- moved R903 398.3 mm to (128.8, 121.2), turned to 180 degrees
- moved D703 395.9 mm to (215.4, 83.1), turned to 90 degrees
- moved C709 389.9 mm to (212.9, 83.1), turned to 90 degrees
- moved R705 389.6 mm to (209.7, 88.1)
- moved R706 388.4 mm to (212.9, 83.1), turned to -90 degrees
- moved D702 387.9 mm to (207.8, 83.1)
- moved D701 387.9 mm to (205.9, 88.1)
- moved R704 381.0 mm to (204.9, 82.7), turned to -90 degrees
- moved C706 378.7 mm to (202.3, 82.7), turned to -90 degrees
- moved R703 378.4 mm to (201.5, 88.4)
- moved R702 375.0 mm to (197.2, 88.4)
- moved C708 371.9 mm to (195.6, 82.7), turned to -90 degrees
- moved C707 370.1 mm to (193.2, 82.7), turned to -90 degrees
- moved C214 369.1 mm to (193.8, 100.8), turned to 180 degrees
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- renumbered R928 to R929, R930 to R931, R931 to R932, R932 to R933, R933 to R934, R934 to R935, R935 to R936, R936 to R937
Connections:
- R928 pad 2: Net-(C931-Pad1) -> Net-(R928-Pad2)
- U1002 pad 36: /Ethernet/RMII_MDIO -> /Ethernet/MDIO
- U201 pad 12: /Ethernet/RMII_MDIO -> /Ethernet/MDIO

Commit message: PCB layout
Parts:
- removed the C813 at (-166.0, -77.8)
- removed the C817 at (-208.9, -27.6)
- removed the C905 at (-41.9, -51.7)
- added C619: 1n, Capacitor_SMD:C_0603_1608Metric_Pad1.08x0.95mm_HandSolder, B.Cu at (156.6, 46.1)
- added C915: 100n, Capacitor_SMD:C_0603_1608Metric_Pad1.08x0.95mm_HandSolder, B.Cu at (142.4, 71.1)
- added C918: 100n, Capacitor_SMD:C_0603_1608Metric_Pad1.08x0.95mm_HandSolder, B.Cu at (119.5, 108.3)
- added C920: 100n, Capacitor_SMD:C_0603_1608Metric_Pad1.08x0.95mm_HandSolder, B.Cu at (132.2, 81.0)
- added C923: 100n, Capacitor_SMD:C_0603_1608Metric_Pad1.08x0.95mm_HandSolder, B.Cu at (138.8, 78.9)
- added C927: 100n, Capacitor_SMD:C_0603_1608Metric_Pad1.08x0.95mm_HandSolder, B.Cu at (147.4, 71.1)
- added D604: BAV99, Package_TO_SOT_SMD:SOT-23, F.Cu at (160.4, 46.1)
- added R611: 100, Resistor_SMD:R_0603_1608Metric_Pad0.98x0.95mm_HandSolder, F.Cu at (156.6, 46.1)
- C1016, C301, C501, C502, C503, C504, C505, C506, C507, C508, C509, C510, C601, C604, C605, C606, C607, C608, C609, C610, C611, C612, C613, C614, C615, C616, C809, R913, R918, R926, R927: moved to B.Cu
- C901: renamed from C912; moved to B.Cu
- C902: renamed from C901; moved to B.Cu
- C904: renamed from C915; moved to B.Cu
- C905: renamed from C903; moved to B.Cu
- C906: renamed from C918; moved to B.Cu
- C907: renamed from C904; moved to B.Cu
- C908: renamed from C906; moved to B.Cu
- C909: renamed from C919; moved to B.Cu
- C910: renamed from C907; moved to B.Cu
- C911: renamed from C921; moved to B.Cu
- C912: renamed from C908; moved to B.Cu
- C913: renamed from C922; moved to B.Cu
- C914: renamed from C909; moved to B.Cu
- C916: renamed from C911; moved to B.Cu
- C917: renamed from C923; moved to B.Cu
- C919: renamed from C925; moved to B.Cu
- C922: renamed from C926; moved to B.Cu
- C924: renamed from C928; moved to B.Cu
- C925: renamed from C929; moved to B.Cu
- C932: renamed from C924; moved to B.Cu
- C936: renamed from C931; moved to B.Cu
- R614: renamed from R613; moved to B.Cu
- R617: renamed from R616; moved to F.Cu
- R908: renamed from R907; moved to B.Cu
- R909: renamed from R908; moved to B.Cu
- R928: renamed from R931; moved to B.Cu
- R936: renamed from R937; moved to B.Cu
- moved C301 440.5 mm to (166.8, 89.8), turned to 180 degrees
- moved C809 435.2 mm to (188.8, 125.5), turned to 180 degrees
- moved R902 423.5 mm to (151.0, 122.7), turned to 180 degrees
- moved C914 412.9 mm to (121.5, 127.6), turned to 90 degrees
- moved U909 409.3 mm to (122.9, 127.6), turned to 180 degrees
- moved U913 407.4 mm to (121.8, 108.0)
- moved C910 407.0 mm to (138.6, 125.3), turned to -90 degrees
- moved U914 406.0 mm to (123.3, 114.4), turned to 90 degrees
- moved C921 406.0 mm to (118.4, 125.0), turned to 90 degrees
- moved R930 402.9 mm to (119.8, 114.3), turned to -90 degrees
- moved C912 402.6 mm to (124.2, 123.6), turned to -90 degrees
- moved C926 401.2 mm to (113.3, 128.5), turned to 180 degrees
- moved U915 400.5 mm to (114.3, 108.8)
- moved U906 398.3 mm to (122.9, 123.4)
- moved C933 398.0 mm to (105.7, 105.4)
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- renumbered C619 to C620, C620 to C621, C621 to C622, C622 to C623, C814 to C813, C815 to C814, C816 to C815, C818 to C816, C819 to C817, C820 to C818, C821 to C819, C822 to C820, C823 to C821, C824 to C822, C825 to C823, C826 to C824, C827 to C825, C902 to C903, C910 to C921, C913 to C926, C914 to C928, C916 to C929, C917 to C930, C920 to C931, C927 to C933, C930 to C934, C933 to C935, C932 to C937, R611 to R612, R612 to R613, R614 to R615, R615 to R616, R617 to R618, R618 to R619, R619 to R620, R620 to R621, R621 to R622, R622 to R623, R623 to R624, R624 to R625, R625 to R626, R626 to R627, R627 to R628, R628 to R629, R629 to R630, R630 to R631, R902 to R901, R901 to R902, R905 to R904, R906 to R905, R904 to R906, R912 to R907, R914 to R910, R909 to R911, R910 to R912, R916 to R914, R917 to R915, R911 to R916, R915 to R917, R928 to R929, R929 to R930, R930 to R931, R933 to R932, R934 to R933, R936 to R934, R932 to R935, R935 to R937, U903 to U902, U902 to U903, U906 to U904, U908 to U905, U904 to U906, U909 to U907, U905 to U908, U907 to U909, U913 to U912, U912 to U913, U915 to U914, U914 to U915
Connections:
- net Net-(R613-Pad2) renamed /Frontend/FILTER_LIM
- net Net-(R615-Pad1) renamed /Frontend/SENS+_LIM
- C823 pad 1: +3V3 -> +3.3V
- C824 pad 1: +3V3 -> +3.3V
- C825 pad 1: +3V3 -> +3.3V
- R614 pad 1: Net-(R613-Pad1) (its old number) -> /Frontend/SENS-_LIM
- R630 pad 2: Net-(R613-Pad1) (its old number) -> /Frontend/SENS-_LIM
- U606 pad 6: Net-(R613-Pad1) (its old number) -> /Frontend/SENS-_LIM
- U804 pad 2: +3V3 -> +3.3V

Commit message: PCB layout
Parts:
- added C909: 100n, Capacitor_SMD:C_0603_1608Metric_Pad1.08x0.95mm_HandSolder, B.Cu at (142.6, 81.2)
- C401, C402, R401: moved to B.Cu
- moved C401 299.1 mm to (142.7, 50.4), turned to 180 degrees
- moved R410 265.4 mm to (137.9, 61.6), turned to -90 degrees
- moved U406 264.2 mm to (142.7, 48.0), turned to -90 degrees
- moved U410 264.1 mm to (126.5, 59.6), turned to -90 degrees
- moved R408 260.5 mm to (137.9, 57.5), turned to 90 degrees
- moved U402 260.2 mm to (116.1, 49.4)
- moved U407 259.4 mm to (133.3, 48.0), turned to 90 degrees
- moved C402 255.5 mm to (142.7, 45.6)
- moved U409 254.7 mm to (126.5, 48.0), turned to -90 degrees
- moved U408 248.5 mm to (133.3, 59.6), turned to -90 degrees
- moved R416 245.6 mm to (121.7, 64.6), turned to -90 degrees
- moved R407 245.6 mm to (137.9, 50.0), turned to 90 degrees
- moved R409 245.4 mm to (137.9, 46.0), turned to 90 degrees
- moved R415 244.9 mm to (121.7, 61.1), turned to -90 degrees
- moved R413 243.1 mm to (121.7, 53.0), turned to -90 degrees
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- renumbered C909 to C908, C911 to C910, C908 to C911, C913 to C912, C910 to C913, C915 to C914, C912 to C915, C914 to C916, C916 to C918, C918 to C920, C920 to C923, C923 to C925, C925 to C926, C926 to C927, C927 to C928, C928 to C929, C929 to C930, C930 to C931, C931 to C932, C932 to C933, C933 to C934, C934 to C935, C935 to C936, C936 to C937, C937 to C938

Commit message: PCB layout
Parts:
- C404, C405, C407, C408, C409, C410, C411, C412, C413, C417, C418, C419, C422, C423, C424, C426, C427, C428, C430, C431, C432, C434, C444, C617, C618, R403: moved to B.Cu
- moved C427 303.5 mm to (133.2, 49.5), turned to 180 degrees
- moved C408 301.0 mm to (133.3, 61.1), turned to 180 degrees
- moved C418 295.9 mm to (113.5, 58.3), turned to 90 degrees
- moved C412 293.4 mm to (126.5, 56.0)
- moved C617 290.3 mm to (159.3, 60.3), turned to 180 degrees
- moved C428 289.5 mm to (133.2, 44.5)
- moved C431 288.3 mm to (109.7, 57.7), turned to -90 degrees
- moved C430 284.9 mm to (104.6, 57.7), turned to 90 degrees
- moved C404 283.3 mm to (126.5, 44.5)
- moved C618 281.6 mm to (159.1, 54.0), turned to 180 degrees
- moved C423 276.7 mm to (113.5, 46.6), turned to 90 degrees
- moved R418 275.5 mm to (89.3, 62.0)
- moved R417 273.8 mm to (75.8, 63.0)
- moved C444 270.0 mm to (109.7, 46.0), turned to -90 degrees
- moved C434 268.7 mm to (104.8, 46.0), turned to 90 degrees
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
Commit message: PCB layout
Parts:
- removed the C438 at (-57.3, -179.5)
- removed the C446 at (-59.2, -166.9)
- C403, C421, C425, C429, C435, C436, C437, C439, C441, C442, C445: moved to B.Cu
- C438: renamed from C443; moved to B.Cu
- C443: renamed from C448; moved to B.Cu
- C446: renamed from C447; moved to B.Cu
- C447: renamed from C449; moved to B.Cu
- C448: renamed from C450; moved to B.Cu
- C449: renamed from C451; moved to B.Cu
- moved U414 319.9 mm to (113.8, 70.6), turned to 180 degrees
- moved U401 314.1 mm to (115.3, 77.3), turned to 180 degrees
- moved C446 302.5 mm to (115.3, 77.3), turned to -90 degrees
- moved R426 301.3 mm to (108.2, 68.8), turned to 90 degrees
- moved R421 300.5 mm to (111.8, 65.9)
- moved C414 300.5 mm to (111.4, 77.3), turned to 90 degrees
- moved R420 299.2 mm to (116.0, 65.9), turned to 180 degrees
- moved R422 294.2 mm to (108.2, 72.4), turned to 90 degrees
- moved C451 294.1 mm to (105.8, 72.4), turned to -90 degrees
- moved C445 293.5 mm to (98.4, 69.7)
- moved C443 293.3 mm to (116.3, 70.6), turned to -90 degrees
- moved C447 292.8 mm to (111.3, 70.6), turned to 90 degrees
- moved C436 290.6 mm to (95.0, 69.7), turned to 180 degrees
- moved C438 289.7 mm to (116.3, 54.7), turned to -90 degrees
- moved R419 289.3 mm to (108.2, 56.5), turned to 90 degrees
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- renumbered C452 to C450, C453 to C451, C454 to C452, C455 to C453
Routing:
- added copper zone on F.Cu, net -15V
