File: HARDWARE/ETH1CSMU2/ETH1CSMU2.kicad_pcb (KiCad board)
At the start: 4 copper layers, 160 x 100 mm, 446 parts, among them J1001 Conn_02x01, J1002 20021111-00010T4LF, J301 C64AC, K301 HE3621A0510, K302 HE3621A0510, K303 HE3621A0510, K304 HE3621A0510, K305 HE3621A0510, K306 HE3621A0510, Q601 MMBT3904, Q602 MMBT3904, Q603 MMBT3904, Q604 MMBT3904, Q801 IRFR5410, Q901 FDV301N, U1001 HDC1080, U1002 STM32F746ZG, U1003 24LC08B-E/MS, U201 LAN8742A, U202 LC03-3.3, U203 LC03-3.3, U301 ULN2003AIDE4, U401 LT1790BCS6-2.5, U402 DG444DY+, U403 REF5040ID, U404 DG444DY+, U405 ADR435ARM, U406 DG419DY, U407 DG419DY, U408 DG419DY, U409 OPA141AID, U410 OPA141AID, U411 DG419DY, U412 DG419DY, U413 OPA141AID, U414 OPA141AID, U415 ADS8681IRUMT, U416 ADS8681IRUMT, U417 AD7980ARM, U418 AD7980ARM, U419 TPS76925, U501 74HCT595PW, U502 74HCT595PW, U503 SN74LVC1T45DRLR, U504 SN74LVC1T45DRLR, U505 SN74LVC1T45DRLR, U506 SN74LVC1T45DRLR, U601 DG419DY, U602 DG419DY, U603 SN74LVC1T45DRLR, U604 SN74LVC1T45DRLR, U605 SN74LVC1T45DRLR, U606 LT1970ACFE, U607 INA823DT, U608 AQY212G2SX, U609 AQY212G2SX, U610 AQY212G2SX, U611 AQY212G2SX, U612 LM7171BIM, U701 TXB0104PW, U702 ADuM5402, U703 74AC125, U801 MAX5902ACEUT, U802 TEL 12-2423, U803 TSR2-2450, U804 NCV1117DT33T5G, U901 DAC8565ICPW, U902 AD9834BRUZ, U903 MC74AC161DR2G, U904 MAX6102EUR, U905 MAX5217GUA+, U906 SN74AHC1G14DBVT, U907 OPA2141AID, U908 MC74AC161DR2G, U909 SN74AUP1G79DCKR, U910 LM7171BIM, U911 OPA141AID, U912 DG409DY+, U913 AD5322ARMZ, U914 LT1790BCS6-2.5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

Commit message: PCB layout
Routing:
- net Net-(R903-Pad1): track 0.00 -> 13.9 mm
- net /MCU/TMS_SWDIO: track 0.00 -> 10.7 mm, vias 0 -> 1
- net /MCU/TCK_SWCLK: track 0.00 -> 10.0 mm, vias 0 -> 1
- net Net-(C201-Pad1): track 0.00 -> 9.60 mm
- net Net-(D201-Pad2): track 0.00 -> 7.69 mm
- net Net-(C1003-Pad1): track 0.00 -> 6.60 mm, vias 0 -> 1
- net Net-(C1005-Pad1): track 0.00 -> 6.58 mm, vias 0 -> 1
- net Net-(C204-Pad1): track 0.00 -> 6.21 mm
- net /MCU/EEPROM_SCL: track 0.00 -> 5.51 mm
- net Net-(C203-Pad1): track 0.00 -> 4.83 mm
- net /Ethernet/MDIO: track 0.00 -> 4.49 mm
- net Net-(D202-Pad2): track 0.00 -> 4.32 mm
- net /Ethernet/MODE2: track 0.00 -> 4.06 mm
- net /Ethernet/MODE1: track 0.00 -> 3.75 mm
- net Net-(R203-Pad1): track 0.00 -> 3.64 mm
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Changed lines of the file:
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@@
   (gr_line (start 228 40) (end 230 42) (layer "Edge.Cuts") (width 0.1))
   (gr_line (start 228 140) (end 230 138) (layer "Edge.Cuts") (width 0.1))
+  (segment (start 165.227 96.139) (end 164.497 95.409) (width 0.127) (layer "F.Cu") (net 1))
+  (segment (start 168.529 96.139) (end 165.227 96.139) (width 0.127) (layer "F.Cu") (net 1))
+  (segment (start 164.497 95.409) (end 164.497 93.8295) (width 0.127) (layer "F.Cu") (net 1))
+  (segment (start 170.446 99.0275) (end 170.446 98.056) (width 0.127) (layer "F.Cu") (net 1))
+  (segment (start 170.446 98.056) (end 168.529 96.139) (width 0.127) (layer "F.Cu") (net 1))
+  (segment (start 168.8775 99.0275) (end 167.132 97.282) (width 0.127) (layer "F.Cu") (net 4))
+  (segment (start 169.946 99.0275) (end 168.8775 99.0275) (width 0.127) (layer "F.Cu") (net 4))
+  (segment (start 167.132 97.282) (end 165.8355 97.282) (width 0.127) (layer "F.Cu") (net 4))
+  (segment (start 170.946 99.0275) (end 170.946 97.921) (width 0.127) (layer "F.Cu") (net 5))
+  (segment (start 168.497 95.472) (end 168.497 93.8295) (width 0.127) (layer "F.Cu") (net 5))
+  (segment (start 170.946 97.921) (end 168.497 95.472) (width 0.127) (layer "F.Cu") (net 5))
+  (segment (start 142.458 116.9615) (end 142.458 115.534) (width 0.127) (layer "F.Cu") (net 37))
+  (segment (start 142.458 115.534) (end 141.732 114.808) (width 0.127) (layer "F.Cu") (net 37))
+  (via (at 141.732 114.808) (size 0.5) (drill 0.2) (layers "F.Cu" "B.Cu") (net 37))
+  (segment (start 141.732 113.35) (end 141.798 113.284) (width 0.127) (layer "B.Cu") (net 37))
+  (segment (start 141.798 110.7835) (end 141.798 113.284) (width 0.127) (layer "B.Cu") (net 37))
+  (segment (start 141.732 110.7175) (end 141.798 110.7835) (width 0.127) (layer "B.Cu") (net 37))
+  (segment (start 141.732 114.808) (end 141.732 113.35) (width 0.127) (layer "B.Cu") (net 37))
+  (segment (start 142.958 115.487) (end 143.637 114.808) (width 0.127) (layer "F.Cu") (net 38))
+  (segment (start 142.958 116.9615) (end 142.958 115.487) (width 0.127) (layer "F.Cu") (net 38))
+  (via (at 143.637 114.808) (size 0.5) (drill 0.2) (layers "F.Cu" "B.Cu") (net 38))
+  (segment (start 143.698 110.7835) (end 143.698 113.284) (width 0.127) (layer "B.Cu") (net 38))
+  (segment (start 143.764 110.7175) (end 143.698 110.7835) (width 0.127) (layer "B.Cu") (net 38))
+  (segment (start 143.637 113.345) (end 143.698 113.284) (width 0.127) (layer "B.Cu") (net 38))
+  (segment (start 143.637 114.808) (end 143.637 113.345) (width 0.127) (layer "B.Cu") (net 38))
+  (segment (start 171.946 99.0275) (end 171.946 96.7485) (width 0.127) (layer "F.Cu") (net 44))
+  (segment (start 171.946 96.7485) (end 173.99 94.7045) (width 0.127) (layer "F.Cu") (net 44))
+  (segment (start 176.4605 94.7045) (end 176.498 94.742) (width 0.127) (layer "F.Cu") (net 44))
+  (segment (start 173.99 94.7045) (end 176.4605 94.7045) (width 0.127) (layer "F.Cu") (net 44))
+  (segment (start 171.446 99.0275) (end 171.446 94.7085) (width 0.127) (layer "F.Cu") (net 46))
+  (segment (start 171.446 94.7085) (end 171.45 94.7045) (width 0.127) (layer "F.Cu") (net 46))
+  (segment (start 132.842 97.79) (end 132.958 97.674) (width 0.127) (layer "F.Cu") (net 107))
+  (segment (start 132.958 97.674) (end 132.958 95.6365) (width 0.127) (layer "F.Cu") (net 107))
+  (via (at 132.842 97.79) (size 0.5) (drill 0.2) (layers "F.Cu" "B.Cu") (net 107))
+  (segment (start 132.842 97.79) (end 132.08 97.028) (width 0.127) (layer "B.Cu") (net 107))
+  (segment (start 132.08 97.028) (end 127.127 97.028) (width 0.127) (layer "B.Cu") (net 107))
+  (segment (start 125.984 95.885) (end 125.095 95.885) (width 0.127) (layer "B.Cu") (net 107))
+  (segment (start 127.127 97.028) (end 125.984 95.885) (width 0.127) (layer "B.Cu") (net 107))
+  (segment (start 132.136731 97.810223) (end 131.875508 97.549) (width 0.127) (layer "F.Cu") (net 108))
+  (segment (start 131.875508 97.549) (end 129.5455 97.549) (width 0.127) (layer "F.Cu") (net 108))
+  (via (at 132.136731 97.810223) (size 0.5) (drill 0.2) (layers "F.Cu" "B.Cu") (net 108))
+  (segment (start 131.862508 97.536) (end 127.127 97.536) (width 0.127) (layer "B.Cu") (net 108))
+  (segment (start 127.127 97.536) (end 126.746 97.155) (width 0.127) (layer "B.Cu") (net 108))
+  (segment (start 132.136731 97.810223) (end 131.862508 97.536) (width 0.127) (layer "B.Cu") (net 108))
+  (segment (start 126.746 97.155) (end 125.095 97.155) (width 0.127) (layer "B.Cu") (net 108))
+  (segment (start 169.2585 100.215) (end 166.993 100.215) (width 0.127) (layer "F.Cu") (net 132))
+  (segment (start 166.993 100.215) (end 166.878 100.33) (width 0.127) (layer "F.Cu") (net 132))
+  (segment (start 166.878 100.33) (end 165.8855 100.33) (width 0.127) (layer "F.Cu") (net 132))
+  (segment (start 169.2585 99.715) (end 168.422 99.715) (width 0.127) (layer "F.Cu") (net 134))
+  (segment (start 167.513 98.806) (end 165.8855 98.806) (width 0.127) (layer "F.Cu") (net 134))
+  (segment (start 168.422 99.715) (end 167.513 98.806) (width 0.127) (layer "F.Cu") (net 134))
+  (segment (start 169.2585 101.215) (end 167.39 101.215) (width 0.127) (layer "F.Cu") (net 136))
+  (segment (start 166.751 101.854) (end 165.8855 101.854) (width 0.127) (layer "F.Cu") (net 136))
+  (segment (start 167.39 101.215) (end 166.751 101.854) (width 0.127) (layer "F.Cu") (net 136))
+  (segment (start 169.2585 101.715) (end 167.5485 101.715) (width 0.127) (layer "F.Cu") (net 137))
+  (segment (start 167.5485 101.715) (end 165.8855 103.378) (width 0.127) (layer "F.Cu") (net 137))
+  (segment (start 170.446 104.1045) (end 169.037 105.5135) (width 0.127) (layer "F.Cu") (net 139))
+  (segment (start 170.446 102.9025) (end 170.446 104.1045) (width 0.127) (layer "F.Cu") (net 139))
+  (segment (start 169.2585 102.215) (end 168.5725 102.215) (width 0.127) (layer "F.Cu") (net 141))
+  (segment (start 168.5725 102.215) (end 165.8855 104.902) (width 0.127) (layer "F.Cu") (net 141))
+  (segment (start 150.8525 127.508) (end 149.733 127.508) (width 0.127) (layer "F.Cu") (net 185))
+  (segment (start 149.733 127.508) (end 149.34025 127.11525) (width 0.127) (layer "F.Cu") (net 185))
+  (segment (start 141.605 124.841) (end 140.589 125.857) (width 0.127) (layer "F.Cu") (net 185))
+  (segment (start 149.34025 127.11525) (end 149.34025 125.99575) (width 0.127) (layer "F.Cu") (net 185))
+  (segment (start 140.589 125.857) (end 140.589 127.316) (width 0.127) (layer "F.Cu") (net 185))
+  (segment (start 149.34025 125.99575) (end 148.1855 124.841) (width 0.127) (layer "F.Cu") (net 185))
+  (segment (start 148.1855 124.841) (end 141.605 124.841) (width 0.127) (layer "F.Cu") (net 185))
+  (segment (start 152.415 127.2455) (end 152.6775 127.508) (width 0.127) (layer "F.Cu") (net 186))
+  (segment (start 152.415 125.818) (end 152.415 127.2455) (width 0.127) (layer "F.Cu") (net 186))
+  (segment (start 141.5405 98.4575) (end 141.478 98.395) (width 0.127) (layer "B.Cu") (net 195))
+  (segment (start 144.1915 98.4575) (end 141.5405 98.4575) (width 0.127) (layer "B.Cu") (net 195))
+  (segment (start 145.6365 98.4575) (end 144.8855 99.2085) (width 0.127) (layer "B.Cu") (net 196))
+  (segment (start 142.733 99.045) (end 141.478 99.045) (width 0.127) (layer "B.Cu") (net 196))
+  (segment (start 146.6045 98.4575) (end 145.6365 98.4575) (width 0.127) (layer "B.Cu") (net 196))
+  (segment (start 144.8855 99.2085) (end 142.8965 99.2085) (width 0.127) (layer "B.Cu") (net 196))
+  (segment (start 142.8965 99.2085) (end 142.733 99.045) (width 0.127) (layer "B.Cu") (net 196))
+  (segment (start 151.115 122.4365) (end 150.8525 122.174) (width 0.127) (layer "F.Cu") (net 417))
+  (segment (start 151.115 124.118) (end 151.115 122.4365) (width 0.127) (layer "F.Cu") (net 417))
   (zone (net 10) (net_name "-15V") (layer "F.Cu") (hatch edge 0.508)
     (connect_pads yes (clearance 0.127))

Commit message: PCB layout
Parts:
- moved C935 14.2 mm to (111.9, 101.5)
- moved R920 14.2 mm to (111.9, 104.0)
- moved Q901 14.2 mm to (116.0, 102.7)
- moved R919 10.2 mm to (119.5, 102.5), turned to 90 degrees
- moved C804 6.74 mm to (199.3, 113.3), turned to 180 degrees
- moved C810 6.48 mm to (199.3, 119.9), turned to 180 degrees
- moved C905 5.34 mm to (113.9, 88.6)
- moved R921 5.34 mm to (111.9, 98.8)
- moved R922 5.34 mm to (116.0, 98.8)
- moved R928 5.34 mm to (116.0, 98.8)
- moved U912 5.34 mm to (113.9, 91.8)
- moved C908 5.34 mm to (114.9, 91.8)
- moved C924 5.34 mm to (112.9, 91.8)
- moved R923 5.34 mm to (119.5, 97.9)
- moved R924 5.34 mm to (119.5, 94.5)
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Connections:
- C701 pad 1: +3V3 -> +3.3V
- C702 pad 1: +3V3 -> +3.3V
- K301 pad 3: Net-(K301-Pad3) -> Net-(U301-Pad16)
- K302 pad 3: Net-(K302-Pad3) -> Net-(U301-Pad15)
- K305 pad 3: Net-(K305-Pad3) -> Net-(U301-Pad12)
- K306 pad 3: Net-(K306-Pad3) -> Net-(U301-Pad11)
- R701 pad 1: +3V3 -> +3.3V
- U301 pad 1: /Connect/CXN_REL6 -> /Connect/CXN_REL1
- U301 pad 11: Net-(K304-Pad3) -> Net-(U301-Pad11)
- U301 pad 12: Net-(K301-Pad3) -> Net-(U301-Pad12)
- U301 pad 13: Net-(K302-Pad3) -> Net-(K304-Pad3)
- U301 pad 15: Net-(K305-Pad3) -> Net-(U301-Pad15)
- U301 pad 16: Net-(K306-Pad3) -> Net-(U301-Pad16)
- U301 pad 2: /Connect/CXN_REL5 -> /Connect/CXN_REL2
- U301 pad 3: /Connect/CXN_REL4 -> /Connect/CXN_REL3
- U301 pad 4: /Connect/CXN_REL3 -> /Connect/CXN_REL4
- U301 pad 5: /Connect/CXN_REL2 -> /Connect/CXN_REL5
- U301 pad 6: /Connect/CXN_REL1 -> /Connect/CXN_REL6
- U417 pad 10: +3V3 -> +3.3V
- U418 pad 10: +3V3 -> +3.3V
- U701 pad 1: +3V3 -> +3.3V
- U902 pad 5: +3V3 -> +3.3V
Routing:
- net +3.3V: track 0.00 -> 98.3 mm, vias 0 -> 44
- net +5V: track 0.00 -> 90.8 mm, vias 0 -> 40
- net /Connect/VOLT_MEAS_SENS: track 0.00 -> 78.0 mm, vias 0 -> 1
- net Net-(U301-Pad16): track 0.00 -> 71.6 mm, vias 0 -> 1
- net /Connect/VOUT_OUT: track 0.00 -> 68.6 mm
- net -15V: track 0.00 -> 68.0 mm, vias 0 -> 62
- net Net-(R616-Pad2): track 0.00 -> 67.4 mm, vias 0 -> 1
- net Net-(U301-Pad15): track 0.00 -> 67.3 mm, vias 0 -> 1
- net Net-(U301-Pad14): track 0.00 -> 63.4 mm, vias 0 -> 1
- net +15V: track 0.00 -> 63.3 mm, vias 0 -> 25
- net Net-(K304-Pad3): track 0.00 -> 59.5 mm, vias 0 -> 1
- net /Frontend/CURR_MEAS: track 0.00 -> 57.2 mm, vias 0 -> 2
- net Net-(U301-Pad12): track 0.00 -> 55.4 mm, vias 0 -> 1
- net Net-(U301-Pad11): track 0.00 -> 51.4 mm, vias 0 -> 1
- net Net-(U602-Pad1): track 0.00 -> 50.4 mm, vias 0 -> 2
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- added copper zone on F.Cu, net +15V
- added copper zone on B.Cu, net -15V
- added copper zone on In1.Cu, net -15V
- added copper zone on In1.Cu, net GND
- added copper zone on In1.Cu, net GND_TRIG

Commit message: PCB layout
Parts:
- moved D1002 6.54 mm to (157.1, 106.2)
- moved R1003 6.54 mm to (157.1, 106.2)
- moved D1001 6.54 mm to (157.1, 108.8)
- moved D1003 6.54 mm to (157.1, 103.4)
- moved R1001 6.54 mm to (157.1, 108.8)
- moved R1005 6.54 mm to (157.1, 103.4)
- moved J1001 6.19 mm to (157.2, 96.6)
- moved R1002 3.98 mm to (157.2, 93.0), turned to 180 degrees
- moved C823 1.69 mm to (160.9, 116.2)
- moved C824 1.69 mm to (160.9, 113.8)
- moved C825 1.69 mm to (160.9, 118.6)
- moved U804 1.42 mm to (168.8, 118.2)
- moved C1012 0.38 mm to (150.9, 95.5)
Connections:
- U1002 pad 10: /Frontend/MCU_nISNK -> /MCU/DDS_DIV2
- U1002 pad 11: /Frontend/MCU_nISRC -> unconnected-(U1002-Pad11)
- U1002 pad 12: /Frontend/MCU_nTDS -> unconnected-(U1002-Pad12)
- U1002 pad 50: /MCU/DDS_DIV2 -> unconnected-(U1002-Pad50)
- U1002 pad 53: /MCU/DDS_DIV4 -> /Frontend/MCU_nISNK
- U1002 pad 54: /MCU/DDS_DIV8 -> /Frontend/MCU_nISRC
- U1002 pad 55: /MCU/~{DDS_DIV10} -> /Frontend/MCU_nTDS
- U1002 pad 58: /Connect/CXN_REL6 -> /MCU/DAC1_LDAC
- U1002 pad 64: /Connect/CXN_REL2 -> /MCU/DAC1_~{RST}
- U1002 pad 65: /Connect/CXN_REL1 -> /Connect/CXN_REL6
- U1002 pad 69: /MCU/DAC1_LDAC -> /Connect/CXN_REL2
- U1002 pad 7: unconnected-(U1002-Pad7) -> /MCU/~{DDS_DIV10}
- U1002 pad 70: /MCU/DAC1_~{RST} -> /Connect/CXN_REL1
- U1002 pad 8: unconnected-(U1002-Pad8) -> /MCU/DDS_DIV8
- U1002 pad 9: unconnected-(U1002-Pad9) -> /MCU/DDS_DIV4
Routing:
- net /MCU/NRST: track 6.65 -> 57.3 mm
- net /Ethernet/RMII_MDC: track 1.04 -> 50.9 mm, vias 1 -> 2
- net /Ethernet/RMII_TXD0: track 2.48 -> 51.1 mm
- net /Ethernet/RMII_TXEN: track 2.63 -> 51.2 mm
- net /Ethernet/RMII_RXD1: track 2.38 -> 50.8 mm
- net /Ethernet/RMII_CRS_DV: track 2.39 -> 50.8 mm
- net /Ethernet/RMII_RXD0: track 2.39 -> 50.8 mm
- net /Ethernet/RMII_TXD1: track 3.03 -> 51.1 mm
- net /Connect/CXN_REL1: track 0.00 -> 28.3 mm, vias 0 -> 2
- net /Connect/CXN_REL2: track 0.00 -> 28.2 mm, vias 0 -> 2
- net /Connect/CXN_REL3: track 0.00 -> 27.8 mm, vias 0 -> 2
- net /Connect/CXN_REL4: track 0.00 -> 27.3 mm, vias 0 -> 2
- net /Connect/CXN_REL5: track 0.00 -> 26.9 mm, vias 0 -> 2
- net /MCU/DDS_DIV8: track 1.20 -> 26.6 mm, vias 1 -> 2
- net /Connect/CXN_REL6: track 0.00 -> 24.7 mm, vias 0 -> 2
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